File: kicad/atari_gravitar_black_widow/atari_gravitar_black_widow.sch (KiCad schematic (older format))
At the start: 2 parts

Commit message: First commit - AVG & VSM
Parts:
- added H7: LS42, symbol Star_Wars_Vector_PCB:LS42
- added J3: LS04, symbol Star_Wars_Vector_PCB:LS04
- added J9: AVG, symbol Star_Wars_Vector_PCB:AVG
- added L4: LS08, symbol Star_Wars_Vector_PCB:LS08
- added N4: S129, symbol Star_Wars_Vector_PCB:S129
- added R20: 10K, symbol Device:R_US
- added R4: LS32, symbol Star_Wars_Vector_PCB:LS32
- added U?: LS74, symbol Star_Wars_Vector_PCB:LS74
- added U?: LS174A, symbol Star_Wars_Vector_PCB:LS174A
Connections:
- new net: J9.35 (ST2), L4.6
- new net: J9.5 (~OP2), R4.6
- new net: R4.8, U?.13 (~1CLR)
- new net: N4.9 (O4), R4.9, U?.6 (3D)
- new net AVG0: J9.36 (AVG0)
- new net AVG1: J9.39 (AVG1)
- new net AVG10: J9.19 (AVG10)
- new net AVG11: J9.20 (AVG11)
- new net AVG12: J9.21 (AVG12)
- new net AVG13: J9.22 (AVG13)
- new net AVG2: J9.40 (AVG2)
- new net AVG3: J9.1 (AVG3)
- new net AVG4: J9.2 (AVG4)
- new net AVG5: J9.3 (AVG5)
- new net AVG6: J9.15 (AVG6)
- new net AVG7: J9.16 (AVG7)
- new net AVG8: J9.17 (AVG8)
- new net AVG9: J9.18 (AVG9)
- new net DVY0: J9.32 (DVY0)
- new net DVY1: J9.31 (DVY1)
- new net DVY10: J9.29 (DVY10)
- new net DVY11: J9.28 (DVY11)
- new net DVY12: J9.27 (DVY12)
- new net DVY2: J9.30 (DVY2)
- new net DVY3: J9.7 (DVY3)
- new net DVY4: J9.8 (DVY4)
- new net DVY5: J9.9 (DVY5)
- new net DVY6: J9.10 (DVY6)
- new net DVY7: J9.11 (DVY7)
- new net DVY8: J9.12 (DVY8)
- new net DVY9: J9.13 (DVY9)
- new net OP1: J9.33 (OP1)
- new net SA: J3.12, R4.10, R4.5
- new net ST0: H7.15 (A0), N4.12 (O1), U?.13 (5D)
- new net ST1: H7.14 (A1), N4.11 (O2), U?.4 (2D)
- new net ST2: H7.13 (A2), L4.4, N4.10 (O3), U?.11 (4D)
- new net ST3: H7.12 (A3), J9.38 (ST3), U?.8 (~2Q)
- new net ~LATCH0: H7.1 (0)
- new net ~LATCH1: H7.2 (1)
- new net ~LATCH2: H7.3 (2)
- new net ~LATCH3: H7.4 (3)
- new net ~OP0: J9.25 (~OPX), J9.26 (~OP0)
- new net ~OP2: R4.4
- new net ~SA: J3.13, L4.5, R20.2
- new net ~STROBE0: H7.5 (4), J9.24 (~STROBE0)
- new net ~STROBE1: H7.6 (5), J9.34 (~STROBE1)
- new net ~STROBE2: H7.7 (6), J9.4 (~STROBE2)
- new net ~STROBE3: H7.9 (7)
- new net ~VGGO: J9.6 (~VGGO)

Commit message: 6B
More sheet 6B (but not all)
Parts:
- added unit 1 of A7
- added N3: LS157, symbol Star_Wars_Vector_PCB:LS157D
- added N5: LS02, symbol Star_Wars_Vector_PCB:LS02
- added R3: LS157, symbol Star_Wars_Vector_PCB:LS157C
- P4: renamed from U?; value LS174A -> LS174
- gave numbers to parts that had none: 1
Connections:
- net AM0: now also R3.3 (B)
- net AM1: now also R3.6 (B)
- net AM2: now also R3.10 (B)
- net AM3: now also R3.13 (B)
- net AM4: now also N3.10 (B)
- net AM5: now also N3.6 (B)
- net AM6: now also N3.3 (B)
- net AM7: now also N3.13 (B)
- net GO: now also N5.9
- net HALT: now also P4.3 (1D)
- net OP0: now also N3.11 (A)
- net OP1: now also N3.5 (A)
- net OP2: now also N3.2 (A)
- net SA: now also N3.1 (S), R3.1 (S)
- net F2: now reaches P4.10 (4Q)
- net F2: now also R3.11 (A)
- net F0: now reaches P4.12 (5Q)
- net F0: now also R3.2 (A)
- net HALT*: now reaches P4.2 (1Q)
- net HALT*: now also N5.8
- net F1: now reaches P4.5 (2Q)
- net F1: now also R3.5 (A)
- net F3: now reaches P4.7 (3Q)
- net F3: now also R3.14 (A)
- net at N4.1 (A6): now also N3.4 (Y)
- net at N4.15 (A7): now also N3.12 (Y)
- net at N4.2 (A5): now also N3.7 (Y)
- net at N4.3 (A4): now also N3.9 (Y)
- net at N4.4 (A3): now also R3.12 (Y)
- net at N4.5 (A0): now also R3.4 (Y)
- net at N4.6 (A1): now also R3.9 (Y)
- net at N4.7 (A2): now also R3.7 (Y)
- new net: N3.14 (A), N5.10
Other:
- moved on the sheet: H7, P4B

Commit message: sheet 6B
Almost done
Parts:
- added B7, K5, K6: LS02, symbol atari_gravitar_black_widow-rescue:LS02-Star_Wars_Vector_PCB
- added J5: S260, symbol atari_gravitar_black_widow-rescue:S260alt-Star_Wars_Vector_PCB
- added K3: LS74, symbol Star_Wars_Vector_PCB:LS74
- added M4: LS27, symbol atari_gravitar_black_widow-rescue:LS27-Star_Wars_Vector_PCB
- N5: symbol Star_Wars_Vector_PCB:LS02 -> atari_gravitar_black_widow-rescue:LS02-Star_Wars_Vector_PCB
Connections:
- net AVG12 is gone; now on net AVG11: J9.21 (AVG12)
- net AVG13 is gone; now on net AVG11: J9.22 (AVG13)
- net ST3 is gone; now on net AVG11: A7.8 (~2Q), H7.12 (A3), J9.38 (ST3)
- net 12MHZ: now also A7.11 (2CLK), A7.3 (1CLK)
- net 3MHZ: now also J5.2, K6.6
- net 6MHZ: now also J5.3, K3.11 (2CLK)
- net AVG0: now also N4.5 (A0), R3.4 (Y)
- net AVG1: now also N4.6 (A1), R3.9 (Y)
- net AVG2: now also N4.7 (A2), R3.7 (Y)
- net AVG3: now also N4.4 (A3), R3.12 (Y)
- net AVG4: now also N3.9 (Y), N4.3 (A4)
- net AVG5: now also N3.7 (Y), N4.2 (A5)
- net AVG6: now also N3.4 (Y), N4.1 (A6)
- net AVG7: now also N3.12 (Y), N4.15 (A7)
- net ST2: now also M4.11
- net ~DISRST: now also P4.1 (C)
- net ~VMEM: now also M4.9
- net at A7.2 (1D): now also A7.12 (2D), B7.13
- net at A7.5 (1Q): now also B7.9
- net at A7.6 (~1Q): now also P4.9 (CK)
- new net: B7.10, B7.11
- new net: B7.12, J5.5
- new net: J5.12, J5.13, K5.1, K5.12
- new net: K5.13, K5.2
- new net: K3.9 (2Q), K5.3, M4.10
- new net: K5.11, M4.8
- new net: K3.12 (2D), K6.4
- new net GND: M4.7 (GND)
- new net SACLK: B7.8, J5.1, K6.5
- new net VCC: M4.14 (VCC)
Other:
- note added: "Address Controller"
- note added: "Decoder Disable"
- note added: "Signature Analysis Flag"
- note added: "State Machine"
- note added: "State Machine Clock"
- note added: "State Machine Clock Logic"
- moved on the sheet: A7A, J3F, N3, N4, N5C, P4B, R20, R3, R4E

Commit message: 6A
Op Code and Intensity Latches
Parts:
- added C6, D6: LS175E, symbol star_wars_arcade_main_pcb:LS175E
Connections:
- net DVY12: now also D6.2 (Q0)
- net DVY4: now also C6.4 (D0), D6.4 (D0)
- net DVY5: now also C6.5 (D1), D6.5 (D1)
- net DVY6: now also C6.12 (D2), D6.12 (D2)
- net DVY7: now also C6.13 (D3), D6.13 (D3)
- net OP0: now also D6.7 (Q1)
- net OP1: now also D6.10 (Q2)
- net OP2: now also D6.15 (Q3)
- net ~LATCH1: now also C6.1 (C), D6.9 (CK)
- net ~LATCH3: now also C6.9 (CK)
- net ~OP0: now also D6.6 (~Q1)
- net ~OP2: now also D6.14 (~Q3)
- new net DVX12: C6.2 (Q0)
- new net Z0: C6.15 (Q3), C6.7 (Q1)
- new net Z1: C6.10 (Q2)
- new net ~DVX12: C6.3 (~Q0)
- new net ~DVY12: D6.3 (~Q0)
- new net ~OP1: D6.11 (~Q2)
- new net ~Z1: C6.11 (~Q2)
- new net ~Z2: C6.14 (~Q3)
- no-connect marks 0 -> 1
Other:
- note added: "Op Code and\nIntensity\nLatches"
Changed lines of the file:
@@
 SACLK
 Wire Bus Line
-	24700 20325 24700 21575
-Wire Bus Line
-	24700 24225 25200 24225
-Wire Bus Line
 	27675 24225 27675 20325
-Wire Bus Line
-	27675 20325 24700 20325
 Wire Wire Line
 	24625 21325 24775 21325
@@
 Address Controller
 Wire Bus Line
-	24700 20325 22475 20325
-Wire Bus Line
 	22475 20325 22475 21575
 Wire Bus Line
 	22475 21575 24700 21575
-Connection ~ 24700 20325
-Connection ~ 24700 21575
-Wire Bus Line
-	24700 21575 24700 24000
 Text Notes 22525 20450 0    50   ~ 0
 Signature Analysis Flag
@@
 Wire Bus Line
 	11625 21600 11625 24675
-Wire Bus Line
-	11625 24675 18850 24675
 Wire Bus Line
 	18850 21600 18850 24675
@@
 Wire Bus Line
 	20500 21600 20500 23450
-Wire Bus Line
-	20500 24675 18850 24675
-Connection ~ 18850 21600
-Connection ~ 18850 24675
 Text Notes 18900 21725 0    50   ~ 0
 State Machine Clock
 Wire Bus Line
-	20500 24675 20500 25025
-Wire Bus Line
-	20500 25025 22425 25025
-Wire Bus Line
 	22425 25025 22900 24000
 Wire Bus Line
@@
 Wire Bus Line
 	22900 23450 20500 23450
-Connection ~ 20500 24675
-Connection ~ 20500 23450
-Wire Bus Line
-	20500 23450 20500 24675
 Text Notes 20575 23575 0    50   ~ 0
 Decoder Disable
 Wire Bus Line
-	20500 25025 17500 25025
-Wire Bus Line
 	17500 25025 17500 30425
 Wire Bus Line
@@
 Wire Bus Line
 	25200 30425 25200 24225
-Connection ~ 20500 25025
-Connection ~ 25200 24225
-Wire Bus Line
-	25200 24225 27675 24225
 Wire Bus Line
 	22900 24000 24700 24000
-Connection ~ 22900 24000
-Connection ~ 24700 24000
-Wire Bus Line
-	24700 24000 24700 24225
 Text Notes 17550 25150 0    50   ~ 0
 State Machine
+$Comp
+L star_wars_arcade_main_pcb:LS175E D6
+U 1 1 61A5F2BD
+P 19175 18275
+F 0 "D6" H 19175 18350 50  0000 C CNN
+F 1 "LS175E" H 19175 18250 50  0000 C CNN
+F 2 "" H 19175 18275 50  0001 C CNN
+F 3 "" H 19175 18275 50  0001 C CNN
+	1    19175 18275
+	1    0    0    -1
+$EndComp
+$Comp
+L star_wars_arcade_main_pcb:LS175E C6
+U 1 1 61A60185
+P 19175 20125
+F 0 "C6" H 19175 20150 50  0000 C CNN
+F 1 "LS175E" H 19175 20050 50  0000 C CNN
+F 2 "" H 19175 20125 50  0001 C CNN
+F 3 "" H 19175 20125 50  0001 C CNN
+	1    19175 20125
+	1    0    0    -1
+$EndComp
+Text GLabel 18700 17575 0    50   Input ~ 0
+~LATCH1
+Wire Wire Line
+	19025 17575 18700 17575
+Text GLabel 18700 19425 0    50   Input ~ 0
+~LATCH3
+Text GLabel 18700 20825 0    50   Input ~ 0
+~LATCH1
+Wire Wire Line
+	18700 19425 19025 19425
+Wire Wire Line
+	19025 20825 18700 20825
+Text GLabel 18300 19925 0    50   Input ~ 0
+DVY7
+Text GLabel 18300 20050 0    50   Input ~ 0
+DVY6
+Text GLabel 18300 20175 0    50   Input ~ 0
+DVY5
+Text GLabel 18300 20300 0    50   Input ~ 0
+DVY4
+Text GLabel 20125 18125 2    50   Output ~ 0
+OP1
+Text GLabel 20125 18425 2    33   Output ~ 0
+~OP0
+Text GLabel 20125 17925 2    50   Output ~ 0
+OP2
+Text GLabel 20125 18325 2    50   Output ~ 0
+OP0
+Text GLabel 20125 18025 2    33   Output ~ 0
+~OP2
+Text GLabel 20125 18225 2    33   Output ~ 0
+~OP1
+Text GLabel 20125 18525 2    50   Output ~ 0
+DVY12
+Text GLabel 20125 18625 2    33   Output ~ 0
+~DVY12
+Text GLabel 18300 18075 0    50   Input ~ 0
+DVY7
+Text GLabel 18300 18200 0    50   Input ~ 0
+DVY6
+Text GLabel 18300 18325 0    50   Input ~ 0
+DVY5
+Text GLabel 18300 18450 0    50   Input ~ 0
+DVY4
+Text GLabel 20125 19775 2    50   Output ~ 0
+Z2
+Text GLabel 20125 19975 2    50   Output ~ 0
+Z1
+Text GLabel 20125 20175 2    50   Output ~ 0
+Z0
+Text GLabel 20125 20475 2    33   Output ~ 0
+~DVX12
+Text GLabel 20125 20075 2    33   Output ~ 0
+~Z1
+Text GLabel 20125 19875 2    33   Output ~ 0
+~Z2
+Wire Bus Line
+	24700 24225 27675 24225
+Wire Bus Line
+	11625 24675 20500 24675
+Wire Bus Line
+	20500 23450 20500 25025
+Wire Bus Line
+	17500 25025 22425 25025
+Wire Bus Line
+	22475 20325 27675 20325
+Wire Bus Line
+	24700 20325 24700 24225
+Text Notes 17975 17350 0    50   ~ 0
+Op Code and\nIntensity\nLatches
+Wire Bus Line
+	17925 21000 17925 17050
+Text Label 18750 17575 0    50   Italic 0
+C794
+Wire Wire Line
+	18300 18075 18525 18075
+Wire Wire Line
+	18525 18200 18300 18200
+Wire Wire Line
+	18300 18325 18525 18325
+Wire Wire Line
+	18525 18450 18300 18450
+Wire Wire Line
+	19825 20475 20125 20475
+Wire Wire Line
+	20125 20375 19825 20375
+Wire Wire Line
+	20125 20175 19825 20175
+Wire Wire Line
+	19825 20075 20125 20075
+Wire Wire Line
+	20125 19975 19825 19975
+Wire Wire Line
+	19825 19875 20125 19875
+Wire Wire Line
+	20125 19775 19825 19775
+Wire Wire Line
+	19825 18625 20125 18625
+Wire Wire Line
+	20125 18525 19825 18525
+Wire Wire Line
+	19825 18425 20125 18425
+Wire Wire Line
+	20125 18325 19825 18325
+Wire Wire Line
+	19825 18225 20125 18225
+Wire Wire Line
+	19825 18125 20125 18125
+Wire Wire Line
+	20125 18025 19825 18025
+Wire Wire Line
+	19825 17925 20125 17925
+Text Label 18350 18075 0    50   Italic 0
+3CC1
+Text Label 18350 18200 0    50   Italic 0
+144P
+Text Label 18350 18325 0    50   Italic 0
+2406
+Text Label 18350 18450 0    50   Italic 0
+A88A
+Text Label 19825 17925 0    50   Italic 0
+OOPH
+Text Label 19825 18025 0    50   Italic 0
+8PC9
+Text Label 19825 18125 0    50   Italic 0
+U5C1
+Text Label 19825 18225 0    50   Italic 0
+7CP5
+Text Label 19825 18325 0    50   Italic 0
+6UUF
+Text Label 19825 18425 0    50   Italic 0
+PIA8
+Text Label 19825 18525 0    50   Italic 0
+4347
+Text Label 19825 18625 0    50   Italic 0
+FH13
+Text Label 19825 19775 0    50   Italic 0
+0482
+Text Label 19825 19875 0    50   Italic 0
+8AH6
+Text Label 19825 19975 0    50   Italic 0
+50H7
+Text Label 19825 20075 0    50   Italic 0
+HP83
+Text Label 19825 20175 0    50   Italic 0
+0482
+NoConn ~ 19825 20275
+Text Label 19825 20375 0    50   Italic 0
+CC14
+Text Label 19825 20475 0    50   Italic 0
+3540
+Wire Wire Line
+	18300 19925 18525 19925
+Wire Wire Line
+	18525 20050 18300 20050
+Wire Wire Line
+	18300 20175 18525 20175
+Wire Wire Line
+	18525 20300 18300 20300
+Text Label 18350 19925 0    50   Italic 0
+3CC1
+Text Label 18350 20050 0    50   Italic 0
+144P
+Text Label 18350 20175 0    50   Italic 0
+2406
+Text Label 18350 20300 0    50   Italic 0
+A88A
+Text Label 18750 19425 0    50   Italic 0
+1C91
+Text Label 18750 20825 0    50   Italic 0
+C794
+Wire Bus Line
+	17925 21000 20500 21000
+Wire Bus Line
+	17925 17050 20500 17050
+Wire Bus Line
+	20500 17050 20500 21000
+Text GLabel 20125 20375 2    50   Output ~ 0
+DVX12
 $EndSCHEMATC

Commit message: Vector Data shifters
Parts:
- added A8, B8, C8, F8, H8, J8: LS194, symbol Star_Wars_Vector_PCB:LS194
- added E7: LS00, symbol Star_Wars_Vector_PCB:LS00
- added F7: LS14, symbol Star_Wars_Vector_PCB:LS14
Connections:
- net 12MHZ: now also A8.11 (CK), B8.11 (CK), C8.11 (CK), F8.11 (CK), H8.11 (CK), J8.11 (CK)
- net DVY0: now also F8.12 (QD)
- net DVY1: now also F8.13 (QC)
- net DVY10: now also H8.14 (QB)
- net DVY11: now also H8.15 (QA)
- net DVY2: now also F8.14 (QB)
- net DVY3: now also F8.15 (QA), J8.7 (L)
- net DVY4: now also J8.12 (QD); no longer C6.4 (D0), D6.4 (D0)
- net DVY5: now also J8.13 (QC); no longer C6.5 (D1), D6.5 (D1)
- net DVY6: now also J8.14 (QB); no longer C6.12 (D2), D6.12 (D2)
- net DVY7: now also H8.7 (L), J8.15 (QA); no longer C6.13 (D3), D6.13 (D3)
- net DVY8: now also H8.12 (QD)
- net DVY9: now also H8.13 (QC)
- net ~LATCH0: now also E7.2, F7.13
- net ~LATCH1: now also A8.1 (C), B8.1 (C), C8.1 (C), E7.4, F7.1, F8.1 (C), H8.1 (C), J8.1 (C)
- net ~LATCH2: now also E7.12, F7.11
- net ~LATCH3: now also E7.9, F7.9
- new net: B8.10 (S1), E7.8
- new net: A8.2 (R), B8.2 (R), C8.2 (R), F8.2 (R), H8.2 (R), J8.2 (R)
- new net: B8.9 (S0), F7.8
- new net: A8.10 (S1), C8.10 (S1), E7.11
- new net: A8.9 (S0), C8.9 (S0), F7.10
- new net: E7.6, H8.10 (S1)
- new net: F7.2, H8.9 (S0)
- new net: E7.3, F8.10 (S1), J8.10 (S1)
- new net: F7.12, F8.9 (S0), J8.9 (S0)
- new net DVG0: A8.6 (D), B8.6 (D), F8.6 (D), H8.6 (D)
- new net DVG1: A8.5 (C), B8.5 (C), F8.5 (C), H8.5 (C)
- new net DVG2: A8.4 (B), B8.4 (B), F8.4 (B), H8.4 (B)
- new net DVG3: A8.3 (A), B8.3 (A), F8.3 (A), H8.3 (A)
- new net DVG4: C6.4 (D0), C8.6 (D), D6.4 (D0), J8.6 (D)
- new net DVG5: C6.5 (D1), C8.5 (C), D6.5 (D1), J8.5 (C)
- new net DVG6: C6.12 (D2), C8.4 (B), D6.12 (D2), J8.4 (B)
- new net DVG7: C6.13 (D3), C8.3 (A), D6.13 (D3), J8.3 (A)
- new net DVX10: B8.14 (QB)
- new net DVX11: B8.15 (QA)
- new net DVX3: A8.15 (QA), C8.14 (QB), C8.7 (L)
- new net DVX4: C8.12 (QD), C8.13 (QC)
- new net DVX7: B8.7 (L), C8.15 (QA)
- new net DVX8: B8.12 (QD)
- new net DVX9: B8.13 (QC)
- new net ~ENORM: E7.1, E7.10, E7.13, E7.5

Commit message: too much information
added wrong (!) imports from Q, Ast, and SW
WIll need to be altered to match Grav
Parts:
- added +12V1, +5V1, +5V2, -15V1, 12MHZ1, 6MHZ1, BLUE1, GND1, GND2, GND3, GND4, GREEN1, RED1, SACLK1, SAEN1, VCTR1, ZREF1, ~SA1, ~VMEM1, ~VROM1: TP, Star_Wars_Vector_PCB:TEST_POINT, symbol Star_Wars_Vector_PCB:TP
- added +15V1: TP1, Star_Wars_Vector_PCB:TEST_POINT, symbol Star_Wars_Vector_PCB:TP
- added A_1, H_2, K_4: LS08, Star_Wars_Vector_PCB:DIP14, symbol Star_Wars_Vector_PCB:LS08
- added A_10, D/E_11, D/E_12, D_10, F_9: 082, Star_Wars_Vector_PCB:DIP8, symbol Star_Wars_Vector_PCB:082
- added A_2: LS20, Star_Wars_Vector_PCB:DIP14, symbol Star_Wars_Vector_PCB:LS20
- added A_3, P_4: LS00, Star_Wars_Vector_PCB:DIP14, symbol Star_Wars_Vector_PCB:LS00
- added A_6: RESET, Asteroids:RST, symbol Asteroids_PCB-rescue:SW_Push
- added B_1, B_2, C_1, D_1, L_5, M_5, M_6, M_7, R_6: LS161, Star_Wars_Vector_PCB:DIP16, symbol Star_Wars_Vector_PCB:LS161
- added B_1: 137290, Star_Wars_Vector_PCB:DIP20, symbol quantum_arcade_pcb:137290
- added B_10, B_7, E_10, E_7: LF13201, Star_Wars_Vector_PCB:DIP16, symbol Star_Wars_Vector_PCB:LF13201
- added B_11, B_12: MC1495LB, Star_Wars_Vector_PCB:DIP14, symbol quantum_arcade_pcb:MC1495LB
- added B_2, C_2: LS244, Asteroids:DIP20, symbol Asteroids:LS244
- added B_2/3, D_2/3: POKEY, Star_Wars_Vector_PCB:DDIP40, symbol quantum_arcade_pcb:POKEY
- added B_4, D_5: LS393, Asteroids:DIP14, symbol Asteroids:LS393
- added B_5: LS04, Asteroids:DIP14, symbol Asteroids:LS04
- added B_6: LS14, Asteroids:DIP14, symbol Asteroids:LS14
- added B_9, F/H_9: AM6012, Star_Wars_Vector_PCB:DIP20, symbol Star_Wars_Vector_PCB:AM6012
- added C1, C10, C11, C111, C112, C12, C13, C14, C15, C16, C17, C18, C2, C20, C21, C22, C23, C26, C28, C29, C3, C30, C31, C4, C41, C42, C43, C44, C49, C5, C52, C53, C57, C6, C60, C61, C66, C7, C8, C84, C85, C9, C91, C94: .1uF, Asteroids:GenericC, symbol Device:C
- added C1, C12, C17, C18, C35, C36, C39, C40, C50, C51, C52, C53, C54, C55, C56, C57, C58, C59, C6, C60, C61, C62, C63, C64, C65, C67, C68, C69, C7, C70, C71, C72, C73, C74, C75, C76, C77, C78, C79, C80, C82: .1uF, Star_Wars_Vector_PCB:GenericComp, symbol Device:C
- added C10, C11, C14, C15, C16, C17, C18, C19, C2, C20, C26, C27, C28, C3, C31, C33, C34, C35, C36, C39, C40, C9: .1uF, quantum_arcade_pcb:GenComp, symbol Device:C
- added C100, C101, C102, C103, C104, C105, C106, C107, C108, C109, C110, C111, C112, C113, C114, C115, C116, C117, C118, C119, C120, C121, C122, C123, C124, C125, C126, C127, C128, C129, C49, C64, C65, C67, C68, C69, C70, C71, C72, C73, C75, C78, C79, C81, C91, C92, C93, C94, C95, C96, C97, C98, C99: .1uf, quantum_arcade_pcb:GenComp, symbol Device:C
- added C117: 22uF, Asteroids:Electrolytic4, symbol Device:C
- added C12, C29: 39pf, quantum_arcade_pcb:CapSmall, symbol Device:C
- added C13, C30, C32: 100pf, quantum_arcade_pcb:CapSmall, symbol Device:C
- added C130: .047uf, quantum_arcade_pcb:GenComp, symbol Device:C
- added C19: 100uF, Asteroids:Electrolytic1, symbol Device:C
- added C21: .0018uF, quantum_arcade_pcb:CapSmall, symbol Device:C
- added C25, C70, C90, C92, C93: 1uF, Asteroids:Electrolytic2C, symbol Device:C
- added C25, C8: .047uF, quantum_arcade_pcb:CapInt, symbol Device:C
- added C37, C47, C66: 150pF, Star_Wars_Vector_PCB:CapBrown, symbol Device:C
- added C37: 150pF, quantum_arcade_pcb:CapSmall, symbol Device:C
- added C38: 39pF, Star_Wars_Vector_PCB:CapBrown, symbol Device:C
- added C38: 39pF, quantum_arcade_pcb:CapSmall, symbol Device:C
- added C4: .01uF, quantum_arcade_pcb:CapSmall, symbol Device:C
- added C41, C5: .01uF, Star_Wars_Vector_PCB:GenericComp, symbol Device:C
- added C41: .01uF, quantum_arcade_pcb:GenComp, symbol Device:C
- added C42: 10pF, Star_Wars_Vector_PCB:CapBrown, symbol Device:C
- added C42: 10pF, quantum_arcade_pcb:CapSmall, symbol Device:C
- added C43, C44, C46, C81: 100uF, Star_Wars_Vector_PCB:LargeCap, symbol Device:CP1
- added C44, C46: 100uf 35V, quantum_arcade_pcb:Cap2, symbol Device:CP1_Small
- added C45, C48: 22uF, Star_Wars_Vector_PCB:CapElec2, symbol Device:CP1
- added C45, C48: 22uf 25V, quantum_arcade_pcb:Cap1, symbol Device:CP1_Small
- added C47: 22uf 35V, quantum_arcade_pcb:Cap3, symbol Device:CP1_Small
- added C74: 1uf, quantum_arcade_pcb:Cap1, symbol Device:CP1_Small
- added C76: 100pf 100V, quantum_arcade_pcb:CapSmall, symbol Device:C
- added C77: 39pf 100V, quantum_arcade_pcb:CapSmall, symbol Device:C
- added C80: .022uf, quantum_arcade_pcb:GenComp, symbol Device:C
- added C82: 100uf 25V, quantum_arcade_pcb:Cap2, symbol Device:CP1_Small
- added C83: 22pF, Star_Wars_Vector_PCB:CapBrown, symbol Device:C
- added C86, C87: 470uF, Asteroids:Electrolytic3, symbol Device:C
- added CR1: 1N914, Asteroids:Diode1, symbol Device:D
- added CR1: 1N914, Star_Wars_Vector_PCB:GenericComp, symbol Device:D
- added CR1: 1N914, quantum_arcade_pcb:Diode, symbol Device:D
- added CR10, CR11, CR12, CR9: 1N4001, Asteroids:GenericD, symbol Device:D
- added CR13, CR14: 1N756A, Asteroids:GenericR, symbol Device:D_Zener
- added CR2: LED, Star_Wars_Vector_PCB:LED, symbol Device:LED
- added CR3, CR4: 1N100, Star_Wars_Vector_PCB:GenericComp, symbol Device:D
- added CR3, CR4, CR6: 1N100, quantum_arcade_pcb:Diode, symbol Device:D
- added CR5: LED, Asteroids:LED, symbol Device:LED
- added CR5: 1N754A, quantum_arcade_pcb:Diode, symbol Device:D_Zener
- added CR7: LED, quantum_arcade_pcb:LED, symbol quantum_arcade_pcb:LED
- added C_11, C_12: MC1495LA, Star_Wars_Vector_PCB:DIP14, symbol quantum_arcade_pcb:MC1495LA
- added C_3: 6502A, Asteroids:6502A, symbol Asteroids:6502A
- added C_4: 9316, Asteroids:DIP16, symbol Asteroids:9316
- added C_5: LS161, Asteroids:DIP16, symbol Asteroids:LS161
- added C_6: LS00, Asteroids:DIP14, symbol Asteroids:LS00
- added D_1, H/J_4: LS138, Star_Wars_Vector_PCB:DIP16, symbol quantum_arcade_pcb:LS138
- added D_4: LS74, Asteroids:DIP14, symbol Asteroids:LS74
- added D_6, D_9: DAC_8, Star_Wars_Vector_PCB:DIP16, symbol Star_Wars_Vector_PCB:DAC_8
- added D_8: LS273, Star_Wars_Vector_PCB:DIP20, symbol quantum_arcade_pcb:LS273
- added E_1, E_3, H_3, J_4, M_8: LS02, Star_Wars_Vector_PCB:DIP14, symbol Star_Wars_Vector_PCB:LS02
- added E_2, F_5, J_5, K_7: LS32, Star_Wars_Vector_PCB:DIP14, symbol Star_Wars_Vector_PCB:LS32
- added E_3: LS245, Asteroids:DIP20, symbol Asteroids:LS245
- added E_5: LS273A, Star_Wars_Vector_PCB:DIP20, symbol Star_Wars_Vector_PCB:LS273A
- added E_6: LS08, Asteroids:DIP14, symbol Asteroids:LS08
- added F/H_4, J_10, K_6, P_5: LS04, Star_Wars_Vector_PCB:DIP14, symbol Star_Wars_Vector_PCB:LS04
- added F_1: LS27, Star_Wars_Vector_PCB:DIP14, symbol Star_Wars_Vector_PCB:LS27
- added F_2, K_9: LS109, Star_Wars_Vector_PCB:DIP16, symbol Star_Wars_Vector_PCB:LS109
- added F_3, L_7: S260, Star_Wars_Vector_PCB:DIP14, symbol Star_Wars_Vector_PCB:S260
- added F_4: LS86, Star_Wars_Vector_PCB:DIP14, symbol Star_Wars_Vector_PCB:LS86
- added F_6: LS273B, Star_Wars_Vector_PCB:DIP20, symbol Star_Wars_Vector_PCB:LS273B
- added F_8: DAC_8A, Star_Wars_Vector_PCB:DIP16, symbol Star_Wars_Vector_PCB:DAC_8A
- added J17: Main_Connector, Star_Wars_Vector_PCB:J17, symbol Star_Wars_Vector_PCB:Main_Connector
- added J20: Edge_Connector_30_Pin, Star_Wars_Vector_PCB:J20, symbol Star_Wars_Vector_PCB:Edge_Connector_30_Pin
- added J20: J20, quantum_arcade_pcb:EdgeCon, symbol quantum_arcade_pcb:J20
- added J_6: LS10, Star_Wars_Vector_PCB:DIP14, symbol Star_Wars_Vector_PCB:LS10
- added K_1: LS245, Star_Wars_Vector_PCB:DIP20, symbol Star_Wars_Vector_PCB:LS245
- added K_10: S86, Star_Wars_Vector_PCB:DIP14, symbol Star_Wars_Vector_PCB:LS86
- added K_2: LS42, Star_Wars_Vector_PCB:DIP16, symbol Star_Wars_Vector_PCB:LS42
- added K_5, L_4: LS74, Star_Wars_Vector_PCB:DIP14, symbol Star_Wars_Vector_PCB:LS74
- added L1, L2, L3: 1uH, Star_Wars_Vector_PCB:Inductor1, symbol Device:L
- added L1: 100uH, quantum_arcade_pcb:Ind, symbol Device:L
- added L_1: 2732_A, Star_Wars_Vector_PCB:DDIP24, symbol Star_Wars_Vector_PCB:2732_A
- added L_3: 137211-001, Star_Wars_Vector_PCB:DDIP24, symbol Star_Wars_Vector_PCB:137211-001
- added L_5: LS175C, Star_Wars_Vector_PCB:DIP16, symbol Star_Wars_Vector_PCB:LS175C
- added L_6: LS175B, Star_Wars_Vector_PCB:DIP16, symbol Star_Wars_Vector_PCB:LS175B
- added L_8: 74LS07, Star_Wars_Vector_PCB:DIP14, symbol Star_Wars_Vector_PCB-rescue:74LS07
- added L_8: S02, Star_Wars_Vector_PCB:DIP14, symbol Star_Wars_Vector_PCB:LS02
- added L_9: LS175, Star_Wars_Vector_PCB:DIP16, symbol quantum_arcade_pcb:LS175
- added M/N_12: TL082, Star_Wars_Vector_PCB:DIP8, symbol Amplifier_Operational:TL082
- added M_1, M_2: LS244_B, Star_Wars_Vector_PCB:DIP20, symbol Star_Wars_Vector_PCB:LS244_B
- added M_4: 06, Star_Wars_Vector_PCB:DIP14, symbol Asteroids:LS06
- added M_5: LS175_A, Star_Wars_Vector_PCB:DIP16, symbol Star_Wars_Vector_PCB:LS175_A
- added M_6: LS191A, Star_Wars_Vector_PCB:DIP16, symbol Star_Wars_Vector_PCB:LS191A
- added M_9: LS244C, Star_Wars_Vector_PCB:DIP20, symbol quantum_arcade_pcb:LS244C
- added N_1: LS244_A, Star_Wars_Vector_PCB:DIP20, symbol Star_Wars_Vector_PCB:LS244_A
- added N_2: LS244_C, Star_Wars_Vector_PCB:DIP20, symbol Star_Wars_Vector_PCB:LS244_C
- added N_3: 2KX8_RAM, Star_Wars_Vector_PCB:DDIP24, symbol quantum_arcade_pcb:2KX8_RAM
- added N_4: S32, Star_Wars_Vector_PCB:DIP14, symbol Star_Wars_Vector_PCB:LS32
- added N_5: LS273B, Star_Wars_Vector_PCB:DIP20, symbol quantum_arcade_pcb:LS273B
- added N_8: LS164, Star_Wars_Vector_PCB:DIP14, symbol Star_Wars_Vector_PCB:LS164
- added PD1, PD2, PD3, PD4: Split_Pad, Asteroids:SP, symbol Asteroids:Split_Pad
- added P_1: LS244, Star_Wars_Vector_PCB:DIP20, symbol Star_Wars_Vector_PCB:LS244
- added P_7: LS163, Star_Wars_Vector_PCB:DIP16, symbol quantum_arcade_pcb:LS163
- added P_8: S04, Star_Wars_Vector_PCB:DIP14, symbol Star_Wars_Vector_PCB:LS04
- added Q1, Q4, Q5, Q6, Q7: 2N3904, Star_Wars_Vector_PCB:GenericTrans, symbol Star_Wars_Vector_PCB-rescue:2N3904
- added Q15, Q16: 2N6044, quantum_arcade_pcb:BigTrans, symbol Device:Q_NPN_BCE
- added Q17: 2N3904, quantum_arcade_pcb:GenTrans, symbol Transistor_BJT:2N3904
- added Q7: 2N3904, quantum_arcade_pcb:GenTrans, symbol Star_Wars_Vector_PCB-rescue:2N3904
- added Q8: 2N3906, Star_Wars_Vector_PCB:GenericTrans, symbol Star_Wars_Vector_PCB-rescue:2N3906
- added Q8: 2N3906, quantum_arcade_pcb:GenTrans, symbol Star_Wars_Vector_PCB-rescue:2N3906
- added R1, R10, R117, R2, R3, R5, R6, R7, R8, R83, R9: 10K, Star_Wars_Vector_PCB:GenericComp, symbol Device:R
- added R10, R11, R12, R13, R14, R15, R16, R17, R18, R28, R33, R9: 10K, Asteroids:GenericR, symbol Device:R
- added R100, R101, R102, R103, R104, R105, R15, R98, R99: 100K, Star_Wars_Vector_PCB:GenericComp, symbol Device:R
- added R106, R30, R31, R58, R85, R86, R89, R93, R95, R96: 7.5K, quantum_arcade_pcb:GenComp, symbol Device:R
- added R107: 150, Star_Wars_Vector_PCB:GenericComp, symbol Device:R
- added R108: 270, quantum_arcade_pcb:CapInt, symbol Device:R_US
- added R109, R110, R111, R82: 1K, Star_Wars_Vector_PCB:GenericComp, symbol Device:R
- added R11, R16: 12K, Star_Wars_Vector_PCB:GenericComp, symbol Device:R
- added R112, R113: 270, Asteroids:GenericR, symbol Device:R
- added R114, R115, R116, R90, R94: 100, Star_Wars_Vector_PCB:GenericComp, symbol Device:R
- added R12: 24K, Star_Wars_Vector_PCB:GenericComp, symbol Device:R
- added R13: 47K, Star_Wars_Vector_PCB:GenericComp, symbol Device:R
- added R14: 820, Star_Wars_Vector_PCB:GenericComp, symbol Device:R
- added R149, R151, R152, R160, R161, R162: 470, quantum_arcade_pcb:GenComp, symbol Device:R_US
- added R153, R155, R156, R157, R158, R159, R166, R167, R168, R169, R176, R205, R210, R214, R218, R219, R220, R221, R222: 1k, quantum_arcade_pcb:GenComp, symbol Device:R_US
- added R163, R173, R177, R178, R215: 10k, quantum_arcade_pcb:GenComp, symbol Device:R_US
- added R164, R165, R179, R223: 220, quantum_arcade_pcb:GenComp, symbol Device:R_US
- added R17: 6.2K, Star_Wars_Vector_PCB:GenericComp, symbol Device:R
- added R174: 68k, quantum_arcade_pcb:GenComp, symbol Device:R_US
- added R175: 15k, quantum_arcade_pcb:GenComp, symbol Device:R_US
- added R180, R181, R182, R183, R184, R185, R186, R187: 100K, quantum_arcade_pcb:GenComp, symbol Device:R
- added R188, R189, R190, R191, R192, R193, R194, R195, R196, R197, R198, R199, R200, R201, R202, R203: 4.7k, quantum_arcade_pcb:GenComp, symbol Device:R_US
- added R20, R21, R22: 470, Star_Wars_Vector_PCB:GenericComp, symbol Device:R
- added R204, R206, R207, R208, R209, R211, R212, R213: 220k, quantum_arcade_pcb:GenComp, symbol Device:R_US
- added R23, R24, R25: 4.7k, Star_Wars_Vector_PCB:GenericComp, symbol Device:R
- added R26, R27, R55: 820, quantum_arcade_pcb:GenComp, symbol Device:R
- added R27, R29: 1K, Asteroids:GenericR, symbol Device:R
- added R30, R31: 330, Asteroids:GenericR, symbol Device:R
- added R32: 470, Asteroids:GenericR, symbol Device:R
- added R32, R33, R38, R51, R59, R62, R63: 470, quantum_arcade_pcb:GenComp, symbol Device:R
- added R34, R60: 2.7k, quantum_arcade_pcb:GenComp, symbol Device:R
- added R35, R54, R61: 680, quantum_arcade_pcb:GenComp, symbol Device:R
- added R36, R44, R45, R50, R64, R69, R70, R77: 2.2k, quantum_arcade_pcb:GenComp, symbol Device:R
- added R37, R39, R52, R65, R66, R78, R79: 3.9k, quantum_arcade_pcb:GenComp, symbol Device:R
- added unit 1 of R4
- added R40, R46, R67, R73: 10k, quantum_arcade_pcb:GenComp, symbol Device:R
- added R41, R71: 5.6k, quantum_arcade_pcb:GenComp, symbol Device:R
- added R42, R43, R68, R72: 10k, Star_Wars_Vector_PCB:PotBlk, symbol Star_Wars_Vector_PCB-rescue:POT
- added R47, R74: 2K, Star_Wars_Vector_PCB:PotBlk, symbol Star_Wars_Vector_PCB-rescue:POT
- added R48, R75: 100k, quantum_arcade_pcb:GenComp, symbol Device:R
- added R49: 1.5k, quantum_arcade_pcb:GenComp, symbol Device:R
- added R53, R80: 1k, quantum_arcade_pcb:GenComp, symbol Device:R
- added R55: 150, Asteroids:GenericR, symbol Device:R
- added R75, R76: 1.30K, Star_Wars_Vector_PCB:GenericComp, symbol Device:R
- added R76: 1.2k, quantum_arcade_pcb:GenComp, symbol Device:R
- added R81: 15K, Star_Wars_Vector_PCB:GenericComp, symbol Device:R
- added R81: 15K, quantum_arcade_pcb:GenComp, symbol Device:R
- added R82: 1K, quantum_arcade_pcb:GenComp, symbol Device:R
- added R83: 10K, quantum_arcade_pcb:GenComp, symbol Device:R
- added R84: 560, Star_Wars_Vector_PCB:GenericComp, symbol Device:R
- added R84: 560, quantum_arcade_pcb:GenComp, symbol Device:R
- added R85, R86, R89, R93, R95, R96: 7.5K, Star_Wars_Vector_PCB:GenericComp, symbol Device:R
- added R87, R91: 6.19K, Star_Wars_Vector_PCB:GenericComp, symbol Device:R
- added R87, R91: 7.5k, quantum_arcade_pcb:GenComp, symbol Device:R
- added R88 (x2), R92 (x2): 200, Star_Wars_Vector_PCB:PotBlk, symbol Star_Wars_Vector_PCB-rescue:POT
- added R90, R94: 100, quantum_arcade_pcb:GenComp, symbol Device:R
- added R97: 3.9K, Star_Wars_Vector_PCB:GenericComp, symbol Device:R
- added R97: 3.9K, quantum_arcade_pcb:GenComp, symbol Device:R
- added RV1, RV2: VDR, quantum_arcade_pcb:GenComp, symbol Device:Varistor
- added R_4, R_5: LS393, Star_Wars_Vector_PCB:DIP14, symbol Asteroids:LS393
- added SW1, SW2: SW_DIP_x08, Star_Wars_Vector_PCB:DIP16, symbol Switch:SW_DIP_x08
- added TP+15V1, TP-15V1, TP12M1, TP5V1, TP5V2, TP6.8V1, TPAUD1, TPAUD2, TPGND1, TPGND2, TPGND3, TPRESET1, TPRESET2, TPWDDIS1, TPXOUT1, TPYOUT1: TP, quantum_arcade_pcb:TP, symbol Star_Wars_Vector_PCB:TP
- added TP1: WDOG_DISABLE, Asteroids:TEST_POINT, symbol Asteroids:AST_TEST
- added TP2: O2, Asteroids:TEST_POINT, symbol Asteroids:AST_TEST
- added TP3: R/W, Asteroids:TEST_POINT, symbol Asteroids:AST_TEST
- added TP4: 6MHz, Asteroids:TEST_POINT, symbol Asteroids:AST_TEST
- added TP5: +5V, Asteroids:TEST_POINT, symbol Asteroids:AST_TEST
- added TP6, TP7: GND, Asteroids:TEST_POINT, symbol Asteroids:AST_TEST
- added U7805: L7805, Asteroids:Volt_Reg, symbol Asteroids_PCB-rescue:L7805
- added U7812: L7812, Asteroids:2N6044, symbol Asteroids_PCB-rescue:L7812
- added U7815: L7815, Asteroids:Volt_Reg, symbol Asteroids_PCB-rescue:L7815
- added U7915: L7915, Asteroids:Volt_Reg, symbol Asteroids_PCB-rescue:L7915
- added VR1: L7815_, Star_Wars_Vector_PCB:VoltReg, symbol Star_Wars_Vector_PCB:L7815_
- added VR1: L7815_, quantum_arcade_pcb:BigTrans, symbol Star_Wars_Vector_PCB:L7815_
- added VR2: L7915_, Star_Wars_Vector_PCB:VoltReg, symbol Star_Wars_Vector_PCB:L7915_
- added VR2: L7915_, quantum_arcade_pcb:BigTrans, symbol Star_Wars_Vector_PCB:L7915_
- added Y1: 12.096MHz, Asteroids:RST, symbol Device:Crystal
- added Y1: 12.096MHz, quantum_arcade_pcb:Crystal, symbol Device:Crystal
Connections:
- net 12MHZ: now also 12MHZ1.1, 12MHZ1.2, B_1.2 (CLK), B_2.2 (CLK), C_1.2 (CLK), D_1.2 (CLK), F_2.12 (Cp), F_2.4 (Cp), M_6.14 (CK), P_1.14 (O2a)
- net 3MHZ: now also N_8.8 (CLK), P_1.9 (O0b)
- net AM0: now also L_1.8 (A0), L_3.8 (A0), M_1.14 (O2a), M_2.14 (O2a)
- net AM1: now also L_1.7 (A1), L_3.7 (A1), M_1.5 (O2b), M_2.5 (O2b)
- net AM2: now also L_1.6 (A2), L_3.6 (A2), M_1.7 (O1b), M_2.7 (O1b)
- net AM3: now also L_1.5 (A3), L_3.5 (A3), M_1.9 (O0b), M_2.9 (O0b)
- net AM4: now also L_1.4 (A4), L_3.4 (A4), M_1.12 (O3a), M_2.12 (O3a)
- net AM5: now also L_1.3 (A5), L_3.3 (A5), M_1.3 (O3b), M_2.3 (O3b)
- net AM6: now also L_1.2 (A6), L_3.2 (A6), M_1.16 (O1a), M_2.16 (O1a)
- net AM7: now also L_1.1 (A7), L_3.1 (A7), M_1.18 (O0a), M_2.18 (O0a)
- net AVG0: now also P_5.9
- net AVG1: now also M_2.15 (I2b)
- net AVG10: now also N_2.13 (I1b)
- net AVG11: now also N_2.11 (I0b), N_2.6 (I2a), N_2.8 (I3a)
- net AVG2: now also M_2.13 (I1b)
- net AVG3: now also M_2.11 (I0b)
- net AVG4: now also M_2.8 (I3a)
- net AVG5: now also M_2.17 (I3b)
- net AVG6: now also M_2.4 (I1a)
- net AVG7: now also M_2.2 (I0a)
- net AVG8: now also N_2.17 (I3b)
- net AVG9: now also N_2.15 (I2b)
- net DVG0: now also K_1.9 (A7), L_1.9 (D0), L_3.9 (D0), R2.2
- net DVG1: now also K_1.8 (A6), L_1.10 (D1), L_3.10 (D1), R9.2
- net DVG2: now also K_1.7 (A5), L_1.11 (D2), L_3.11 (D2), R8.2
- net DVG3: now also K_1.6 (A4), L_1.13 (D3), L_3.13 (D3), R7.2
- net DVG4: now also K_1.5 (A3), L_1.14 (D4), L_3.14 (D4), R6.2
- net DVG5: now also K_1.4 (A2), L_1.15 (D5), L_3.15 (D5), R5.2
- net DVG6: now also K_1.3 (A1), L_1.16 (D6), L_3.16 (D6), R4.2
- net DVG7: now also K_1.2 (A0), L_1.17 (D7), L_3.17 (D7), R3.2
- net DVX10: now also B_9.3 (B3), K_10.9
- net DVX11: now also F_4.10, K_10.10
- net DVX12: now also F_4.9
- net DVX3: now also B_9.10 (B10), B_9.7 (B7)
- net DVX4: now also B_9.8 (B8), B_9.9 (B9)
- net DVX7: now also B_9.6 (B6)
- net DVX8: now also B_9.5 (B5)
- net DVX9: now also B_9.4 (B4)
- net DVY0: now also D_8.14 (D5), E_5.7 (D2), F_6.13 (D4)
- net DVY1: now also D_8.13 (D4), E_5.4 (D1), F_6.14 (D5)
- net DVY10: now also F/H_9.3 (B3), K_10.5, L_5.5 (D1), L_6.12 (D2), L_6.5 (D1), L_9.4 (D0), L_9.5 (D1)
- net DVY11: now also F_4.2, K_10.4, L_5.4 (D0)
- net DVY12: now also F_4.1, J_5.2
- net VCC renamed +5V
- new net: B_5.6, C_3.6 (NMI_), C_5.9 (LD)
- new net: CR5.2 (A), R55.2
- new net: C86.1, CR10.2 (A), CR9.2 (A), U7915.2 (VI)
- new net: B_4.1 (1CK), C_4.11 (QD)
- new net: B_5.8, C_4.2 (CK)
- new net: B_5.12, B_5.9, R30.2, Y1.1
- new net: B_5.11, R31.2, Y1.2
- new net: B_5.13, C18.2, R30.1, R32.1
- new net: B_5.10, C18.1, R31.1
- new net: B_4.13 (2CK), B_4.6 (1QD)
- new net: A_6.2, B_6.13, C25.1, CR1.2 (A), R33.2
- new net: B_6.11, B_6.12
- new net: B_6.10, C_6.5, D_4.10 (~1PRE_)
- new net: C_6.6, D_5.12 (2CLR), D_5.2 (1CLR)
- new net: D_5.13 (2CK), D_5.6 (1QD)
- new net: D_4.11 (2CLK), D_5.8 (2QD)
- new net: E_6.10, R28.2, TP1.1, TP1.2
- new net: D_4.12 (2D), E_6.8
- new net: B_5.5, C_5.15 (RCO)
- new net: B_2.19 (OEb), PD2.2, R18.2
- new net: C_2.19 (OEb), PD3.2, R17.2
- new net: CR2.2 (A), R107.2
- new net: H_2.4, K_2.7 (6)
- new net: H_2.5, K_2.9 (7)
- new net: N_1.14 (O2a), P_5.3, R1.2
- new net: A_3.1, P_5.4
- new net: M_2.6 (I2a), P_5.8
- new net: F_3.5, J_6.10, K_5.13 (~1CLR)
- new net: F_3.2, F_4.8
- new net: F_1.12, F_2.14 (J)
- new net: E_2.3, F_1.13, H_3.8
- new net: F_2.2 (J), H_3.10
- new net: F_2.7 (~Q), H_2.12
- new net: E_3.13, E_3.3, P_5.13
- new net: M_6.11 (LD), P_5.12
- new net: E_3.2, M_6.12 (M/M), M_6.4 (G)
- new net: J_5.1, J_5.12, J_5.8
- new net: B_1.9 (LD), B_2.9 (LD), C_1.9 (LD), D_1.9 (LD), H_3.13
- new net: A_3.5, E_1.1
- new net: A_3.6, C_1.6 (D)
- new net: A_2.6, A_3.10
- new net: A_2.13, A_3.8
- new net: A_2.10, C_1.15 (RCO), C_2.10
- new net: L_8.11, L_8.13, L_8.3, M_8.10
- new net: L_8.2, L_8.4, Q4.2 (B), R23.2
- new net: L_5.15 (Q3), L_8.5
- new net: L_8.10, L_8.6, Q5.2 (B), R24.2
- new net: L_8.12, L_8.8, Q6.2 (B), R25.2
- new net: L_5.10 (Q2), L_8.9
- new net: L1.2, Q4.1 (E), R20.2, RED1.1, RED1.2
- new net: GREEN1.1, GREEN1.2, L2.2, Q5.1 (E), R21.2
- new net: BLUE1.1, BLUE1.2, L3.2, Q6.1 (E), R22.2
- new net: Q1.2 (B), R117.2
- new net: L_5.2 (Q0), R117.1
- new net: L1.1, R114.1
- new net: L2.1, R115.1
- new net: L3.1, R116.1
- new net: D_6.5 (B1), E_5.15 (Q5), R98.1
- new net: D_6.6 (B2), E_5.16 (Q6), R99.1
- new net: D_6.7 (B3), E_5.19 (Q7), R100.1
- new net: D_6.8 (B4), E_5.9 (Q3), R101.1
- new net: D_6.9 (B5), E_5.12 (Q4), R102.2
- new net: D_6.10 (B6), E_5.2 (Q0), R103.2
- new net: D_6.11 (B7), E_5.5 (Q1), R104.2
- new net: D_6.12 (B8), E_5.6 (Q2), R105.2
- new net: C41.2, D_6.16 (C)
- new net: D_6.15 (VR-), R97.2
- new net: D_6.14 (VR+), R95.2, R96.2
- new net: C37.1, Q7.2 (B), R81.1 (x2)
- new net: C38.2, Q7.3 (C), R82.1, R83.2 (x2)
- new net: C38.1, Q8.2 (B), R83.1 (x2)
- new net: Q8.3 (C), R84.2, R85.2, R86.2 (x2)
- new net: C42.2, CR1.1 (K), D_6.4 (IO), R85.1, R86.1, R87.2, R89.2, R91.2, R93.2
- new net: C47.2, R75.2, R87.1
- new net: R75.1, R88.3
- new net: R89.1, R90.2 (x2)
- new net: C66.2, R76.2, R91.1
- new net: R76.1, R92.3
- new net: R93.1, R94.2 (x2)
- new net: 6MHZ1.1, 6MHZ1.2, P_1.7 (O1b)
- new net: F_6.16 (Q6), F_8.10 (B6)
- new net: F_6.15 (Q5), F_8.11 (B7)
- new net: F_6.12 (Q4), F_8.12 (B8)
- new net: C5.1, F_8.14 (VR+), R11.1, R12.1, R13.1
- new net: F_8.15 (VR-), R17.2
- new net: C83.2, F_8.4 (IO), F_9.2 (-), R15.1, R16.2
- new net: F_6.9 (Q3), F_8.5 (B1)
- new net: F_6.6 (Q2), F_8.6 (B2)
- new net: F_6.5 (Q1), F_8.7 (B3)
- new net: F_6.2 (Q0), F_8.8 (B4)
- new net: F_6.19 (Q7), F_8.9 (B5)
- new net: M_5.10 (Q2), R11.2
- new net: J_6.2, M_5.11 (~Q2)
- new net: J_6.13, M_5.14 (~Q3)
- new net: M_5.15 (Q3), R13.2
- new net: J_6.1, M_5.6 (~Q1)
- new net: M_5.7 (Q1), R12.2
- new net: C5.2, R14.1
- new net: J_6.12, K_6.5
- new net: L_6.15 (Q3), M_6.15 (A)
- new net: L_6.2 (Q0), M_6.1 (B)
- new net: L_6.7 (Q1), M_6.10 (C)
- new net: L_5.7 (Q1), L_8.1
- new net: B_1.14 (QA), E_1.3
- new net: D_1.11 (QD), D_1.5 (C)
- new net: D_1.12 (QC), D_1.4 (B)
- new net: D_1.13 (QB), D_1.3 (A)
- new net: C_1.14 (QA), D_1.6 (D)
- new net: C_1.11 (QD), C_1.5 (C)
- new net: C_1.12 (QC), C_1.4 (B)
- new net: C_1.13 (QB), C_1.3 (A)
- new net: B_1.11 (QD), B_1.5 (C)
- new net: B_1.12 (QC), B_1.4 (B)
- new net: B_1.13 (QB), B_1.3 (A)
- new net: A_2.1, B_1.15 (RCO), C_2.11
- new net: A_2.2, B_1.6 (D), B_2.14 (QA)
- new net: B_2.10 (ET), B_2.7 (EP), C_2.8
- new net: A_2.5, B_2.12 (QC), B_2.4 (B)
- new net: A_2.4, B_2.13 (QB), B_2.3 (A)
- new net: M_8.2, N_8.11 (QF)
- new net: M_8.3, N_8.10 (QE)
- new net: F_3.1, F_4.3
- new net: J_10.5, M_7.15 (RCO)
- new net: E_10.1, J_10.10
- new net: C21.2, R54.2
- new net: F/H_9.15 (VR-), R55.2
- new net: C25.1, D_10.7, E_10.11, E_10.3, R58.2
- new net: D_10.1, E_10.14, R106.1
- new net: D_10.2 (-), R106.2, R58.1
- new net: E_10.15, E_10.2, R59.2, R62.2
- new net: C_12.2, D/E_12.5 (+), R69.1, R71.2
- new net: C29.2, C30.2, C_12.14, D/E_12.6 (-), R70.1, R73.2
- new net: C29.1, C30.1, D/E_12.7, R73.1, R74.1, R74.2
- new net: D/E_12.3 (+), R74.3, RV2.1
- new net: C_12.10, R65.2
- new net: C_12.11, R65.1
- new net: C_12.12, C_12.8, R63.2
- new net: C_12.13, R67.2
- new net: C_12.3, R66.2
- new net: C_12.4, R60.2, R61.2
- new net: C_12.5, R64.2
- new net: C_12.6, R64.1
- new net: C_12.9, R59.1
- new net: B_12.10, R77.2
- new net: B_12.11, R77.1
- new net: B_12.12, B_12.8, R78.2
- new net: B_12.13, B_12.3, R79.2
- new net: B_12.4, B_12.9, R62.1
- new net: B_12.5, R75.2, R76.2
- new net: B_12.6, C32.2, R75.1, R76.1
- new net: R66.1, R68.3
- new net: R71.1, R72.3
- new net: C4.2, R26.2
- new net: B_9.15 (VR-), R27.2
- new net: A_10.7, B_10.11, B_10.3, C8.1, R30.2
- new net: A_10.1, B_10.14, R31.1
- new net: A_10.2 (-), R30.1, R31.2
- new net: B_10.15, B_10.2, R32.2, R33.2
- new net: B_10.1, J_10.12
- new net: C_11.2, D/E_11.5 (+), R41.2, R44.1
- new net: C12.2, C13.2, C_11.14, D/E_11.6 (-), R45.1, R46.2
- new net: C12.1, C13.1, D/E_11.7, R46.1, R47.1, R47.2
- new net: D/E_11.3 (+), R47.3, RV1.1
- new net: C_11.10, R37.2
- new net: C_11.11, R37.1
- new net: C_11.12, C_11.8, R38.2
- new net: C_11.13, R40.2
- new net: C_11.3, R39.2
- new net: C_11.4, R34.2, R35.2
- new net: C_11.5, R36.2
- new net: C_11.6, R36.1
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Other:
- note added: "ADDRESS DECODERS"
- note added: "AUDIO OUTPUT"
- note added: "CENTER FLAG"
- note added: "CLOCK"
- note added: "CLOCK CIRCUIT"
- note added: "COIN DOOR AND CONTROL PANEL INPUT"
- note added: "COIN DOOR AND CONTROL PANEL OUTPUT"
- note added: "Center Flag"
- note added: "DAC Reference And Bipolar Current Sources"
- note added: "Go Flag"
- note added: "MPU CIRCUITRY"
- note added: "Misc."
- note added: "NMI COUNTER"
- note added: "NORMALIZATION FLAG"
- note added: "NOT LOADED"
- note added: "Normalization Flag"
- note added: "POWER INPUT"
- note added: "POWER RESET AND WATCHDOG TIMER"
- note added: "POWER-ON RESET AND WATCHDOG"
- note added: "PROGRAM RAM"
- note added: "Power Input"
- note added: "R-G-B Output"
- note added: "Signature Analysis"
- note added: "VECTOR FLAG"
- note added: "VECTOR HALT FLAG"
- note added: "VECTOR SCALING"
- note added: "VECTOR TIMER"
- note added: "Vector Address Decoder\n"
- note added: "Vector Address Selector\n"
- note added: "Vector Flag"
- note added: "Vector Interface Buffer"
- note added: "Vector Memory Data Buffer"
- note added: "Vector RAM\n"
- note added: "Vector ROM\n"
- note added: "Vector Scaling"
- note added: "Vector Timer"
- note added: "X-Axis Output"
- note added: "Y-Axis Output"
- note added: "Z-Intensity And Blanking"
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