File: kicad/atari_gravitar_black_widow/atari_gravitar_black_widow.sch (KiCad schematic (older format))
At the start: 657 parts, among them J17 Main_Connector, J20 Edge_Connector_30_Pin, J20 J20, J3 LS04, J5 S260, J8 LS194, J9 AVG, K3 LS74, K5 LS02, K6 LS02, M4 LS27, P4 LS174, Q1 2N3904, Q15 2N6044, Q16 2N6044, Q17 2N3904, Q4 2N3904, Q5 2N3904, Q6 2N3904, Q7 2N3904, Q8 2N3906, SW1 SW_DIP_x08, SW2 SW_DIP_x08, U7805 L7805, U7812 L7812, U7815 L7815, U7915 L7915, Y1 12.096MHz

Commit message: Added PCB connectors to schematic
Parts:
- removed +12V1, +5V1, +5V2, -15V1, 12MHZ1, 6MHZ1, BLUE1, GND1, GND2, GND3, GND4, GREEN1, RED1, SACLK1, SAEN1, VCTR1, ZREF1, ~SA1, ~VMEM1, ~VROM1: TP, Star_Wars_Vector_PCB:TEST_POINT, symbol Star_Wars_Vector_PCB:TP
- removed +15V1: TP1, Star_Wars_Vector_PCB:TEST_POINT, symbol Star_Wars_Vector_PCB:TP
- removed A_1, H_2, K_4: LS08, Star_Wars_Vector_PCB:DIP14, symbol Star_Wars_Vector_PCB:LS08
- removed A_10, D/E_11, D/E_12, D_10, F_9: 082, Star_Wars_Vector_PCB:DIP8, symbol Star_Wars_Vector_PCB:082
- removed A_2: LS20, Star_Wars_Vector_PCB:DIP14, symbol Star_Wars_Vector_PCB:LS20
- removed A_3, P_4: LS00, Star_Wars_Vector_PCB:DIP14, symbol Star_Wars_Vector_PCB:LS00
- removed A_6: RESET, Asteroids:RST, symbol Asteroids_PCB-rescue:SW_Push
- removed B_1, B_2, C_1, D_1, L_5, R_6: LS161, Star_Wars_Vector_PCB:DIP16, symbol Star_Wars_Vector_PCB:LS161
- removed B_1: 137290, Star_Wars_Vector_PCB:DIP20, symbol quantum_arcade_pcb:137290
- removed B_10, B_7, E_10, E_7: LF13201, Star_Wars_Vector_PCB:DIP16, symbol Star_Wars_Vector_PCB:LF13201
- removed B_11, B_12: MC1495LB, Star_Wars_Vector_PCB:DIP14, symbol quantum_arcade_pcb:MC1495LB
- removed B_2, C_2: LS244, Asteroids:DIP20, symbol Asteroids:LS244
- removed B_2/3, D_2/3: POKEY, Star_Wars_Vector_PCB:DDIP40, symbol quantum_arcade_pcb:POKEY
- removed B_4, D_5: LS393, Asteroids:DIP14, symbol Asteroids:LS393
- removed B_5: LS04, Asteroids:DIP14, symbol Asteroids:LS04
- removed B_6: LS14, Asteroids:DIP14, symbol Asteroids:LS14
- removed B_9, F/H_9: AM6012, Star_Wars_Vector_PCB:DIP20, symbol Star_Wars_Vector_PCB:AM6012
- removed C1, C10, C11, C111, C112, C12, C13, C14, C15, C16, C17, C18, C2, C20, C21, C22, C23, C26, C28, C29, C3, C30, C31, C4, C41, C42, C43, C44, C49, C5, C52, C53, C57, C6, C60, C61, C66, C7, C8, C84, C85, C9, C91, C94: .1uF, Asteroids:GenericC, symbol Device:C
- removed C1, C12, C17, C18, C35, C36, C39, C40, C50, C51, C52, C53, C54, C55, C56, C57, C58, C59, C6, C60, C61, C62, C63, C64, C65, C67, C68, C69, C7, C70, C71, C72, C73, C74, C75, C76, C77, C78, C79, C80, C82: .1uF, Star_Wars_Vector_PCB:GenericComp, symbol Device:C
- removed C10, C11, C14, C15, C16, C17, C18, C19, C2, C20, C26, C27, C28, C3, C31, C33, C34, C35, C36, C39, C40, C9: .1uF, quantum_arcade_pcb:GenComp, symbol Device:C
- removed C100, C101, C102, C103, C104, C105, C106, C107, C108, C109, C110, C111, C112, C113, C114, C115, C116, C117, C118, C119, C120, C121, C122, C123, C124, C125, C126, C127, C128, C129, C49, C64, C65, C67, C68, C69, C70, C71, C72, C73, C75, C78, C79, C81, C91, C92, C93, C94, C95, C96, C97, C98, C99: .1uf, quantum_arcade_pcb:GenComp, symbol Device:C
- removed C117: 22uF, Asteroids:Electrolytic4, symbol Device:C
- removed C12, C29: 39pf, quantum_arcade_pcb:CapSmall, symbol Device:C
- removed C13, C30, C32: 100pf, quantum_arcade_pcb:CapSmall, symbol Device:C
- removed C130: .047uf, quantum_arcade_pcb:GenComp, symbol Device:C
- removed C19: 100uF, Asteroids:Electrolytic1, symbol Device:C
- removed C21: .0018uF, quantum_arcade_pcb:CapSmall, symbol Device:C
- removed C25, C70, C90, C92, C93: 1uF, Asteroids:Electrolytic2C, symbol Device:C
- removed C25, C8: .047uF, quantum_arcade_pcb:CapInt, symbol Device:C
- removed C37, C47, C66: 150pF, Star_Wars_Vector_PCB:CapBrown, symbol Device:C
- removed C37: 150pF, quantum_arcade_pcb:CapSmall, symbol Device:C
- removed C38: 39pF, Star_Wars_Vector_PCB:CapBrown, symbol Device:C
- removed C38: 39pF, quantum_arcade_pcb:CapSmall, symbol Device:C
- removed C4: .01uF, quantum_arcade_pcb:CapSmall, symbol Device:C
- removed C41, C5: .01uF, Star_Wars_Vector_PCB:GenericComp, symbol Device:C
- removed C41: .01uF, quantum_arcade_pcb:GenComp, symbol Device:C
- removed C42: 10pF, Star_Wars_Vector_PCB:CapBrown, symbol Device:C
- removed C42: 10pF, quantum_arcade_pcb:CapSmall, symbol Device:C
- removed C43, C44, C46, C81: 100uF, Star_Wars_Vector_PCB:LargeCap, symbol Device:CP1
- removed C44, C46: 100uf 35V, quantum_arcade_pcb:Cap2, symbol Device:CP1_Small
- removed C45, C48: 22uF, Star_Wars_Vector_PCB:CapElec2, symbol Device:CP1
- removed C45, C48: 22uf 25V, quantum_arcade_pcb:Cap1, symbol Device:CP1_Small
- removed C47: 22uf 35V, quantum_arcade_pcb:Cap3, symbol Device:CP1_Small
- removed C74: 1uf, quantum_arcade_pcb:Cap1, symbol Device:CP1_Small
- removed C76: 100pf 100V, quantum_arcade_pcb:CapSmall, symbol Device:C
- removed C77: 39pf 100V, quantum_arcade_pcb:CapSmall, symbol Device:C
- removed C80: .022uf, quantum_arcade_pcb:GenComp, symbol Device:C
- removed C82: 100uf 25V, quantum_arcade_pcb:Cap2, symbol Device:CP1_Small
- removed C83: 22pF, Star_Wars_Vector_PCB:CapBrown, symbol Device:C
- removed C86, C87: 470uF, Asteroids:Electrolytic3, symbol Device:C
- removed CR1: 1N914, Asteroids:Diode1, symbol Device:D
- removed CR1: 1N914, Star_Wars_Vector_PCB:GenericComp, symbol Device:D
- removed CR1: 1N914, quantum_arcade_pcb:Diode, symbol Device:D
- removed CR10, CR11, CR12, CR9: 1N4001, Asteroids:GenericD, symbol Device:D
- removed CR13, CR14: 1N756A, Asteroids:GenericR, symbol Device:D_Zener
- removed CR2: LED, Star_Wars_Vector_PCB:LED, symbol Device:LED
- removed CR3, CR4: 1N100, Star_Wars_Vector_PCB:GenericComp, symbol Device:D
- removed CR3, CR4, CR6: 1N100, quantum_arcade_pcb:Diode, symbol Device:D
- removed CR5: LED, Asteroids:LED, symbol Device:LED
- removed CR5: 1N754A, quantum_arcade_pcb:Diode, symbol Device:D_Zener
- removed CR7: LED, quantum_arcade_pcb:LED, symbol quantum_arcade_pcb:LED
- removed C_11, C_12: MC1495LA, Star_Wars_Vector_PCB:DIP14, symbol quantum_arcade_pcb:MC1495LA
- removed C_3: 6502A, Asteroids:6502A, symbol Asteroids:6502A
- removed C_4: 9316, Asteroids:DIP16, symbol Asteroids:9316
- removed C_5: LS161, Asteroids:DIP16, symbol Asteroids:LS161
- removed C_6: LS00, Asteroids:DIP14, symbol Asteroids:LS00
- removed D_1, H/J_4: LS138, Star_Wars_Vector_PCB:DIP16, symbol quantum_arcade_pcb:LS138
- removed D_4: LS74, Asteroids:DIP14, symbol Asteroids:LS74
- removed D_6, D_9: DAC_8, Star_Wars_Vector_PCB:DIP16, symbol Star_Wars_Vector_PCB:DAC_8
- removed D_8: LS273, Star_Wars_Vector_PCB:DIP20, symbol quantum_arcade_pcb:LS273
- removed E_1, E_3, H_3: LS02, Star_Wars_Vector_PCB:DIP14, symbol Star_Wars_Vector_PCB:LS02
- removed E_2, F_5, J_5: LS32, Star_Wars_Vector_PCB:DIP14, symbol Star_Wars_Vector_PCB:LS32
- removed E_3: LS245, Asteroids:DIP20, symbol Asteroids:LS245
- removed E_5: LS273A, Star_Wars_Vector_PCB:DIP20, symbol Star_Wars_Vector_PCB:LS273A
- removed E_6: LS08, Asteroids:DIP14, symbol Asteroids:LS08
- removed F/H_4, K_6, P_5: LS04, Star_Wars_Vector_PCB:DIP14, symbol Star_Wars_Vector_PCB:LS04
- removed F_1: LS27, Star_Wars_Vector_PCB:DIP14, symbol Star_Wars_Vector_PCB:LS27
- removed F_2, K_9: LS109, Star_Wars_Vector_PCB:DIP16, symbol Star_Wars_Vector_PCB:LS109
- removed F_3, L_7: S260, Star_Wars_Vector_PCB:DIP14, symbol Star_Wars_Vector_PCB:S260
- removed F_4: LS86, Star_Wars_Vector_PCB:DIP14, symbol Star_Wars_Vector_PCB:LS86
- removed F_6: LS273B, Star_Wars_Vector_PCB:DIP20, symbol Star_Wars_Vector_PCB:LS273B
- removed F_8: DAC_8A, Star_Wars_Vector_PCB:DIP16, symbol Star_Wars_Vector_PCB:DAC_8A
- removed J17: Main_Connector, Star_Wars_Vector_PCB:J17, symbol Star_Wars_Vector_PCB:Main_Connector
- removed J20: Edge_Connector_30_Pin, Star_Wars_Vector_PCB:J20, symbol Star_Wars_Vector_PCB:Edge_Connector_30_Pin
- removed J20: J20, quantum_arcade_pcb:EdgeCon, symbol quantum_arcade_pcb:J20
- removed J?: J20, symbol quantum_arcade_pcb:J20
- removed J?: cat_box_con, symbol atari_grav_bw:cat_box_con
- removed unit 5 of J_10
- removed unit 6 of J_10
- removed unit 3 of J_4
- removed unit 1 of J_4
- removed J_6: LS10, Star_Wars_Vector_PCB:DIP14, symbol Star_Wars_Vector_PCB:LS10
- removed K_1: LS245, Star_Wars_Vector_PCB:DIP20, symbol Star_Wars_Vector_PCB:LS245
- removed K_10: S86, Star_Wars_Vector_PCB:DIP14, symbol Star_Wars_Vector_PCB:LS86
- removed K_2: LS42, Star_Wars_Vector_PCB:DIP16, symbol Star_Wars_Vector_PCB:LS42
- removed K_5, L_4: LS74, Star_Wars_Vector_PCB:DIP14, symbol Star_Wars_Vector_PCB:LS74
- removed unit 3 of K_7
- removed L1, L2, L3: 1uH, Star_Wars_Vector_PCB:Inductor1, symbol Device:L
- removed L1: 100uH, quantum_arcade_pcb:Ind, symbol Device:L
- removed L_1: 2732_A, Star_Wars_Vector_PCB:DDIP24, symbol Star_Wars_Vector_PCB:2732_A
- removed L_3: 137211-001, Star_Wars_Vector_PCB:DDIP24, symbol Star_Wars_Vector_PCB:137211-001
- removed L_5: LS175C, Star_Wars_Vector_PCB:DIP16, symbol Star_Wars_Vector_PCB:LS175C
- removed L_6: LS175B, Star_Wars_Vector_PCB:DIP16, symbol Star_Wars_Vector_PCB:LS175B
- removed L_8: 74LS07, Star_Wars_Vector_PCB:DIP14, symbol Star_Wars_Vector_PCB-rescue:74LS07
- removed unit 3 of L_8
- removed unit 5 of L_8
- removed unit 6 of L_8
- removed unit 1 of L_8
- removed M/N_12: TL082, Star_Wars_Vector_PCB:DIP8, symbol Amplifier_Operational:TL082
- removed M_1, M_2: LS244_B, Star_Wars_Vector_PCB:DIP20, symbol Star_Wars_Vector_PCB:LS244_B
- removed M_4: 06, Star_Wars_Vector_PCB:DIP14, symbol Asteroids:LS06
- removed M_5: LS175_A, Star_Wars_Vector_PCB:DIP16, symbol Star_Wars_Vector_PCB:LS175_A
- removed M_6: LS191A, Star_Wars_Vector_PCB:DIP16, symbol Star_Wars_Vector_PCB:LS191A
- removed unit 3 of M_8
- removed M_9: LS244C, Star_Wars_Vector_PCB:DIP20, symbol quantum_arcade_pcb:LS244C
- removed N_1: LS244_A, Star_Wars_Vector_PCB:DIP20, symbol Star_Wars_Vector_PCB:LS244_A
- removed N_2: LS244_C, Star_Wars_Vector_PCB:DIP20, symbol Star_Wars_Vector_PCB:LS244_C
- removed N_3: 2KX8_RAM, Star_Wars_Vector_PCB:DDIP24, symbol quantum_arcade_pcb:2KX8_RAM
- removed N_4: S32, Star_Wars_Vector_PCB:DIP14, symbol Star_Wars_Vector_PCB:LS32
- removed N_5: LS273B, Star_Wars_Vector_PCB:DIP20, symbol quantum_arcade_pcb:LS273B
- removed N_8: LS164, Star_Wars_Vector_PCB:DIP14, symbol Star_Wars_Vector_PCB:LS164
- removed PD1, PD2, PD3, PD4: Split_Pad, Asteroids:SP, symbol Asteroids:Split_Pad
- removed P_1: LS244, Star_Wars_Vector_PCB:DIP20, symbol Star_Wars_Vector_PCB:LS244
- removed P_7: LS163, Star_Wars_Vector_PCB:DIP16, symbol quantum_arcade_pcb:LS163
- removed unit 5 of P_8
- removed unit 1 of P_8
- removed Q1, Q4, Q5, Q6, Q7: 2N3904, Star_Wars_Vector_PCB:GenericTrans, symbol Star_Wars_Vector_PCB-rescue:2N3904
- removed Q15, Q16: 2N6044, quantum_arcade_pcb:BigTrans, symbol Device:Q_NPN_BCE
- removed Q17: 2N3904, quantum_arcade_pcb:GenTrans, symbol Transistor_BJT:2N3904
- removed Q7: 2N3904, quantum_arcade_pcb:GenTrans, symbol Star_Wars_Vector_PCB-rescue:2N3904
- removed Q8: 2N3906, Star_Wars_Vector_PCB:GenericTrans, symbol Star_Wars_Vector_PCB-rescue:2N3906
- removed Q8: 2N3906, quantum_arcade_pcb:GenTrans, symbol Star_Wars_Vector_PCB-rescue:2N3906
- removed R1, R10, R117, R2, R3, R5, R6, R7, R8, R83, R9: 10K, Star_Wars_Vector_PCB:GenericComp, symbol Device:R
- removed R10, R11, R12, R13, R14, R15, R16, R17, R18, R28, R33, R9: 10K, Asteroids:GenericR, symbol Device:R
- removed R100, R101, R102, R103, R104, R105, R15, R98, R99: 100K, Star_Wars_Vector_PCB:GenericComp, symbol Device:R
- removed R106, R30, R31, R58, R85, R86, R89, R93, R95, R96: 7.5K, quantum_arcade_pcb:GenComp, symbol Device:R
- removed R107: 150, Star_Wars_Vector_PCB:GenericComp, symbol Device:R
- removed R108: 270, quantum_arcade_pcb:CapInt, symbol Device:R_US
- removed R109, R110, R111, R82: 1K, Star_Wars_Vector_PCB:GenericComp, symbol Device:R
- removed R11, R16: 12K, Star_Wars_Vector_PCB:GenericComp, symbol Device:R
- removed R112, R113: 270, Asteroids:GenericR, symbol Device:R
- removed R114, R115, R116, R90, R94: 100, Star_Wars_Vector_PCB:GenericComp, symbol Device:R
- removed R12: 24K, Star_Wars_Vector_PCB:GenericComp, symbol Device:R
- removed R13: 47K, Star_Wars_Vector_PCB:GenericComp, symbol Device:R
- removed R14: 820, Star_Wars_Vector_PCB:GenericComp, symbol Device:R
- removed R149, R151, R152, R160, R161, R162: 470, quantum_arcade_pcb:GenComp, symbol Device:R_US
- removed R153, R155, R156, R157, R158, R159, R166, R167, R168, R169, R176, R205, R210, R214, R218, R219, R220, R221, R222: 1k, quantum_arcade_pcb:GenComp, symbol Device:R_US
- removed R163, R173, R177, R178, R215: 10k, quantum_arcade_pcb:GenComp, symbol Device:R_US
- removed R164, R165, R179, R223: 220, quantum_arcade_pcb:GenComp, symbol Device:R_US
- removed R17: 6.2K, Star_Wars_Vector_PCB:GenericComp, symbol Device:R
- removed R174: 68k, quantum_arcade_pcb:GenComp, symbol Device:R_US
- removed R175: 15k, quantum_arcade_pcb:GenComp, symbol Device:R_US
- removed R180, R181, R182, R183, R184, R185, R186, R187: 100K, quantum_arcade_pcb:GenComp, symbol Device:R
- removed R188, R189, R190, R191, R192, R193, R194, R195, R196, R197, R198, R199, R200, R201, R202, R203: 4.7k, quantum_arcade_pcb:GenComp, symbol Device:R_US
- removed R20, R21, R22: 470, Star_Wars_Vector_PCB:GenericComp, symbol Device:R
- removed R204, R206, R207, R208, R209, R211, R212, R213: 220k, quantum_arcade_pcb:GenComp, symbol Device:R_US
- removed R23, R24, R25: 4.7k, Star_Wars_Vector_PCB:GenericComp, symbol Device:R
- removed R26, R27, R55: 820, quantum_arcade_pcb:GenComp, symbol Device:R
- removed R27, R29: 1K, Asteroids:GenericR, symbol Device:R
- removed R30, R31: 330, Asteroids:GenericR, symbol Device:R
- removed R32: 470, Asteroids:GenericR, symbol Device:R
- removed R32, R33, R38, R51, R59, R62, R63: 470, quantum_arcade_pcb:GenComp, symbol Device:R
- removed R34, R60: 2.7k, quantum_arcade_pcb:GenComp, symbol Device:R
- removed R35, R54, R61: 680, quantum_arcade_pcb:GenComp, symbol Device:R
- removed R36, R44, R45, R50, R64, R69, R70, R77: 2.2k, quantum_arcade_pcb:GenComp, symbol Device:R
- removed R37, R39, R52, R65, R66, R78, R79: 3.9k, quantum_arcade_pcb:GenComp, symbol Device:R
- removed unit 1 of R4
- removed R40, R46, R67, R73: 10k, quantum_arcade_pcb:GenComp, symbol Device:R
- removed R41, R71: 5.6k, quantum_arcade_pcb:GenComp, symbol Device:R
- removed R42, R43, R68, R72: 10k, Star_Wars_Vector_PCB:PotBlk, symbol Star_Wars_Vector_PCB-rescue:POT
- removed R47, R74: 2K, Star_Wars_Vector_PCB:PotBlk, symbol Star_Wars_Vector_PCB-rescue:POT
- removed R48, R75: 100k, quantum_arcade_pcb:GenComp, symbol Device:R
- removed R49: 1.5k, quantum_arcade_pcb:GenComp, symbol Device:R
- removed R53, R80: 1k, quantum_arcade_pcb:GenComp, symbol Device:R
- removed R55: 150, Asteroids:GenericR, symbol Device:R
- removed R75, R76: 1.30K, Star_Wars_Vector_PCB:GenericComp, symbol Device:R
- removed R76: 1.2k, quantum_arcade_pcb:GenComp, symbol Device:R
- removed R81: 15K, Star_Wars_Vector_PCB:GenericComp, symbol Device:R
- removed R81: 15K, quantum_arcade_pcb:GenComp, symbol Device:R
- removed R82: 1K, quantum_arcade_pcb:GenComp, symbol Device:R
- removed R83: 10K, quantum_arcade_pcb:GenComp, symbol Device:R
- removed R84: 560, Star_Wars_Vector_PCB:GenericComp, symbol Device:R
- removed R84: 560, quantum_arcade_pcb:GenComp, symbol Device:R
- removed R85, R86, R89, R93, R95, R96: 7.5K, Star_Wars_Vector_PCB:GenericComp, symbol Device:R
- removed R87, R91: 6.19K, Star_Wars_Vector_PCB:GenericComp, symbol Device:R
- removed R87, R91: 7.5k, quantum_arcade_pcb:GenComp, symbol Device:R
- removed R88 (x2), R92 (x2): 200, Star_Wars_Vector_PCB:PotBlk, symbol Star_Wars_Vector_PCB-rescue:POT
- removed R90, R94: 100, quantum_arcade_pcb:GenComp, symbol Device:R
- removed R97: 3.9K, Star_Wars_Vector_PCB:GenericComp, symbol Device:R
- removed R97: 3.9K, quantum_arcade_pcb:GenComp, symbol Device:R
- removed RV1, RV2: VDR, quantum_arcade_pcb:GenComp, symbol Device:Varistor
- removed R_4, R_5: LS393, Star_Wars_Vector_PCB:DIP14, symbol Asteroids:LS393
- removed SW1, SW2: SW_DIP_x08, Star_Wars_Vector_PCB:DIP16, symbol Switch:SW_DIP_x08
- removed TP+15V1, TP-15V1, TP12M1, TP5V1, TP5V2, TP6.8V1, TPAUD1, TPAUD2, TPGND1, TPGND2, TPGND3, TPRESET1, TPRESET2, TPWDDIS1, TPXOUT1, TPYOUT1: TP, quantum_arcade_pcb:TP, symbol Star_Wars_Vector_PCB:TP
- removed TP1: WDOG_DISABLE, Asteroids:TEST_POINT, symbol Asteroids:AST_TEST
- removed TP2: O2, Asteroids:TEST_POINT, symbol Asteroids:AST_TEST
- removed TP3: R/W, Asteroids:TEST_POINT, symbol Asteroids:AST_TEST
- removed TP4: 6MHz, Asteroids:TEST_POINT, symbol Asteroids:AST_TEST
- removed TP5: +5V, Asteroids:TEST_POINT, symbol Asteroids:AST_TEST
- removed TP6, TP7: GND, Asteroids:TEST_POINT, symbol Asteroids:AST_TEST
- removed U7805: L7805, Asteroids:Volt_Reg, symbol Asteroids_PCB-rescue:L7805
- removed U7812: L7812, Asteroids:2N6044, symbol Asteroids_PCB-rescue:L7812
- removed U7815: L7815, Asteroids:Volt_Reg, symbol Asteroids_PCB-rescue:L7815
- removed U7915: L7915, Asteroids:Volt_Reg, symbol Asteroids_PCB-rescue:L7915
- removed VR1: L7815_, Star_Wars_Vector_PCB:VoltReg, symbol Star_Wars_Vector_PCB:L7815_
- removed VR1: L7815_, quantum_arcade_pcb:BigTrans, symbol Star_Wars_Vector_PCB:L7815_
- removed VR2: L7915_, Star_Wars_Vector_PCB:VoltReg, symbol Star_Wars_Vector_PCB:L7915_
- removed VR2: L7915_, quantum_arcade_pcb:BigTrans, symbol Star_Wars_Vector_PCB:L7915_
- removed Y1: 12.096MHz, Asteroids:RST, symbol Device:Crystal
- removed Y1: 12.096MHz, quantum_arcade_pcb:Crystal, symbol Device:Crystal
- added J17: cat_box_con, symbol atari_grav_bw:cat_box_con
- added J19: J19, symbol atari_grav_bw:J19
- added J20: J20, symbol atari_grav_bw:J20
- added R_6: LS161A, symbol atari_grav_bw:LS161A
Connections:
- net +10V: now also J20.18 (+10.3V_UNREG), J20.E (+10.3V_UNREG)
- net +24V: now also J20.3 (+22VDC), J20.X (+22VDC)
- net +5V: now also J17.45 (+5V), J17.46 (+5V), J17.47 (+5V), J17.48 (+5V), J17.49 (+5V), J17.50 (+5V), J20.2 (+5V), J20.21 (+5V), J20.B (+5V), J20.Y (+5V), R_6.16 (VCC); no longer M4.14 (VCC)
- net -24V: now also J20.4 (-22VDC), J20.W (-22VDC)
- net 12M: no longer M_5.2 (CLK), M_6.2 (CLK), M_7.2 (CLK)
- net A0: now also J17.17 (A0)
- net A1: now also J17.18 (A1)
- net A10: now also J17.7 (A10)
- net A11: now also J17.8 (A11)
- net A12: now also J17.21 (A12)
- net A13: now also J17.22 (A13)
- net A14: now also J17.19 (A14)
- net A15: now also J17.20 (A15)
- net A2: now also J17.15 (A2)
- net A3: now also J17.16 (A3)
- net A4: now also J17.13 (A4)
- net A5: now also J17.14 (A5)
- net A6: now also J17.11 (A6)
- net A7: now also J17.12 (A7)
- net A8: now also J17.9 (A8)
- net A9: now also J17.10 (A9)
- net BLUE: now also J19.9 (BLUE)
- net COINL: now also J20.16 (COINL)
- net COINR: now also J20.U (COINR)
- net D0: now also J17.29 (D0)
- net D1: now also J17.30 (D1)
- net D2: now also J17.27 (D2)
- net D3: now also J17.28 (D3)
- net D4: now also J17.25 (D4)
- net D5: now also J17.26 (D5)
- net D6: now also J17.23 (D6)
- net D7: now also J17.24 (D7)
- net GND: now also J17.1 (GND), J17.2 (GND), J17.3 (GND), J17.34 (GND), J17.4 (GND), J17.5 (GND), J17.6 (GND), J19.1 (GND), J19.2 (GND), J19.H (GND), J19.J (GND), J19.K (GND), J19.L (GND), J19.M (GND), J20.1 (GND), J20.12 (GND), J20.13 (GND), J20.22 (GND), J20.A (GND), J20.N (GND), J20.P (GND), J20.Z (GND), R_6.8 (GND)
- net GREEN: now also J19.8 (GREEN)
- net PR221: no longer M_6.1 (C), M_7.1 (C)
- net RED: now also J19.7 (RED)
- net START1: now also J20.M (START1)
- net START2: now also J20.11 (START2)
- net XOUT: now also J19.A (XOUT)
- net YOUT: now also J19.B (YOUT)
- net ~RESET: now also J20.V (~RESET)
- net at M_5.10 (ET), M_5.7 (EP), M_6.7 (EP)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: now also R_6.15 (RCO)
- net at M_5.14 (QA): now also R_6.6 (D)
- net at J_4.4, M_5.9 (LD), M_6.9 (LD)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: now also R_6.9 (LD)
- net PR219: no longer names the net of M_5.1 (C)
- new net: R_6.10 (ET), R_6.7 (EP)
- new net: R_6.11 (QD), R_6.5 (C)
- new net: R_6.12 (QC), R_6.4 (B)
- new net: R_6.13 (QB), R_6.3 (A)
- new net AUD1: J19.12 (AUD1)
- new net AUD2: J19.11 (AUD2)
- new net CABINET: J20.R (CABINET)
- new net CAT_STROBE: J17.35 (CAT_STB)
- new net COIN_AUX: J20.S (COIN_AUX)
- new net COIN_CNTRL: J20.H (COIN_CNTRL)
- new net COIN_CNTRR: J20.6 (COIN_CNTRR)
- new net COIN_LOCKOUT: J20.F (COIN_LOCKOUT)
- new net FIRE1: J19.4 (FIRE1)
- new net FIRE2: J20.9 (FIRE2)
- new net PHASE0: J17.33 (PHASE0)
- new net PHASE2: J17.31 (PHASE2)
- new net PLAYER1_LED: J20.7 (PLAYER1_LED)
- new net PLAYER2_LED: J20.J (PLAYER2_LED)
- new net PR55: R_6.1 (C)
- new net ROT_LEFT1: J19.E (ROT_LEFT1)
- new net ROT_LEFT2: J20.8 (ROT_LEFT2)
- new net ROT_RIGHT1: J19.5 (ROT_RIGHT1)
- new net ROT_RIGHT2: J20.K (ROT_RIGHT2)
- new net R~W: J17.32 (R/~W)
- new net SELF_TEST: J20.T (SELF_TEST)
- new net SHIELDS1: J19.3 (SHIELDS1)
- new net SHIELDS2: J20.L (SHIELDS2)
- new net SLAM: J20.14 (SLAM)
- new net THRUST1: J19.6 (THRUST1)
- new net THRUST2: J20.10 (THRUST2)
- new net VCC: M4.14 (VCC)
- new net Z_OUT: J19.10 (Z_OUT)
- new net ~DISDAT: J17.36 (~DISDAT)
- no-connect marks 110 -> 33
Other:
- note removed: "ADDRESS DECODERS"
- note removed: "AUDIO OUTPUT"
- note removed: "CENTER FLAG"
- note removed: "CLOCK"
- note removed: "CLOCK CIRCUIT"
- note removed: "COIN DOOR AND CONTROL PANEL INPUT"
- note removed: "COIN DOOR AND CONTROL PANEL OUTPUT"
- note removed: "Center Flag"
- note removed: "DAC Reference And Bipolar Current Sources"
- note removed: "Go Flag"
- note removed: "MPU CIRCUITRY"
- note removed: "Misc."
- note removed: "NMI COUNTER"
- note removed: "NORMALIZATION FLAG"
- note removed: "NOT LOADED"
- note removed: "Normalization Flag"
- note removed: "POWER INPUT"
- note removed: "POWER RESET AND WATCHDOG TIMER"
- note removed: "POWER-ON RESET AND WATCHDOG"
- note removed: "PROGRAM RAM"
- note removed: "Power Input"
- note removed: "R-G-B Output"
- note removed: "Signature Analysis"
- note removed: "VECTOR FLAG"
- note removed: "VECTOR HALT FLAG"
- note removed: "Vector Address Decoder\n"
- note removed: "Vector Address Selector\n"
- note removed: "Vector Flag"
- note removed: "Vector Interface Buffer"
- note removed: "Vector Memory Data Buffer"
- note removed: "Vector RAM\n"
- note removed: "Vector ROM\n"
- note removed: "Vector Scaling"
- note removed: "Vector Timer"
- note removed: "X-Axis Output"
- note removed: "Y-Axis Output"
- note removed: "Z-Intensity And Blanking"
- moved on the sheet: J_10C, J_4B, K_7B, L_8B, L_8D, L_9, M_5, M_6, M_7, M_8, P_8F

Commit message: Completed sheet 6A
Parts:
- removed A8, B8, C8, F8, H8, J8: LS194, symbol Star_Wars_Vector_PCB:LS194
- removed C6, D6: LS175E, symbol star_wars_arcade_main_pcb:LS175E
- removed E7: LS00, symbol Star_Wars_Vector_PCB:LS00
- removed F7: LS14, symbol Star_Wars_Vector_PCB:LS14
Connections:
- no-connect marks 33 -> 32
Other:
- note removed: "Op Code and\nIntensity\nLatches"
- moved on the sheet: J_10C, J_4B, K_7B, L_8B, L_8D, L_9, M_5, M_6, M_7, M_8, P_8F, R_6
