File: kicad/atari_gravitar_black_widow/atari_gravitar_black_widow.sch (KiCad schematic (older format))
At the start: 32 parts, among them J17 cat_box_con, J19 J19, J20 J20, J3 LS04, J5 S260, J9 AVG, K3 LS74, K5 LS02, K6 LS02, M4 LS27, P4 LS174

Commit message: Rearranged the schematic sheets layout
Parts:
- removed A7, K3: LS74, symbol Star_Wars_Vector_PCB:LS74
- removed B7, K5, K6, N5: LS02, symbol atari_gravitar_black_widow-rescue:LS02-Star_Wars_Vector_PCB
- removed H7: LS42, symbol Star_Wars_Vector_PCB:LS42
- removed J17: cat_box_con, symbol atari_grav_bw:cat_box_con
- removed J19: J19, symbol atari_grav_bw:J19
- removed J20: J20, symbol atari_grav_bw:J20
- removed J3: LS04, symbol Star_Wars_Vector_PCB:LS04
- removed J5: S260, symbol atari_gravitar_black_widow-rescue:S260alt-Star_Wars_Vector_PCB
- removed J9: AVG, symbol Star_Wars_Vector_PCB:AVG
- removed J_10: LS04, Star_Wars_Vector_PCB:DIP14, symbol Star_Wars_Vector_PCB:LS04
- removed J_4: LS02, Star_Wars_Vector_PCB:DIP14, symbol Star_Wars_Vector_PCB:LS02
- removed K_7: LS32, Star_Wars_Vector_PCB:DIP14, symbol Star_Wars_Vector_PCB:LS32
- removed L4: LS08, symbol Star_Wars_Vector_PCB:LS08
- removed L_8: S02, Star_Wars_Vector_PCB:DIP14, symbol Star_Wars_Vector_PCB:LS02
- removed L_9: LS175, Star_Wars_Vector_PCB:DIP16, symbol quantum_arcade_pcb:LS175
- removed M4: LS27, symbol atari_gravitar_black_widow-rescue:LS27-Star_Wars_Vector_PCB
- removed M_5, M_6, M_7: LS161, Star_Wars_Vector_PCB:DIP16, symbol Star_Wars_Vector_PCB:LS161
- removed M_8: LS191A, Star_Wars_Vector_PCB:DIP16, symbol Star_Wars_Vector_PCB:LS191A
- removed N3: LS157, symbol Star_Wars_Vector_PCB:LS157D
- removed N4: S129, symbol Star_Wars_Vector_PCB:S129
- removed P4: LS174, symbol Star_Wars_Vector_PCB:LS174A
- removed P_8: S04, Star_Wars_Vector_PCB:DIP14, symbol Star_Wars_Vector_PCB:LS04
- removed R20: 10K, symbol Device:R_US
- removed R3: LS157, symbol Star_Wars_Vector_PCB:LS157C
- removed R4: LS32, symbol Star_Wars_Vector_PCB:LS32
- removed R_6: LS161A, symbol atari_grav_bw:LS161A
Connections:
- net labels removed: (OU9A), +10V, +24V, +5V, -24V, 0000, 0000', 0108, 0863, 08A0, 12C7, 12M, 12MHZ, 1C91, 2946, 29PP, 3A9A, 3MHZ, 4596, 4760, 69F0, 6MHZ, 7862, 79P4, 8834, 8P54', 8PUH, A0, A1, A10, A11, A12, A13, A14, A15, A2, A3, A4, A5, A6, A7, A736, A8, A9, AM0, AM1, AM2, AM3, AM4, AM5, AM6, AM7, AUD1, AUD2, AVG0, AVG1, AVG10, AVG11, AVG12, AVG13, AVG2, AVG3, AVG4, AVG5, AVG6, AVG7, AVG8, AVG9, BLUE, C592, C794, CABINET, CAT_STROBE, CF31, CNTR, COINL, COINR, COIN_AUX, COIN_CNTRL, COIN_CNTRR, COIN_LOCKOUT, D0, D1, D2, D3, D4, D5, D6, D7, DVY0, DVY1, DVY10, DVY11, DVY12, DVY2, DVY3, DVY4, DVY5, DVY6, DVY7, DVY8, DVY9, F0, F1, F2, F3, F61C, FIRE1, FIRE2, GND, GO, GREEN, H10F, H381, HALT, HALT*, HF91, HH53, NORM, OP0, OP1, OP2, PHASE0, PHASE2, PLAYER1_LED, PLAYER2_LED, PR221, PR55, RED, ROT_LEFT1, ROT_LEFT2, ROT_RIGHT1, ROT_RIGHT2, R~W, SA, SACLK, SCALE, SCALELO, SELF_TEST, SHIELDS1, SHIELDS2, SLAM, ST0, ST1, ST2, ST3, START1, START2, THRUST1, THRUST2, U467, U9H9, VCTR, VGCK, XOUT, YOUT, Z_OUT, ~DISDAT, ~DISRST, ~LATCH0, ~LATCH1, ~LATCH2, ~LATCH3, ~OP0, ~OP2, ~RESET, ~SA, ~STOP, ~STROBE0, ~STROBE1, ~STROBE2, ~STROBE3, ~VGGO, ~VMEM
- wire segments 282 -> 0
- no-connect marks 32 -> 0
Other:
- note added: "Atari\nGravitar/\nBlack Widow\nPCB"
- note added: "DONE"
- note removed: "Address Controller"
- note removed: "Decoder Disable"
- note removed: "Signature Analysis Flag"
- note removed: "State Machine"
- note removed: "State Machine Clock"
- note removed: "State Machine Clock Logic"
- note removed: "VECTOR SCALING"
- note removed: "VECTOR TIMER"

Commit message: Completed sheet 3B
Changed lines of the file:
@@
 Text Notes 11975 3775 0    400  ~ 80
 Atari\nGravitar/\nBlack Widow\nPCB
+Text Notes 1450 2525 0    200  ~ 40
+DONE
 $EndSCHEMATC

Commit message: Completed sheet 6B
Changed lines of the file:
@@
 Text Notes 1450 2525 0    200  ~ 40
 DONE
+Text Notes 7000 5825 0    200  ~ 40
+DONE
 $EndSCHEMATC

Commit message: More Sheet 7a
Other:
- note added: "JBB\nIN \nPROGRESS\n"
Changed lines of the file:
@@
 $EndSheet
 $Sheet
-S 6125 4450 2500 2500
+S 6125 4475 2500 2500
 U 6B32D4FA
 F0 "Sheet6B" 200
@@
 Text Notes 1450 2525 0    200  ~ 40
 DONE
-Text Notes 7000 5825 0    200  ~ 40
+Text Notes 7000 5850 0    200  ~ 40
 DONE
+Text Notes 9475 5900 0    200  ~ 40
+JBB\nIN \nPROGRESS\n
 $EndSCHEMATC
