File: kicad/atari_gravitar_black_widow/Sheet6A.sch (KiCad schematic (older format))
At the start: 16 parts

Commit message: Rearranged the schematic sheets layout
Parts:
- gave numbers to parts that had none: 10
Other:
- moved on the sheet: A_8, B_8, C_6, C_8, D_6, E_7A, E_7B, E_7C, E_7D, F_7A, F_7D, F_7E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

Commit message: Completed sheet 6B
Other:
- note added: "0000'"
- note removed: "0000"
Changed lines of the file:
@@
 $EndComp
 Text Notes 5750 13900 0    50   ~ 0
-0000
+0000'
 Text Notes 5750 14025 0    50   ~ 0
 C794
