File: kicad/atari_gravitar_black_widow/Sheet6B.sch (KiCad schematic (older format))
At the start: 22 parts

Commit message: Completed sheet 6B
Parts:
- removed A? (x2), K?: LS74, symbol Star_Wars_Vector_PCB:LS74
- removed B? (x2), K? (x3), N?: LS02, symbol atari_gravitar_black_widow-rescue:LS02-Star_Wars_Vector_PCB
- removed H?: LS42, symbol Star_Wars_Vector_PCB:LS42
- removed J?: AVG, symbol Star_Wars_Vector_PCB:AVG
- removed J?: S260, symbol atari_gravitar_black_widow-rescue:S260alt-Star_Wars_Vector_PCB
- removed J?: LS04, symbol Star_Wars_Vector_PCB:LS04
- removed L?: LS08, symbol Star_Wars_Vector_PCB:LS08
- removed M?: LS27, symbol atari_gravitar_black_widow-rescue:LS27-Star_Wars_Vector_PCB
- removed N?: S129, symbol Star_Wars_Vector_PCB:S129
- removed N?: LS157, symbol Star_Wars_Vector_PCB:LS157D
- removed P?: LS174, symbol Star_Wars_Vector_PCB:LS174A
- removed R? (x2): LS32, symbol Star_Wars_Vector_PCB:LS32
- removed R?: LS157, symbol Star_Wars_Vector_PCB:LS157C
- added A_7, K_3: LS74, symbol atari_grav_bw:LS74
- added B_7, K_5, K_6, N_5: LS02, symbol atari_grav_bw:LS02
- added H_7: LS42, symbol atari_grav_bw:LS42
- added J_3: LS04, symbol atari_grav_bw:LS04
- added J_5: S260, symbol atari_grav_bw:S260
- added J_9: AVG, symbol atari_grav_bw:AVG
- added L_4: LS08, symbol atari_grav_bw:LS08
- added M_4: LS27, symbol atari_grav_bw:LS27
- added N_3: LS157A, symbol atari_grav_bw:LS157A
- added N_4: S129, symbol atari_grav_bw:S129
- added P_4: LS174A, symbol atari_grav_bw:LS174A
- added R_3: LS157B, symbol atari_grav_bw:LS157B
- added R_4: LS32, symbol atari_grav_bw:LS32
- added TPSACLK1, TP~SA1: TP, symbol atari_grav_bw:TP
- gave numbers to parts that had none: 1
Connections:
- net 12MHZ: now also A_7.11 (2CLK), A_7.3 (1CLK)
- net 3MHZ: now also J_5.2, K_6.6
- net 6MHZ: now also J_5.3, K_3.11 (2CLK)
- net AM0: now also R_3.2 (A)
- net AM1: now also R_3.6 (B)
- net AM2: now also R_3.10 (B)
- net AM3: now also R_3.13 (B)
- net AM4: now also N_3.10 (B)
- net AM5: now also N_3.6 (B)
- net AM6: now also N_3.3 (B)
- net AM7: now also N_3.13 (B)
- net AVG0: now also J_9.36 (AVG0)
- net AVG1: now also J_9.39 (AVG1)
- net AVG10: now also J_9.19 (AVG10)
- net AVG11: now also J_9.20 (AVG11)
- net AVG2: now also J_9.40 (AVG2)
- net AVG3: now also J_9.1 (AVG3)
- net AVG4: now also J_9.2 (AVG4)
- net AVG5: now also J_9.3 (AVG5)
- net AVG6: now also J_9.15 (AVG6)
- net AVG7: now also J_9.16 (AVG7)
- net AVG8: now also J_9.17 (AVG8)
- net AVG9: now also J_9.18 (AVG9)
- net DVY0: now also J_9.32 (DVY0)
- net DVY1: now also J_9.31 (DVY1)
- net DVY10: now also J_9.29 (DVY10)
- net DVY11: now also J_9.28 (DVY11)
- net DVY12: now also J_9.27 (DVY12)
- net DVY2: now also J_9.30 (DVY2)
- net DVY3: now also J_9.7 (DVY3)
- net DVY4: now also J_9.8 (DVY4)
- net DVY5: now also J_9.9 (DVY5)
- net DVY6: now also J_9.10 (DVY6)
- net DVY7: now also J_9.11 (DVY7)
- net DVY8: now also J_9.12 (DVY8)
- net DVY9: now also J_9.13 (DVY9)
- net F0: now also P_4.12 (5Q), R_3.3 (B)
- net F1: now also P_4.5 (2Q), R_3.5 (A)
- net F2: now also P_4.10 (4Q), R_3.11 (A)
- net F3: now also P_4.7 (3Q), R_3.14 (A)
- net GND: now also H_7.8 (GND), J_5.7 (GND), J_9.14 (GND), K_5.7 (GND), N_3.15 (G), N_3.8 (GND), N_4.13 (CE1), N_4.14 (CE2), P_4.8 (GND), R_3.15 (G), R_3.8 (GND)
- net GO: now also N_5.9
- net HALT: now also P_4.3 (1D)
- net HALT*: now also N_5.8, P_4.2 (1Q)
- net OP0: now also N_3.11 (A)
- net OP1: now also J_9.33 (OP1), N_3.5 (A)
- net OP2: now also N_3.2 (A)
- net SA: now also J_3.12, N_3.1 (S), R_3.1 (S), R_4.10, R_4.5
- net ST0: now also H_7.15 (A0), N_4.12 (O1), P_4.13 (5D)
- net ST1: now also H_7.14 (A1), N_4.11 (O2), P_4.4 (2D)
- net ST2: now also H_7.13 (A2), L_4.4, M_4.11, N_4.10 (O3), P_4.11 (4D)
- net ~DISRST: now also P_4.1 (C)
- net ~LATCH0: now also H_7.1 (0)
- net ~LATCH1: now also H_7.2 (1)
- net ~LATCH2: now also H_7.3 (2)
- net ~LATCH3: now also H_7.4 (3)
- net ~OP0: now also J_9.25 (~OPX), J_9.26 (~OP0)
- net ~OP2: now also R_4.4
- net ~SA: now also J_3.13, L_4.5, TP~SA1.1, TP~SA1.2
- net ~STROBE0: now also H_7.5 (4), J_9.24 (~STROBE0)
- net ~STROBE1: now also H_7.6 (5), J_9.34 (~STROBE1)
- net ~STROBE2: now also H_7.7 (6), J_9.4 (~STROBE2)
- net ~STROBE3: now also H_7.9 (7)
- net ~VGGO: now also J_9.6 (~VGGO)
- net ~VMEM: now also M_4.9
- net +5V: now reaches R20.1
- net +5V: now also H_7.16 (VCC), J_5.14 (VCC), J_9.37 (VDD), K_5.14 (VCC), N_3.16 (VCC), N_4.16 (VCC), P_4.16 (VCC), R_3.16 (VCC)
- new net: J_9.5 (~OP2), R_4.6
- new net: J_9.35 (ST2), L_4.6
- new net: K_3.9 (2Q), K_5.3, M_4.10
- new net: K_5.11, M_4.8
- new net: K_3.12 (2D), K_6.4
- new net: J_5.12, J_5.13, K_5.1, K_5.12
- new net: K_5.13, K_5.2
- new net: B_7.12, J_5.5
- new net: B_7.10, B_7.11
- new net: A_7.5 (1Q), B_7.9
- new net: A_7.12 (2D), A_7.2 (1D), B_7.13
- new net: A_7.6 (~1Q), P_4.9 (CK)
- new net: A_7.13 (~1CLR), R_4.8
- new net: N_4.9 (O4), P_4.6 (3D), R_4.9
- new net: N_3.14 (A), N_5.10
- new net: N_3.12 (Y), N_4.15 (A7)
- new net: N_3.4 (Y), N_4.1 (A6)
- new net: N_3.7 (Y), N_4.2 (A5)
- new net: N_3.9 (Y), N_4.3 (A4)
- new net: N_4.4 (A3), R_3.12 (Y)
- new net: N_4.7 (A2), R_3.4 (Y)
- new net: N_4.6 (A1), R_3.7 (Y)
- new net: N_4.5 (A0), R_3.9 (Y)
- new net AVG12: J_9.21 (AVG12)
- new net AVG13: J_9.22 (AVG13)
- new net PR23: K_3.10 (~1PRE_), K_3.13 (~1CLR)
- new net PR82: A_7.10 (~1PRE_), A_7.4 (~1PRE_)
- new net PR83: A_7.1 (~1CLR)
- new net ST3: A_7.8 (~2Q), H_7.12 (A3), J_9.38 (ST3)
- new net VGCK: B_7.8, J_5.1, K_6.5, TPSACLK1.1, TPSACLK1.2
- no-connect marks 0 -> 7
Other:
- note added: "(00PH)"
- note added: "(068C)"
- note added: "(08A0)"
- note added: "(0H0H)"
- note added: "(0U9A)"
- note added: "(1C91)"
- note added: "(1H6F)"
- note added: "(389H)"
- note added: "(3F47)"
- note added: "(4347)"
- note added: "(4760)"
- note added: "(4HPH)"
- note added: "(6608)"
- note added: "(6682)"
- note added: "(69F0)"
- note added: "(6UUF)"
- note added: "(8P54)"
- note added: "(8PC9)"
- note added: "(8PUH)"
- note added: "(A262)"
- note added: "(A736)"
- note added: "(C592)"
- note added: "(CF31)"
- note added: "(F580)"
- note added: "(H2P1)"
- note added: "(H381)"
- note added: "(HF91)"
- note added: "(P1A8)"
- note added: "(PA7F)"
- note added: "(U5C1)"
- note added: "0000"
- note added: "0000'"
- note added: "0108"
- note added: "0863"
- note added: "12C7"
- note added: "1U34"
- note added: "2946"
- note added: "29PP"
- note added: "3A95"
- note added: "3A9A"
- note added: "4596"
- note added: "7862"
- note added: "79P4"
- note added: "8834"
- note added: "8P54"
- note added: "8P54'"
- note added: "ADDRESS CONTROLLER"
- note added: "C794"
- note added: "DECODER DISABLE"
- note added: "F61C"
- note added: "H10F"
- note added: "H381"
- note added: "HH53"
- note added: "SIGNATURE ANALYSIS FLAG"
- note added: "STATE MACHINE"
- note added: "STATE MACHINE CLOCK LOGIC"
- note added: "STATE MACHINE\nCLOCK"
- note added: "U0H9"
- note added: "U467"
- note added: "UUUU"
- note removed: "Address Controller"
- note removed: "Decoder Disable"
- note removed: "Signature Analysis Flag"
- note removed: "State Machine"
- note removed: "State Machine Clock"
- note removed: "State Machine Clock Logic"
- moved on the sheet: R20
