File: kicad/atari_gravitar_black_widow/Sheet7A.sch (KiCad schematic (older format))
At the start: 12 parts

Commit message: Worked on sheet 7A
Parts:
- removed J_?: LS02, Star_Wars_Vector_PCB:DIP14, symbol Star_Wars_Vector_PCB:LS02
- removed J_?: LS04, Star_Wars_Vector_PCB:DIP14, symbol Star_Wars_Vector_PCB:LS04
- removed K_?: LS32, Star_Wars_Vector_PCB:DIP14, symbol Star_Wars_Vector_PCB:LS32
- removed L_?: LS175, Star_Wars_Vector_PCB:DIP16, symbol quantum_arcade_pcb:LS175
- removed L_? (x2): S02, Star_Wars_Vector_PCB:DIP14, symbol Star_Wars_Vector_PCB:LS02
- removed M_? (x3): LS161, Star_Wars_Vector_PCB:DIP16, symbol Star_Wars_Vector_PCB:LS161
- removed M_?: LS191A, Star_Wars_Vector_PCB:DIP16, symbol Star_Wars_Vector_PCB:LS191A
- removed P_?: S04, Star_Wars_Vector_PCB:DIP14, symbol Star_Wars_Vector_PCB:LS04
- removed R_?: LS161A, symbol atari_grav_bw:LS161A
- added E_3, L_3: LS00, symbol atari_grav_bw:LS00
- added F_5: LS11, symbol atari_grav_bw:LS11
- added H_3: LS20A, symbol atari_grav_bw:LS20A
- added H_5: LS20, symbol atari_grav_bw:LS20
- added K_5, K_6: LS02, symbol atari_grav_bw:LS02
- added L_6: LS08, symbol atari_grav_bw:LS08
- added M_6, N_6, P_6, R_6: LS161A, symbol atari_grav_bw:LS161A
Connections:
- net labels added: ~SCALELD
- net labels removed: 12M, CNTR, DVY10, DVY8, DVY9, NORM, OP2, PR221, SCALE, SCALELO, VCTR, ~DISRST, ~STROBE1
- wire segments 122 -> 152
- no-connect marks 13 -> 3
Other:
- note added: "0AP1"
- note added: "0P9F"
- note added: "13CF"
- note added: "2F31"
- note added: "2HC6"
- note added: "2PPC"
- note added: "60P6"
- note added: "66HF"
- note added: "6859"
- note added: "6P29"
- note added: "7579"
- note added: "8P54"
- note added: "8P54'"
- note added: "919P"
- note added: "9PP2"
- note added: "C87F"
- note added: "CCF4"
- note added: "HF49"
- note added: "P60H"
- note added: "P724"
- note added: "P88C"
- note added: "PC8A"
- note removed: "VECTOR SCALING"

Commit message: JBB worked on sheet 7a
Parts:
- added U?: LS175, symbol atari_grav_bw:LS175
- added U?: LS191, symbol atari_grav_bw:LS191
Connections:
- wire segments 152 -> 153
Other:
- moved on the sheet: E_3B, F_5B, H_3A, H_5A, K_5B, K_6C, L_3A, L_6A, M_6, N_6, P_6, R_6

Commit message: JBB Sheet 7a
Parts:
- added U? (x3): LS02, symbol atari_grav_bw:LS02
- added U? (x2): LS32, symbol atari_grav_bw:LS32
- added U?: LS00, symbol atari_grav_bw:LS00
- added U?: LS04, symbol atari_grav_bw:LS04
- gave numbers to parts that had none: 2
Connections:
- wire segments 153 -> 176
- no-connect marks 3 -> 12
Other:
- moved on the sheet: C_7, D_7
Changed lines of the file:
@@
 PR55
-Wire Wire Line
-	7150 10625 6350 10625
 Wire Wire Line
 	7900 11625 7775 11625
@@
 Text GLabel 22125 9925 2    50   Input ~ 0
 ~SCALELD
-Wire Wire Line
-	22125 9925 6350 9925
 Wire Wire Line
 	7150 10425 7150 9800
@@
 13CF
 Wire Notes Line
-	1725 8100 6200 8100
-Wire Notes Line
-	1700 8125 1675 8125
-Wire Notes Line
-	1700 12425 1700 8125
-Wire Notes Line
-	6200 12425 1700 12425
-Wire Notes Line
-	6200 8100 6200 12425
-$Comp
-L atari_grav_bw:LS175 U?
+	1600 8525 6075 8525
+Wire Notes Line
+	1575 8550 1550 8550
+Wire Notes Line
+	1575 12850 1575 8550
+Wire Notes Line
+	6075 12850 1575 12850
+Wire Notes Line
+	6075 8525 6075 12850
+Wire Wire Line
+	1550 11575 1550 11775
+$Comp
+L atari_grav_bw:LS191 C_7
+U 1 1 61E3075F
+P 4625 11775
+F 0 "C_7" H 4600 11800 50  0000 C CNN
+F 1 "LS191" H 4600 11650 50  0000 C CNN
+F 2 "" H 4625 11775 50  0001 C CNN
+F 3 "" H 4625 11775 50  0001 C CNN
+	1    4625 11775
+	1    0    0    -1
+$EndComp
+Wire Wire Line
+	3925 11775 2900 11775
+$Comp
+L atari_grav_bw:LS175 D_7
 U 1 1 61DFA64A
-P 2325 11500
-F 0 "U?" H 2325 12481 50  0000 C CNN
-F 1 "LS175" H 2325 12390 50  0000 C CNN
-F 2 "" H 2325 11500 50  0001 C CNN
-F 3 "" H 2325 11500 50  0001 C CNN
-	1    2325 11500
-	1    0    0    -1
-$EndComp
-Wire Wire Line
-	1675 11150 1675 11350
-$Comp
-L atari_grav_bw:LS191 U?
-U 1 1 61E3075F
-P 4750 11475
-F 0 "U?" H 4750 10636 50  0000 C CNN
-F 1 "LS191" H 4750 10545 50  0000 C CNN
-F 2 "" H 4750 11475 50  0001 C CNN
-F 3 "" H 4750 11475 50  0001 C CNN
-	1    4750 11475
-	1    0    0    -1
-$EndComp
+P 2200 11925
+F 0 "D_7" H 2150 12025 50  0000 C CNN
+F 1 "LS175" H 2175 11875 50  0000 C CNN
+F 2 "" H 2200 11925 50  0001 C CNN
+F 3 "" H 2200 11925 50  0001 C CNN
+	1    2200 11925
+	1    0    0    -1
+$EndComp
+NoConn ~ 2900 11575
+NoConn ~ 2900 11675
+NoConn ~ 2900 11875
+NoConn ~ 2900 12075
+NoConn ~ 2900 12275
+NoConn ~ 5325 11525
+NoConn ~ 5325 11675
+NoConn ~ 5325 11825
+NoConn ~ 5325 11975
+Wire Wire Line
+	3925 11925 3025 11925
+Wire Wire Line
+	3025 11925 3025 11975
+Wire Wire Line
+	3025 11975 2900 11975
+Wire Wire Line
+	3925 12075 3650 12075
+Wire Wire Line
+	3650 12075 3650 12175
+Wire Wire Line
+	3650 12175 2900 12175
+$Comp
+L atari_grav_bw:LS02 U?
+U 2 1 61E940EB
+P 5475 10625
+F 0 "U?" H 5475 10991 50  0000 C CNN
+F 1 "LS02" H 5475 10900 50  0000 C CNN
+F 2 "" H 5475 10625 50  0001 C CNN
+F 3 "" H 5475 10625 50  0001 C CNN
+	2    5475 10625
+	1    0    0    -1
+$EndComp
+$Comp
+L atari_grav_bw:LS32 U?
+U 2 1 61EADD35
+P 5450 9925
+F 0 "U?" H 5450 10225 50  0000 C CNN
+F 1 "LS32" H 5450 10134 50  0000 C CNN
+F 2 "" H 5450 9925 50  0001 C CNN
+F 3 "" H 5450 9925 50  0001 C CNN
+	2    5450 9925
+	1    0    0    -1
+$EndComp
+$Comp
+L atari_grav_bw:LS32 U?
+U 3 1 61EAF1AE
+P 5425 9250
+F 0 "U?" H 5425 9550 50  0000 C CNN
+F 1 "LS32" H 5425 9459 50  0000 C CNN
+F 2 "" H 5425 9250 50  0001 C CNN
+F 3 "" H 5425 9250 50  0001 C CNN
+	3    5425 9250
+	1    0    0    -1
+$EndComp
+$Comp
+L atari_grav_bw:LS00 U?
+U 2 1 61EB1716
+P 3975 9550
+F 0 "U?" H 3975 9915 50  0000 C CNN
+F 1 "LS00" H 3975 9824 50  0000 C CNN
+F 2 "" H 3975 9550 50  0001 C CNN
+F 3 "" H 3975 9550 50  0001 C CNN
+	2    3975 9550
+	1    0    0    -1
+$EndComp
+$Comp
+L atari_grav_bw:LS02 U?
+U 1 1 61EB33A3
+P 3925 8825
+F 0 "U?" H 4569 8884 50  0000 L CNN
+F 1 "LS02" H 4569 8793 50  0000 L CNN
+F 2 "" H 3925 8825 50  0001 C CNN
+F 3 "" H 3925 8825 50  0001 C CNN
+	1    3925 8825
+	1    0    0    -1
+$EndComp
+$Comp
+L atari_grav_bw:LS02 U?
+U 2 1 61EB3F53
+P 2450 9450
+F 0 "U?" H 2450 9816 50  0000 C CNN
+F 1 "LS02" H 2450 9725 50  0000 C CNN
+F 2 "" H 2450 9450 50  0001 C CNN
+F 3 "" H 2450 9450 50  0001 C CNN
+	2    2450 9450
+	1    0    0    -1
+$EndComp
+$Comp
+L atari_grav_bw:LS04 U?
+U 4 1 61EB53A6
+P 4525 10425
+F 0 "U?" V 4479 10603 50  0000 L CNN
+F 1 "LS04" V 4570 10603 50  0000 L CNN
+F 2 "" H 4525 10425 50  0001 C CNN
+F 3 "" H 4525 10425 50  0001 C CNN
+	4    4525 10425
+	0    1    1    0
+$EndComp
+Wire Wire Line
+	5075 9175 4925 9175
+Wire Wire Line
+	4925 9175 4925 10000
+Wire Wire Line
+	4925 10000 5100 10000
+Wire Wire Line
+	4525 8825 4525 9975
+Wire Wire Line
+	4525 10875 4525 11025
+Wire Wire Line
+	4525 10100 4800 10100
+Wire Wire Line
+	4800 10100 4800 10725
+Wire Wire Line
+	4800 10725 4875 10725
+Wire Wire Line
+	4875 10525 4875 10725
+Wire Wire Line
+	4875 11225 5475 11225
+Wire Wire Line
+	5475 11225 5475 12700
+Wire Wire Line
+	5475 12700 4525 12700
+Wire Wire Line
+	4525 12700 4525 12525
+Connection ~ 4875 10725
+Wire Wire Line
+	4875 10725 4875 11225
+Wire Wire Line
+	6075 10625 7150 10625
+Wire Wire Line
+	5800 9925 22125 9925
+Wire Wire Line
+	3375 9650 3375 9450
+Wire Wire Line
+	3375 9450 3050 9450
+Connection ~ 3375 9450
 $EndSCHEMATC

Commit message: More Sheet 7a
Parts:
- added L_5: LS74, symbol atari_grav_bw:LS74
- added unit 4 of L_6
- added R82: 4.7K, symbol Device:R
- F_3: renamed from U?; value LS04 -> S04
- gave numbers to parts that had none: 4
Connections:
- net labels added: DVY10, DVY8, DVY9, ~DVY12, ~RESET, ~STROBE1, ~STROBE2, ~VGGO, ~VGRST
- wire segments 176 -> 204
- no-connect marks 12 -> 13
Other:
- note added: "Halt\nFlag\n"
- note added: "VECTOR SCALING\n"
Changed lines of the file:
@@
 Wire Notes Line
 	6075 8525 6075 12850
-Wire Wire Line
-	1550 11575 1550 11775
 $Comp
 L atari_grav_bw:LS191 C_7
@@
 	3650 12175 2900 12175
 $Comp
-L atari_grav_bw:LS02 U?
-U 2 1 61E940EB
-P 5475 10625
-F 0 "U?" H 5475 10991 50  0000 C CNN
-F 1 "LS02" H 5475 10900 50  0000 C CNN
-F 2 "" H 5475 10625 50  0001 C CNN
-F 3 "" H 5475 10625 50  0001 C CNN
-	2    5475 10625
-	1    0    0    -1
-$EndComp
-$Comp
-L atari_grav_bw:LS32 U?
-U 2 1 61EADD35
-P 5450 9925
-F 0 "U?" H 5450 10225 50  0000 C CNN
-F 1 "LS32" H 5450 10134 50  0000 C CNN
-F 2 "" H 5450 9925 50  0001 C CNN
-F 3 "" H 5450 9925 50  0001 C CNN
-	2    5450 9925
-	1    0    0    -1
-$EndComp
-$Comp
-L atari_grav_bw:LS32 U?
-U 3 1 61EAF1AE
-P 5425 9250
-F 0 "U?" H 5425 9550 50  0000 C CNN
-F 1 "LS32" H 5425 9459 50  0000 C CNN
-F 2 "" H 5425 9250 50  0001 C CNN
-F 3 "" H 5425 9250 50  0001 C CNN
-	3    5425 9250
-	1    0    0    -1
-$EndComp
-$Comp
-L atari_grav_bw:LS00 U?
+L atari_grav_bw:LS00 L_3
 U 2 1 61EB1716
 P 3975 9550
-F 0 "U?" H 3975 9915 50  0000 C CNN
-F 1 "LS00" H 3975 9824 50  0000 C CNN
+F 0 "L_3" H 3950 9625 50  0000 C CNN
+F 1 "LS00" H 3950 9525 50  0000 C CNN
 F 2 "" H 3975 9550 50  0001 C CNN
 F 3 "" H 3975 9550 50  0001 C CNN
@@
 $EndComp
 $Comp
-L atari_grav_bw:LS02 U?
-U 1 1 61EB33A3
+L atari_grav_bw:LS02 B_7
+U 1 2 61EB33A3
 P 3925 8825
-F 0 "U?" H 4569 8884 50  0000 L CNN
-F 1 "LS02" H 4569 8793 50  0000 L CNN
+F 0 "B_7" H 3925 8900 50  0000 L CNN
+F 1 "LS02" H 3925 8800 50  0000 L CNN
 F 2 "" H 3925 8825 50  0001 C CNN
 F 3 "" H 3925 8825 50  0001 C CNN
 	1    3925 8825
-	1    0    0    -1
-$EndComp
-$Comp
-L atari_grav_bw:LS02 U?
-U 2 1 61EB3F53
+	1    0    0    1
+$EndComp
+$Comp
+L atari_grav_bw:LS02 N_5
+U 2 2 61EB3F53
 P 2450 9450
-F 0 "U?" H 2450 9816 50  0000 C CNN
-F 1 "LS02" H 2450 9725 50  0000 C CNN
+F 0 "N_5" H 2425 9500 50  0000 C CNN
+F 1 "LS02" H 2425 9400 50  0000 C CNN
 F 2 "" H 2450 9450 50  0001 C CNN
 F 3 "" H 2450 9450 50  0001 C CNN
@@
 $EndComp
 $Comp
-L atari_grav_bw:LS04 U?
+L atari_grav_bw:LS04 F_3
 U 4 1 61EB53A6
 P 4525 10425
-F 0 "U?" V 4479 10603 50  0000 L CNN
-F 1 "LS04" V 4570 10603 50  0000 L CNN
+F 0 "F_3" V 4325 10225 50  0000 L CNN
+F 1 "S04" V 4650 10225 50  0000 L CNN
 F 2 "" H 4525 10425 50  0001 C CNN
 F 3 "" H 4525 10425 50  0001 C CNN
@@
 $EndComp
 Wire Wire Line
-	5075 9175 4925 9175
-Wire Wire Line
-	4925 9175 4925 10000
-Wire Wire Line
-	4925 10000 5100 10000
-Wire Wire Line
 	4525 8825 4525 9975
 Wire Wire Line
 	4525 10875 4525 11025
 Wire Wire Line
-	4525 10100 4800 10100
-Wire Wire Line
-	4800 10100 4800 10725
-Wire Wire Line
-	4800 10725 4875 10725
-Wire Wire Line
-	4875 10525 4875 10725
-Wire Wire Line
-	4875 11225 5475 11225
-Wire Wire Line
-	5475 11225 5475 12700
-Wire Wire Line
 	5475 12700 4525 12700
 Wire Wire Line
 	4525 12700 4525 12525
-Connection ~ 4875 10725
-Wire Wire Line
-	4875 10725 4875 11225
-Wire Wire Line
-	6075 10625 7150 10625
+Wire Wire Line
+	6075 10625 6250 10625
 Wire Wire Line
 	5800 9925 22125 9925
@@
 	3375 9450 3050 9450
 Connection ~ 3375 9450
+$Comp
+L atari_grav_bw:LS32 J_6
+U 3 2 61EAF1AE
+P 5425 9250
+F 0 "J_6" H 5400 9225 50  0000 C CNN
+F 1 "LS32" H 5400 9325 50  0000 C CNN
+F 2 "" H 5425 9250 50  0001 C CNN
+F 3 "" H 5425 9250 50  0001 C CNN
+	3    5425 9250
+	1    0    0    1
+$EndComp
+$Comp
+L atari_grav_bw:LS32 J_6
+U 2 2 61EADD35
+P 5450 9925
+F 0 "J_6" H 5425 9900 50  0000 C CNN
+F 1 "LS32" H 5425 10000 50  0000 C CNN
+F 2 "" H 5450 9925 50  0001 C CNN
+F 3 "" H 5450 9925 50  0001 C CNN
+	2    5450 9925
+	1    0    0    1
+$EndComp
+Wire Wire Line
+	4825 9350 4825 9550
+Wire Wire Line
+	4825 9825 4850 9825
+Wire Wire Line
+	4850 10025 1450 10025
+Wire Wire Line
+	1850 9550 1450 9550
+Wire Wire Line
+	1850 9350 1850 8925
+Wire Wire Line
+	3325 8725 1450 8725
+Wire Wire Line
+	3325 8925 1850 8925
+Connection ~ 1850 8925
+Wire Wire Line
+	1850 8925 1850 8275
+Wire Wire Line
+	4575 9550 4825 9550
+Connection ~ 4825 9550
+Wire Wire Line
+	4825 9550 4825 9825
+Wire Wire Line
+	4825 9150 4825 8300
+Wire Wire Line
+	6025 9250 6350 9250
+NoConn ~ 4875 12525
+Wire Wire Line
+	4325 12525 4325 12975
+Wire Wire Line
+	6250 11125 6250 10625
+Wire Wire Line
+	2050 11125 6250 11125
+Connection ~ 6250 10625
+Wire Wire Line
+	6250 10625 7150 10625
+$Comp
+L atari_grav_bw:LS02 B_7
+U 2 2 61E940EB
+P 5475 10625
+F 0 "B_7" H 5450 10600 50  0000 C CNN
+F 1 "LS02" H 5450 10700 50  0000 C CNN
+F 2 "" H 5475 10625 50  0001 C CNN
+F 3 "" H 5475 10625 50  0001 C CNN
+	2    5475 10625
+	1    0    0    1
+$EndComp
+Wire Wire Line
+	1500 11775 1475 11775
+Wire Wire Line
+	1500 11575 1475 11575
+Wire Wire Line
+	1475 11575 1475 11775
+Connection ~ 1475 11575
+Wire Wire Line
+	1475 11575 1450 11575
+Connection ~ 1475 11775
+Wire Wire Line
+	1475 11775 1450 11775
+Wire Wire Line
+	1500 11925 1425 11925
+Wire Wire Line
+	1500 12075 1425 12075
+Wire Wire Line
+	4525 10200 4875 10200
+Wire Wire Line
+	4875 10200 4875 10525
+Wire Wire Line
+	4875 10725 4850 10725
+Wire Wire Line
+	4725 10725 4725 11025
+Wire Wire Line
+	5475 10900 4850 10900
+Wire Wire Line
+	4850 10900 4850 10725
+Wire Wire Line
+	5475 10900 5475 12700
+Connection ~ 4850 10725
+Wire Wire Line
+	4850 10725 4725 10725
+Text Notes 2250 10550 0    100  ~ 20
+VECTOR SCALING\n
+$Comp
+L Device:R R82
+U 1 1 620FF205
+P 4625 10875
+F 0 "R82" H 4695 10921 50  0000 L CNN
+F 1 "4.7K" H 4695 10830 50  0000 L CNN
+F 2 "" V 4555 10875 50  0001 C CNN
+F 3 "~" H 4625 10875 50  0001 C CNN
+	1    4625 10875
+	1    0    0    -1
+$EndComp
+Wire Notes Line
+	3625 8425 7400 8425
+Wire Notes Line
+	7400 8425 7400 6950
+Wire Notes Line
+	7400 6950 3625 6950
+Wire Notes Line
+	3625 6950 3625 8425
+Text Notes 4000 8200 0    100  ~ 20
+Halt\nFlag\n
+$Comp
+L atari_grav_bw:LS08 L_6
+U 4 2 6211CB8D
+P 4300 7175
+F 0 "L_6" H 4275 7075 50  0000 C CNN
+F 1 "LS08" H 4275 7175 50  0000 C CNN
+F 2 "" H 4300 7175 50  0001 C CNN
+F 3 "" H 4300 7175 50  0001 C CNN
+	4    4300 7175
+	1    0    0    1
+$EndComp
+$Comp
+L atari_grav_bw:LS74 L_5
+U 1 1 6212B505
+P 6750 7800
+F 0 "L_5" H 6800 7850 50  0000 L CNN
+F 1 "LS74" H 6800 7750 50  0000 L CNN
+F 2 "" H 6775 7550 300 0001 C CNN
+F 3 "" H 6775 7550 300 0001 C CNN
+	1    6750 7800
+	1    0    0    -1
+$EndComp
+Wire Wire Line
+	4900 7175 6175 7175
+Wire Wire Line
+	6600 7175 6600 7200
+Wire Wire Line
+	3700 7075 1950 7075
+Wire Wire Line
+	3700 7275 1950 7275
+Wire Wire Line
+	2050 12725 6175 12725
+Wire Wire Line
+	6175 12725 6175 7175
+Connection ~ 6175 7175
+Wire Wire Line
+	6175 7175 6600 7175
+Wire Wire Line
+	6600 8400 1950 8400
+Text GLabel 1950 7075 0    50   Input ~ 0
+~RESET
+Text GLabel 1950 7275 0    50   Input ~ 0
+~VGRST
+Text GLabel 1450 8725 0    50   Input ~ 0
+~STROBE1
+Text GLabel 1450 9550 0    50   Input ~ 0
+~STROBE2
+Text GLabel 1450 10025 0    50   Input ~ 0
+~DVY12
+Text GLabel 1450 11775 0    50   Input ~ 0
+DVY10
+Text GLabel 1425 11925 0    50   Input ~ 0
+DVY9
+Text GLabel 1425 12075 0    50   Input ~ 0
+DVY8
+Text GLabel 1950 8400 0    50   Input ~ 0
+~VGGO
 $EndSCHEMATC

Commit message: Power for John
sheet 7B
Parts:
- removed R82: 4.7K, symbol Device:R
Connections:
- net labels added: PR82
Changed lines of the file:
@@
 Text Notes 2250 10550 0    100  ~ 20
 VECTOR SCALING\n
-$Comp
-L Device:R R82
-U 1 1 620FF205
-P 4625 10875
-F 0 "R82" H 4695 10921 50  0000 L CNN
-F 1 "4.7K" H 4695 10830 50  0000 L CNN
-F 2 "" V 4555 10875 50  0001 C CNN
-F 3 "~" H 4625 10875 50  0001 C CNN
-	1    4625 10875
-	1    0    0    -1
-$EndComp
 Wire Notes Line
 	3625 8425 7400 8425
@@
 Text GLabel 1950 8400 0    50   Input ~ 0
 ~VGGO
+Text GLabel 4625 11025 1    50   Input ~ 0
+PR82
+$Comp
+L power:GND #PWR?
+U 1 1 61DA4F12
+P 8100 7925
+AR Path="/6B0E57BF/61DA4F12" Ref="#PWR?"  Part="1"
+AR Path="/6B32D907/61DA4F12" Ref="#PWR?"  Part="1"
+F 0 "#PWR?" H 8100 7675 50  0001 C CNN
+F 1 "GND" H 8250 7850 50  0000 C CNN
+F 2 "" H 8100 7925 50  0001 C CNN
+F 3 "" H 8100 7925 50  0001 C CNN
+	1    8100 7925
+	1    0    0    -1
+$EndComp
+$Comp
+L power:+5V #PWR?
+U 1 1 61DA4F18
+P 8125 7725
+AR Path="/6B0E57BF/61DA4F18" Ref="#PWR?"  Part="1"
+AR Path="/6B32D907/61DA4F18" Ref="#PWR?"  Part="1"
+F 0 "#PWR?" H 8125 7575 50  0001 C CNN
+F 1 "+5V" H 8250 7800 50  0000 C CNN
+F 2 "" H 8125 7725 50  0001 C CNN
+F 3 "" H 8125 7725 50  0001 C CNN
+	1    8125 7725
+	1    0    0    -1
+$EndComp
+$Comp
+L power:+5V #PWR?
+U 1 1 61DB1F66
+P 7000 7400
+AR Path="/6B0E57BF/61DB1F66" Ref="#PWR?"  Part="1"
+AR Path="/6B32D907/61DB1F66" Ref="#PWR?"  Part="1"
+F 0 "#PWR?" H 7000 7250 50  0001 C CNN
+F 1 "+5V" H 7125 7475 50  0000 C CNN
+F 2 "" H 7000 7400 50  0001 C CNN
+F 3 "" H 7000 7400 50  0001 C CNN
+	1    7000 7400
+	1    0    0    -1
+$EndComp
+$Comp
+L power:GND #PWR?
+U 1 1 61DB2F01
+P 7000 8200
+AR Path="/6B0E57BF/61DB2F01" Ref="#PWR?"  Part="1"
+AR Path="/6B32D907/61DB2F01" Ref="#PWR?"  Part="1"
+F 0 "#PWR?" H 7000 7950 50  0001 C CNN
+F 1 "GND" H 7150 8125 50  0000 C CNN
+F 2 "" H 7000 8200 50  0001 C CNN
+F 3 "" H 7000 8200 50  0001 C CNN
+	1    7000 8200
+	1    0    0    -1
+$EndComp
+$Comp
+L power:+5V #PWR?
+U 1 1 61DB3B89
+P 4825 11025
+AR Path="/6B0E57BF/61DB3B89" Ref="#PWR?"  Part="1"
+AR Path="/6B32D907/61DB3B89" Ref="#PWR?"  Part="1"
+F 0 "#PWR?" H 4825 10875 50  0001 C CNN
+F 1 "+5V" H 4950 11100 50  0000 C CNN
+F 2 "" H 4825 11025 50  0001 C CNN
+F 3 "" H 4825 11025 50  0001 C CNN
+	1    4825 11025
+	1    0    0    -1
+$EndComp
+$Comp
+L power:GND #PWR?
+U 1 1 61DC0F1C
+P 4375 11025
+AR Path="/6B0E57BF/61DC0F1C" Ref="#PWR?"  Part="1"
+AR Path="/6B32D907/61DC0F1C" Ref="#PWR?"  Part="1"
+F 0 "#PWR?" H 4375 10775 50  0001 C CNN
+F 1 "GND" H 4525 10950 50  0000 C CNN
+F 2 "" H 4375 11025 50  0001 C CNN
+F 3 "" H 4375 11025 50  0001 C CNN
+	1    4375 11025
+	-1   0    0    1
+$EndComp
+$Comp
+L power:GND #PWR?
+U 1 1 61DDA98B
+P 2375 12425
+AR Path="/6B0E57BF/61DDA98B" Ref="#PWR?"  Part="1"
+AR Path="/6B32D907/61DDA98B" Ref="#PWR?"  Part="1"
+F 0 "#PWR?" H 2375 12175 50  0001 C CNN
+F 1 "GND" H 2525 12350 50  0000 C CNN
+F 2 "" H 2375 12425 50  0001 C CNN
+F 3 "" H 2375 12425 50  0001 C CNN
+	1    2375 12425
+	1    0    0    -1
+$EndComp
+$Comp
+L power:+5V #PWR?
+U 1 1 61DDBC08
+P 2375 11425
+AR Path="/6B0E57BF/61DDBC08" Ref="#PWR?"  Part="1"
+AR Path="/6B32D907/61DDBC08" Ref="#PWR?"  Part="1"
+F 0 "#PWR?" H 2375 11275 50  0001 C CNN
+F 1 "+5V" H 2500 11500 50  0000 C CNN
+F 2 "" H 2375 11425 50  0001 C CNN
+F 3 "" H 2375 11425 50  0001 C CNN
+	1    2375 11425
+	1    0    0    -1
+$EndComp
 $EndSCHEMATC

Commit message: SHEET 7A
Parts:
- added U?: LS32, symbol atari_grav_bw:LS32
- added U?: LS02, symbol atari_grav_bw:LS02
- added U?: LS109, symbol Star_Wars_Vector_PCB:LS109
Other:
- note added: "CENTER FLAG\n"
- note added: "GO FLAG\n"
- note added: "NORMALIZATION FLAG\n\n"
- note added: "VECTOR FLAG\n"
Changed lines of the file:
@@
 Wire Notes Line
 	7400 6950 3625 6950
-Wire Notes Line
-	3625 6950 3625 8425
 Text Notes 4000 8200 0    100  ~ 20
 Halt\nFlag\n
@@
 L power:GND #PWR?
 U 1 1 61DA4F12
-P 8100 7925
+P 6375 1450
 AR Path="/6B0E57BF/61DA4F12" Ref="#PWR?"  Part="1"
 AR Path="/6B32D907/61DA4F12" Ref="#PWR?"  Part="1"
-F 0 "#PWR?" H 8100 7675 50  0001 C CNN
-F 1 "GND" H 8250 7850 50  0000 C CNN
-F 2 "" H 8100 7925 50  0001 C CNN
-F 3 "" H 8100 7925 50  0001 C CNN
-	1    8100 7925
+F 0 "#PWR?" H 6375 1200 50  0001 C CNN
+F 1 "GND" H 6525 1375 50  0000 C CNN
+F 2 "" H 6375 1450 50  0001 C CNN
+F 3 "" H 6375 1450 50  0001 C CNN
+	1    6375 1450
 	1    0    0    -1
 $EndComp
@@
 L power:+5V #PWR?
 U 1 1 61DA4F18
-P 8125 7725
+P 6400 1250
 AR Path="/6B0E57BF/61DA4F18" Ref="#PWR?"  Part="1"
 AR Path="/6B32D907/61DA4F18" Ref="#PWR?"  Part="1"
-F 0 "#PWR?" H 8125 7575 50  0001 C CNN
-F 1 "+5V" H 8250 7800 50  0000 C CNN
-F 2 "" H 8125 7725 50  0001 C CNN
-F 3 "" H 8125 7725 50  0001 C CNN
-	1    8125 7725
+F 0 "#PWR?" H 6400 1100 50  0001 C CNN
+F 1 "+5V" H 6525 1325 50  0000 C CNN
+F 2 "" H 6400 1250 50  0001 C CNN
+F 3 "" H 6400 1250 50  0001 C CNN
+	1    6400 1250
 	1    0    0    -1
 $EndComp
@@
 	1    0    0    -1
 $EndComp
+Wire Notes Line
+	7400 7800 13525 7800
+Wire Notes Line
+	13525 7800 13525 9675
+Wire Notes Line
+	10925 9675 10925 5525
+Wire Notes Line
+	3625 5575 3625 8425
+Wire Notes Line
+	12025 3225 2550 3225
+Wire Notes Line
+	2550 3225 2550 5550
+Wire Notes Line
+	2550 5550 12025 5550
+Wire Notes Line
+	12025 4675 16950 4675
+Wire Notes Line
+	16950 4675 16950 825
+Wire Notes Line
+	16950 825  12025 825
+Wire Notes Line
+	12025 825  12025 5550
+Text Notes 4950 5975 0    100  ~ 20
+VECTOR FLAG\n
+Text Notes 6125 3775 0    100  ~ 20
+CENTER FLAG\n
+Text Notes 10925 8825 0    100  ~ 20
+GO FLAG\n
+Text Notes 12125 1750 0    100  ~ 20
+NORMALIZATION FLAG\n\n
+$Comp
+L atari_grav_bw:LS32 U?
+U 1 2 61E7524F
+P 3675 4625
+F 0 "U?" H 3675 4990 50  0000 C CNN
+F 1 "LS32" H 3675 4899 50  0000 C CNN
+F 2 "" H 3675 4625 50  0001 C CNN
+F 3 "" H 3675 4625 50  0001 C CNN
+	1    3675 4625
+	1    0    0    -1
+$EndComp
+$Comp
+L atari_grav_bw:LS02 U?
+U 3 2 61E91B85
+P 4600 3800
+F 0 "U?" H 4600 3434 50  0000 C CNN
+F 1 "LS02" H 4600 3525 50  0000 C CNN
+F 2 "" H 4600 3800 50  0001 C CNN
+F 3 "" H 4600 3800 50  0001 C CNN
+	3    4600 3800
+	1    0    0    1
+$EndComp
+$Comp
+L Star_Wars_Vector_PCB:LS109 U?
+U 2 1 61EA090B
+P 8650 4450
+F 0 "U?" H 8650 5431 50  0000 C CNN
+F 1 "LS109" H 8650 5340 50  0000 C CNN
+F 2 "" H 8650 4450 50  0001 C CNN
+F 3 "" H 8650 4450 50  0001 C CNN
+	2    8650 4450
+	1    0    0    -1
+$EndComp

Commit message: SHEET 7A
Parts:
- removed U?: LS109, symbol Star_Wars_Vector_PCB:LS109
- added E_5: LS109A, symbol atari_grav_bw:LS109A
- added unit 2 of L_6
- gave numbers to parts that had none: 2
Changed lines of the file:
@@
 NORMALIZATION FLAG\n\n
 $Comp
-L atari_grav_bw:LS32 U?
+L atari_grav_bw:LS32 M_5
 U 1 2 61E7524F
 P 3675 4625
-F 0 "U?" H 3675 4990 50  0000 C CNN
-F 1 "LS32" H 3675 4899 50  0000 C CNN
+F 0 "M_5" H 3650 4750 50  0000 C CNN
+F 1 "LS32" H 3650 4625 50  0000 C CNN
 F 2 "" H 3675 4625 50  0001 C CNN
 F 3 "" H 3675 4625 50  0001 C CNN
@@
 $EndComp
 $Comp
-L atari_grav_bw:LS02 U?
+L atari_grav_bw:LS02 K_5
 U 3 2 61E91B85
 P 4600 3800
-F 0 "U?" H 4600 3434 50  0000 C CNN
-F 1 "LS02" H 4600 3525 50  0000 C CNN
+F 0 "K_5" H 4575 3700 50  0000 C CNN
+F 1 "LS02" H 4575 3800 50  0000 C CNN
 F 2 "" H 4600 3800 50  0001 C CNN
 F 3 "" H 4600 3800 50  0001 C CNN
@@
 $EndComp
 $Comp
-L Star_Wars_Vector_PCB:LS109 U?
-U 2 1 61EA090B
-P 8650 4450
-F 0 "U?" H 8650 5431 50  0000 C CNN
-F 1 "LS109" H 8650 5340 50  0000 C CNN
-F 2 "" H 8650 4450 50  0001 C CNN
-F 3 "" H 8650 4450 50  0001 C CNN
-	2    8650 4450
+L atari_grav_bw:LS109A E_5
+U 2 1 61D49212
+P 8725 4425
+F 0 "E_5" H 8725 4575 50  0000 C CNN
+F 1 "LS109A" H 8725 4425 50  0000 C CNN
+F 2 "" H 8725 4425 50  0001 C CNN
+F 3 "" H 8725 4425 50  0001 C CNN
+	2    8725 4425
 	1    0    0    -1
 $EndComp
+$Comp
+L Star_Wars_Vector_PCB:LS08 L_6
+U 2 1 61D58647
+P 10850 4675
+F 0 "L_6" H 10850 4625 50  0000 C CNN
+F 1 "LS08" H 10850 4725 50  0000 C CNN
+F 2 "" H 10850 4675 50  0001 C CNN
+F 3 "" H 10850 4675 50  0001 C CNN
+	2    10850 4675
+	1    0    0    1
+$EndComp
 $EndSCHEMATC
