File: kicad/atari_gravitar_black_widow/Sheet7A.sch (KiCad schematic (older format))
At the start: 27 parts

Commit message: 7A
Parts:
- added K_4: LS10, symbol atari_grav_bw:LS10
- A_6: renamed from U?; value LS74 -> S74
- B6, B_6: renamed from U?; value LS86 -> S86
Connections:
- wire segments 204 -> 220
- no-connect marks 13 -> 14
Other:
- moved on the sheet: A_6A, B6A, B_6B
Changed lines of the file:
@@
 	7150 10425 7150 9800
 Wire Wire Line
-	7150 9800 16875 9800
-Wire Wire Line
-	16875 9800 16875 9425
+	7150 9800 15600 9800
 Wire Wire Line
 	14625 12175 15175 12175
@@
 PR82
 $Comp
-L power:GND #PWR?
-U 1 1 61DA4F12
-P 6375 1450
-AR Path="/6B0E57BF/61DA4F12" Ref="#PWR?"  Part="1"
-AR Path="/6B32D907/61DA4F12" Ref="#PWR?"  Part="1"
-F 0 "#PWR?" H 6375 1200 50  0001 C CNN
-F 1 "GND" H 6525 1375 50  0000 C CNN
-F 2 "" H 6375 1450 50  0001 C CNN
-F 3 "" H 6375 1450 50  0001 C CNN
-	1    6375 1450
-	1    0    0    -1
-$EndComp
-$Comp
-L power:+5V #PWR?
-U 1 1 61DA4F18
-P 6400 1250
-AR Path="/6B0E57BF/61DA4F18" Ref="#PWR?"  Part="1"
-AR Path="/6B32D907/61DA4F18" Ref="#PWR?"  Part="1"
-F 0 "#PWR?" H 6400 1100 50  0001 C CNN
-F 1 "+5V" H 6525 1325 50  0000 C CNN
-F 2 "" H 6400 1250 50  0001 C CNN
-F 3 "" H 6400 1250 50  0001 C CNN
-	1    6400 1250
-	1    0    0    -1
-$EndComp
-$Comp
 L power:+5V #PWR?
 U 1 1 61DB1F66
@@
 Text Notes 10925 8825 0    100  ~ 20
 GO FLAG\n
-Text Notes 12125 1750 0    100  ~ 20
+Text Notes 12325 1425 0    100  ~ 20
 NORMALIZATION FLAG\n\n
 $Comp
@@
 $EndComp
 $Comp
-L Star_Wars_Vector_PCB:LS86 U?
-U 2 1 61D76815
-P 12950 2175
-F 0 "U?" H 12950 1810 50  0000 C CNN
-F 1 "LS86" H 12950 1901 50  0000 C CNN
-F 2 "" H 12950 2175 50  0001 C CNN
-F 3 "" H 12950 2175 50  0001 C CNN
-	2    12950 2175
-	1    0    0    1
-$EndComp
-$Comp
-L Star_Wars_Vector_PCB:LS86 U?
+L Star_Wars_Vector_PCB:LS86 B6
 U 1 1 61D8458C
-P 12975 3500
-F 0 "U?" H 12975 3109 50  0000 C CNN
-F 1 "LS86" H 12975 3200 50  0000 C CNN
-F 2 "" H 12975 3500 50  0001 C CNN
-F 3 "" H 12975 3500 50  0001 C CNN
-	1    12975 3500
-	1    0    0    1
-$EndComp
-$Comp
-L atari_grav_bw:LS74 U?
+P 12975 3250
+F 0 "B6" H 13000 3175 50  0000 C CNN
+F 1 "S86" H 13025 3275 50  0000 C CNN
+F 2 "" H 12975 3250 50  0001 C CNN
+F 3 "" H 12975 3250 50  0001 C CNN
+	1    12975 3250
+	1    0    0    1
+$EndComp
+$Comp
+L atari_grav_bw:LS74 A_6
 U 1 1 61D9391A
-P 15550 2650
-F 0 "U?" H 16194 2696 50  0000 L CNN
-F 1 "LS74" H 16194 2605 50  0000 L CNN
-F 2 "" H 15575 2400 300 0001 C CNN
-F 3 "" H 15575 2400 300 0001 C CNN
-	1    15550 2650
-	1    0    0    -1
-$EndComp
-Text GLabel 1200 825  0    50   Input ~ 0
+P 14675 1900
+F 0 "A_6" H 14650 1975 50  0000 L CNN
+F 1 "S74" H 14650 1875 50  0000 L CNN
+F 2 "" H 14700 1650 300 0001 C CNN
+F 3 "" H 14700 1650 300 0001 C CNN
+	1    14675 1900
+	1    0    0    -1
+$EndComp
+Text GLabel 1975 950  0    50   Input ~ 0
 ~SA
-Text GLabel 1250 1100 0    50   Input ~ 0
+Text GLabel 1975 1800 0    50   Input ~ 0
 ~OP0
-Text GLabel 1425 1400 0    50   Input ~ 0
+Text GLabel 1975 2000 0    50   Input ~ 0
 ~STROBE0
-Text GLabel 1325 1675 0    50   Input ~ 0
+Text GLabel 1975 2650 0    50   Input ~ 0
 DVY12
-Text GLabel 1325 1900 0    50   Input ~ 0
+Text GLabel 1975 2850 0    50   Input ~ 0
 DVY11
-Text GLabel 1325 2150 0    50   Input ~ 0
+Text GLabel 1975 3150 0    50   Input ~ 0
 DVX12
-Text GLabel 1325 2425 0    50   Input ~ 0
+Text GLabel 1975 3350 0    50   Input ~ 0
 DXV11
 Text GLabel 1325 2675 0    50   Input ~ 0
@@
 Text GLabel 1275 3650 0    50   Input ~ 0
 OP0
+$Comp
+L atari_grav_bw:LS10 K_4
+U 3 1 61D4B7A1
+P 16350 2000
+F 0 "K_4" H 16300 2125 50  0000 C CNN
+F 1 "LS10" H 16300 2000 50  0000 C CNN
+F 2 "" H 16350 2000 50  0001 C CNN
+F 3 "" H 16350 2000 50  0001 C CNN
+	3    16350 2000
+	1    0    0    -1
+$EndComp
+$Comp
+L power:+5V #PWR?
+U 1 1 61DA4F18
+P 14925 1500
+AR Path="/6B0E57BF/61DA4F18" Ref="#PWR?"  Part="1"
+AR Path="/6B32D907/61DA4F18" Ref="#PWR?"  Part="1"
+F 0 "#PWR?" H 14925 1350 50  0001 C CNN
+F 1 "+5V" H 15050 1575 50  0000 C CNN
+F 2 "" H 14925 1500 50  0001 C CNN
+F 3 "" H 14925 1500 50  0001 C CNN
+	1    14925 1500
+	1    0    0    -1
+$EndComp
+Wire Wire Line
+	1975 1800 14075 1800
+$Comp
+L power:GND #PWR?
+U 1 1 61D89427
+P 14925 2300
+AR Path="/6B0E57BF/61D89427" Ref="#PWR?"  Part="1"
+AR Path="/6B32D907/61D89427" Ref="#PWR?"  Part="1"
+F 0 "#PWR?" H 14925 2050 50  0001 C CNN
+F 1 "GND" H 15075 2225 50  0000 C CNN
+F 2 "" H 14925 2300 50  0001 C CNN
+F 3 "" H 14925 2300 50  0001 C CNN
+	1    14925 2300
+	1    0    0    -1
+$EndComp
+Wire Wire Line
+	14075 2000 1975 2000
+Text GLabel 14525 1300 1    50   Input ~ 0
+PR82
+Wire Wire Line
+	15600 1800 15275 1800
+Wire Wire Line
+	15600 1800 15600 2000
+Wire Wire Line
+	15750 2000 15600 2000
+Connection ~ 15600 2000
+Wire Wire Line
+	15600 2000 15600 9800
+Wire Wire Line
+	15750 1850 15750 950
+Wire Wire Line
+	15750 950  1975 950
+NoConn ~ 15275 2000
+Wire Wire Line
+	15750 2150 15450 2150
+Wire Wire Line
+	15450 2150 15450 2750
+Wire Wire Line
+	15450 2750 14525 2750
+Wire Wire Line
+	14525 2500 14525 2750
+Connection ~ 14525 2750
+Wire Wire Line
+	14525 2750 13575 2750
+Wire Wire Line
+	12375 3150 1975 3150
+Wire Wire Line
+	12375 3350 1975 3350
+Wire Wire Line
+	12375 2850 1975 2850
+Wire Wire Line
+	12375 2650 1975 2650
+$Comp
+L Star_Wars_Vector_PCB:LS86 B_6
+U 2 1 61D76815
+P 12975 2750
+F 0 "B_6" H 13000 2725 50  0000 C CNN
+F 1 "S86" H 13000 2650 50  0000 C CNN
+F 2 "" H 12975 2750 50  0001 C CNN
+F 3 "" H 12975 2750 50  0001 C CNN
+	2    12975 2750
+	1    0    0    -1
+$EndComp
 $EndSCHEMATC

Commit message: 7a
Parts:
- added U?: S260A, symbol atari_grav_bw:S260A
Connections:
- net labels added: GO, HALT, NORM, VCTR, ~CENTER, ~ENORM, ~STATCLK, ~VCTR
- wire segments 220 -> 241
Other:
- moved on the sheet: E_5B, L_6B
Changed lines of the file:
@@
 	7150 10425 7150 9800
-Wire Wire Line
-	7150 9800 15600 9800
 Wire Wire Line
 	14625 12175 15175 12175
@@
 L atari_grav_bw:LS109A E_5
 U 2 1 61D49212
-P 8725 4425
-F 0 "E_5" H 8725 4575 50  0000 C CNN
-F 1 "LS109A" H 8725 4425 50  0000 C CNN
-F 2 "" H 8725 4425 50  0001 C CNN
-F 3 "" H 8725 4425 50  0001 C CNN
-	2    8725 4425
+P 8850 4525
+F 0 "E_5" H 8850 4675 50  0000 C CNN
+F 1 "LS109A" H 8850 4525 50  0000 C CNN
+F 2 "" H 8850 4525 50  0001 C CNN
+F 3 "" H 8850 4525 50  0001 C CNN
+	2    8850 4525
 	1    0    0    -1
 $EndComp
@@
 L Star_Wars_Vector_PCB:LS08 L_6
 U 2 1 61D58647
-P 10850 4675
-F 0 "L_6" H 10850 4625 50  0000 C CNN
-F 1 "LS08" H 10850 4725 50  0000 C CNN
-F 2 "" H 10850 4675 50  0001 C CNN
-F 3 "" H 10850 4675 50  0001 C CNN
-	2    10850 4675
+P 10850 4800
+F 0 "L_6" H 10850 4750 50  0000 C CNN
+F 1 "LS08" H 10850 4850 50  0000 C CNN
+F 2 "" H 10850 4800 50  0001 C CNN
+F 3 "" H 10850 4800 50  0001 C CNN
+	2    10850 4800
 	1    0    0    1
 $EndComp
@@
 Text GLabel 1975 3350 0    50   Input ~ 0
 DXV11
-Text GLabel 1325 2675 0    50   Input ~ 0
+Text GLabel 1975 4425 0    50   Input ~ 0
 SCALE
 Text GLabel 1250 2925 0    50   Input ~ 0
@@
 	15600 1800 15600 2000
 Wire Wire Line
-	15750 2000 15600 2000
-Connection ~ 15600 2000
-Wire Wire Line
-	15600 2000 15600 9800
+	15750 2000 15700 2000
 Wire Wire Line
 	15750 1850 15750 950
@@
 NoConn ~ 15275 2000
 Wire Wire Line
-	15750 2150 15450 2150
-Wire Wire Line
-	15450 2150 15450 2750
-Wire Wire Line
-	15450 2750 14525 2750
-Wire Wire Line
 	14525 2500 14525 2750
-Connection ~ 14525 2750
-Wire Wire Line
-	14525 2750 13575 2750
 Wire Wire Line
 	12375 3150 1975 3150
@@
 	1    0    0    -1
 $EndComp
+Text GLabel 20325 2000 2    50   Input ~ 0
+~ENORM
+Text GLabel 20325 3000 2    50   Input ~ 0
+NORM
+Text GLabel 22000 1325 2    50   Input ~ 0
+~CENTER
+Text GLabel 20325 6300 2    50   Input ~ 0
+VCTR
+Text GLabel 22025 1750 2    50   Input ~ 0
+~VCTR
+Text GLabel 22000 1950 2    50   Input ~ 0
+HALT
+Text GLabel 22025 2125 2    50   Input ~ 0
+GO
+Text GLabel 22000 2375 2    50   Input ~ 0
+~STATCLK
+Text GLabel 22025 2550 2    50   Input ~ 0
+~SCALELD
+Text GLabel 22000 2825 2    50   Input ~ 0
+~STOP
+Wire Wire Line
+	16950 2000 20325 2000
+$Comp
+L power:GND #PWR?
+U 1 1 620431A5
+P 19675 675
+AR Path="/6B0E57BF/620431A5" Ref="#PWR?"  Part="1"
+AR Path="/6B32D907/620431A5" Ref="#PWR?"  Part="1"
+F 0 "#PWR?" H 19675 425 50  0001 C CNN
+F 1 "GND" H 19825 600 50  0000 C CNN
+F 2 "" H 19675 675 50  0001 C CNN
+F 3 "" H 19675 675 50  0001 C CNN
+	1    19675 675
+	1    0    0    -1
+$EndComp
+$Comp
+L power:+5V #PWR?
+U 1 1 62058461
+P 19725 1125
+F 0 "#PWR?" H 19725 975 50  0001 C CNN
+F 1 "+5V" H 19850 1200 50  0000 C CNN
+F 2 "" H 19725 1125 50  0001 C CNN
+F 3 "" H 19725 1125 50  0001 C CNN
+	1    19725 1125
+	1    0    0    -1
+$EndComp
+$Comp
+L power:+5V #PWR?
+U 1 1 62067DCB
+P 12900 3450
+F 0 "#PWR?" H 12900 3300 50  0001 C CNN
+F 1 "+5V" H 13025 3525 50  0000 C CNN
+F 2 "" H 12900 3450 50  0001 C CNN
+F 3 "" H 12900 3450 50  0001 C CNN
+	1    12900 3450
+	-1   0    0    1
+$EndComp
+$Comp
+L power:GND #PWR?
+U 1 1 62076A63
+P 12900 3050
+AR Path="/6B0E57BF/62076A63" Ref="#PWR?"  Part="1"
+AR Path="/6B32D907/62076A63" Ref="#PWR?"  Part="1"
+F 0 "#PWR?" H 12900 2800 50  0001 C CNN
+F 1 "GND" H 13050 2975 50  0000 C CNN
+F 2 "" H 12900 3050 50  0001 C CNN
+F 3 "" H 12900 3050 50  0001 C CNN
+	1    12900 3050
+	-1   0    0    1
+$EndComp
+Wire Wire Line
+	15750 4225 15325 4225
+Wire Wire Line
+	14525 2750 15325 2750
+Wire Wire Line
+	15325 2750 15325 4225
+Connection ~ 15325 4225
+Wire Wire Line
+	15325 4225 15125 4225
+Wire Wire Line
+	13575 2750 13800 2750
+Wire Wire Line
+	13800 2750 13800 3925
+Wire Wire Line
+	13575 3250 13575 4025
+Wire Wire Line
+	15750 2150 15750 4225
+Wire Wire Line
+	15700 2000 15700 3000
+Wire Wire Line
+	7150 9800 15700 9800
+Connection ~ 15700 2000
+Wire Wire Line
+	15700 2000 15600 2000
+Wire Wire Line
+	15700 3000 20325 3000
+Connection ~ 15700 3000
+Wire Wire Line
+	15700 3000 15700 9800
+Wire Wire Line
+	13575 4225 13575 6300
+Wire Wire Line
+	10050 6300 13575 6300
+Connection ~ 13575 6300
+Wire Wire Line
+	13575 6300 20325 6300
+Wire Wire Line
+	10325 4525 10325 4275
+Wire Wire Line
+	10325 4275 9600 4275
+Wire Wire Line
+	14075 4225 13575 4225
+Wire Wire Line
+	1975 4425 14025 4425
+Wire Wire Line
+	13575 4025 14025 4025
+Wire Wire Line
+	13800 3925 13975 3925
+$Comp
+L atari_grav_bw:S260A U?
+U 2 1 61D62188
+P 14525 4225
+F 0 "U?" H 14525 4750 50  0000 C CNN
+F 1 "S260A" H 14525 4659 50  0000 C CNN
+F 2 "" H 14525 4225 50  0001 C CNN
+F 3 "" H 14525 4225 50  0001 C CNN
+	2    14525 4225
+	1    0    0    -1
+$EndComp
+Wire Wire Line
+	13925 4525 11775 4525
+Wire Wire Line
+	11775 4525 11775 8925
+Wire Wire Line
+	11775 8925 12225 8925
+Connection ~ 11775 4525
+Wire Wire Line
+	11775 4525 10325 4525
 $EndSCHEMATC
