File: kicad/atari_gravitar_black_widow/SheetMisc.sch (KiCad schematic (older format))
At the start: 3 parts, among them J17 cat_box_con, J19 J19, J20 J20

Commit message: Completed sheet 3B
Parts:
- added R_8: 082, symbol atari_grav_bw:082
Connections:
- net +10V: now also R_8.4 (VSS)
- net GND: now also R_8.8 (VCC)
- no-connect marks 19 -> 22
Changed lines of the file:
@@
 Text GLabel 6925 2225 0    50   Input ~ 0
 AUD1
+$Comp
+L atari_grav_bw:082 R_8
+U 2 1 6C1085DD
+P 10350 1425
+F 0 "R_8" H 10375 1575 50  0000 L CNN
+F 1 "082" H 10375 1300 50  0000 L CNN
+F 2 "" H 10350 1425 50  0001 C CNN
+F 3 "" H 10350 1425 50  0001 C CNN
+	2    10350 1425
+	1    0    0    -1
+$EndComp
+$Comp
+L power:+10V #PWR?
+U 1 1 6C109596
+P 10300 1300
+F 0 "#PWR?" H 10300 1150 50  0001 C CNN
+F 1 "+10V" H 10315 1473 50  0000 C CNN
+F 2 "" H 10300 1300 50  0001 C CNN
+F 3 "" H 10300 1300 50  0001 C CNN
+	1    10300 1300
+	1    0    0    -1
+$EndComp
+$Comp
+L power:GND #PWR?
+U 1 1 6C1099FF
+P 10300 1550
+F 0 "#PWR?" H 10300 1300 50  0001 C CNN
+F 1 "GND" H 10305 1377 50  0000 C CNN
+F 2 "" H 10300 1550 50  0001 C CNN
+F 3 "" H 10300 1550 50  0001 C CNN
+	1    10300 1550
+	1    0    0    -1
+$EndComp
+NoConn ~ 10650 1425
+NoConn ~ 10050 1325
+NoConn ~ 10050 1525
 $EndSCHEMATC

Commit message: More Sheet 7a
Changed lines of the file:
@@
 NoConn ~ 10050 1325
 NoConn ~ 10050 1525
+Text GLabel 1575 4525 0    50   Input ~ 0
+~RESET
+Text GLabel 1575 4750 0    50   Input ~ 0
+~VGRST
+Text GLabel 1650 4950 0    50   Input ~ 0
+~STROBE1
+Text GLabel 1650 5200 0    50   Input ~ 0
+~STROBE2
+Text GLabel 1550 5450 0    50   Input ~ 0
+~DVY12
+Text GLabel 1550 5800 0    50   Input ~ 0
+DVY10
+Text GLabel 1525 5975 0    50   Input ~ 0
+DVY9
+Text GLabel 1525 6175 0    50   Input ~ 0
+DVY8
+Text GLabel 1525 6400 0    50   Input ~ 0
+~VGGO
 $EndSCHEMATC

Commit message: 7A
Changed lines of the file:
@@
 NoConn ~ 10050 1325
 NoConn ~ 10050 1525
-Text GLabel 1575 4525 0    50   Input ~ 0
+Text GLabel 1800 7575 0    50   Input ~ 0
 ~RESET
-Text GLabel 1575 4750 0    50   Input ~ 0
+Text GLabel 1800 7800 0    50   Input ~ 0
 ~VGRST
-Text GLabel 1650 4950 0    50   Input ~ 0
+Text GLabel 1875 8000 0    50   Input ~ 0
 ~STROBE1
-Text GLabel 1650 5200 0    50   Input ~ 0
+Text GLabel 1875 8250 0    50   Input ~ 0
 ~STROBE2
-Text GLabel 1550 5450 0    50   Input ~ 0
+Text GLabel 1775 8500 0    50   Input ~ 0
 ~DVY12
-Text GLabel 1550 5800 0    50   Input ~ 0
+Text GLabel 1775 8850 0    50   Input ~ 0
 DVY10
-Text GLabel 1525 5975 0    50   Input ~ 0
+Text GLabel 1750 9025 0    50   Input ~ 0
 DVY9
-Text GLabel 1525 6175 0    50   Input ~ 0
+Text GLabel 1750 9225 0    50   Input ~ 0
 DVY8
-Text GLabel 1525 6400 0    50   Input ~ 0
+Text GLabel 1750 9450 0    50   Input ~ 0
 ~VGGO
+Text GLabel 1650 4525 0    50   Input ~ 0
+~SA
+Text GLabel 1700 4800 0    50   Input ~ 0
+~OP0
+Text GLabel 1875 5100 0    50   Input ~ 0
+~STROBE0
+Text GLabel 1775 5375 0    50   Input ~ 0
+DVY12
+Text GLabel 1775 5600 0    50   Input ~ 0
+DVY11
+Text GLabel 1775 5850 0    50   Input ~ 0
+DVX12
+Text GLabel 1775 6125 0    50   Input ~ 0
+DXV11
+Text GLabel 1775 6375 0    50   Input ~ 0
+SCALE
+Text GLabel 1700 6625 0    50   Input ~ 0
+~OP2
+Text GLabel 1750 6900 0    50   Input ~ 0
+VGCK
+Text GLabel 1875 7075 0    50   Input ~ 0
+~STROBE3
+Text GLabel 1725 7225 0    50   Input ~ 0
+OP2
+Text GLabel 1725 7350 0    50   Input ~ 0
+OP0
 $EndSCHEMATC

Commit message: 7a
Changed lines of the file:
@@
 Text GLabel 1725 7350 0    50   Input ~ 0
 OP0
+Text GLabel 4700 4575 2    50   Input ~ 0
+~ENORM
+Text GLabel 4775 4775 2    50   Input ~ 0
+NORM
+Text GLabel 4825 5000 2    50   Input ~ 0
+~CENTER
+Text GLabel 4775 5200 2    50   Input ~ 0
+VCTR
+Text GLabel 4850 5425 2    50   Input ~ 0
+~VCTR
+Text GLabel 4825 5625 2    50   Input ~ 0
+HALT
+Text GLabel 4850 5800 2    50   Input ~ 0
+GO
+Text GLabel 4825 6050 2    50   Input ~ 0
+~STATCLK
+Text GLabel 4850 6225 2    50   Input ~ 0
+~SCALELD
+Text GLabel 4825 6500 2    50   Input ~ 0
+~STOP
+Text GLabel 1525 9800 0    50   Input ~ 0
+12MHZ
+Text GLabel 1475 9950 0    50   Input ~ 0
+~OP1
+Text GLabel 1475 10100 0    50   Input ~ 0
+~SA
+Text GLabel 1450 10225 0    50   Input ~ 0
+OP1
 $EndSCHEMATC
