File: kicad/atari_gravitar_black_widow/atari_gravitar_black_widow.kicad_sch (KiCad schematic)
At the start: 0 parts

Commit message: 7a draft
Other:
- note added: "JBB draft done"
- note removed: "JBB IN PROGRESS"
Changed lines of the file:
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@@
     (effects (font (size 5.08 5.08) (thickness 1.016) bold) (justify left bottom))
   )
-  (text "JBB\nIN \nPROGRESS\n" (at 240.665 149.86 0)
+  (text "JBB\ndraft done\n" (at 240.665 149.86 0)
     (effects (font (size 5.08 5.08) (thickness 1.016) bold) (justify left bottom))
   )

Commit message: start 8a
Other:
- note added: "JBB In progress"

Commit message: 8A
Other:
- note added: "JBB DONE Needs Review"
- note removed: "JBB draft done"

Commit message: 8B COMPLETED
Other:
- note removed: "JBB In progress"
