File: kicad/atari_gravitar_black_widow/Sheet8B.kicad_sch (KiCad schematic)
At the start: 57 parts

Commit message: 20 errors left
Parts:
- removed J_?: LS04, Star_Wars_Vector_PCB:DIP14, symbol Star_Wars_Vector_PCB:LS04
- added K_9: LS04, symbol atari_grav_bw:LS04
- added TPYOUT1: TP, symbol atari_grav_bw:TP
- R215: renamed from R?; value 6.8k -> 68
- gave numbers to parts that had none: 49
Connections:
- net +5V: now also K_9.14 (VCC)
- net -15V: now also D/E_12.4 (VSS)
- net GND: now also K_9.7 (GND)
- net INVERTY: now also K_9.1
- net YOUT: now also TPYOUT1.1, TPYOUT1.2
- net at E_10.1: now also K_9.2
- no-connect marks 4 -> 7
Other:
- moved on the sheet: C81, C82, NOTEB

Commit message: Fixed most errors
Parts:
- removed A/B_12: MC1495LB, Star_Wars_Vector_PCB:DIP14, symbol quantum_arcade_pcb:MC1495LB
- removed C1: 100pf, quantum_arcade_pcb:CapSmall, symbol Device:C
- removed C130, C131, C134, C135, C64, C66, C81, C82, C83, C84: .1uF, quantum_arcade_pcb:GenComp, symbol Device:C
- removed C132: 39pf, quantum_arcade_pcb:CapSmall, symbol Device:C
- removed C136: 1000pf, quantum_arcade_pcb:GenComp, symbol Device:C
- removed C65: .01uF, quantum_arcade_pcb:CapSmall, symbol Device:C
- removed C72: .047uF, quantum_arcade_pcb:CapInt, symbol Device:C
- removed C_12: MC1495LA, Star_Wars_Vector_PCB:DIP14, symbol quantum_arcade_pcb:MC1495LA
- removed D/E_12: 082A, symbol atari_grav_bw:082A
- removed D_10: 082, Star_Wars_Vector_PCB:DIP8, symbol Star_Wars_Vector_PCB:082
- removed E_10, NOTE: LF13201, Star_Wars_Vector_PCB:DIP16, symbol Star_Wars_Vector_PCB:LF13201
- removed F_9: AM6012, Star_Wars_Vector_PCB:DIP20, symbol Star_Wars_Vector_PCB:AM6012
- removed K_9: LS04, symbol atari_grav_bw:LS04
- removed R190: 2.2K, quantum_arcade_pcb:GenComp, symbol Device:R
- removed R191: 100k, quantum_arcade_pcb:GenComp, symbol Device:R
- removed R193, R194, R199, R209: 470, quantum_arcade_pcb:GenComp, symbol Device:R
- removed R196, R197, R198, R207: 2.2k, quantum_arcade_pcb:GenComp, symbol Device:R
- removed R200: 12K, quantum_arcade_pcb:GenComp, symbol Device:R
- removed R202: 10k, quantum_arcade_pcb:GenComp, symbol Device:R
- removed R202, R206, R208: 3.9k, quantum_arcade_pcb:GenComp, symbol Device:R
- removed R203, R83: 680, quantum_arcade_pcb:GenComp, symbol Device:R
- removed R204: 1k, quantum_arcade_pcb:GenComp, symbol Device:R
- removed R205: 2.7k, quantum_arcade_pcb:GenComp, symbol Device:R
- removed R210: 2K, Star_Wars_Vector_PCB:PotBlk, symbol Star_Wars_Vector_PCB-rescue:POT
- removed R211: 5.6k, quantum_arcade_pcb:GenComp, symbol Device:R
- removed R212, R213: 10k, Star_Wars_Vector_PCB:PotBlk, symbol Star_Wars_Vector_PCB-rescue:POT
- removed R214: 100, quantum_arcade_pcb:GenComp, symbol Device:R
- removed R215: 68, quantum_arcade_pcb:GenComp, symbol Device:R
- removed R216: 6.8k, quantum_arcade_pcb:GenComp, symbol Device:R
- removed R84: 820, quantum_arcade_pcb:GenComp, symbol Device:R
- removed R96, R97: 7.5K, quantum_arcade_pcb:GenComp, symbol Device:R
- removed RV1: VDR, quantum_arcade_pcb:GenComp, symbol Device:Varistor
- removed TPYOUT1: TP, symbol atari_grav_bw:TP
Connections:
- no-connect marks 7 -> 0
Other:
- note removed: "NOT LOADED"
- note removed: "NOTE"
- note removed: "Y-AXIS OUTPUT"

Commit message: 8B COMPLETED
Parts:
- added A_? (x2): 082, Star_Wars_Vector_PCB:DIP8, symbol Star_Wars_Vector_PCB:082
- added B_? (x4): LF13201, Star_Wars_Vector_PCB:DIP16, symbol Star_Wars_Vector_PCB:LF13201
- added B_?: MC1495LB, Star_Wars_Vector_PCB:DIP14, symbol quantum_arcade_pcb:MC1495LB
- added B_?: AM6012, Star_Wars_Vector_PCB:DIP20, symbol Star_Wars_Vector_PCB:AM6012
- added C136: 1000pf, quantum_arcade_pcb:GenComp, symbol Device:C
- added C? (x10): .1uF, quantum_arcade_pcb:GenComp, symbol Device:C
- added C?: 39pf, quantum_arcade_pcb:CapSmall, symbol Device:C
- added C?: .01uF, quantum_arcade_pcb:CapSmall, symbol Device:C
- added C?: .047uF, quantum_arcade_pcb:CapInt, symbol Device:C
- added C?: 100pf, quantum_arcade_pcb:CapSmall, symbol Device:C
- added C_?: MC1495LA, Star_Wars_Vector_PCB:DIP14, symbol quantum_arcade_pcb:MC1495LA
- added J_?: LS04, Star_Wars_Vector_PCB:DIP14, symbol Star_Wars_Vector_PCB:LS04
- added R? (x2): 6.8k, quantum_arcade_pcb:GenComp, symbol Device:R
- added R?: 2.7k, quantum_arcade_pcb:GenComp, symbol Device:R
- added R?: 5.6k, quantum_arcade_pcb:GenComp, symbol Device:R
- added R? (x2): 680, quantum_arcade_pcb:GenComp, symbol Device:R
- added R? (x3): 3.9k, quantum_arcade_pcb:GenComp, symbol Device:R
- added R? (x2): 10k, Star_Wars_Vector_PCB:PotBlk, symbol Star_Wars_Vector_PCB-rescue:POT
- added R?: 10k, quantum_arcade_pcb:GenComp, symbol Device:R
- added R?: 2.2K, quantum_arcade_pcb:GenComp, symbol Device:R
- added R? (x4): 470, quantum_arcade_pcb:GenComp, symbol Device:R
- added R?: 12K, quantum_arcade_pcb:GenComp, symbol Device:R
- added R?: 1k, quantum_arcade_pcb:GenComp, symbol Device:R
- added R? (x2): 7.5K, quantum_arcade_pcb:GenComp, symbol Device:R
- added R?: 820, quantum_arcade_pcb:GenComp, symbol Device:R
- added R?: 100k, quantum_arcade_pcb:GenComp, symbol Device:R
- added R? (x4): 2.2k, quantum_arcade_pcb:GenComp, symbol Device:R
- added R?: 100, quantum_arcade_pcb:GenComp, symbol Device:R
- added R?: 2K, Star_Wars_Vector_PCB:PotBlk, symbol Star_Wars_Vector_PCB-rescue:POT
- added RV?: VDR, quantum_arcade_pcb:GenComp, symbol Device:Varistor
- added U? (x2): 082A, symbol atari_grav_bw:082A
Connections:
- new net: A_?.1, B_?.14, R?.1
- new net: B_?.15, B_?.2, R?.2, R?.2
- new net: R?.1, R?.1, U?.2 (-)
- new net: C_?.4, R?.2, R?.2
- new net: R?.1, R?.3 (x2)
- new net: C_?.2, R?.1, R?.2, U?.5 (+)
- new net: C_?.3, R?.2
- new net: A_?.7, B_?.11, B_?.3, C?.1, R?.2
- new net: C?.2, C?.2, C_?.14, R?.1, R?.2, U?.6 (-)
- new net: C_?.13, R?.2
- new net: B_?.6, R?.1, R?.1
- new net: B_?.5, R?.2, R?.2
- new net: C_?.9, R?.1
- new net: R?.1, R?.2, U?.1
- new net: C_?.12, C_?.8, R?.2
- new net: B_?.4, B_?.9, R?.1
- new net: A_?.2 (-), R?.1, R?.2
- new net: B_?.10, R?.2
- new net: B_?.11, R?.1
- new net: B_?.12, B_?.8, R?.2
- new net: B_?.13, B_?.3, R?.2
- new net: B_?.1, J_?.12
- new net: B_?.15 (VR-), R?.2
- new net: C?.2, R?.2
- new net: C_?.10, R?.2
- new net: C_?.11, R?.1
- new net: C_?.5, R?.2
- new net: C_?.6, R?.1
- new net: R?.3, RV?.1, U?.3 (+)
- new net +15V: A_?.8 (VCC), B_?.13, B_?.2, C?.1, C?.2, C?.2, C?.2, R?.1, R?.2, R?.2, U?.8 (VCC)
- new net +5V: B_?.20 (VCC), C?.1
- new net +6V: B_?.1, C_?.1
- new net -15V: A_?.4 (VSS), B_?.17 (V-), B_?.4, B_?.7, C?.1, C?.2, C?.2, C?.2, C?.2, C_?.7
- new net DVX10: B_?.4 (B4)
- new net DVX11: B_?.3 (B3)
- new net DVX3: B_?.11 (B11)
- new net DVX4: B_?.10 (B10)
- new net DVX5: B_?.9 (B9)
- new net DVX6: B_?.8 (B8)
- new net DVX7: B_?.7 (B7)
- new net DVX8: B_?.6 (B6)
- new net DVX9: B_?.5 (B5)
- new net GND: A_?.3 (+), A_?.5 (+), B_?.1 (B1), B_?.12 (B12), B_?.13 (GND), B_?.19 (~{IO}), B_?.5, C136.1, C?.1, C?.1, C?.1, C?.1, C?.1, C?.1, C?.1, C?.1, C?.2, C?.2, C?.2, R?.1, R?.1, R?.1, R?.1, R?.1, R?.1, R?.1, R?.1, R?.2, R?.2, R?.2, RV?.2
- new net INVERTY: B_?.16, J_?.13
- new net YBIP: A_?.6 (-), B_?.10, B_?.18 (IO), C136.2, C?.2
- new net YCOR: B_?.14, R?.1, R?.2
- new net YLIN: C?.1, C?.1, R?.1, R?.1, R?.2, U?.7
- new net YOUT: R?.2
- new net YREF: B_?.14 (VR+), R?.1
- new net ~{CENTER}: B_?.9
- new net ~{DVX12}: B_?.2 (B2)
- no-connect marks 0 -> 4
Other:
- note added: "NOT LOADED"
- note added: "NOTE"
- note added: "Y-AXIS OUTPUT"
