File: kicad/atari_gravitar_black_widow/Sheet7A.kicad_sch (KiCad schematic)
At the start: 27 parts

Commit message: REVIEW 4A DONE
Parts:
- K_4: value LS10 -> S10
Changed lines of the file:
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@@
     (in_bom yes) (on_board yes)
     (property "Reference" "K_4" (id 0) (at 414.02 47.625 0))
-    (property "Value" "LS10" (id 1) (at 414.02 50.8 0))
+    (property "Value" "S10" (id 1) (at 414.02 50.8 0))
     (property "Footprint" "" (id 2) (at 415.29 50.8 0)
       (effects (font (size 1.27 1.27)) hide)

Commit message: REVIEWS AND FINALS
Parts:
- added HALT1, ~{VCTR}1: TP, symbol atari_grav_bw:TP
Connections:
- net 12MHZ: now also C_7.14 (CK)
- net HALT: now also HALT1.1, HALT1.2
- net ~{SCALELD}: now also D_7.9 (CK); no longer J_6.6
- net at D_7.1 (C), L_5.4 (~{1PRE_}): no longer C_7.14 (CK)
- net at B_7.4, K_6.9: no longer D_7.9 (CK)
- new net: ~{VCTR}1.1, ~{VCTR}1.2
Other:
- note added: "Center Flag"
- note added: "Go Flag"
- note added: "Normalization Flag"
- note added: "Vector Flag"
- note added: "Vector Scaling"
- note added: "Vector Timer"
- note removed: "CENTER FLAG"
- note removed: "GO FLAG"
- note removed: "NORMALIZATION FLAG"
- note removed: "VECTOR FLAG"
- note removed: "VECTOR SCALING"
- note removed: "VECTOR TIMER"
Changed lines of the file:
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@@
   (junction (at 37.465 299.085) (diameter 0) (color 0 0 0 0)
   )
-  (junction (at 158.75 269.875) (diameter 0) (color 0 0 0 0)
-  )
   (junction (at 563.245 262.89) (diameter 0) (color 0 0 0 0)
   )
@@
   (junction (at 122.555 242.57) (diameter 0) (color 0 0 0 0)
   )
+  (junction (at 505.333 195.58) (diameter 0) (color 0 0 0 0)
+  )
   (junction (at 261.62 318.77) (diameter 0) (color 0 0 0 0)
   )
@@
   (junction (at 66.04 133.985) (diameter 0) (color 0 0 0 0)
   )
-  (junction (at 153.67 252.095) (diameter 0) (color 0 0 0 0)
-  )
   (junction (at 212.09 267.335) (diameter 0) (color 0 0 0 0)
   )
@@
   (junction (at 197.485 292.735) (diameter 0) (color 0 0 0 0)
   )
+  (junction (at 516.382 186.436) (diameter 0) (color 0 0 0 0)
+  )
   (junction (at 344.805 160.02) (diameter 0) (color 0 0 0 0)
   )
@@
   (junction (at 398.78 50.8) (diameter 0) (color 0 0 0 0)
   )
+  (junction (at 109.855 318.77) (diameter 0) (color 0 0 0 0)
+  )
   (junction (at 481.965 269.875) (diameter 0) (color 0 0 0 0)
   )
+  (junction (at 158.75 252.095) (diameter 0) (color 0 0 0 0)
+  )
   (junction (at 95.25 167.005) (diameter 0) (color 0 0 0 0)
   )
@@
   (junction (at 315.595 294.64) (diameter 0) (color 0 0 0 0)
   )
-  (junction (at 109.855 323.215) (diameter 0) (color 0 0 0 0)
-  )
   (junction (at 273.05 255.905) (diameter 0) (color 0 0 0 0)
   )
-  (junction (at 109.855 318.135) (diameter 0) (color 0 0 0 0)
+  (junction (at 516.382 212.471) (diameter 0) (color 0 0 0 0)
   )
   (junction (at 464.185 280.035) (diameter 0) (color 0 0 0 0)
@@
     (stroke (width 0) (type default) (color 0 0 0 0))
   )
+  (wire (pts (xy 109.855 318.135) (xy 109.855 318.77))
+    (stroke (width 0) (type default) (color 0 0 0 0))
+  )
   (wire (pts (xy 315.595 294.64) (xy 315.595 295.275))
     (stroke (width 0) (type default) (color 0 0 0 0))
@@
     (stroke (width 0) (type default) (color 0 0 0 0))
   )
-  (wire (pts (xy 109.855 311.785) (xy 109.855 318.135))
-    (stroke (width 0) (type default) (color 0 0 0 0))
-  )
-  (wire (pts (xy 153.67 252.095) (xy 561.975 252.095))
-    (stroke (width 0) (type default) (color 0 0 0 0))
-  )
   (wire (pts (xy 495.935 283.21) (xy 495.935 291.465))
     (stroke (width 0) (type default) (color 0 0 0 0))
@@
     (stroke (width 0) (type default) (color 0 0 0 0))
   )
+  (wire (pts (xy 505.333 195.58) (xy 516.255 195.58))
+    (stroke (width 0) (type default) (color 0 0 0 0))
+  )
   (wire (pts (xy 400.05 24.13) (xy 50.165 24.13))
     (stroke (width 0) (type default) (color 0 0 0 0))
   )
-  (wire (pts (xy 109.855 323.215) (xy 156.845 323.215))
-    (stroke (width 0) (type default) (color 0 0 0 0))
-  )
   (wire (pts (xy 275.59 316.865) (xy 253.365 316.865))
     (stroke (width 0) (type default) (color 0 0 0 0))
@@
     (stroke (width 0) (type default) (color 0 0 0 0))
   )
-  (wire (pts (xy 158.75 269.875) (xy 181.61 269.875))
+  (wire (pts (xy 154.305 269.875) (xy 181.61 269.875))
     (stroke (width 0) (type default) (color 0 0 0 0))
   )
@@
     (stroke (width 0) (type default) (color 0 0 0 0))
   )
+  (wire (pts (xy 516.382 212.471) (xy 520.192 212.471))
+    (stroke (width 0) (type default) (color 0 0 0 0))
+  )
   (wire (pts (xy 404.495 261.62) (xy 404.495 291.465))
     (stroke (width 0) (type default) (color 0 0 0 0))
@@
     (stroke (width 0) (type default) (color 0 0 0 0))
   )
+  (wire (pts (xy 158.75 252.095) (xy 158.75 282.575))
+    (stroke (width 0) (type default) (color 0 0 0 0))
+  )
   (wire (pts (xy 398.78 50.8) (xy 396.24 50.8))
     (stroke (width 0) (type default) (color 0 0 0 0))
@@
     (stroke (width 0) (type default) (color 0 0 0 0))
   )
-  (wire (pts (xy 158.75 282.575) (xy 158.75 269.875))
+  (wire (pts (xy 505.333 172.593) (xy 505.333 186.436))
+    (stroke (width 0) (type default) (color 0 0 0 0))
+  )
+  (wire (pts (xy 516.382 186.436) (xy 520.192 186.436))
     (stroke (width 0) (type default) (color 0 0 0 0))
   )
@@
     (stroke (width 0) (type default) (color 0 0 0 0))
   )
-  (wire (pts (xy 52.07 323.215) (xy 109.855 323.215))
+  (wire (pts (xy 52.07 323.215) (xy 156.845 323.215))
+    (stroke (width 0) (type default) (color 0 0 0 0))
+  )
+  (wire (pts (xy 153.67 252.095) (xy 158.75 252.095))
+    (stroke (width 0) (type default) (color 0 0 0 0))
+  )
+  (wire (pts (xy 109.855 318.77) (xy 184.15 318.77))
     (stroke (width 0) (type default) (color 0 0 0 0))
   )
@@
     (stroke (width 0) (type default) (color 0 0 0 0))
   )
-  (wire (pts (xy 186.69 195.58) (xy 516.255 195.58))
+  (wire (pts (xy 505.333 186.436) (xy 516.382 186.436))
+    (stroke (width 0) (type default) (color 0 0 0 0))
+  )
+  (wire (pts (xy 186.69 195.58) (xy 505.333 195.58))
     (stroke (width 0) (type default) (color 0 0 0 0))
   )
@@
     (stroke (width 0) (type default) (color 0 0 0 0))
   )
+  (wire (pts (xy 158.75 252.095) (xy 561.975 252.095))
+    (stroke (width 0) (type default) (color 0 0 0 0))
+  )
   (wire (pts (xy 98.425 131.445) (xy 105.41 131.445))
     (stroke (width 0) (type default) (color 0 0 0 0))
@@
     (stroke (width 0) (type default) (color 0 0 0 0))
   )
-  (wire (pts (xy 154.305 269.875) (xy 158.75 269.875))
-    (stroke (width 0) (type default) (color 0 0 0 0))
-  )
   (wire (pts (xy 366.395 309.245) (xy 366.395 314.325))
     (stroke (width 0) (type default) (color 0 0 0 0))
@@
     (stroke (width 0) (type default) (color 0 0 0 0))
   )
-  (wire (pts (xy 147.32 252.095) (xy 153.67 252.095))
-    (stroke (width 0) (type default) (color 0 0 0 0))
-  )
   (wire (pts (xy 459.105 307.975) (xy 459.105 313.055))
     (stroke (width 0) (type default) (color 0 0 0 0))
@@
     (stroke (width 0) (type default) (color 0 0 0 0))
   )
+  (wire (pts (xy 505.333 212.471) (xy 516.382 212.471))
+    (stroke (width 0) (type default) (color 0 0 0 0))
+  )
   (wire (pts (xy 38.1 299.085) (xy 37.465 299.085))
     (stroke (width 0) (type default) (color 0 0 0 0))
@@
     (stroke (width 0) (type default) (color 0 0 0 0))
   )
-  (wire (pts (xy 36.83 318.77) (xy 184.15 318.77))
+  (wire (pts (xy 36.83 318.77) (xy 109.855 318.77))
     (stroke (width 0) (type default) (color 0 0 0 0))
   )
@@
     (stroke (width 0) (type default) (color 0 0 0 0))
   )
-  (wire (pts (xy 109.855 318.135) (xy 109.855 323.215))
-    (stroke (width 0) (type default) (color 0 0 0 0))
-  )
   (wire (pts (xy 184.15 318.77) (xy 200.66 318.77))
     (stroke (width 0) (type default) (color 0 0 0 0))
@@
     (stroke (width 0) (type default) (color 0 0 0 0))
   )
+  (wire (pts (xy 505.333 195.58) (xy 505.333 212.471))
+    (stroke (width 0) (type default) (color 0 0 0 0))
+  )
   (wire (pts (xy 456.565 316.23) (xy 398.145 316.23))
     (stroke (width 0) (type default) (color 0 0 0 0))
@@
     (stroke (width 0) (type default) (color 0 0 0 0))
   )
-  (text "GO FLAG\n" (at 277.495 224.155 0)
+  (text "Go Flag" (at 277.495 224.155 0)
     (effects (font (size 2.54 2.54) (thickness 0.508) bold) (justify left bottom))
   )
@@
     (effects (font (size 1.27 1.27)) (justify left bottom))
   )
-  (text "CENTER FLAG\n" (at 155.575 95.885 0)
+  (text "Center Flag\n\n" (at 155.575 95.885 0)
     (effects (font (size 2.54 2.54) (thickness 0.508) bold) (justify left bottom))
   )
@@
     (effects (font (size 1.27 1.27)) (justify left bottom))
   )
-  (text "VECTOR TIMER" (at 430.53 337.82 0)
+  (text "Vector Timer" (at 430.53 337.82 0)
     (effects (font (size 2.54 2.54) (thickness 0.508) bold) (justify left bottom))
   )
@@
     (effects (font (size 1.27 1.27)) (justify left bottom))
   )
-  (text "VECTOR FLAG\n" (at 125.73 151.765 0)
+  (text "Vector Flag" (at 125.73 151.765 0)
     (effects (font (size 2.54 2.54) (thickness 0.508) bold) (justify left bottom))
   )
@@
     (effects (font (size 1.27 1.27)) (justify left bottom))
   )
-  (text "VECTOR SCALING\n" (at 57.15 267.97 0)
+  (text "Vector Scaling\n\n" (at 57.15 267.97 0)
     (effects (font (size 2.54 2.54) (thickness 0.508) bold) (justify left bottom))
   )
@@
     (effects (font (size 1.27 1.27)) (justify left bottom))
   )
-  (text "NORMALIZATION FLAG\n\n" (at 313.055 36.195 0)
+  (text "Normalization Flag\n\n" (at 313.055 36.195 0)
     (effects (font (size 2.54 2.54) (thickness 0.508) bold) (justify left bottom))
   )
@@
     (pin "1")
   )
+  (symbol (lib_id "atari_grav_bw:TP") (at 518.287 207.391 0) (unit 1)
+    (in_bom yes) (on_board yes)
+    (property "Reference" "HALT1" (id 0) (at 519.811 204.724 0)
+      (effects (font (size 1.524 1.524)) (justify left))
+    )
+    (property "Value" "TP" (id 1) (at 516.382 206.121 0)
+      (effects (font (size 1.524 1.524)) hide)
+    )
+    (property "Footprint" "" (id 2) (at 516.382 208.661 0)
+      (effects (font (size 1.524 1.524)) hide)
+    )
+    (property "Datasheet" "" (id 3) (at 516.382 208.661 0)
+      (effects (font (size 1.524 1.524)) hide)
+    )
+    (pin "1")
+    (pin "2")
+  )
+  (symbol (lib_id "atari_grav_bw:TP") (at 518.287 181.356 0) (unit 1)
+    (in_bom yes) (on_board yes)
+    (property "Reference" "~{VCTR}1" (id 0) (at 519.811 179.578 0)
+      (effects (font (size 1.524 1.524)) (justify left))
+    )
+    (property "Value" "TP" (id 1) (at 516.382 180.086 0)
+      (effects (font (size 1.524 1.524)) hide)
+    )
+    (property "Footprint" "" (id 2) (at 516.382 182.626 0)
+      (effects (font (size 1.524 1.524)) hide)
+    )
+    (property "Datasheet" "" (id 3) (at 516.382 182.626 0)
+      (effects (font (size 1.524 1.524)) hide)
+    )
+    (pin "1")
+    (pin "2")
+  )
 )

Commit message: 20 errors left
Parts:
- J_5: value S260A -> S260
- M_4: value LS27A -> LS27
Changed lines of the file:
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@@
     (in_bom yes) (on_board yes)
     (property "Reference" "M_4" (id 0) (at 132.08 160.655 0))
-    (property "Value" "LS27A" (id 1) (at 132.715 163.83 0))
+    (property "Value" "LS27" (id 1) (at 132.715 163.83 0))
     (property "Footprint" "" (id 2) (at 132.715 163.195 0)
       (effects (font (size 1.27 1.27)) hide)
@@
     (in_bom yes) (on_board yes)
     (property "Reference" "J_5" (id 0) (at 368.935 105.41 0))
-    (property "Value" "S260A" (id 1) (at 368.3 108.585 0))
+    (property "Value" "S260" (id 1) (at 368.3 108.585 0))
     (property "Footprint" "" (id 2) (at 368.935 107.315 0)
       (effects (font (size 1.27 1.27)) hide)

Commit message: 19 errors left
Connections:
- net ~{VCTR}: now also ~{VCTR}1.1, ~{VCTR}1.2
Changed lines of the file:
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@@
   (junction (at 197.485 292.735) (diameter 0) (color 0 0 0 0)
   )
-  (junction (at 516.382 186.436) (diameter 0) (color 0 0 0 0)
-  )
   (junction (at 344.805 160.02) (diameter 0) (color 0 0 0 0)
   )
@@
   (junction (at 407.035 259.08) (diameter 0) (color 0 0 0 0)
   )
+  (junction (at 505.333 172.72) (diameter 0) (color 0 0 0 0)
+  )
   (junction (at 105.41 131.445) (diameter 0) (color 0 0 0 0)
   )
@@
   )
   (junction (at 273.05 255.905) (diameter 0) (color 0 0 0 0)
+  )
+  (junction (at 516.382 186.563) (diameter 0) (color 0 0 0 0)
   )
   (junction (at 516.382 212.471) (diameter 0) (color 0 0 0 0)
@@
     (stroke (width 0) (type default) (color 0 0 0 0))
   )
+  (wire (pts (xy 505.333 172.72) (xy 516.255 172.72))
+    (stroke (width 0) (type default) (color 0 0 0 0))
+  )
   (wire (pts (xy 495.935 283.21) (xy 495.935 291.465))
     (stroke (width 0) (type default) (color 0 0 0 0))
@@
     (stroke (width 0) (type default) (color 0 0 0 0))
   )
-  (wire (pts (xy 255.27 172.72) (xy 516.255 172.72))
+  (wire (pts (xy 255.27 172.72) (xy 505.333 172.72))
     (stroke (width 0) (type default) (color 0 0 0 0))
   )
@@
     (stroke (width 0) (type default) (color 0 0 0 0))
   )
+  (wire (pts (xy 505.333 186.563) (xy 516.382 186.563))
+    (stroke (width 0) (type default) (color 0 0 0 0))
+  )
   (wire (pts (xy 123.825 251.46) (xy 114.935 251.46))
     (stroke (width 0) (type default) (color 0 0 0 0))
@@
     (stroke (width 0) (type default) (color 0 0 0 0))
   )
-  (wire (pts (xy 505.333 172.593) (xy 505.333 186.436))
-    (stroke (width 0) (type default) (color 0 0 0 0))
-  )
-  (wire (pts (xy 516.382 186.436) (xy 520.192 186.436))
+  (wire (pts (xy 505.333 172.72) (xy 505.333 186.563))
+    (stroke (width 0) (type default) (color 0 0 0 0))
+  )
+  (wire (pts (xy 516.382 186.563) (xy 520.192 186.563))
     (stroke (width 0) (type default) (color 0 0 0 0))
   )
@@
   )
   (wire (pts (xy 389.255 69.85) (xy 389.255 107.315))
-    (stroke (width 0) (type default) (color 0 0 0 0))
-  )
-  (wire (pts (xy 505.333 186.436) (xy 516.382 186.436))
     (stroke (width 0) (type default) (color 0 0 0 0))
   )
@@
     (pin "2")
   )
-  (symbol (lib_id "atari_grav_bw:TP") (at 518.287 181.356 0) (unit 1)
-    (in_bom yes) (on_board yes)
-    (property "Reference" "~{VCTR}1" (id 0) (at 519.811 179.578 0)
+  (symbol (lib_id "atari_grav_bw:TP") (at 518.287 181.483 0) (unit 1)
+    (in_bom yes) (on_board yes)
+    (property "Reference" "~{VCTR}1" (id 0) (at 519.811 179.705 0)
       (effects (font (size 1.524 1.524)) (justify left))
     )
-    (property "Value" "TP" (id 1) (at 516.382 180.086 0)
+    (property "Value" "TP" (id 1) (at 516.382 180.213 0)
       (effects (font (size 1.524 1.524)) hide)
     )
-    (property "Footprint" "" (id 2) (at 516.382 182.626 0)
+    (property "Footprint" "" (id 2) (at 516.382 182.753 0)
       (effects (font (size 1.524 1.524)) hide)
     )
-    (property "Datasheet" "" (id 3) (at 516.382 182.626 0)
+    (property "Datasheet" "" (id 3) (at 516.382 182.753 0)
       (effects (font (size 1.524 1.524)) hide)
     )

Commit message: Fixed most errors
Connections:
- net ~{DISRST}: now reaches D_7.1 (C), L_5.4 (~{1PRE_})
Changed lines of the file:
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@@
   (junction (at 140.97 80.01) (diameter 0) (color 0 0 0 0)
+  )
+  (junction (at 167.64 182.245) (diameter 0) (color 0 0 0 0)
   )
   (junction (at 255.905 292.735) (diameter 0) (color 0 0 0 0)
@@
     (stroke (width 0) (type default) (color 0 0 0 0))
   )
+  (wire (pts (xy 167.64 182.245) (xy 170.561 182.245))
+    (stroke (width 0) (type default) (color 0 0 0 0))
+  )
   (polyline (pts (xy 154.305 216.535) (xy 154.305 326.39))
     (stroke (width 0) (type default) (color 0 0 0 0))
@@
       (effects (font (size 1.27 1.27)) hide)
     )
+  )
+  (global_label "~{DISRST}" (shape input) (at 170.561 182.245 0) (fields_autoplaced)
+    (effects (font (size 0.8382 0.8382)) (justify left))
+    (property "Intersheet References" "${INTERSHEET_REFS}" (id 0) (at 237.871 568.325 0)
+      (effects (font (size 1.27 1.27)) hide)
+    )
