File: kicad/atari_gravitar_black_widow/Sheet7A.kicad_sch (KiCad schematic)
At the start: 28 parts

Commit message: lots o' traces
Parts:
- renumbered TP~{VCTR}1 to TPVCTR1
Connections:
- net +5V: no longer E_5.5 (Sd)
- net VCTR: now also TPVCTR1.1, TPVCTR1.2
- net ~{SA}: now also E_5.11 (Sd)
- net ~{VCTR}: no longer TPVCTR1.1, TPVCTR1.2
- new net PR23: E_5.5 (Sd)
- no-connect marks 15 -> 14
Other:
- moved on the sheet: E_5B, TPVCTR1
Changed lines of the file:
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@@
   (junction (at 184.15 318.77) (diameter 0) (color 0 0 0 0)
   )
+  (junction (at 505.3327 160.02) (diameter 0) (color 0 0 0 0)
+  )
   (junction (at 454.025 321.31) (diameter 0) (color 0 0 0 0)
   )
@@
   (junction (at 407.035 259.08) (diameter 0) (color 0 0 0 0)
   )
-  (junction (at 505.333 172.72) (diameter 0) (color 0 0 0 0)
-  )
   (junction (at 105.41 131.445) (diameter 0) (color 0 0 0 0)
   )
@@
   (junction (at 273.05 255.905) (diameter 0) (color 0 0 0 0)
   )
-  (junction (at 516.382 186.563) (diameter 0) (color 0 0 0 0)
+  (junction (at 516.3817 151.1308) (diameter 0) (color 0 0 0 0)
   )
   (junction (at 516.382 212.471) (diameter 0) (color 0 0 0 0)
@@
   )
   (no_connect (at 464.185 307.975))
-  (no_connect (at 224.79 94.615))
   (no_connect (at 135.255 296.545))
   (no_connect (at 73.66 294.005))
@@
     (stroke (width 0) (type default) (color 0 0 0 0))
   )
-  (wire (pts (xy 505.333 172.72) (xy 516.255 172.72))
+  (wire (pts (xy 255.27 172.72) (xy 516.255 172.72))
     (stroke (width 0) (type default) (color 0 0 0 0))
   )
@@
     (stroke (width 0) (type default) (color 0 0 0 0))
   )
+  (wire (pts (xy 505.3327 160.02) (xy 516.255 160.02))
+    (stroke (width 0) (type default) (color 0 0 0 0))
+  )
   (wire (pts (xy 46.99 226.695) (xy 46.99 191.77))
     (stroke (width 0) (type default) (color 0 0 0 0))
@@
     (stroke (width 0) (type default) (color 0 0 0 0))
   )
-  (wire (pts (xy 255.27 172.72) (xy 505.333 172.72))
-    (stroke (width 0) (type default) (color 0 0 0 0))
-  )
   (wire (pts (xy 224.79 135.255) (xy 259.715 135.255))
     (stroke (width 0) (type default) (color 0 0 0 0))
@@
     (stroke (width 0) (type default) (color 0 0 0 0))
   )
-  (wire (pts (xy 197.485 125.095) (xy 204.47 125.095))
+  (wire (pts (xy 197.4939 121.2939) (xy 204.4789 121.2939))
     (stroke (width 0) (type default) (color 0 0 0 0))
   )
@@
     (stroke (width 0) (type default) (color 0 0 0 0))
   )
-  (wire (pts (xy 344.805 160.02) (xy 516.255 160.02))
+  (wire (pts (xy 344.805 160.02) (xy 505.3327 160.02))
     (stroke (width 0) (type default) (color 0 0 0 0))
   )
@@
     (stroke (width 0) (type default) (color 0 0 0 0))
   )
-  (wire (pts (xy 505.333 186.563) (xy 516.382 186.563))
+  (wire (pts (xy 505.3327 151.1308) (xy 516.3817 151.1308))
     (stroke (width 0) (type default) (color 0 0 0 0))
   )
@@
     (stroke (width 0) (type default) (color 0 0 0 0))
   )
-  (wire (pts (xy 197.485 172.72) (xy 197.485 125.095))
+  (wire (pts (xy 197.485 172.72) (xy 197.4939 121.2939))
     (stroke (width 0) (type default) (color 0 0 0 0))
   )
@@
     (stroke (width 0) (type default) (color 0 0 0 0))
   )
-  (wire (pts (xy 505.333 172.72) (xy 505.333 186.563))
-    (stroke (width 0) (type default) (color 0 0 0 0))
-  )
-  (wire (pts (xy 516.382 186.563) (xy 520.192 186.563))
+  (wire (pts (xy 505.3327 160.02) (xy 505.3327 151.1308))
+    (stroke (width 0) (type default) (color 0 0 0 0))
+  )
+  (wire (pts (xy 516.3817 151.1308) (xy 520.1917 151.1308))
     (stroke (width 0) (type default) (color 0 0 0 0))
   )
@@
   )
   (wire (pts (xy 396.24 45.72) (xy 387.985 45.72))
+    (stroke (width 0) (type default) (color 0 0 0 0))
+  )
+  (wire (pts (xy 204.4789 121.2939) (xy 205.74 121.285))
     (stroke (width 0) (type default) (color 0 0 0 0))
   )
@@
     )
   )
+  (global_label "PR23" (shape input) (at 238.76 148.59 0) (fields_autoplaced)
+    (effects (font (size 1.27 1.27)) (justify left))
+    (property "Intersheet References" "${INTERSHEET_REFS}" (id 0) (at 246.0432 148.5106 0)
+      (effects (font (size 1.27 1.27)) (justify left) hide)
+    )
+  )
   (global_label "DVY8" (shape input) (at 36.195 306.705 180) (fields_autoplaced)
     (effects (font (size 1.27 1.27)) (justify right))
@@
     )
   )
+  (global_label "~{SA}" (shape input) (at 224.79 94.615 0) (fields_autoplaced)
+    (effects (font (size 1.27 1.27)) (justify left))
+    (property "Intersheet References" "${INTERSHEET_REFS}" (id 0) (at 229.4123 94.5356 0)
+      (effects (font (size 1.27 1.27)) (justify left) hide)
+    )
+  )
   (global_label "PR82" (shape input) (at 117.475 280.035 90) (fields_autoplaced)
     (effects (font (size 1.27 1.27)) (justify left))
@@
     )
   )
-  (symbol (lib_id "atari_grav_bw:LS109A") (at 224.79 114.935 0) (unit 2)
+  (symbol (lib_name "LS109A_1") (lib_id "atari_grav_bw:LS109A") (at 224.79 114.935 0) (unit 2)
     (in_bom yes) (on_board yes)
     (property "Reference" "E_5" (id 0) (at 224.79 111.125 0))
@@
     (pin "6")
   )
-  (symbol (lib_id "power:+5V") (at 238.76 148.59 0) (unit 1)
-    (in_bom yes) (on_board yes)
-    (property "Reference" "#PWR0266" (id 0) (at 238.76 152.4 0)
-      (effects (font (size 1.27 1.27)) hide)
-    )
-    (property "Value" "+5V" (id 1) (at 241.935 146.685 0))
-    (property "Footprint" "" (id 2) (at 238.76 148.59 0)
-      (effects (font (size 1.27 1.27)) hide)
-    )
-    (property "Datasheet" "" (id 3) (at 238.76 148.59 0)
-      (effects (font (size 1.27 1.27)) hide)
-    )
-    (pin "1")
-  )
   (symbol (lib_id "Star_Wars_Vector_PCB:LS32") (at 137.795 234.95 0) (mirror x) (unit 3) (convert 2)
     (in_bom yes) (on_board yes)
@@
       (effects (font (size 1.27 1.27)) hide)
     )
-    (property "Value" "+5V" (id 1) (at 237.49 154.305 0))
+    (property "Value" "+5V" (id 1) (at 232.41 152.3746 0))
     (property "Footprint" "" (id 2) (at 234.315 156.21 0)
       (effects (font (size 1.27 1.27)) hide)
@@
     (pin "7")
   )
-  (symbol (lib_id "atari_grav_bw:TP") (at 518.287 181.483 0) (unit 1)
-    (in_bom yes) (on_board yes)
-    (property "Reference" "TP~{VCTR}1" (id 0) (at 519.811 179.705 0)
+  (symbol (lib_id "atari_grav_bw:TP") (at 518.2867 146.0508 0) (unit 1)
+    (in_bom yes) (on_board yes)
+    (property "Reference" "TPVCTR1" (id 0) (at 519.8107 144.2728 0)
       (effects (font (size 1.524 1.524)) (justify left))
     )
-    (property "Value" "TP" (id 1) (at 516.382 180.213 0)
+    (property "Value" "TP" (id 1) (at 516.3817 144.7808 0)
       (effects (font (size 1.524 1.524)) hide)
     )
-    (property "Footprint" "quantum_arcade_pcb:TP" (id 2) (at 516.382 182.753 0)
+    (property "Footprint" "quantum_arcade_pcb:TP" (id 2) (at 516.3817 147.3208 0)
       (effects (font (size 1.524 1.524)) hide)
     )
-    (property "Datasheet" "" (id 3) (at 516.382 182.753 0)
+    (property "Datasheet" "" (id 3) (at 516.3817 147.3208 0)
       (effects (font (size 1.524 1.524)) hide)
     )
