File: kicad/atari_gravitar_black_widow/Sheet3B.kicad_sch (KiCad schematic)
At the start: 106 parts, among them Q1 2N3904, Y1 12.096 MHZ

Commit message: reviewed first two sheets
see notes on individual sheets
Parts:
- renumbered TP+15V1 to TP+15V, TP+6.8V1 to TP+6.8V, TP-15V1 to TP-15V, TP~POR1 to TP/POR, TP~RESET1 to TP/RESET, TP~WDDIS1 to TP/WDDIS, TP12MHZ1 to TP12MHZ, TPRESET1 to TPRESET, TPPHI0 to TPΦ0
Connections:
- net 12MHZ: now reaches E_4.5 (UP), F_3.10, TP12MHZ.1, TP12MHZ.2
Other:
- note added: "1/14 (am): Added 12MHz and Φ0 globals. Should /WDDIS also have a global label? Should /POR also have a gloabl label?"
Changed lines of the file:
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@@
     (effects (font (size 2.54 2.54) (thickness 0.508) bold) (justify left bottom))
+  )
+  (text "1/14 (am):\n\nAdded 12MHz and Φ0 globals.\n\nShould /WDDIS also have a global label?\n\nShould /POR also have a gloabl label?"
+    (at 531.495 236.855 0)
+    (effects (font (size 1.27 1.27)) (justify left bottom))
   )
   (global_label "3KHZ" (shape input) (at 440.055 195.58 0) (fields_autoplaced)
@@
     )
   )
+  (global_label "Φ0" (shape input) (at 434.34 161.925 0) (fields_autoplaced)
+    (effects (font (size 1.27 1.27)) (justify left))
+    (property "Intersheet References" "${INTERSHEET_REFS}" (id 0) (at 439.2042 161.8456 0)
+      (effects (font (size 1.27 1.27)) (justify left) hide)
+    )
+  )
   (global_label "PR23" (shape input) (at 359.41 131.445 90) (fields_autoplaced)
     (effects (font (size 1.27 1.27)) (justify left))
@@
     (property "Intersheet References" "${INTERSHEET_REFS}" (id 0) (at 0 0 0)
       (effects (font (size 1.27 1.27)) hide)
+    )
+  )
+  (global_label "12MHZ" (shape input) (at 434.34 132.715 0) (fields_autoplaced)
+    (effects (font (size 1.27 1.27)) (justify left))
+    (property "Intersheet References" "${INTERSHEET_REFS}" (id 0) (at 443.0747 132.6356 0)
+      (effects (font (size 1.27 1.27)) (justify left) hide)
     )
   )
@@
   (symbol (lib_id "atari_grav_bw:TP") (at 518.795 285.115 0) (unit 1)
     (in_bom yes) (on_board yes)
-    (property "Reference" "TP~RESET1" (id 0) (at 513.715 278.765 0)
+    (property "Reference" "TP/RESET" (id 0) (at 513.715 278.765 0)
       (effects (font (size 1.524 1.524)) (justify left))
     )
@@
   (symbol (lib_id "atari_grav_bw:TP") (at 507.365 281.305 0) (unit 1)
     (in_bom yes) (on_board yes)
-    (property "Reference" "TPRESET1" (id 0) (at 502.285 274.955 0)
+    (property "Reference" "TPRESET" (id 0) (at 502.285 274.955 0)
       (effects (font (size 1.524 1.524)) (justify left))
     )
@@
   (symbol (lib_id "atari_grav_bw:TP") (at 507.365 240.665 0) (unit 1)
     (in_bom yes) (on_board yes)
-    (property "Reference" "TP~POR1" (id 0) (at 503.555 234.315 0)
+    (property "Reference" "TP/POR" (id 0) (at 503.555 234.315 0)
       (effects (font (size 1.524 1.524)) (justify left))
     )
@@
   (symbol (lib_id "atari_grav_bw:TP") (at 432.435 156.845 0) (unit 1)
     (in_bom yes) (on_board yes)
-    (property "Reference" "TPPHI0" (id 0) (at 428.625 150.495 0)
+    (property "Reference" "TPΦ0" (id 0) (at 428.625 150.495 0)
       (effects (font (size 1.524 1.524)) (justify left))
     )
@@
   (symbol (lib_id "atari_grav_bw:TP") (at 432.435 127.635 0) (unit 1)
     (in_bom yes) (on_board yes)
-    (property "Reference" "TP12MHZ1" (id 0) (at 435.4576 127.8382 0)
+    (property "Reference" "TP12MHZ" (id 0) (at 435.4576 127.8382 0)
       (effects (font (size 1.524 1.524)) (justify left))
     )
@@
   (symbol (lib_id "atari_grav_bw:TP") (at 131.445 116.84 0) (unit 1)
     (in_bom yes) (on_board yes)
-    (property "Reference" "TP-15V1" (id 0) (at 134.4676 117.0432 0)
+    (property "Reference" "TP-15V" (id 0) (at 134.4676 117.0432 0)
       (effects (font (size 1.524 1.524)) (justify left))
     )
@@
   (symbol (lib_id "atari_grav_bw:TP") (at 145.415 139.065 0) (unit 1)
     (in_bom yes) (on_board yes)
-    (property "Reference" "TP+15V1" (id 0) (at 148.4376 139.2682 0)
+    (property "Reference" "TP+15V" (id 0) (at 148.4376 139.2682 0)
       (effects (font (size 1.524 1.524)) (justify left))
     )
@@
   (symbol (lib_id "atari_grav_bw:TP") (at 95.885 164.465 0) (unit 1)
     (in_bom yes) (on_board yes)
-    (property "Reference" "TP+6.8V1" (id 0) (at 90.17 158.115 0)
+    (property "Reference" "TP+6.8V" (id 0) (at 90.17 158.115 0)
       (effects (font (size 1.524 1.524)) (justify left))
     )
@@
   (symbol (lib_id "atari_grav_bw:TP") (at 507.365 225.425 0) (unit 1)
     (in_bom yes) (on_board yes)
-    (property "Reference" "TP~WDDIS1" (id 0) (at 502.92 219.075 0)
+    (property "Reference" "TP/WDDIS" (id 0) (at 502.92 219.075 0)
       (effects (font (size 1.524 1.524)) (justify left))
     )

Commit message: Fri Night
various reviews
Parts:
- renumbered E_3 to E3, E_4 to E4, F_3 to F3, F_4 to F4, F_7 to F7, H_4 to H4, K_3 to K3, L_4 to L4, R_8 to R8, TP6MHZ1 to TP6MHZ, TPΦ0 to TPPHI0
Other:
- note added: "Clock"
- note added: "Power Input"
- note added: "Power-On Reset"
- note added: "Watchdog"
- note removed: "1/14 (am): Added 12MHz and Φ0 globals. Should /WDDIS also have a global label? Should /POR also have a gloabl label?"
- note removed: "CLOCK"
- note removed: "POWER INPUT"
- note removed: "POWER-ON RESET"
- note removed: "WATCHDOG"
Changed lines of the file:
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@@
     (stroke (width 0) (type default) (color 0 0 0 0))
   )
-  (text "POWER-ON RESET" (at 300.99 192.405 0)
+  (text "Power-On Reset" (at 300.99 192.405 0)
     (effects (font (size 2.54 2.54) (thickness 0.508) bold) (justify left bottom))
   )
-  (text "POWER INPUT" (at 119.38 273.685 0)
+  (text "Power Input" (at 119.38 273.685 0)
     (effects (font (size 2.54 2.54) (thickness 0.508) bold) (justify left bottom))
   )
-  (text "CLOCK" (at 238.76 123.19 0)
+  (text "Clock" (at 238.76 123.19 0)
     (effects (font (size 2.54 2.54) (thickness 0.508) bold) (justify left bottom))
   )
-  (text "WATCHDOG" (at 367.665 218.44 0)
+  (text "Watchdog" (at 367.665 218.44 0)
     (effects (font (size 2.54 2.54) (thickness 0.508) bold) (justify left bottom))
-  )
-  (text "1/14 (am):\n\nAdded 12MHz and Φ0 globals.\n\nShould /WDDIS also have a global label?\n\nShould /POR also have a gloabl label?"
-    (at 531.495 236.855 0)
-    (effects (font (size 1.27 1.27)) (justify left bottom))
   )
   (global_label "3KHZ" (shape input) (at 440.055 195.58 0) (fields_autoplaced)
@@
   (symbol (lib_id "atari_grav_bw:LS04") (at 333.375 146.05 0) (unit 5)
     (in_bom yes) (on_board yes)
-    (property "Reference" "F_3" (id 0) (at 337.185 143.51 0))
+    (property "Reference" "F3" (id 0) (at 337.185 143.51 0))
     (property "Value" "S04" (id 1) (at 337.185 147.955 0))
     (property "Footprint" "" (id 2) (at 333.375 146.05 0)
@@
   (symbol (lib_id "atari_grav_bw:LS193A") (at 369.57 148.59 0) (unit 1)
     (in_bom yes) (on_board yes)
-    (property "Reference" "E_4" (id 0) (at 368.935 147.32 0)
+    (property "Reference" "E4" (id 0) (at 368.935 147.32 0)
       (effects (font (size 1.27 1.27)) (justify left))
     )
@@
   (symbol (lib_id "atari_grav_bw:082") (at 277.495 219.075 0) (unit 1)
     (in_bom yes) (on_board yes)
-    (property "Reference" "R_8" (id 0) (at 280.035 215.265 0))
-    (property "Value" "082" (id 1) (at 280.035 222.25 0))
+    (property "Reference" "R8" (id 0) (at 280.67 215.9 0))
+    (property "Value" "082" (id 1) (at 280.67 222.25 0))
     (property "Footprint" "" (id 2) (at 277.495 219.075 0)
       (effects (font (size 1.27 1.27)) hide)
@@
   (symbol (lib_id "atari_grav_bw:LS393A") (at 386.715 193.04 0) (unit 1)
     (in_bom yes) (on_board yes)
-    (property "Reference" "F_4" (id 0) (at 386.715 192.405 0))
+    (property "Reference" "F4" (id 0) (at 386.715 192.405 0))
     (property "Value" "LS393A" (id 1) (at 386.715 194.31 0))
     (property "Footprint" "" (id 2) (at 386.715 193.04 0)
@@
   (symbol (lib_id "atari_grav_bw:LS393B") (at 428.625 264.16 0) (unit 1)
     (in_bom yes) (on_board yes)
-    (property "Reference" "H_4" (id 0) (at 428.625 262.89 0))
+    (property "Reference" "H4" (id 0) (at 428.625 262.89 0))
     (property "Value" "LS393B" (id 1) (at 428.625 265.43 0))
     (property "Footprint" "" (id 2) (at 428.625 264.16 0)
@@
   (symbol (lib_id "atari_grav_bw:LS14") (at 325.755 245.745 0) (unit 2)
     (in_bom yes) (on_board yes)
-    (property "Reference" "F_7" (id 0) (at 328.93 243.205 0))
+    (property "Reference" "F7" (id 0) (at 328.93 243.205 0))
     (property "Value" "LS14" (id 1) (at 328.93 248.285 0))
     (property "Footprint" "" (id 2) (at 328.295 245.745 0)
@@
   (symbol (lib_id "atari_grav_bw:LS14") (at 356.87 245.745 0) (unit 3)
     (in_bom yes) (on_board yes)
-    (property "Reference" "F_7" (id 0) (at 360.045 243.205 0))
+    (property "Reference" "F7" (id 0) (at 360.045 243.205 0))
     (property "Value" "LS14" (id 1) (at 360.045 248.285 0))
     (property "Footprint" "" (id 2) (at 359.41 245.745 0)
@@
   (symbol (lib_id "atari_grav_bw:LS00") (at 393.7 256.54 0) (mirror x) (unit 1) (convert 2)
     (in_bom yes) (on_board yes)
-    (property "Reference" "E_3" (id 0) (at 393.065 257.81 0)
+    (property "Reference" "E3" (id 0) (at 393.065 257.81 0)
       (effects (font (size 1.27 1.27)) (justify left))
     )
@@
   (symbol (lib_id "atari_grav_bw:LS08") (at 429.895 231.14 0) (unit 3)
     (in_bom yes) (on_board yes)
-    (property "Reference" "L_4" (id 0) (at 429.895 233.045 0))
+    (property "Reference" "L4" (id 0) (at 429.895 233.045 0))
     (property "Value" "LS08" (id 1) (at 429.895 230.505 0))
     (property "Footprint" "" (id 2) (at 429.895 231.14 0)
@@
   (symbol (lib_id "atari_grav_bw:LS74") (at 469.9 264.16 0) (unit 1)
     (in_bom yes) (on_board yes)
-    (property "Reference" "K_3" (id 0) (at 467.36 262.89 0)
+    (property "Reference" "K3" (id 0) (at 467.36 262.89 0)
       (effects (font (size 1.27 1.27)) (justify left))
     )
@@
   (symbol (lib_id "atari_grav_bw:TP") (at 432.435 156.845 0) (unit 1)
     (in_bom yes) (on_board yes)
-    (property "Reference" "TPΦ0" (id 0) (at 428.625 150.495 0)
+    (property "Reference" "TPPHI0" (id 0) (at 428.625 150.495 0)
       (effects (font (size 1.524 1.524)) (justify left))
     )
@@
   (symbol (lib_id "atari_grav_bw:TP") (at 432.435 180.975 0) (unit 1)
     (in_bom yes) (on_board yes)
-    (property "Reference" "TP6MHZ1" (id 0) (at 427.355 174.625 0)
+    (property "Reference" "TP6MHZ" (id 0) (at 427.355 174.625 0)
       (effects (font (size 1.524 1.524)) (justify left))
     )

Commit message: 20 errors left
Parts:
- renumbered R8 to R_8
Changed lines of the file:
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@@
   (symbol (lib_id "atari_grav_bw:082") (at 277.495 219.075 0) (unit 1)
     (in_bom yes) (on_board yes)
-    (property "Reference" "R8" (id 0) (at 280.67 215.9 0))
+    (property "Reference" "R_8" (id 0) (at 280.67 215.9 0))
     (property "Value" "082" (id 1) (at 280.67 222.25 0))
     (property "Footprint" "" (id 2) (at 277.495 219.075 0)

Commit message: Fixed most errors
Parts:
- renumbered TP+15V to TP+15V1, TP+6.8V to TP+6.8V1, TP-15V to TP-15V1, TP/POR to TP/POR1, TP/RESET to TP/RESET1, TP/WDDIS to TP/WDDIS1, TP12MHZ to TP12MHZ1, TP6MHZ to TP6MHZ1, TPPHI0 to TPPHI01, TPRESET to TPRESET1
Changed lines of the file:
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@@
   (junction (at 136.525 181.61) (diameter 0) (color 0 0 0 0)
   )
+  (junction (at 88.9 169.545) (diameter 0) (color 0 0 0 0)
+  )
   (junction (at 306.705 158.115) (diameter 0) (color 0 0 0 0)
   )
@@
     (stroke (width 0) (type default) (color 0 0 0 0))
   )
+  (wire (pts (xy 88.9 167.005) (xy 88.9 169.545))
+    (stroke (width 0) (type default) (color 0 0 0 0))
+  )
   (wire (pts (xy 136.525 166.37) (xy 136.525 165.1))
     (stroke (width 0) (type default) (color 0 0 0 0))
@@
     (pin "6")
   )
-  (symbol (lib_id "power:GND") (at 476.25 274.32 0) (unit 1)
-    (in_bom yes) (on_board yes)
-    (property "Reference" "#PWR0124" (id 0) (at 476.25 280.67 0)
-      (effects (font (size 1.27 1.27)) hide)
-    )
-    (property "Value" "GND" (id 1) (at 476.377 278.7142 0))
-    (property "Footprint" "" (id 2) (at 476.25 274.32 0)
-      (effects (font (size 1.27 1.27)) hide)
-    )
-    (property "Datasheet" "" (id 3) (at 476.25 274.32 0)
-      (effects (font (size 1.27 1.27)) hide)
-    )
-    (pin "1")
-  )
   (symbol (lib_id "power:+5V") (at 476.25 254 0) (unit 1)
     (in_bom yes) (on_board yes)
@@
   (symbol (lib_id "atari_grav_bw:TP") (at 518.795 285.115 0) (unit 1)
     (in_bom yes) (on_board yes)
-    (property "Reference" "TP/RESET" (id 0) (at 513.715 278.765 0)
+    (property "Reference" "TP/RESET1" (id 0) (at 513.715 278.765 0)
       (effects (font (size 1.524 1.524)) (justify left))
     )
@@
   (symbol (lib_id "atari_grav_bw:TP") (at 507.365 281.305 0) (unit 1)
     (in_bom yes) (on_board yes)
-    (property "Reference" "TPRESET" (id 0) (at 502.285 274.955 0)
+    (property "Reference" "TPRESET1" (id 0) (at 502.285 274.955 0)
       (effects (font (size 1.524 1.524)) (justify left))
     )
@@
   (symbol (lib_id "atari_grav_bw:TP") (at 507.365 240.665 0) (unit 1)
     (in_bom yes) (on_board yes)
-    (property "Reference" "TP/POR" (id 0) (at 503.555 234.315 0)
+    (property "Reference" "TP/POR1" (id 0) (at 503.555 234.315 0)
       (effects (font (size 1.524 1.524)) (justify left))
     )
@@
   (symbol (lib_id "atari_grav_bw:TP") (at 432.435 156.845 0) (unit 1)
     (in_bom yes) (on_board yes)
-    (property "Reference" "TPPHI0" (id 0) (at 428.625 150.495 0)
+    (property "Reference" "TPPHI01" (id 0) (at 428.625 150.495 0)
       (effects (font (size 1.524 1.524)) (justify left))
     )
@@
   (symbol (lib_id "atari_grav_bw:TP") (at 432.435 180.975 0) (unit 1)
     (in_bom yes) (on_board yes)
-    (property "Reference" "TP6MHZ" (id 0) (at 427.355 174.625 0)
+    (property "Reference" "TP6MHZ1" (id 0) (at 427.355 174.625 0)
       (effects (font (size 1.524 1.524)) (justify left))
     )
@@
   (symbol (lib_id "atari_grav_bw:TP") (at 432.435 127.635 0) (unit 1)
     (in_bom yes) (on_board yes)
-    (property "Reference" "TP12MHZ" (id 0) (at 435.4576 127.8382 0)
+    (property "Reference" "TP12MHZ1" (id 0) (at 435.4576 127.8382 0)
       (effects (font (size 1.524 1.524)) (justify left))
     )
@@
   (symbol (lib_id "atari_grav_bw:TP") (at 131.445 116.84 0) (unit 1)
     (in_bom yes) (on_board yes)
-    (property "Reference" "TP-15V" (id 0) (at 134.4676 117.0432 0)
+    (property "Reference" "TP-15V1" (id 0) (at 134.4676 117.0432 0)
       (effects (font (size 1.524 1.524)) (justify left))
     )
@@
   (symbol (lib_id "atari_grav_bw:TP") (at 145.415 139.065 0) (unit 1)
     (in_bom yes) (on_board yes)
-    (property "Reference" "TP+15V" (id 0) (at 148.4376 139.2682 0)
+    (property "Reference" "TP+15V1" (id 0) (at 148.4376 139.2682 0)
       (effects (font (size 1.524 1.524)) (justify left))
     )
@@
   (symbol (lib_id "atari_grav_bw:TP") (at 95.885 164.465 0) (unit 1)
     (in_bom yes) (on_board yes)
-    (property "Reference" "TP+6.8V" (id 0) (at 90.17 158.115 0)
+    (property "Reference" "TP+6.8V1" (id 0) (at 90.17 158.115 0)
       (effects (font (size 1.524 1.524)) (justify left))
     )
@@
   (symbol (lib_id "atari_grav_bw:TP") (at 507.365 225.425 0) (unit 1)
     (in_bom yes) (on_board yes)
-    (property "Reference" "TP/WDDIS" (id 0) (at 502.92 219.075 0)
+    (property "Reference" "TP/WDDIS1" (id 0) (at 502.92 219.075 0)
       (effects (font (size 1.524 1.524)) (justify left))
     )
@@
     (pin "2")
   )
+  (symbol (lib_id "power:PWR_FLAG") (at 88.9 167.005 0) (unit 1)
+    (in_bom yes) (on_board yes) (fields_autoplaced)
+    (property "Reference" "#FLG0107" (id 0) (at 88.9 165.1 0)
+      (effects (font (size 1.27 1.27)) hide)
+    )
+    (property "Value" "PWR_FLAG" (id 1) (at 88.9 163.4005 0))
+    (property "Footprint" "" (id 2) (at 88.9 167.005 0)
+      (effects (font (size 1.27 1.27)) hide)
+    )
+    (property "Datasheet" "~" (id 3) (at 88.9 167.005 0)
+      (effects (font (size 1.27 1.27)) hide)
+    )
+    (pin "1")
+  )
+  (symbol (lib_id "power:GND") (at 476.25 274.32 0) (unit 1)
+    (in_bom yes) (on_board yes) (fields_autoplaced)
+    (property "Reference" "#PWR0124" (id 0) (at 476.25 280.67 0)
+      (effects (font (size 1.27 1.27)) hide)
+    )
+    (property "Value" "GND" (id 1) (at 476.25 278.8825 0))
+    (property "Footprint" "" (id 2) (at 476.25 274.32 0)
+      (effects (font (size 1.27 1.27)) hide)
+    )
+    (property "Datasheet" "" (id 3) (at 476.25 274.32 0)
+      (effects (font (size 1.27 1.27)) hide)
+    )
+    (pin "1")
+  )
 )

Commit message: Worked on removing the warnings
Parts:
- removed C110: 2.2uf 35V, symbol Device:CP1
- removed C111, C121: 22uf 25V, symbol Device:CP1
- removed C117: 100uf 25V, symbol Device:CP1
- removed C119, C120: 100uf 35V, symbol Device:CP1
- added C110: 2.2uf 35V, symbol Device:C_Polarized_US
- added C111, C121: 22uf 25V, symbol Device:C_Polarized_US
- added C117: 100uf 25V, symbol Device:C_Polarized_US
- added C119, C120: 100uf 35V, symbol Device:C_Polarized_US
Connections:
- net +10V: now also R_8.8 (VCC)
- net +15V: now also C121.1
- net +24V: now also C120.1
- net +5V: now also C117.1
- net -15V: now also C111.2
- net -24V: now also C110.2, C119.2
- net GND: now also R_8.4 (VSS), C110.1, C111.1, C117.2, C119.1, C120.2, C121.2

Commit message: Removed more warnings - 25 warnings remain
Parts:
- Q1: footprint Package_TO_SOT_THT:TO-92_Inline -> (none)
Changed lines of the file:
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@@
       (effects (font (size 1.27 1.27)) (justify left))
     )
-    (property "Footprint" "Package_TO_SOT_THT:TO-92_Inline" (id 2) (at 309.245 147.955 0)
+    (property "Footprint" "" (id 2) (at 309.245 147.955 0)
       (effects (font (size 1.27 1.27) italic) (justify left) hide)
     )
