File: kicad/atari_gravitar_black_widow/Sheet3B.kicad_sch (KiCad schematic)
At the start: 106 parts, among them K3 LS74, Q1 2N3904, Y1 12.096 MHZ

Commit message: Fixed all warnings and errors
Parts:
- renumbered E3 to E_3, E4 to E_4, F3 to F_3, F4 to F_4, F7 to F_7, H4 to H_4, K3 to K_3, L4 to L_4
Changed lines of the file:
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@@
   (symbol (lib_id "atari_grav_bw:LS04") (at 333.375 146.05 0) (unit 5)
     (in_bom yes) (on_board yes)
-    (property "Reference" "F3" (id 0) (at 337.185 143.51 0))
+    (property "Reference" "F_3" (id 0) (at 337.185 143.51 0))
     (property "Value" "S04" (id 1) (at 337.185 147.955 0))
     (property "Footprint" "" (id 2) (at 333.375 146.05 0)
@@
   (symbol (lib_id "atari_grav_bw:LS193A") (at 369.57 148.59 0) (unit 1)
     (in_bom yes) (on_board yes)
-    (property "Reference" "E4" (id 0) (at 368.935 147.32 0)
+    (property "Reference" "E_4" (id 0) (at 368.935 147.32 0)
       (effects (font (size 1.27 1.27)) (justify left))
     )
@@
   (symbol (lib_id "atari_grav_bw:LS393A") (at 386.715 193.04 0) (unit 1)
     (in_bom yes) (on_board yes)
-    (property "Reference" "F4" (id 0) (at 386.715 192.405 0))
+    (property "Reference" "F_4" (id 0) (at 386.715 192.405 0))
     (property "Value" "LS393A" (id 1) (at 386.715 194.31 0))
     (property "Footprint" "" (id 2) (at 386.715 193.04 0)
@@
   (symbol (lib_id "atari_grav_bw:LS393B") (at 428.625 264.16 0) (unit 1)
     (in_bom yes) (on_board yes)
-    (property "Reference" "H4" (id 0) (at 428.625 262.89 0))
+    (property "Reference" "H_4" (id 0) (at 428.625 262.89 0))
     (property "Value" "LS393B" (id 1) (at 428.625 265.43 0))
     (property "Footprint" "" (id 2) (at 428.625 264.16 0)
@@
   (symbol (lib_id "atari_grav_bw:LS14") (at 325.755 245.745 0) (unit 2)
     (in_bom yes) (on_board yes)
-    (property "Reference" "F7" (id 0) (at 328.93 243.205 0))
+    (property "Reference" "F_7" (id 0) (at 328.93 243.205 0))
     (property "Value" "LS14" (id 1) (at 328.93 248.285 0))
     (property "Footprint" "" (id 2) (at 328.295 245.745 0)
@@
   (symbol (lib_id "atari_grav_bw:LS14") (at 356.87 245.745 0) (unit 3)
     (in_bom yes) (on_board yes)
-    (property "Reference" "F7" (id 0) (at 360.045 243.205 0))
+    (property "Reference" "F_7" (id 0) (at 360.045 243.205 0))
     (property "Value" "LS14" (id 1) (at 360.045 248.285 0))
     (property "Footprint" "" (id 2) (at 359.41 245.745 0)
@@
   (symbol (lib_id "atari_grav_bw:LS00") (at 393.7 256.54 0) (mirror x) (unit 1) (convert 2)
     (in_bom yes) (on_board yes)
-    (property "Reference" "E3" (id 0) (at 393.065 257.81 0)
+    (property "Reference" "E_3" (id 0) (at 393.065 257.81 0)
       (effects (font (size 1.27 1.27)) (justify left))
     )
@@
   (symbol (lib_id "atari_grav_bw:LS08") (at 429.895 231.14 0) (unit 3)
     (in_bom yes) (on_board yes)
-    (property "Reference" "L4" (id 0) (at 429.895 233.045 0))
+    (property "Reference" "L_4" (id 0) (at 429.895 233.045 0))
     (property "Value" "LS08" (id 1) (at 429.895 230.505 0))
     (property "Footprint" "" (id 2) (at 429.895 231.14 0)
@@
   (symbol (lib_id "atari_grav_bw:LS74") (at 469.9 264.16 0) (unit 1)
     (in_bom yes) (on_board yes)
-    (property "Reference" "K3" (id 0) (at 467.36 262.89 0)
-      (effects (font (size 1.27 1.27)) (justify left))
-    )
+    (property "Reference" "K_3" (id 0) (at 467.36 262.89 0)
+      (effects (font (size 1.27 1.27)) (justify left))
+    )

Commit message: more ttl placements
Parts:
- E_3, F_3, F_4, F_7, H_4: footprint (none) -> Star_Wars_Vector_PCB:DIP14
- E_4: footprint (none) -> Star_Wars_Vector_PCB:DIP16
Changed lines of the file:
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@@
     (property "Reference" "F_3" (id 0) (at 337.185 143.51 0))
     (property "Value" "S04" (id 1) (at 337.185 147.955 0))
-    (property "Footprint" "" (id 2) (at 333.375 146.05 0)
+    (property "Footprint" "Star_Wars_Vector_PCB:DIP14" (id 2) (at 333.375 146.05 0)
       (effects (font (size 1.27 1.27)) hide)
     )
@@
       (effects (font (size 1.27 1.27)) (justify left))
     )
-    (property "Footprint" "" (id 2) (at 369.57 148.59 0)
+    (property "Footprint" "Star_Wars_Vector_PCB:DIP16" (id 2) (at 369.57 148.59 0)
       (effects (font (size 1.27 1.27)) hide)
     )
@@
     (property "Reference" "F_4" (id 0) (at 386.715 192.405 0))
     (property "Value" "LS393A" (id 1) (at 386.715 194.31 0))
-    (property "Footprint" "" (id 2) (at 386.715 193.04 0)
+    (property "Footprint" "Star_Wars_Vector_PCB:DIP14" (id 2) (at 386.715 193.04 0)
       (effects (font (size 1.27 1.27)) hide)
     )
@@
     (property "Reference" "H_4" (id 0) (at 428.625 262.89 0))
     (property "Value" "LS393B" (id 1) (at 428.625 265.43 0))
-    (property "Footprint" "" (id 2) (at 428.625 264.16 0)
+    (property "Footprint" "Star_Wars_Vector_PCB:DIP14" (id 2) (at 428.625 264.16 0)
       (effects (font (size 1.27 1.27)) hide)
     )
@@
     (property "Reference" "F_7" (id 0) (at 328.93 243.205 0))
     (property "Value" "LS14" (id 1) (at 328.93 248.285 0))
-    (property "Footprint" "" (id 2) (at 328.295 245.745 0)
+    (property "Footprint" "Star_Wars_Vector_PCB:DIP14" (id 2) (at 328.295 245.745 0)
       (effects (font (size 1.27 1.27)) hide)
     )
@@
     (property "Reference" "F_7" (id 0) (at 360.045 243.205 0))
     (property "Value" "LS14" (id 1) (at 360.045 248.285 0))
-    (property "Footprint" "" (id 2) (at 359.41 245.745 0)
+    (property "Footprint" "Star_Wars_Vector_PCB:DIP14" (id 2) (at 359.41 245.745 0)
       (effects (font (size 1.27 1.27)) hide)
     )
@@
       (effects (font (size 1.27 1.27)) (justify left))
     )
-    (property "Footprint" "" (id 2) (at 393.7 256.54 0)
-      (effects (font (size 1.27 1.27)) hide)
-    )
+    (property "Footprint" "Star_Wars_Vector_PCB:DIP14" (id 2) (at 393.7 256.54 0)
+      (effects (font (size 1.27 1.27)) hide)
+    )

Commit message: more chip layouts
Parts:
- K_3: footprint (none) -> Star_Wars_Vector_PCB:DIP14
Changed lines of the file:
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@@
       (effects (font (size 1.27 1.27)) (justify left))
     )
-    (property "Footprint" "" (id 2) (at 470.535 270.51 0)
+    (property "Footprint" "Star_Wars_Vector_PCB:DIP14" (id 2) (at 470.535 270.51 0)
       (effects (font (size 7.62 7.62)) hide)
     )

Commit message: placements
Parts:
- L_4: footprint (none) -> Star_Wars_Vector_PCB:DIP14
- R_8: footprint (none) -> Star_Wars_Vector_PCB:DIP8
Changed lines of the file:
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@@
     (property "Reference" "L_4" (id 0) (at 429.895 233.045 0))
     (property "Value" "LS08" (id 1) (at 429.895 230.505 0))
-    (property "Footprint" "" (id 2) (at 429.895 231.14 0)
+    (property "Footprint" "Star_Wars_Vector_PCB:DIP14" (id 2) (at 429.895 231.14 0)
       (effects (font (size 1.27 1.27)) hide)
     )
@@
       (effects (font (size 1.27 1.27)) (justify left))
     )
-    (property "Footprint" "" (id 2) (at 277.495 219.075 0)
-      (effects (font (size 1.27 1.27)) hide)
-    )
+    (property "Footprint" "Star_Wars_Vector_PCB:DIP8" (id 2) (at 277.495 219.075 0)
+      (effects (font (size 1.27 1.27)) hide)
+    )

Commit message: TEST POINTS PLACED
Parts:
- TP+15V1, TP+5V1, TP+5V2, TP+6.8V1, TP-15V1, TP/POR1, TP/RESET1, TP/WDDIS1, TP12MHZ1, TP6MHZ1, TPGND1, TPGND2, TPGND3, TPGND4, TPGND5, TPGND6, TPPHI01, TPRESET1: footprint (none) -> quantum_arcade_pcb:TP
Changed lines of the file:
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@@
       (effects (font (size 1.524 1.524)) hide)
     )
-    (property "Footprint" "" (id 2) (at 516.89 286.385 0)
+    (property "Footprint" "quantum_arcade_pcb:TP" (id 2) (at 516.89 286.385 0)
       (effects (font (size 1.524 1.524)) hide)
     )
@@
       (effects (font (size 1.524 1.524)) hide)
     )
-    (property "Footprint" "" (id 2) (at 505.46 282.575 0)
+    (property "Footprint" "quantum_arcade_pcb:TP" (id 2) (at 505.46 282.575 0)
       (effects (font (size 1.524 1.524)) hide)
     )
@@
       (effects (font (size 1.524 1.524)) hide)
     )
-    (property "Footprint" "" (id 2) (at 505.46 241.935 0)
+    (property "Footprint" "quantum_arcade_pcb:TP" (id 2) (at 505.46 241.935 0)
       (effects (font (size 1.524 1.524)) hide)
     )
@@
       (effects (font (size 1.524 1.524)) hide)
     )
-    (property "Footprint" "" (id 2) (at 430.53 158.115 0)
+    (property "Footprint" "quantum_arcade_pcb:TP" (id 2) (at 430.53 158.115 0)
       (effects (font (size 1.524 1.524)) hide)
     )
@@
       (effects (font (size 1.524 1.524)) hide)
     )
-    (property "Footprint" "" (id 2) (at 430.53 182.245 0)
+    (property "Footprint" "quantum_arcade_pcb:TP" (id 2) (at 430.53 182.245 0)
       (effects (font (size 1.524 1.524)) hide)
     )
@@
       (effects (font (size 1.524 1.524)) hide)
     )
-    (property "Footprint" "" (id 2) (at 430.53 128.905 0)
+    (property "Footprint" "quantum_arcade_pcb:TP" (id 2) (at 430.53 128.905 0)
       (effects (font (size 1.524 1.524)) hide)
     )
@@
       (effects (font (size 1.524 1.524)) hide)
     )
-    (property "Footprint" "" (id 2) (at 129.54 118.11 0)
+    (property "Footprint" "quantum_arcade_pcb:TP" (id 2) (at 129.54 118.11 0)
       (effects (font (size 1.524 1.524)) hide)
     )
@@
       (effects (font (size 1.524 1.524)) hide)
     )
-    (property "Footprint" "" (id 2) (at 143.51 140.335 0)
+    (property "Footprint" "quantum_arcade_pcb:TP" (id 2) (at 143.51 140.335 0)
       (effects (font (size 1.524 1.524)) hide)
     )
@@
       (effects (font (size 1.524 1.524)) hide)
     )
-    (property "Footprint" "" (id 2) (at 93.98 165.735 0)
+    (property "Footprint" "quantum_arcade_pcb:TP" (id 2) (at 93.98 165.735 0)
       (effects (font (size 1.524 1.524)) hide)
     )
@@
       (effects (font (size 1.524 1.524)) hide)
     )
-    (property "Footprint" "" (id 2) (at 68.58 288.925 0)
+    (property "Footprint" "quantum_arcade_pcb:TP" (id 2) (at 68.58 288.925 0)
       (effects (font (size 1.524 1.524)) hide)
     )
@@
       (effects (font (size 1.524 1.524)) hide)
     )
-    (property "Footprint" "" (id 2) (at 78.105 288.925 0)
+    (property "Footprint" "quantum_arcade_pcb:TP" (id 2) (at 78.105 288.925 0)
       (effects (font (size 1.524 1.524)) hide)
     )
@@
       (effects (font (size 1.524 1.524)) hide)
     )
-    (property "Footprint" "" (id 2) (at 90.17 288.925 0)
+    (property "Footprint" "quantum_arcade_pcb:TP" (id 2) (at 90.17 288.925 0)
       (effects (font (size 1.524 1.524)) hide)
     )
@@
       (effects (font (size 1.524 1.524)) hide)
     )
-    (property "Footprint" "" (id 2) (at 99.06 288.925 0)
+    (property "Footprint" "quantum_arcade_pcb:TP" (id 2) (at 99.06 288.925 0)
       (effects (font (size 1.524 1.524)) hide)
     )
@@
       (effects (font (size 1.524 1.524)) hide)
     )
-    (property "Footprint" "" (id 2) (at 107.95 288.925 0)
+    (property "Footprint" "quantum_arcade_pcb:TP" (id 2) (at 107.95 288.925 0)
       (effects (font (size 1.524 1.524)) hide)
     )
@@
       (effects (font (size 1.524 1.524)) hide)
     )
-    (property "Footprint" "" (id 2) (at 116.84 288.925 0)
+    (property "Footprint" "quantum_arcade_pcb:TP" (id 2) (at 116.84 288.925 0)
       (effects (font (size 1.524 1.524)) hide)
     )
@@
       (effects (font (size 1.524 1.524)) hide)
     )
-    (property "Footprint" "" (id 2) (at 125.73 288.925 0)
+    (property "Footprint" "quantum_arcade_pcb:TP" (id 2) (at 125.73 288.925 0)
       (effects (font (size 1.524 1.524)) hide)
     )
@@
       (effects (font (size 1.524 1.524)) hide)
     )
-    (property "Footprint" "" (id 2) (at 134.62 288.925 0)
+    (property "Footprint" "quantum_arcade_pcb:TP" (id 2) (at 134.62 288.925 0)
       (effects (font (size 1.524 1.524)) hide)
     )
@@
       (effects (font (size 1.524 1.524)) hide)
     )
-    (property "Footprint" "" (id 2) (at 505.46 226.695 0)
-      (effects (font (size 1.524 1.524)) hide)
-    )
+    (property "Footprint" "quantum_arcade_pcb:TP" (id 2) (at 505.46 226.695 0)
+      (effects (font (size 1.524 1.524)) hide)
+    )

Commit message: PLACED C1-C15
Parts:
- C1, C10, C11, C12, C13, C14, C15, C2, C3, C4, C5, C6, C7, C8: footprint (none) -> Star_Wars_Vector_PCB:GenericComp
Changed lines of the file:
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@@
       (effects (font (size 1.27 1.27)) (justify left))
     )
-    (property "Footprint" "" (id 2) (at 108.9152 173.99 0)
+    (property "Footprint" "Star_Wars_Vector_PCB:GenericComp" (id 2) (at 108.9152 173.99 0)
       (effects (font (size 1.27 1.27)) hide)
     )
@@
       (effects (font (size 1.27 1.27)) (justify left))
     )
-    (property "Footprint" "" (id 2) (at 118.4402 173.99 0)
+    (property "Footprint" "Star_Wars_Vector_PCB:GenericComp" (id 2) (at 118.4402 173.99 0)
       (effects (font (size 1.27 1.27)) hide)
     )
@@
       (effects (font (size 1.27 1.27)) (justify left))
     )
-    (property "Footprint" "" (id 2) (at 127.9652 173.99 0)
+    (property "Footprint" "Star_Wars_Vector_PCB:GenericComp" (id 2) (at 127.9652 173.99 0)
       (effects (font (size 1.27 1.27)) hide)
     )
@@
       (effects (font (size 1.27 1.27)) (justify left))
     )
-    (property "Footprint" "" (id 2) (at 137.4902 173.99 0)
+    (property "Footprint" "Star_Wars_Vector_PCB:GenericComp" (id 2) (at 137.4902 173.99 0)
       (effects (font (size 1.27 1.27)) hide)
     )
@@
       (effects (font (size 1.27 1.27)) (justify left))
     )
-    (property "Footprint" "" (id 2) (at 147.0152 173.99 0)
+    (property "Footprint" "Star_Wars_Vector_PCB:GenericComp" (id 2) (at 147.0152 173.99 0)
       (effects (font (size 1.27 1.27)) hide)
     )
@@
       (effects (font (size 1.27 1.27)) (justify left))
     )
-    (property "Footprint" "" (id 2) (at 108.9152 190.5 0)
+    (property "Footprint" "Star_Wars_Vector_PCB:GenericComp" (id 2) (at 108.9152 190.5 0)
       (effects (font (size 1.27 1.27)) hide)
     )
@@
       (effects (font (size 1.27 1.27)) (justify left))
     )
-    (property "Footprint" "" (id 2) (at 118.4402 190.5 0)
+    (property "Footprint" "Star_Wars_Vector_PCB:GenericComp" (id 2) (at 118.4402 190.5 0)
       (effects (font (size 1.27 1.27)) hide)
     )
@@
       (effects (font (size 1.27 1.27)) (justify left))
     )
-    (property "Footprint" "" (id 2) (at 127.9652 190.5 0)
+    (property "Footprint" "Star_Wars_Vector_PCB:GenericComp" (id 2) (at 127.9652 190.5 0)
       (effects (font (size 1.27 1.27)) hide)
     )
@@
       (effects (font (size 1.27 1.27)) (justify left))
     )
-    (property "Footprint" "" (id 2) (at 137.4902 190.5 0)
+    (property "Footprint" "Star_Wars_Vector_PCB:GenericComp" (id 2) (at 137.4902 190.5 0)
       (effects (font (size 1.27 1.27)) hide)
     )
@@
       (effects (font (size 1.27 1.27)) (justify left))
     )
-    (property "Footprint" "" (id 2) (at 147.0152 190.5 0)
+    (property "Footprint" "Star_Wars_Vector_PCB:GenericComp" (id 2) (at 147.0152 190.5 0)
       (effects (font (size 1.27 1.27)) hide)
     )
@@
       (effects (font (size 1.27 1.27)) (justify left))
     )
-    (property "Footprint" "" (id 2) (at 108.9152 207.01 0)
+    (property "Footprint" "Star_Wars_Vector_PCB:GenericComp" (id 2) (at 108.9152 207.01 0)
       (effects (font (size 1.27 1.27)) hide)
     )
@@
       (effects (font (size 1.27 1.27)) (justify left))
     )
-    (property "Footprint" "" (id 2) (at 118.4402 207.01 0)
+    (property "Footprint" "Star_Wars_Vector_PCB:GenericComp" (id 2) (at 118.4402 207.01 0)
       (effects (font (size 1.27 1.27)) hide)
     )
@@
       (effects (font (size 1.27 1.27)) (justify left))
     )
-    (property "Footprint" "" (id 2) (at 127.9652 207.01 0)
+    (property "Footprint" "Star_Wars_Vector_PCB:GenericComp" (id 2) (at 127.9652 207.01 0)
       (effects (font (size 1.27 1.27)) hide)
     )
@@
       (effects (font (size 1.27 1.27)) (justify left))
     )
-    (property "Footprint" "" (id 2) (at 137.4902 207.01 0)
-      (effects (font (size 1.27 1.27)) hide)
-    )
+    (property "Footprint" "Star_Wars_Vector_PCB:GenericComp" (id 2) (at 137.4902 207.01 0)
+      (effects (font (size 1.27 1.27)) hide)
+    )
