File: kicad/atari_gravitar_black_widow/Sheet5B.kicad_sch (KiCad schematic)
At the start: 0 parts

Commit message: Sheet 5B
needs signatures
Parts:
- added J3: LS04, Star_Wars_Vector_PCB:DIP14, symbol Star_Wars_Vector_PCB:LS04
- added J6, M5: LS32, symbol atari_grav_bw:LS32
- added J7: LS139, symbol Asteroids:LS139
- added K7: 2016, Star_Wars_Vector_PCB:DDIP24, symbol Star_Wars_Vector_PCB:137211-001
- added K8, L8, L?, M8: LS157A, symbol atari_grav_bw:LS157A
- added L7: 2716, Star_Wars_Vector_PCB:DDIP24, symbol Star_Wars_Vector_PCB:2732_A
- added M/N7, N/P7, R7: 2532, Star_Wars_Vector_PCB:DDIP24, symbol Star_Wars_Vector_PCB:2732_A
- added P8: LS245, Star_Wars_Vector_PCB:DIP20, symbol Star_Wars_Vector_PCB:LS245
- added R61, R62, R63, R64, R65, R66, R67, R68: 10K, Star_Wars_Vector_PCB:GenericComp, symbol Device:R
Connections:
- new net: J7.1 (1G), J7.12 (2Y0)
- new net +5V: J7.16 (VCC), K7.24 (5V0), L7.21 (VPP), L7.24 (5V0), L8.16 (VCC), L?.16 (VCC), M/N7.21 (VPP), M/N7.24 (5V0), M8.16 (VCC), N/P7.21 (VPP), N/P7.24 (5V0), P8.20 (VCC), R61.1, R62.1, R63.1, R64.1, R65.1, R66.1, R67.1, R68.1, R7.21 (VPP), R7.24 (5V0)
- new net AB0: L?.2 (A)
- new net AB1: L?.5 (A)
- new net AB10: M8.14 (A)
- new net AB11: K8.14 (A)
- new net AB12: K8.2 (A)
- new net AB2: L?.11 (A)
- new net AB3: L?.14 (A)
- new net AB4: L8.2 (A)
- new net AB5: L8.5 (A)
- new net AB6: L8.11 (A)
- new net AB7: L8.14 (A)
- new net AB9: M8.11 (A)
- new net AM0: K7.8 (A0), L7.8 (A0), L?.4 (Y), M/N7.8 (A0), N/P7.8 (A0), R7.8 (A0)
- new net AM1: K7.7 (A1), L7.7 (A1), L?.7 (Y), M/N7.7 (A1), N/P7.7 (A1), R7.7 (A1)
- new net AM10: J3.3, K7.19 (A10), L7.19 (A10), M/N7.19 (A10), M8.12 (Y), N/P7.19 (A10), R7.19 (A10)
- new net AM11: J7.2 (1A), K8.12 (Y), M/N7.18 (A11), N/P7.18 (A11), R7.18 (A11)
- new net AM12: J7.14 (2A), K8.4 (Y)
- new net AM13: J7.13 (2B), M8.4 (Y)
- new net AM2: K7.6 (A2), L7.6 (A2), L?.9 (Y), M/N7.6 (A2), N/P7.6 (A2), R7.6 (A2)
- new net AM3: K7.5 (A3), L7.5 (A3), L?.12 (Y), M/N7.5 (A3), N/P7.5 (A3), R7.5 (A3)
- new net AM4: K7.4 (A4), L7.4 (A4), L8.4 (Y), M/N7.4 (A4), N/P7.4 (A4), R7.4 (A4)
- new net AM5: K7.3 (A5), L7.3 (A5), L8.7 (Y), M/N7.3 (A5), N/P7.3 (A5), R7.3 (A5)
- new net AM6: K7.2 (A6), L7.2 (A6), L8.9 (Y), M/N7.2 (A6), N/P7.2 (A6), R7.2 (A6)
- new net AM7: K7.1 (A7), L7.1 (A7), L8.12 (Y), M/N7.1 (A7), N/P7.1 (A7), R7.1 (A7)
- new net AM8: K7.23 (A8), L7.23 (A8), M/N7.23 (A8), M8.7 (Y), N/P7.23 (A8), R7.23 (A8)
- new net AM9: K7.22 (A9), L7.22 (A9), M/N7.22 (A9), M8.9 (Y), N/P7.22 (A9), R7.22 (A9)
- new net AVG0: L?.3 (B)
- new net AVG1: L?.6 (B)
- new net AVG10: M8.13 (B)
- new net AVG11: K8.13 (B)
- new net AVG12: K8.3 (B)
- new net AVG13: M8.3 (B)
- new net AVG2: L?.10 (B)
- new net AVG3: L?.13 (B)
- new net AVG4: L8.3 (B)
- new net AVG5: L8.6 (B)
- new net AVG6: L8.10 (B)
- new net AVG7: L8.13 (B)
- new net AVG9: M8.10 (B)
- new net DVG0: K7.9 (D0), L7.9 (D0), M/N7.9 (D0), N/P7.9 (D0), P8.17 (B1), R68.2, R7.9 (D0)
- new net DVG1: K7.10 (D1), L7.10 (D1), M/N7.10 (D1), N/P7.10 (D1), P8.18 (B0), R67.2, R7.10 (D1)
- new net DVG2: K7.11 (D2), L7.11 (D2), M/N7.11 (D2), N/P7.11 (D2), P8.16 (B2), R66.2, R7.11 (D2)
- new net DVG3: K7.13 (D3), L7.13 (D3), M/N7.13 (D3), N/P7.13 (D3), P8.15 (B3), R65.2, R7.13 (D3)
- new net DVG4: K7.14 (D4), L7.14 (D4), M/N7.14 (D4), N/P7.14 (D4), P8.14 (B4), R64.2, R7.14 (D4)
- new net DVG5: K7.15 (D5), L7.15 (D5), M/N7.15 (D5), N/P7.15 (D5), P8.11 (B7), R63.2, R7.15 (D5)
- new net DVG6: K7.16 (D6), L7.16 (D6), M/N7.16 (D6), N/P7.16 (D6), P8.12 (B6), R62.2, R7.16 (D6)
- new net DVG7: K7.17 (D7), L7.17 (D7), M/N7.17 (D7), N/P7.17 (D7), P8.13 (B5), R61.2, R7.17 (D7)
- new net GND: J7.15 (2G), J7.3 (1B), J7.8 (GND), K7.12 (GND), K7.20 (~{OE}), L7.12 (GND), L8.15 (G), L8.8 (GND), L?.15 (G), L?.8 (GND), M/N7.12 (GND), M8.15 (G), M8.8 (GND), N/P7.12 (GND), P8.10 (GND), R7.12 (GND)
- new net PR82: K8.10 (B), K8.6 (B)
- new net ~{AB13}: M8.2 (A)
- new net ~{BUFFEN}: K8.7 (Y), P8.19 (G)
- new net ~{BΦ2}: K8.5 (A)
- new net ~{R}/WB: P8.1 (DIR)
- new net ~{VMEM}: K8.1 (S), L8.1 (S), L?.1 (S), M8.1 (S)
- new net ~{VRAM}: J7.4 (1Y0), K7.18 (~{CE})
- new net ~{VROM0}: J7.5 (1Y1), L7.20 (CS)
- new net ~{VROM1}: J7.11 (2Y1), M/N7.20 (CS)
- new net ~{VROM2}: J7.10 (2Y2), N/P7.20 (CS)
- new net ~{VROM3}: J7.9 (2Y3), R7.20 (CS)
- new net ~{VW}: K7.21 (~{WE})
- new net ~{WRITE}: K8.11 (A)
- no-connect marks 0 -> 2
Other:
- note added: "Vector Address Decoder"
- note added: "Vector Address Selector"
- note added: "Vector Memory Data Buffer"
- note added: "Vector RAM"
- note added: "Vector ROM"

Commit message: REVIEWS AND FINALS
Connections:
- net +5V: now also K8.16 (VCC)
- net AB8: now also M8.5 (A)
- net AVG8: now also M8.6 (B)
- net GND: now also K8.15 (G), K8.8 (GND)
Changed lines of the file:
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@@
   )
   (text "Vector RAM" (at 186.69 142.24 0)
-    (effects (font (size 5.08 5.08)) (justify left bottom))
+    (effects (font (size 5.08 5.08) (thickness 1.016) bold) (justify left bottom))
   )
   (text "Vector ROM\n" (at 172.72 40.64 0)
-    (effects (font (size 5.08 5.08)) (justify left bottom))
+    (effects (font (size 5.08 5.08) (thickness 1.016) bold) (justify left bottom))
   )
   (text "Vector Address Selector\n" (at 31.115 153.035 0)
-    (effects (font (size 5.08 5.08)) (justify left bottom))
+    (effects (font (size 5.08 5.08) (thickness 1.016) bold) (justify left bottom))
   )
   (text "Vector Address Decoder\n" (at 37.465 34.29 0)
-    (effects (font (size 5.08 5.08)) (justify left bottom))
+    (effects (font (size 5.08 5.08) (thickness 1.016) bold) (justify left bottom))
   )
   (text "Vector Memory Data Buffer" (at 455.295 37.465 0)
-    (effects (font (size 5.08 5.08)) (justify left bottom))
+    (effects (font (size 5.08 5.08) (thickness 1.016) bold) (justify left bottom))
   )
   (global_label "~{BUFFEN}" (shape input) (at 96.52 177.165 0) (fields_autoplaced)
@@
     )
   )
-  (global_label "AVG8" (shape input) (at 51.435 257.81 180) (fields_autoplaced)
-    (effects (font (size 1.524 1.524)) (justify right))
-    (property "Intersheet References" "${INTERSHEET_REFS}" (id 0) (at -316.865 59.69 0)
+  (global_label "AVG8" (shape input) (at 51.435 258.445 180) (fields_autoplaced)
+    (effects (font (size 1.524 1.524)) (justify right))
+    (property "Intersheet References" "${INTERSHEET_REFS}" (id 0) (at -316.865 60.325 0)
       (effects (font (size 1.27 1.27)) hide)
     )
@@
     )
   )
-  (global_label "AB8" (shape input) (at 51.435 255.27 180) (fields_autoplaced)
-    (effects (font (size 1.524 1.524)) (justify right))
-    (property "Intersheet References" "${INTERSHEET_REFS}" (id 0) (at -220.345 59.69 0)
+  (global_label "AB8" (shape input) (at 51.435 255.905 180) (fields_autoplaced)
+    (effects (font (size 1.524 1.524)) (justify right))
+    (property "Intersheet References" "${INTERSHEET_REFS}" (id 0) (at -220.345 60.325 0)
       (effects (font (size 1.27 1.27)) hide)
     )
@@
     (pin "1")
   )
-  (symbol (lib_id "power:GND") (at 70.485 203.835 0) (unit 1)
-    (in_bom yes) (on_board yes)
-    (property "Reference" "#PWR0478" (id 0) (at 70.485 210.185 0)
-      (effects (font (size 1.27 1.27)) hide)
-    )
-    (property "Value" "GND" (id 1) (at 70.485 207.645 0))
-    (property "Footprint" "" (id 2) (at 70.485 203.835 0)
-      (effects (font (size 1.27 1.27)) hide)
-    )
-    (property "Datasheet" "" (id 3) (at 70.485 203.835 0)
+  (symbol (lib_id "power:GND") (at 69.85 203.835 0) (unit 1)
+    (in_bom yes) (on_board yes)
+    (property "Reference" "#PWR0478" (id 0) (at 69.85 210.185 0)
+      (effects (font (size 1.27 1.27)) hide)
+    )
+    (property "Value" "GND" (id 1) (at 69.85 207.645 0))
+    (property "Footprint" "" (id 2) (at 69.85 203.835 0)
+      (effects (font (size 1.27 1.27)) hide)
+    )
+    (property "Datasheet" "" (id 3) (at 69.85 203.835 0)
       (effects (font (size 1.27 1.27)) hide)
     )
@@
     (pin "2")
   )
-  (symbol (lib_id "power:GND") (at 75.565 196.215 0) (unit 1)
-    (in_bom yes) (on_board yes)
-    (property "Reference" "#PWR0477" (id 0) (at 75.565 202.565 0)
-      (effects (font (size 1.27 1.27)) hide)
-    )
-    (property "Value" "GND" (id 1) (at 75.565 200.025 0))
-    (property "Footprint" "" (id 2) (at 75.565 196.215 0)
-      (effects (font (size 1.27 1.27)) hide)
-    )
-    (property "Datasheet" "" (id 3) (at 75.565 196.215 0)
+  (symbol (lib_id "power:GND") (at 74.93 196.215 0) (unit 1)
+    (in_bom yes) (on_board yes)
+    (property "Reference" "#PWR0477" (id 0) (at 74.93 202.565 0)
+      (effects (font (size 1.27 1.27)) hide)
+    )
+    (property "Value" "GND" (id 1) (at 74.93 200.025 0))
+    (property "Footprint" "" (id 2) (at 74.93 196.215 0)
+      (effects (font (size 1.27 1.27)) hide)
+    )
+    (property "Datasheet" "" (id 3) (at 74.93 196.215 0)
       (effects (font (size 1.27 1.27)) hide)
     )
@@
     (pin "9")
   )
-  (symbol (lib_id "power:+5V") (at 70.485 165.735 0) (unit 1)
-    (in_bom yes) (on_board yes)
-    (property "Reference" "#PWR0469" (id 0) (at 70.485 169.545 0)
-      (effects (font (size 1.27 1.27)) hide)
-    )
-    (property "Value" "+5V" (id 1) (at 70.485 162.179 0))
-    (property "Footprint" "" (id 2) (at 70.485 165.735 0)
-      (effects (font (size 1.27 1.27)) hide)
-    )
-    (property "Datasheet" "" (id 3) (at 70.485 165.735 0)
-      (effects (font (size 1.27 1.27)) hide)
-    )
+  (symbol (lib_id "power:+5V") (at 69.85 165.735 0) (unit 1)
+    (in_bom yes) (on_board yes)
+    (property "Reference" "#PWR0469" (id 0) (at 69.85 169.545 0)
+      (effects (font (size 1.27 1.27)) hide)
+    )
+    (property "Value" "+5V" (id 1) (at 69.85 162.179 0))
+    (property "Footprint" "" (id 2) (at 69.85 165.735 0)
+      (effects (font (size 1.27 1.27)) hide)
+    )
+    (property "Datasheet" "" (id 3) (at 69.85 165.735 0)
+      (effects (font (size 1.27 1.27)) hide)
+    )

Commit message: 20 errors left
Parts:
- gave numbers to parts that had none: 1
- renumbered R7 to R_7
Connections:
- net DB1: now reaches P8.2 (A0)
- net DB0: now reaches P8.3 (A1)
- net DB2: now reaches P8.4 (A2)
- net DB3: now reaches P8.5 (A3)
- net DB4: now reaches P8.6 (A4)
- net DB7: now reaches P8.7 (A5)
- net DB6: now reaches P8.8 (A6)
- net DB5: now reaches P8.9 (A7)
Changed lines of the file:
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@@
+    )
+  )
+  (global_label "DB5" (shape input) (at 541.655 67.945 0) (fields_autoplaced)
+    (effects (font (size 1.27 1.27)) (justify left))
+    (property "Intersheet References" "${INTERSHEET_REFS}" (id 0) (at 547.7287 67.8656 0)
+      (effects (font (size 1.27 1.27)) (justify left) hide)
     )
   )
@@
     (property "Intersheet References" "${INTERSHEET_REFS}" (id 0) (at 284.1914 64.0538 0)
       (effects (font (size 1.3 1.3)) (justify left) hide)
+    )
+  )
+  (global_label "DB4" (shape input) (at 541.655 70.485 0) (fields_autoplaced)
+    (effects (font (size 1.27 1.27)) (justify left))
+    (property "Intersheet References" "${INTERSHEET_REFS}" (id 0) (at 547.7287 70.4056 0)
+      (effects (font (size 1.27 1.27)) (justify left) hide)
     )
   )
@@
     )
   )
+  (global_label "DB7" (shape input) (at 541.655 62.865 0) (fields_autoplaced)
+    (effects (font (size 1.27 1.27)) (justify left))
+    (property "Intersheet References" "${INTERSHEET_REFS}" (id 0) (at 547.7287 62.7856 0)
+      (effects (font (size 1.27 1.27)) (justify left) hide)
+    )
+  )
   (global_label "AM1" (shape input) (at 88.265 366.395 0) (fields_autoplaced)
     (effects (font (size 1.524 1.524)) (justify left))
@@
     )
   )
+  (global_label "DB3" (shape input) (at 541.655 73.025 0) (fields_autoplaced)
+    (effects (font (size 1.27 1.27)) (justify left))
+    (property "Intersheet References" "${INTERSHEET_REFS}" (id 0) (at 547.7287 72.9456 0)
+      (effects (font (size 1.27 1.27)) (justify left) hide)
+    )
+  )
   (global_label "AM4" (shape input) (at 179.07 74.295 180) (fields_autoplaced)
     (effects (font (size 1.3 1.3)) (justify right))
@@
     )
   )
+  (global_label "DB2" (shape input) (at 541.655 75.565 0) (fields_autoplaced)
+    (effects (font (size 1.27 1.27)) (justify left))
+    (property "Intersheet References" "${INTERSHEET_REFS}" (id 0) (at 547.7287 75.4856 0)
+      (effects (font (size 1.27 1.27)) (justify left) hide)
+    )
+  )
   (global_label "AB5" (shape input) (at 51.435 311.15 180) (fields_autoplaced)
     (effects (font (size 1.524 1.524)) (justify right))
@@
     )
   )
+  (global_label "DB6" (shape input) (at 541.655 65.405 0) (fields_autoplaced)
+    (effects (font (size 1.27 1.27)) (justify left))
+    (property "Intersheet References" "${INTERSHEET_REFS}" (id 0) (at 547.7287 65.3256 0)
+      (effects (font (size 1.27 1.27)) (justify left) hide)
+    )
+  )
+  (global_label "DB1" (shape input) (at 541.655 78.105 0) (fields_autoplaced)
+    (effects (font (size 1.27 1.27)) (justify left))
+    (property "Intersheet References" "${INTERSHEET_REFS}" (id 0) (at 547.7287 78.0256 0)
+      (effects (font (size 1.27 1.27)) (justify left) hide)
+    )
+  )
   (global_label "DVG7" (shape input) (at 403.86 61.595 0) (fields_autoplaced)
     (effects (font (size 1.3 1.3)) (justify left))
@@
     (property "Intersheet References" "${INTERSHEET_REFS}" (id 0) (at 299.8529 81.8338 0)
       (effects (font (size 1.3 1.3)) (justify right) hide)
+    )
+  )
+  (global_label "DB0" (shape input) (at 541.655 80.645 0) (fields_autoplaced)
+    (effects (font (size 1.27 1.27)) (justify left))
+    (property "Intersheet References" "${INTERSHEET_REFS}" (id 0) (at 547.7287 80.5656 0)
+      (effects (font (size 1.27 1.27)) (justify left) hide)
     )
   )
@@
   (symbol (lib_id "Star_Wars_Vector_PCB:2732_A") (at 196.215 70.485 0) (unit 1)
     (in_bom yes) (on_board yes)
-    (property "Reference" "R7" (id 0) (at 196.215 71.755 0)
+    (property "Reference" "R_7" (id 0) (at 196.215 71.755 0)
       (effects (font (size 1.524 1.524)))
     )
@@
   (symbol (lib_name "LS157A_2") (lib_id "atari_grav_bw:LS157A") (at 69.85 362.585 0) (unit 1)
     (in_bom yes) (on_board yes)
-    (property "Reference" "L?" (id 0) (at 68.58 361.315 0)
+    (property "Reference" "N_8" (id 0) (at 68.58 361.315 0)
       (effects (font (size 1.27 1.27)) (justify left))
     )

Commit message: Removed more warnings - 25 warnings remain
Parts:
- removed L7: 2716, Star_Wars_Vector_PCB:DDIP24, symbol Star_Wars_Vector_PCB:2732_A
- removed L8, N_8: LS157A, symbol atari_grav_bw:LS157A
- removed M/N7, N/P7, R_7: 2532, Star_Wars_Vector_PCB:DDIP24, symbol Star_Wars_Vector_PCB:2732_A
- added L_7: 2716, symbol atari_grav_bw:2716
- added L_8, N_8: LS157D, symbol atari_grav_bw:LS157D
- added M/N_7, N/P_7, R_7: 2532B, symbol atari_grav_bw:2532B
- added TPSAEN1: TP, symbol atari_grav_bw:TP
- J_3: renamed from J3; footprint Star_Wars_Vector_PCB:DIP14 -> (none)
- K_7: renamed from K7; footprint Star_Wars_Vector_PCB:DDIP24 -> (none)
- P_8: renamed from P8; footprint Star_Wars_Vector_PCB:DIP20 -> (none)
- R61, R62, R63, R64, R65, R66, R67, R68: footprint Star_Wars_Vector_PCB:GenericComp -> (none)
- renumbered J6 to J_6, J7 to J_7, K8 to K_8, M5 to M_5, M8 to M_8
Connections:
- net +5V: now also L_7.21 (VPP), L_7.24 (5V0), L_8.16 (VCC), M/N_7.21 (VPP), M/N_7.24 (5V0), N/P_7.21 (VPP), N/P_7.24 (5V0), N_8.16 (VCC), R_7.21 (VPP), R_7.24 (5V0)
- net AB0: now also N_8.2 (A)
- net AB1: now also N_8.5 (A)
- net AB2: now also N_8.11 (A)
- net AB3: now also N_8.14 (A)
- net AB4: now also L_8.2 (A)
- net AB5: now also L_8.5 (A)
- net AB6: now also L_8.11 (A)
- net AB7: now also L_8.14 (A)
- net AM0: now also L_7.8 (A0), M/N_7.8 (A0), N/P_7.8 (A0), N_8.4 (Y), R_7.8 (A0)
- net AM1: now also L_7.7 (A1), M/N_7.7 (A1), N/P_7.7 (A1), N_8.7 (Y), R_7.7 (A1)
- net AM10: now also L_7.19 (A10), M/N_7.19 (A10), N/P_7.19 (A10), R_7.19 (A10)
- net AM11: now also M/N_7.18 (A11), N/P_7.18 (A11), R_7.18 (A11)
- net AM2: now also L_7.6 (A2), M/N_7.6 (A2), N/P_7.6 (A2), N_8.9 (Y), R_7.6 (A2)
- net AM3: now also L_7.5 (A3), M/N_7.5 (A3), N/P_7.5 (A3), N_8.12 (Y), R_7.5 (A3)
- net AM4: now also L_7.4 (A4), L_8.4 (Y), M/N_7.4 (A4), N/P_7.4 (A4), R_7.4 (A4)
- net AM5: now also L_7.3 (A5), L_8.7 (Y), M/N_7.3 (A5), N/P_7.3 (A5), R_7.3 (A5)
- net AM6: now also L_7.2 (A6), L_8.9 (Y), M/N_7.2 (A6), N/P_7.2 (A6), R_7.2 (A6)
- net AM7: now also L_7.1 (A7), L_8.12 (Y), M/N_7.1 (A7), N/P_7.1 (A7), R_7.1 (A7)
- net AM8: now also L_7.23 (A8), M/N_7.23 (A8), N/P_7.23 (A8), R_7.23 (A8)
- net AM9: now also L_7.22 (A9), M/N_7.22 (A9), N/P_7.22 (A9), R_7.22 (A9)
- net AVG0: now also N_8.3 (B)
- net AVG1: now also N_8.6 (B)
- net AVG2: now also N_8.10 (B)
- net AVG3: now also N_8.13 (B)
- net AVG4: now also L_8.3 (B)
- net AVG5: now also L_8.6 (B)
- net AVG6: now also L_8.10 (B)
- net AVG7: now also L_8.13 (B)
- net DVG0: now also L_7.9 (D0), M/N_7.9 (D0), N/P_7.9 (D0), R_7.9 (D0)
- net DVG1: now also L_7.10 (D1), M/N_7.10 (D1), N/P_7.10 (D1), R_7.10 (D1)
- net DVG2: now also L_7.11 (D2), M/N_7.11 (D2), N/P_7.11 (D2), R_7.11 (D2)
- net DVG3: now also L_7.13 (D3), M/N_7.13 (D3), N/P_7.13 (D3), R_7.13 (D3)
- net DVG4: now also L_7.14 (D4), M/N_7.14 (D4), N/P_7.14 (D4), R_7.14 (D4)
- net DVG5: now also L_7.15 (D5), M/N_7.15 (D5), N/P_7.15 (D5), R_7.15 (D5)
- net DVG6: now also L_7.16 (D6), M/N_7.16 (D6), N/P_7.16 (D6), R_7.16 (D6)
- net DVG7: now also L_7.17 (D7), M/N_7.17 (D7), N/P_7.17 (D7), R_7.17 (D7)
- net GND: now also L_7.12 (GND), L_8.15 (G), L_8.8 (GND), M/N_7.12 (GND), N/P_7.12 (GND), N_8.15 (G), N_8.8 (GND), R_7.12 (GND)
- net ~{VMEM}: now also L_8.1 (S), N_8.1 (S)
- net ~{VROM0}: now also L_7.20 (CS)
- net ~{VROM1}: now also M/N_7.20 (CS)
- net ~{VROM2}: now also N/P_7.20 (CS)
- net ~{VROM3}: now also R_7.20 (CS)
- new net: TPSAEN1.1, TPSAEN1.2

Commit message: Fixed all warnings and errors
Parts:
- removed J_7: LS139, symbol Asteroids:LS139
- removed K_8, M_8: LS157A, symbol atari_grav_bw:LS157A
- removed P_8: LS245, symbol Star_Wars_Vector_PCB:LS245
- added J_7: LS139, symbol atari_grav_bw:LS139
- added K_8: LS157F, symbol atari_grav_bw:LS157F
- added M_8: LS157E, symbol atari_grav_bw:LS157E
- added P_8: LS245A, symbol atari_grav_bw:LS245A
Connections:
- net +5V: now also J_7.16 (VCC), K_8.16 (VCC), M_8.16 (VCC), P_8.20 (VCC)
- net AB10: now also M_8.14 (A)
- net AB11: now also K_8.14 (A)
- net AB12: now also K_8.2 (A)
- net AB8: now also M_8.5 (A)
- net AB9: now also M_8.11 (A)
- net AM10: now also M_8.12 (Y)
- net AM11: now also J_7.2 (1A), K_8.12 (Y)
- net AM12: now also J_7.14 (2A), K_8.4 (Y)
- net AM13: now also J_7.13 (2B), M_8.4 (Y)
- net AM8: now also M_8.7 (Y)
- net AM9: now also M_8.9 (Y)
- net AVG10: now also M_8.13 (B)
- net AVG11: now also K_8.13 (B)
- net AVG12: now also K_8.3 (B)
- net AVG13: now also M_8.3 (B)
- net AVG8: now also M_8.6 (B)
- net AVG9: now also M_8.10 (B)
- net DB0: now also P_8.3 (A1)
- net DB1: now also P_8.2 (A0)
- net DB2: now also P_8.4 (A2)
- net DB3: now also P_8.5 (A3)
- net DB4: now also P_8.6 (A4)
- net DB5: now also P_8.9 (A7)
- net DB6: now also P_8.8 (A6)
- net DB7: now also P_8.7 (A5)
- net DVG0: now also P_8.17 (B1)
- net DVG1: now also P_8.18 (B0)
- net DVG2: now also P_8.16 (B2)
- net DVG3: now also P_8.15 (B3)
- net DVG4: now also P_8.14 (B4)
- net DVG5: now also P_8.11 (B7)
- net DVG6: now also P_8.12 (B6)
- net DVG7: now also P_8.13 (B5)
- net GND: now also J_7.15 (2G), J_7.3 (1B), J_7.8 (GND), K_8.15 (G), K_8.8 (GND), M_8.15 (G), M_8.8 (GND), P_8.10 (GND)
- net PR82: now also K_8.10 (B), K_8.6 (B)
- net ~{AB13}: now also M_8.2 (A)
- net ~{BUFFEN}: now also K_8.7 (Y), P_8.19 (G)
- net ~{BΦ2}: now also K_8.5 (A)
- net ~{R}/WB: now also P_8.1 (DIR)
- net ~{VMEM}: now also K_8.1 (S), M_8.1 (S)
- net ~{VRAM}: now also J_7.4 (1Y0)
- net ~{VROM0}: now also J_7.5 (1Y1)
- net ~{VROM1}: now also J_7.11 (2Y1)
- net ~{VROM2}: now also J_7.10 (2Y2)
- net ~{VROM3}: now also J_7.9 (2Y3)
- net ~{WRITE}: now also K_8.11 (A)
- new net: J_7.1 (1G), J_7.12 (2Y0)
Other:
- moved on the sheet: J_3B, J_6D, TPSAEN1
