File: kicad/atari_gravitar_black_widow/Sheet5B.kicad_sch (KiCad schematic)
At the start: 28 parts

Commit message: Fixed 5c issues
Parts:
- renumbered R68 to R66, R66 to R68
Connections:
- net DVG6: now also P_8.12 (B6), R62.2
Changed lines of the file:
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@@
   (junction (at 492.76 73.025) (diameter 0) (color 0 0 0 0)
+  )
+  (junction (at 479.425 65.405) (diameter 0) (color 0 0 0 0)
   )
   (junction (at 488.315 45.72) (diameter 0) (color 0 0 0 0)
@@
     (stroke (width 0) (type default) (color 0 0 0 0))
   )
+  (wire (pts (xy 472.948 65.405) (xy 479.425 65.405))
+    (stroke (width 0) (type default) (color 0 0 0 0))
+  )
   (wire (pts (xy 64.77 269.24) (xy 47.625 269.24))
     (stroke (width 0) (type default) (color 0 0 0 0))
@@
     (stroke (width 0) (type default) (color 0 0 0 0))
   )
-  (wire (pts (xy 479.09 65.405) (xy 509.905 65.405))
-    (stroke (width 0) (type default) (color 0 0 0 0))
-  )
   (wire (pts (xy 473.075 67.945) (xy 483.87 67.945))
     (stroke (width 0) (type default) (color 0 0 0 0))
@@
     (stroke (width 0) (type default) (color 0 0 0 0))
   )
-  (wire (pts (xy 479.65 65.36) (xy 479.09 65.405))
-    (stroke (width 0) (type default) (color 0 0 0 0))
-  )
   (wire (pts (xy 109.728 105.41) (xy 109.728 224.79))
     (stroke (width 0) (type default) (color 0 0 0 0))
@@
     (stroke (width 0) (type default) (color 0 0 0 0))
   )
-  (wire (pts (xy 473 65.36) (xy 479.65 65.36))
-    (stroke (width 0) (type default) (color 0 0 0 0))
-  )
   (wire (pts (xy 525.78 97.155) (xy 509.27 97.155))
     (stroke (width 0) (type default) (color 0 0 0 0))
@@
   )
   (wire (pts (xy 94.615 191.135) (xy 96.52 191.135))
+    (stroke (width 0) (type default) (color 0 0 0 0))
+  )
+  (wire (pts (xy 479.425 65.405) (xy 509.905 65.405))
     (stroke (width 0) (type default) (color 0 0 0 0))
   )
@@
     )
   )
-  (global_label "DVG6" (shape input) (at 473 65.365 180) (fields_autoplaced)
-    (effects (font (size 1.3 1.3)) (justify right))
-    (property "Intersheet References" "${INTERSHEET_REFS}" (id 0) (at 465.6686 65.2838 0)
+  (global_label "DVG6" (shape input) (at 472.948 65.405 180) (fields_autoplaced)
+    (effects (font (size 1.3 1.3)) (justify right))
+    (property "Intersheet References" "${INTERSHEET_REFS}" (id 0) (at 465.6166 65.3238 0)
       (effects (font (size 1.3 1.3)) (justify right) hide)
     )
@@
   (symbol (lib_id "Device:R") (at 497.205 52.07 0) (unit 1)
     (in_bom yes) (on_board yes)
-    (property "Reference" "R66" (id 0) (at 499.237 52.07 90))
+    (property "Reference" "R68" (id 0) (at 499.237 52.07 90))
     (property "Value" "10K" (id 1) (at 497.205 52.07 90))
     (property "Footprint" "Star_Wars_Vector_PCB:GenericComp" (id 2) (at 495.427 52.07 90)
@@
   (symbol (lib_id "Device:R") (at 506.095 52.07 0) (unit 1)
     (in_bom yes) (on_board yes)
-    (property "Reference" "R68" (id 0) (at 508.127 52.07 90))
+    (property "Reference" "R66" (id 0) (at 508.127 52.07 90))
     (property "Value" "10K" (id 1) (at 506.095 52.07 90))
     (property "Footprint" "Star_Wars_Vector_PCB:GenericComp" (id 2) (at 504.317 52.07 90)
