File: kicad/atari_gravitar_black_widow/Sheet5A.kicad_sch (KiCad schematic)
At the start: 120 parts, among them J6 LS32, P10 DIP SW, Q2 2N6044, Q3 2N6044, Q4 2N6044

Commit message: Fixed all warnings and errors
Parts:
- removed P10: DIP SW, symbol Switch:SW_DIP_x01
- removed P_10: DIP SW, symbol Switch:SW_DIP_x03
- added P_10: SW4POS, symbol atari_grav_bw:SW4POS
- renumbered B4 to B_4, B5 to B_5, C/D3 to C/D_3, D4 to D_4, D5 to D_5, J6 to J_6
Connections:
- net COIN_CNTRL: now also P_10.8
- net COIN_CNTRR: now also P_10.1
- net GND: now also P_10.5, P_10.6, P_10.7
- net at L_9.15 (I2b), R138.2: now also P_10.4
- net at L_9.13 (I1b), R137.2: now also P_10.3
- net at L_9.11 (I0b), R136.2: now also P_10.2
Other:
- moved on the sheet: J_6A

Commit message: first traces.
Parts:
- B_3, C/D_3: footprint (none) -> Star_Wars_Vector_PCB:DDIP40
Changed lines of the file:
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@@
     (property "Reference" "B_3" (id 0) (at 358.14 86.995 0))
     (property "Value" "POKEY" (id 1) (at 358.14 89.535 0))
-    (property "Footprint" "" (id 2) (at 358.14 92.075 0)
+    (property "Footprint" "Star_Wars_Vector_PCB:DDIP40" (id 2) (at 358.14 92.075 0)
       (effects (font (size 1.27 1.27)) hide)
     )
@@
     (property "Reference" "C/D_3" (id 0) (at 358.14 149.225 0))
     (property "Value" "POKEY" (id 1) (at 358.14 151.765 0))
-    (property "Footprint" "" (id 2) (at 358.14 154.305 0)
-      (effects (font (size 1.27 1.27)) hide)
-    )
+    (property "Footprint" "Star_Wars_Vector_PCB:DDIP40" (id 2) (at 358.14 154.305 0)
+      (effects (font (size 1.27 1.27)) hide)
+    )

Commit message: place ttl
Parts:
- B_5: footprint (none) -> Star_Wars_Vector_PCB:DIP14
Changed lines of the file:
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@@
     (property "Reference" "B_5" (id 0) (at 483.235 176.53 0))
     (property "Value" "LM324A" (id 1) (at 479.425 179.705 0))
-    (property "Footprint" "" (id 2) (at 479.425 182.245 0)
+    (property "Footprint" "Star_Wars_Vector_PCB:DIP14" (id 2) (at 479.425 182.245 0)
       (effects (font (size 1.27 1.27)) hide)
     )
@@
     (property "Reference" "B_5" (id 0) (at 516.89 177.165 0))
     (property "Value" "LM324A" (id 1) (at 513.08 180.34 0))
-    (property "Footprint" "" (id 2) (at 513.08 182.88 0)
+    (property "Footprint" "Star_Wars_Vector_PCB:DIP14" (id 2) (at 513.08 182.88 0)
       (effects (font (size 1.27 1.27)) hide)
     )
@@
     (property "Reference" "B_5" (id 0) (at 516.89 183.515 0))
     (property "Value" "LM324A" (id 1) (at 513.08 180.34 0))
-    (property "Footprint" "" (id 2) (at 513.08 177.8 0)
+    (property "Footprint" "Star_Wars_Vector_PCB:DIP14" (id 2) (at 513.08 177.8 0)
       (effects (font (size 1.27 1.27)) hide)
     )
@@
     (property "Reference" "B_5" (id 0) (at 453.39 173.355 0))
     (property "Value" "LM324A" (id 1) (at 450.215 177.165 0))
-    (property "Footprint" "" (id 2) (at 450.215 179.705 0)
+    (property "Footprint" "Star_Wars_Vector_PCB:DIP14" (id 2) (at 450.215 179.705 0)
       (effects (font (size 1.27 1.27)) hide)
     )
@@
     (property "Reference" "B_5" (id 0) (at 415.925 170.815 0))
     (property "Value" "LM324A" (id 1) (at 412.75 174.625 0))
-    (property "Footprint" "" (id 2) (at 412.75 177.165 0)
-      (effects (font (size 1.27 1.27)) hide)
-    )
+    (property "Footprint" "Star_Wars_Vector_PCB:DIP14" (id 2) (at 412.75 177.165 0)
+      (effects (font (size 1.27 1.27)) hide)
+    )

Commit message: more ttl placements
Parts:
- D_5: footprint (none) -> Star_Wars_Vector_PCB:DIP14
Changed lines of the file:
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@@
     (property "Reference" "D_5" (id 0) (at 494.03 113.665 0))
     (property "Value" "LM324A" (id 1) (at 490.855 117.475 0))
-    (property "Footprint" "" (id 2) (at 490.855 120.015 0)
+    (property "Footprint" "Star_Wars_Vector_PCB:DIP14" (id 2) (at 490.855 120.015 0)
       (effects (font (size 1.27 1.27)) hide)
     )
@@
     (property "Reference" "D_5" (id 0) (at 466.725 111.125 0))
     (property "Value" "LM324A" (id 1) (at 463.55 114.935 0))
-    (property "Footprint" "" (id 2) (at 463.55 117.475 0)
+    (property "Footprint" "Star_Wars_Vector_PCB:DIP14" (id 2) (at 463.55 117.475 0)
       (effects (font (size 1.27 1.27)) hide)
     )
@@
     (property "Reference" "D_5" (id 0) (at 421.64 109.22 0))
     (property "Value" "LM324A" (id 1) (at 417.83 112.395 0))
-    (property "Footprint" "" (id 2) (at 417.83 114.935 0)
+    (property "Footprint" "Star_Wars_Vector_PCB:DIP14" (id 2) (at 417.83 114.935 0)
       (effects (font (size 1.27 1.27)) hide)
     )
@@
     (property "Reference" "D_5" (id 0) (at 421.64 115.57 0))
     (property "Value" "LM324A" (id 1) (at 417.83 112.395 0))
-    (property "Footprint" "" (id 2) (at 417.83 109.855 0)
-      (effects (font (size 1.27 1.27)) hide)
-    )
+    (property "Footprint" "Star_Wars_Vector_PCB:DIP14" (id 2) (at 417.83 109.855 0)
+      (effects (font (size 1.27 1.27)) hide)
+    )

Commit message: more chip layouts
Parts:
- J_6: footprint (none) -> Star_Wars_Vector_PCB:DIP14
Changed lines of the file:
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@@
     (property "Reference" "J_6" (id 0) (at 88.9 142.24 0))
     (property "Value" "LS32" (id 1) (at 88.9 144.78 0))
-    (property "Footprint" "" (id 2) (at 88.9 143.51 0)
+    (property "Footprint" "Star_Wars_Vector_PCB:DIP14" (id 2) (at 88.9 143.51 0)
       (effects (font (size 1.27 1.27)) hide)
     )

Commit message: placements
Parts:
- L_9, M_9, N_9, R_9: footprint (none) -> Star_Wars_Vector_PCB:DIP20
Changed lines of the file:
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@@
       (effects (font (size 1.27 1.27)) (justify left))
     )
-    (property "Footprint" "" (id 2) (at 194.945 316.865 0)
+    (property "Footprint" "Star_Wars_Vector_PCB:DIP20" (id 2) (at 194.945 316.865 0)
       (effects (font (size 1.27 1.27)) hide)
     )
@@
       (effects (font (size 1.27 1.27)) (justify left))
     )
-    (property "Footprint" "" (id 2) (at 306.705 284.48 0)
+    (property "Footprint" "Star_Wars_Vector_PCB:DIP20" (id 2) (at 306.705 284.48 0)
       (effects (font (size 1.27 1.27)) hide)
     )
@@
       (effects (font (size 1.27 1.27)) (justify left))
     )
-    (property "Footprint" "" (id 2) (at 194.945 103.505 0)
+    (property "Footprint" "Star_Wars_Vector_PCB:DIP20" (id 2) (at 194.945 103.505 0)
       (effects (font (size 1.27 1.27)) hide)
     )
@@
       (effects (font (size 1.27 1.27)) (justify left))
     )
-    (property "Footprint" "" (id 2) (at 194.945 210.185 0)
-      (effects (font (size 1.27 1.27)) hide)
-    )
+    (property "Footprint" "Star_Wars_Vector_PCB:DIP20" (id 2) (at 194.945 210.185 0)
+      (effects (font (size 1.27 1.27)) hide)
+    )

Commit message: LAST OF TP PLACEMENT
Parts:
- added TPAUD21, TPYAUD11: TP, quantum_arcade_pcb:TP, symbol atari_grav_bw:TP
Connections:
- net AUD1: now also TPYAUD11.1, TPYAUD11.2
- net AUD2: now also TPAUD21.1, TPAUD21.2
Changed lines of the file:
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@@
   (junction (at 146.05 100.965) (diameter 0) (color 0 0 0 0)
   )
+  (junction (at 534.543 156.845) (diameter 0) (color 0 0 0 0)
+  )
   (junction (at 318.77 140.335) (diameter 0) (color 0 0 0 0)
   )
@@
   (junction (at 153.67 216.535) (diameter 0) (color 0 0 0 0)
   )
+  (junction (at 534.543 164.465) (diameter 0) (color 0 0 0 0)
+  )
   (junction (at 532.13 180.34) (diameter 0) (color 0 0 0 0)
   )
@@
   (junction (at 142.875 203.2) (diameter 0) (color 0 0 0 0)
   )
+  (junction (at 542.544 129.413) (diameter 0) (color 0 0 0 0)
+  )
   (junction (at 132.715 130.81) (diameter 0) (color 0 0 0 0)
   )
   (junction (at 377.19 295.91) (diameter 0) (color 0 0 0 0)
   )
+  (junction (at 541.655 192.532) (diameter 0) (color 0 0 0 0)
+  )
   (junction (at 160.655 212.09) (diameter 0) (color 0 0 0 0)
   )
@@
     (stroke (width 0) (type default) (color 0 0 0 0))
   )
+  (wire (pts (xy 534.543 164.465) (xy 534.543 192.532))
+    (stroke (width 0) (type default) (color 0 0 0 0))
+  )
   (wire (pts (xy 318.77 61.595) (xy 318.77 78.105))
     (stroke (width 0) (type default) (color 0 0 0 0))
@@
     (stroke (width 0) (type default) (color 0 0 0 0))
   )
-  (wire (pts (xy 532.13 164.465) (xy 538.48 164.465))
+  (wire (pts (xy 532.13 164.465) (xy 534.543 164.465))
     (stroke (width 0) (type default) (color 0 0 0 0))
   )
@@
     (stroke (width 0) (type default) (color 0 0 0 0))
   )
+  (wire (pts (xy 534.543 156.845) (xy 534.543 129.413))
+    (stroke (width 0) (type default) (color 0 0 0 0))
+  )
   (wire (pts (xy 146.685 237.49) (xy 146.685 234.95))
     (stroke (width 0) (type default) (color 0 0 0 0))
@@
     (stroke (width 0) (type default) (color 0 0 0 0))
   )
+  (wire (pts (xy 534.543 164.465) (xy 538.48 164.465))
+    (stroke (width 0) (type default) (color 0 0 0 0))
+  )
   (wire (pts (xy 69.85 344.17) (xy 73.66 344.17))
     (stroke (width 0) (type default) (color 0 0 0 0))
   )
+  (wire (pts (xy 534.543 129.413) (xy 542.544 129.413))
+    (stroke (width 0) (type default) (color 0 0 0 0))
+  )
   (wire (pts (xy 118.745 300.355) (xy 125.73 300.355))
     (stroke (width 0) (type default) (color 0 0 0 0))
@@
     (stroke (width 0) (type default) (color 0 0 0 0))
   )
+  (wire (pts (xy 534.543 192.532) (xy 541.655 192.532))
+    (stroke (width 0) (type default) (color 0 0 0 0))
+  )
   (wire (pts (xy 314.325 47.625) (xy 314.325 53.975))
     (stroke (width 0) (type default) (color 0 0 0 0))
@@
     (stroke (width 0) (type default) (color 0 0 0 0))
   )
+  (wire (pts (xy 534.543 156.845) (xy 488.315 156.845))
+    (stroke (width 0) (type default) (color 0 0 0 0))
+  )
   (wire (pts (xy 324.485 285.75) (xy 339.09 285.75))
     (stroke (width 0) (type default) (color 0 0 0 0))
@@
     (stroke (width 0) (type default) (color 0 0 0 0))
   )
-  (wire (pts (xy 538.48 156.845) (xy 488.315 156.845))
+  (wire (pts (xy 538.48 156.845) (xy 534.543 156.845))
     (stroke (width 0) (type default) (color 0 0 0 0))
   )
@@
     (stroke (width 0) (type default) (color 0 0 0 0))
   )
+  (wire (pts (xy 541.655 192.532) (xy 545.465 192.532))
+    (stroke (width 0) (type default) (color 0 0 0 0))
+  )
   (wire (pts (xy 80.01 75.565) (xy 86.36 75.565))
     (stroke (width 0) (type default) (color 0 0 0 0))
@@
     (stroke (width 0) (type default) (color 0 0 0 0))
   )
+  (wire (pts (xy 542.544 129.413) (xy 546.354 129.413))
+    (stroke (width 0) (type default) (color 0 0 0 0))
+  )
   (wire (pts (xy 146.685 220.98) (xy 177.165 220.98))
     (stroke (width 0) (type default) (color 0 0 0 0))
@@
     )
     (pin "1")
+    (pin "2")
+  )
+  (symbol (lib_id "atari_grav_bw:TP") (at 544.449 124.333 0) (unit 1)
+    (in_bom yes) (on_board yes)
+    (property "Reference" "TPYAUD11" (id 0) (at 539.496 131.191 0)
+      (effects (font (size 1.524 1.524)) (justify left))
+    )
+    (property "Value" "TP" (id 1) (at 542.544 123.063 0)
+      (effects (font (size 1.524 1.524)) hide)
+    )
+    (property "Footprint" "quantum_arcade_pcb:TP" (id 2) (at 542.544 125.603 0)
+      (effects (font (size 1.524 1.524)) hide)
+    )
+    (property "Datasheet" "" (id 3) (at 542.544 125.603 0)
+      (effects (font (size 1.524 1.524)) hide)
+    )
+    (pin "1")
+    (pin "2")
+  )
+  (symbol (lib_id "atari_grav_bw:TP") (at 543.56 187.452 0) (unit 1)
+    (in_bom yes) (on_board yes)
+    (property "Reference" "TPAUD21" (id 0) (at 538.607 194.31 0)
+      (effects (font (size 1.524 1.524)) (justify left))
+    )
+    (property "Value" "TP" (id 1) (at 541.655 186.182 0)
+      (effects (font (size 1.524 1.524)) hide)
+    )
+    (property "Footprint" "quantum_arcade_pcb:TP" (id 2) (at 541.655 188.722 0)
+      (effects (font (size 1.524 1.524)) hide)
+    )
+    (property "Datasheet" "" (id 3) (at 541.655 188.722 0)
+      (effects (font (size 1.524 1.524)) hide)
+    )
+    (pin "1")

Commit message: C16-30
Parts:
- C27, C28, C29, C30, C33, C34, C35, C44: footprint (none) -> Star_Wars_Vector_PCB:GenericComp
- C31, C32: footprint (none) -> Star_Wars_Vector_PCB:SmallCap
- C39: footprint (none) -> Star_Wars_Vector_PCB:CapElec2
Changed lines of the file:
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@@
       (effects (font (size 1.27 1.27)) (justify left))
     )
-    (property "Footprint" "" (id 2) (at 348.2848 186.69 0)
+    (property "Footprint" "Star_Wars_Vector_PCB:GenericComp" (id 2) (at 348.2848 186.69 0)
       (effects (font (size 1.27 1.27)) hide)
     )
@@
       (effects (font (size 1.27 1.27)) (justify left))
     )
-    (property "Footprint" "" (id 2) (at 338.7598 186.69 0)
+    (property "Footprint" "Star_Wars_Vector_PCB:CapElec2" (id 2) (at 338.7598 186.69 0)
       (effects (font (size 1.27 1.27)) hide)
     )
@@
       (effects (font (size 1.27 1.27)) (justify left))
     )
-    (property "Footprint" "" (id 2) (at 429.26 173.6598 0)
+    (property "Footprint" "Star_Wars_Vector_PCB:GenericComp" (id 2) (at 429.26 173.6598 0)
       (effects (font (size 1.27 1.27)) hide)
     )
@@
       (effects (font (size 1.27 1.27)) (justify left))
     )
-    (property "Footprint" "" (id 2) (at 445.135 111.4298 0)
+    (property "Footprint" "Star_Wars_Vector_PCB:GenericComp" (id 2) (at 445.135 111.4298 0)
       (effects (font (size 1.27 1.27)) hide)
     )
@@
       (effects (font (size 1.27 1.27)) (justify left))
     )
-    (property "Footprint" "" (id 2) (at 428.2948 104.14 0)
+    (property "Footprint" "Star_Wars_Vector_PCB:GenericComp" (id 2) (at 428.2948 104.14 0)
       (effects (font (size 1.27 1.27)) hide)
     )
@@
       (effects (font (size 1.27 1.27)) (justify left))
     )
-    (property "Footprint" "" (id 2) (at 417.83 151.4348 0)
+    (property "Footprint" "Star_Wars_Vector_PCB:GenericComp" (id 2) (at 417.83 151.4348 0)
       (effects (font (size 1.27 1.27)) hide)
     )
@@
       (effects (font (size 1.27 1.27)) (justify left))
     )
-    (property "Footprint" "" (id 2) (at 385.7498 109.855 0)
+    (property "Footprint" "Star_Wars_Vector_PCB:SmallCap" (id 2) (at 385.7498 109.855 0)
       (effects (font (size 1.27 1.27)) hide)
     )
@@
       (effects (font (size 1.27 1.27)) (justify left))
     )
-    (property "Footprint" "" (id 2) (at 385.7498 172.085 0)
+    (property "Footprint" "Star_Wars_Vector_PCB:SmallCap" (id 2) (at 385.7498 172.085 0)
       (effects (font (size 1.27 1.27)) hide)
     )
@@
       (effects (font (size 1.27 1.27)) (justify left))
     )
-    (property "Footprint" "" (id 2) (at 495.935 100.6348 0)
+    (property "Footprint" "Star_Wars_Vector_PCB:GenericComp" (id 2) (at 495.935 100.6348 0)
       (effects (font (size 1.27 1.27)) hide)
     )
@@
       (effects (font (size 1.27 1.27)) (justify left))
     )
-    (property "Footprint" "" (id 2) (at 468.63 100.6348 0)
+    (property "Footprint" "Star_Wars_Vector_PCB:GenericComp" (id 2) (at 468.63 100.6348 0)
       (effects (font (size 1.27 1.27)) hide)
     )
@@
       (effects (font (size 1.27 1.27)) (justify left))
     )
-    (property "Footprint" "" (id 2) (at 523.5448 171.45 0)
-      (effects (font (size 1.27 1.27)) hide)
-    )
+    (property "Footprint" "Star_Wars_Vector_PCB:GenericComp" (id 2) (at 523.5448 171.45 0)
+      (effects (font (size 1.27 1.27)) hide)
+    )
