File: kicad/atari_gravitar_black_widow/Sheet4A.kicad_sch (KiCad schematic)
At the start: 23 parts

Commit message: first traces.
Parts:
- C_2: footprint (none) -> Star_Wars_Vector_PCB:DDIP40
Changed lines of the file:
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@@
       (effects (font (size 1.524 1.524)) (justify left))
     )
-    (property "Footprint" "" (id 2) (at 113.03 161.29 0)
+    (property "Footprint" "Star_Wars_Vector_PCB:DDIP40" (id 2) (at 113.03 161.29 0)
       (effects (font (size 1.524 1.524)) hide)
     )

Commit message: place ttl
Parts:
- B_1: footprint (none) -> Star_Wars_Vector_PCB:DIP20
Changed lines of the file:
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@@
       (effects (font (size 1.27 1.27)) (justify left))
     )
-    (property "Footprint" "" (id 2) (at 210.058 114.3 0)
+    (property "Footprint" "Star_Wars_Vector_PCB:DIP20" (id 2) (at 210.058 114.3 0)
       (effects (font (size 1.27 1.27)) hide)
     )

Commit message: more ttl placements
Parts:
- C_1, F_2: footprint (none) -> Star_Wars_Vector_PCB:DIP20
- F_3: footprint (none) -> Star_Wars_Vector_PCB:DIP14
Changed lines of the file:
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@@
     (property "Reference" "F_3" (id 0) (at 257.81 88.519 0))
     (property "Value" "S04" (id 1) (at 250.825 91.694 0))
-    (property "Footprint" "" (id 2) (at 251.46 91.694 0)
+    (property "Footprint" "Star_Wars_Vector_PCB:DIP14" (id 2) (at 251.46 91.694 0)
       (effects (font (size 1.27 1.27)) hide)
     )
@@
       (effects (font (size 1.27 1.27)) (justify left))
     )
-    (property "Footprint" "" (id 2) (at 210.185 228.6 0)
+    (property "Footprint" "Star_Wars_Vector_PCB:DIP20" (id 2) (at 210.185 228.6 0)
       (effects (font (size 1.27 1.27)) hide)
     )
@@
     (property "Reference" "F_3" (id 0) (at 278.13 106.045 0))
     (property "Value" "S04" (id 1) (at 278.13 107.95 0))
-    (property "Footprint" "" (id 2) (at 279.146 106.68 0)
+    (property "Footprint" "Star_Wars_Vector_PCB:DIP14" (id 2) (at 279.146 106.68 0)
       (effects (font (size 1.27 1.27)) hide)
     )
@@
       (effects (font (size 1.27 1.27)) (justify left))
     )
-    (property "Footprint" "" (id 2) (at 210.058 173.99 0)
+    (property "Footprint" "Star_Wars_Vector_PCB:DIP20" (id 2) (at 210.058 173.99 0)
       (effects (font (size 5.08 5.08)) hide)
     )

Commit message: more chip layouts
Parts:
- J_3, J_4, K_4, L_3: footprint (none) -> Star_Wars_Vector_PCB:DIP14
Changed lines of the file:
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@@
     (property "Reference" "K_4" (id 0) (at 283.337 42.037 0))
     (property "Value" "S10" (id 1) (at 283.337 45.085 0))
-    (property "Footprint" "" (id 2) (at 283.21 44.704 0)
+    (property "Footprint" "Star_Wars_Vector_PCB:DIP14" (id 2) (at 283.21 44.704 0)
       (effects (font (size 1.27 1.27)) hide)
     )
@@
     (property "Reference" "L_3" (id 0) (at 91.567 251.46 0))
     (property "Value" "LS00" (id 1) (at 91.567 253.873 0))
-    (property "Footprint" "" (id 2) (at 91.694 254 0)
+    (property "Footprint" "Star_Wars_Vector_PCB:DIP14" (id 2) (at 91.694 254 0)
       (effects (font (size 1.27 1.27)) hide)
     )
@@
     (property "Reference" "J_3" (id 0) (at 294.767 56.261 0))
     (property "Value" "LS04" (id 1) (at 289.179 59.944 0))
-    (property "Footprint" "" (id 2) (at 290.068 59.944 0)
+    (property "Footprint" "Star_Wars_Vector_PCB:DIP14" (id 2) (at 290.068 59.944 0)
       (effects (font (size 1.27 1.27)) hide)
     )
@@
       (effects (font (size 1.524 1.524)))
     )
-    (property "Footprint" "" (id 2) (at 72.898 220.599 0)
-      (effects (font (size 1.524 1.524)) hide)
-    )
+    (property "Footprint" "Star_Wars_Vector_PCB:DIP14" (id 2) (at 72.898 220.599 0)
+      (effects (font (size 1.524 1.524)) hide)
+    )

Commit message: placements
Parts:
- P_3, R_1, R_2: footprint (none) -> Star_Wars_Vector_PCB:DIP16
- R_4: footprint (none) -> Star_Wars_Vector_PCB:DIP14
Changed lines of the file:
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@@
       (effects (font (size 1.27 1.27)) (justify left))
     )
-    (property "Footprint" "" (id 2) (at 454.914 161.29 0)
+    (property "Footprint" "Star_Wars_Vector_PCB:DIP16" (id 2) (at 454.914 161.29 0)
       (effects (font (size 1.27 1.27)) hide)
     )
@@
       (effects (font (size 1.27 1.27)) (justify left))
     )
-    (property "Footprint" "" (id 2) (at 455.93 242.57 0)
+    (property "Footprint" "Star_Wars_Vector_PCB:DIP16" (id 2) (at 455.93 242.57 0)
       (effects (font (size 1.27 1.27)) hide)
     )
@@
       (effects (font (size 1.27 1.27)) (justify left))
     )
-    (property "Footprint" "" (id 2) (at 455.676 91.948 0)
+    (property "Footprint" "Star_Wars_Vector_PCB:DIP16" (id 2) (at 455.676 91.948 0)
       (effects (font (size 1.27 1.27)) hide)
     )
@@
     (property "Reference" "R_4" (id 0) (at 178.435 279.4 0))
     (property "Value" "LS32" (id 1) (at 178.435 281.94 0))
-    (property "Footprint" "" (id 2) (at 178.435 280.67 0)
-      (effects (font (size 1.27 1.27)) hide)
-    )
+    (property "Footprint" "Star_Wars_Vector_PCB:DIP14" (id 2) (at 178.435 280.67 0)
+      (effects (font (size 1.27 1.27)) hide)
+    )

Commit message: TEST POINTS PLACED
Parts:
- TPPHI2, TPR/~{W}1, TP~{ROM0}1, TP~{ROM1}1, TP~{ROM2}1, TP~{ROM3}1, TP~{ROM4}1, TP~{ROM5}1, TP~{VMEM}1: footprint (none) -> quantum_arcade_pcb:TP
Changed lines of the file:
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@@
       (effects (font (size 1.524 1.524)) hide)
     )
-    (property "Footprint" "" (id 2) (at 342.9 67.945 0)
+    (property "Footprint" "quantum_arcade_pcb:TP" (id 2) (at 342.9 67.945 0)
       (effects (font (size 1.524 1.524)) hide)
     )
@@
       (effects (font (size 1.524 1.524)) hide)
     )
-    (property "Footprint" "" (id 2) (at 561.34 293.37 0)
+    (property "Footprint" "quantum_arcade_pcb:TP" (id 2) (at 561.34 293.37 0)
       (effects (font (size 1.524 1.524)) hide)
     )
@@
       (effects (font (size 1.524 1.524)) hide)
     )
-    (property "Footprint" "" (id 2) (at 544.83 272.415 0)
+    (property "Footprint" "quantum_arcade_pcb:TP" (id 2) (at 544.83 272.415 0)
       (effects (font (size 1.524 1.524)) hide)
     )
@@
       (effects (font (size 1.524 1.524)) hide)
     )
-    (property "Footprint" "" (id 2) (at 544.83 258.445 0)
+    (property "Footprint" "quantum_arcade_pcb:TP" (id 2) (at 544.83 258.445 0)
       (effects (font (size 1.524 1.524)) hide)
     )
@@
       (effects (font (size 1.524 1.524)) hide)
     )
-    (property "Footprint" "" (id 2) (at 328.295 64.135 0)
+    (property "Footprint" "quantum_arcade_pcb:TP" (id 2) (at 328.295 64.135 0)
       (effects (font (size 1.524 1.524)) hide)
     )
@@
       (effects (font (size 1.524 1.524)) hide)
     )
-    (property "Footprint" "" (id 2) (at 561.34 265.43 0)
+    (property "Footprint" "quantum_arcade_pcb:TP" (id 2) (at 561.34 265.43 0)
       (effects (font (size 1.524 1.524)) hide)
     )
@@
       (effects (font (size 1.524 1.524)) hide)
     )
-    (property "Footprint" "" (id 2) (at 544.83 300.355 0)
+    (property "Footprint" "quantum_arcade_pcb:TP" (id 2) (at 544.83 300.355 0)
       (effects (font (size 1.524 1.524)) hide)
     )
@@
       (effects (font (size 1.524 1.524)) hide)
     )
-    (property "Footprint" "" (id 2) (at 561.34 279.4 0)
+    (property "Footprint" "quantum_arcade_pcb:TP" (id 2) (at 561.34 279.4 0)
       (effects (font (size 1.524 1.524)) hide)
     )
@@
       (effects (font (size 1.524 1.524)) hide)
     )
-    (property "Footprint" "" (id 2) (at 544.83 286.385 0)
-      (effects (font (size 1.524 1.524)) hide)
-    )
+    (property "Footprint" "quantum_arcade_pcb:TP" (id 2) (at 544.83 286.385 0)
+      (effects (font (size 1.524 1.524)) hide)
+    )

Commit message: resistor placements R1-R153
Parts:
- R19: footprint (none) -> Star_Wars_Vector_PCB:GenericComp
Changed lines of the file:
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@@
     (property "Reference" "R19" (id 0) (at 96.012 181.102 90))
     (property "Value" "1k" (id 1) (at 96.012 179.07 90))
-    (property "Footprint" "" (id 2) (at 96.012 177.292 90)
+    (property "Footprint" "Star_Wars_Vector_PCB:GenericComp" (id 2) (at 96.012 177.292 90)
       (effects (font (size 1.27 1.27)) hide)
     )

Commit message: ALL PARTS PLACED!!
Parts:
- J_4: footprint Star_Wars_Vector_PCB:DIP14 -> Star_Wars_Vector_PCB:DIP16
Changed lines of the file:
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@@
       (effects (font (size 1.524 1.524)))
     )
-    (property "Footprint" "Star_Wars_Vector_PCB:DIP14" (id 2) (at 72.898 220.599 0)
+    (property "Footprint" "Star_Wars_Vector_PCB:DIP16" (id 2) (at 72.898 220.599 0)
       (effects (font (size 1.524 1.524)) hide)
     )
