File: kicad/atari_gravitar_black_widow/Sheet8A.kicad_sch (KiCad schematic)
At the start: 87 parts, among them Q11 2N3906, Q12 2N3904

Commit message: LAST OF TP PLACEMENT
Parts:
- added TPXOUT1: TP, quantum_arcade_pcb:TP, symbol atari_grav_bw:TP
Connections:
- net XOUT: now also TPXOUT1.1, TPXOUT1.2
Changed lines of the file:
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@@
   (junction (at 122.555 261.62) (diameter 0) (color 0 0 0 0)
   )
+  (junction (at 566.928 98.425) (diameter 0) (color 0 0 0 0)
+  )
   (junction (at 438.785 83.185) (diameter 0) (color 0 0 0 0)
   )
@@
     (stroke (width 0) (type default) (color 0 0 0 0))
   )
+  (wire (pts (xy 566.928 98.425) (xy 570.738 98.425))
+    (stroke (width 0) (type default) (color 0 0 0 0))
+  )
   (wire (pts (xy 487.045 102.235) (xy 487.045 84.455))
     (stroke (width 0) (type default) (color 0 0 0 0))
@@
     (stroke (width 0) (type default) (color 0 0 0 0))
   )
-  (wire (pts (xy 563.2196 96.8756) (xy 566.0136 96.8756))
-    (stroke (width 0) (type default) (color 0 0 0 0))
-  )
   (wire (pts (xy 317.5 99.695) (xy 317.5 100.965))
     (stroke (width 0) (type default) (color 0 0 0 0))
@@
     (stroke (width 0) (type default) (color 0 0 0 0))
   )
-  (wire (pts (xy 566.0136 96.8756) (xy 566.0136 96.9264))
-    (stroke (width 0) (type default) (color 0 0 0 0))
-  )
   (wire (pts (xy 456.565 133.985) (xy 456.565 137.16))
     (stroke (width 0) (type default) (color 0 0 0 0))
@@
     (stroke (width 0) (type default) (color 0 0 0 0))
   )
+  (wire (pts (xy 566.039 84.455) (xy 566.039 98.425))
+    (stroke (width 0) (type default) (color 0 0 0 0))
+  )
   (wire (pts (xy 277.495 97.79) (xy 289.56 97.79))
     (stroke (width 0) (type default) (color 0 0 0 0))
@@
     (stroke (width 0) (type default) (color 0 0 0 0))
   )
+  (wire (pts (xy 566.039 98.425) (xy 566.928 98.425))
+    (stroke (width 0) (type default) (color 0 0 0 0))
+  )
   (wire (pts (xy 461.645 67.945) (xy 461.645 73.025))
     (stroke (width 0) (type default) (color 0 0 0 0))
@@
     (pin "1")
   )
+  (symbol (lib_id "atari_grav_bw:TP") (at 568.833 93.345 0) (unit 1)
+    (in_bom yes) (on_board yes)
+    (property "Reference" "TPXOUT1" (id 0) (at 563.88 100.203 0)
+      (effects (font (size 1.524 1.524)) (justify left))
+    )
+    (property "Value" "TP" (id 1) (at 566.928 92.075 0)
+      (effects (font (size 1.524 1.524)) hide)
+    )
+    (property "Footprint" "quantum_arcade_pcb:TP" (id 2) (at 566.928 94.615 0)
+      (effects (font (size 1.524 1.524)) hide)
+    )
+    (property "Datasheet" "" (id 3) (at 566.928 94.615 0)
+      (effects (font (size 1.524 1.524)) hide)
+    )
+    (pin "1")
+    (pin "2")
+  )
   (symbol (lib_id "power:GND") (at 173.355 201.295 0) (unit 1)

Commit message: PLACED C1-C15
Parts:
- A/B_9: footprint quantum_arcade_pcb:TP -> Star_Wars_Vector_PCB:DIP20
Changed lines of the file:
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@@
     (property "Reference" "A/B_9" (id 0) (at 262.255 96.52 0))
     (property "Value" "AM6012" (id 1) (at 262.255 103.505 0))
-    (property "Footprint" "quantum_arcade_pcb:TP" (id 2) (at 262.255 95.25 0)
+    (property "Footprint" "Star_Wars_Vector_PCB:DIP20" (id 2) (at 262.255 95.25 0)
       (effects (font (size 1.27 1.27)) hide)
     )

Commit message: more cap placements
Parts:
- C122, C123, C124, C125, C70, C71, C73, C76, C77, C78, C86, C87, C88, C89: footprint (none) -> Star_Wars_Vector_PCB:GenericComp
Changed lines of the file:
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@@
       (effects (font (size 1.27 1.27)) (justify left))
     )
-    (property "Footprint" "" (id 2) (at 142.875 246.0752 0)
+    (property "Footprint" "Star_Wars_Vector_PCB:GenericComp" (id 2) (at 142.875 246.0752 0)
       (effects (font (size 1.27 1.27)) hide)
     )
@@
       (effects (font (size 1.27 1.27)) (justify left))
     )
-    (property "Footprint" "" (id 2) (at 544.195 77.4192 0)
+    (property "Footprint" "Star_Wars_Vector_PCB:GenericComp" (id 2) (at 544.195 77.4192 0)
       (effects (font (size 1.27 1.27)) hide)
     )
@@
       (effects (font (size 1.27 1.27)) (justify left))
     )
-    (property "Footprint" "" (id 2) (at 254.635 77.8002 0)
+    (property "Footprint" "Star_Wars_Vector_PCB:GenericComp" (id 2) (at 254.635 77.8002 0)
       (effects (font (size 1.27 1.27)) hide)
     )
@@
       (effects (font (size 1.27 1.27)) (justify left))
     )
-    (property "Footprint" "" (id 2) (at 294.9448 93.345 0)
+    (property "Footprint" "Star_Wars_Vector_PCB:GenericComp" (id 2) (at 294.9448 93.345 0)
       (effects (font (size 1.27 1.27)) hide)
     )
@@
       (effects (font (size 1.27 1.27)) (justify left))
     )
-    (property "Footprint" "" (id 2) (at 112.395 220.6752 0)
+    (property "Footprint" "Star_Wars_Vector_PCB:GenericComp" (id 2) (at 112.395 220.6752 0)
       (effects (font (size 1.27 1.27)) hide)
     )
@@
       (effects (font (size 1.27 1.27)) (justify left))
     )
-    (property "Footprint" "" (id 2) (at 528.6502 157.48 0)
+    (property "Footprint" "Star_Wars_Vector_PCB:GenericComp" (id 2) (at 528.6502 157.48 0)
       (effects (font (size 1.27 1.27)) hide)
     )
@@
       (effects (font (size 1.27 1.27)) (justify left))
     )
-    (property "Footprint" "" (id 2) (at 544.195 93.4212 0)
+    (property "Footprint" "Star_Wars_Vector_PCB:GenericComp" (id 2) (at 544.195 93.4212 0)
       (effects (font (size 1.27 1.27)) hide)
     )
@@
       (effects (font (size 1.27 1.27)) (justify left))
     )
-    (property "Footprint" "" (id 2) (at 520.3952 157.48 0)
+    (property "Footprint" "Star_Wars_Vector_PCB:GenericComp" (id 2) (at 520.3952 157.48 0)
       (effects (font (size 1.27 1.27)) hide)
     )
@@
       (effects (font (size 1.27 1.27)) (justify left))
     )
-    (property "Footprint" "" (id 2) (at 288.5948 106.68 0)
+    (property "Footprint" "Star_Wars_Vector_PCB:GenericComp" (id 2) (at 288.5948 106.68 0)
       (effects (font (size 1.27 1.27)) hide)
     )
@@
       (effects (font (size 1.27 1.27)) (justify left))
     )
-    (property "Footprint" "" (id 2) (at 365.76 94.3102 0)
+    (property "Footprint" "Star_Wars_Vector_PCB:GenericComp" (id 2) (at 365.76 94.3102 0)
       (effects (font (size 1.27 1.27)) hide)
     )
@@
       (effects (font (size 1.27 1.27)) (justify left))
     )
-    (property "Footprint" "" (id 2) (at 493.0648 144.78 0)
+    (property "Footprint" "Star_Wars_Vector_PCB:GenericComp" (id 2) (at 493.0648 144.78 0)
       (effects (font (size 1.27 1.27)) hide)
     )
@@
       (effects (font (size 1.27 1.27)) (justify left))
     )
-    (property "Footprint" "" (id 2) (at 468.63 157.1752 0)
+    (property "Footprint" "Star_Wars_Vector_PCB:GenericComp" (id 2) (at 468.63 157.1752 0)
       (effects (font (size 1.27 1.27)) hide)
     )
@@
       (effects (font (size 1.27 1.27)) (justify left))
     )
-    (property "Footprint" "" (id 2) (at 112.395 262.5852 0)
+    (property "Footprint" "Star_Wars_Vector_PCB:GenericComp" (id 2) (at 112.395 262.5852 0)
       (effects (font (size 1.27 1.27)) hide)
     )
@@
       (effects (font (size 1.27 1.27)) (justify left))
     )
-    (property "Footprint" "" (id 2) (at 365.76 111.4552 0)
-      (effects (font (size 1.27 1.27)) hide)
-    )
+    (property "Footprint" "Star_Wars_Vector_PCB:GenericComp" (id 2) (at 365.76 111.4552 0)
+      (effects (font (size 1.27 1.27)) hide)
+    )

Commit message: more cap placements
Parts:
- C112, C113, C127, C85: footprint (none) -> Star_Wars_Vector_PCB:CapBrown
- C77: footprint Star_Wars_Vector_PCB:GenericComp -> quantum_arcade_pcb:CapSmall
- C80: footprint (none) -> Star_Wars_Vector_PCB:CapYellow
Changed lines of the file:
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@@
       (effects (font (size 1.27 1.27)) (justify left))
     )
-    (property "Footprint" "" (id 2) (at 151.765 185.1152 0)
+    (property "Footprint" "Star_Wars_Vector_PCB:CapBrown" (id 2) (at 151.765 185.1152 0)
       (effects (font (size 1.27 1.27)) hide)
     )
@@
       (effects (font (size 1.27 1.27)) (justify left))
     )
-    (property "Footprint" "Star_Wars_Vector_PCB:GenericComp" (id 2) (at 288.5948 106.68 0)
+    (property "Footprint" "quantum_arcade_pcb:CapSmall" (id 2) (at 288.5948 106.68 0)
       (effects (font (size 1.27 1.27)) hide)
     )
@@
       (effects (font (size 1.27 1.27)) (justify left))
     )
-    (property "Footprint" "" (id 2) (at 328.93 77.1652 0)
+    (property "Footprint" "Star_Wars_Vector_PCB:CapYellow" (id 2) (at 328.93 77.1652 0)
       (effects (font (size 1.27 1.27)) hide)
     )
@@
       (effects (font (size 1.27 1.27)) (justify left))
     )
-    (property "Footprint" "" (id 2) (at 493.395 110.1852 0)
+    (property "Footprint" "Star_Wars_Vector_PCB:CapBrown" (id 2) (at 493.395 110.1852 0)
       (effects (font (size 1.27 1.27)) hide)
     )
@@
       (effects (font (size 1.27 1.27)) (justify left))
     )
-    (property "Footprint" "" (id 2) (at 120.65 192.1002 0)
+    (property "Footprint" "Star_Wars_Vector_PCB:CapBrown" (id 2) (at 120.65 192.1002 0)
       (effects (font (size 1.27 1.27)) hide)
     )
@@
       (effects (font (size 1.27 1.27)) (justify left))
     )
-    (property "Footprint" "" (id 2) (at 190.8048 231.775 0)
-      (effects (font (size 1.27 1.27)) hide)
-    )
+    (property "Footprint" "Star_Wars_Vector_PCB:CapBrown" (id 2) (at 190.8048 231.775 0)
+      (effects (font (size 1.27 1.27)) hide)
+    )

Commit message: resistor placements R1-R153
Parts:
- C128, R100, R101, R159, R160, R161, R74, R75, R76, R77, R78, R79, R80, R81, R87, R88, R89, R90, R91, R94, R95: footprint (none) -> Star_Wars_Vector_PCB:GenericComp
- R98, R99: footprint (none) -> Star_Wars_Vector_PCB:PotBlk
Changed lines of the file:
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@@
       (effects (font (size 1.27 1.27)) (justify right))
     )
-    (property "Footprint" "" (id 2) (at 222.25 193.04 0)
+    (property "Footprint" "Star_Wars_Vector_PCB:PotBlk" (id 2) (at 222.25 193.04 0)
       (effects (font (size 1.27 1.27)) hide)
     )
@@
     (property "Reference" "R95" (id 0) (at 281.305 109.982 90))
     (property "Value" "820" (id 1) (at 281.305 107.95 90))
-    (property "Footprint" "" (id 2) (at 281.305 106.172 90)
+    (property "Footprint" "Star_Wars_Vector_PCB:GenericComp" (id 2) (at 281.305 106.172 90)
       (effects (font (size 1.27 1.27)) hide)
     )
@@
     (property "Reference" "R161" (id 0) (at 124.46 198.247 90))
     (property "Value" "15K" (id 1) (at 124.46 196.215 90))
-    (property "Footprint" "" (id 2) (at 124.46 194.437 90)
+    (property "Footprint" "Star_Wars_Vector_PCB:GenericComp" (id 2) (at 124.46 194.437 90)
       (effects (font (size 1.27 1.27)) hide)
     )
@@
     (property "Reference" "R77" (id 0) (at 85.598 257.175 90))
     (property "Value" "100K" (id 1) (at 87.63 257.175 90))
-    (property "Footprint" "" (id 2) (at 89.408 257.175 90)
+    (property "Footprint" "Star_Wars_Vector_PCB:GenericComp" (id 2) (at 89.408 257.175 90)
       (effects (font (size 1.27 1.27)) hide)
     )
@@
     (property "Reference" "R90" (id 0) (at 222.25 204.47 90))
     (property "Value" "100" (id 1) (at 222.25 206.375 90))
-    (property "Footprint" "" (id 2) (at 222.25 204.597 90)
+    (property "Footprint" "Star_Wars_Vector_PCB:GenericComp" (id 2) (at 222.25 204.597 90)
       (effects (font (size 1.27 1.27)) hide)
     )
@@
     (property "Reference" "R100" (id 0) (at 348.615 99.187 90))
     (property "Value" "7.5K" (id 1) (at 348.615 97.155 90))
-    (property "Footprint" "" (id 2) (at 348.615 95.377 90)
+    (property "Footprint" "Star_Wars_Vector_PCB:GenericComp" (id 2) (at 348.615 95.377 90)
       (effects (font (size 1.27 1.27)) hide)
     )
@@
       (effects (font (size 1.27 1.27)) (justify right))
     )
-    (property "Footprint" "" (id 2) (at 222.25 214.63 0)
+    (property "Footprint" "Star_Wars_Vector_PCB:PotBlk" (id 2) (at 222.25 214.63 0)
       (effects (font (size 1.27 1.27)) hide)
     )
@@
     (property "Reference" "R76" (id 0) (at 81.153 257.175 90))
     (property "Value" "100K" (id 1) (at 83.185 257.175 90))
-    (property "Footprint" "" (id 2) (at 84.963 257.175 90)
+    (property "Footprint" "Star_Wars_Vector_PCB:GenericComp" (id 2) (at 84.963 257.175 90)
       (effects (font (size 1.27 1.27)) hide)
     )
@@
     (property "Reference" "R79" (id 0) (at 85.598 226.695 90))
     (property "Value" "100K" (id 1) (at 87.63 226.695 90))
-    (property "Footprint" "" (id 2) (at 89.408 226.695 90)
+    (property "Footprint" "Star_Wars_Vector_PCB:GenericComp" (id 2) (at 89.408 226.695 90)
       (effects (font (size 1.27 1.27)) hide)
     )
@@
     (property "Reference" "R159" (id 0) (at 155.575 191.262 90))
     (property "Value" "10K" (id 1) (at 155.575 189.23 90))
-    (property "Footprint" "" (id 2) (at 155.575 187.452 90)
+    (property "Footprint" "Star_Wars_Vector_PCB:GenericComp" (id 2) (at 155.575 187.452 90)
       (effects (font (size 1.27 1.27)) hide)
     )
@@
     (property "Reference" "R88" (id 0) (at 166.37 245.872 90))
     (property "Value" "7.5K" (id 1) (at 166.37 243.84 90))
-    (property "Footprint" "" (id 2) (at 166.37 242.062 90)
+    (property "Footprint" "Star_Wars_Vector_PCB:GenericComp" (id 2) (at 166.37 242.062 90)
       (effects (font (size 1.27 1.27)) hide)
     )
@@
     (property "Reference" "R80" (id 0) (at 81.153 226.695 90))
     (property "Value" "100K" (id 1) (at 83.185 226.695 90))
-    (property "Footprint" "" (id 2) (at 84.963 226.695 90)
+    (property "Footprint" "Star_Wars_Vector_PCB:GenericComp" (id 2) (at 84.963 226.695 90)
       (effects (font (size 1.27 1.27)) hide)
     )
@@
     (property "Reference" "R91" (id 0) (at 222.25 226.06 90))
     (property "Value" "100" (id 1) (at 222.25 227.965 90))
-    (property "Footprint" "" (id 2) (at 222.25 226.187 90)
+    (property "Footprint" "Star_Wars_Vector_PCB:GenericComp" (id 2) (at 222.25 226.187 90)
       (effects (font (size 1.27 1.27)) hide)
     )
@@
     (property "Reference" "R81" (id 0) (at 76.708 226.695 90))
     (property "Value" "100K" (id 1) (at 78.74 226.695 90))
-    (property "Footprint" "" (id 2) (at 80.518 226.695 90)
+    (property "Footprint" "Star_Wars_Vector_PCB:GenericComp" (id 2) (at 80.518 226.695 90)
       (effects (font (size 1.27 1.27)) hide)
     )
@@
     (property "Reference" "R89" (id 0) (at 147.955 253.492 90))
     (property "Value" "3.9K" (id 1) (at 147.955 251.46 90))
-    (property "Footprint" "" (id 2) (at 147.955 249.682 90)
+    (property "Footprint" "Star_Wars_Vector_PCB:GenericComp" (id 2) (at 147.955 249.682 90)
       (effects (font (size 1.27 1.27)) hide)
     )
@@
       (effects (font (size 1.27 1.27)) (justify left))
     )
-    (property "Footprint" "" (id 2) (at 493.395 119.0752 0)
+    (property "Footprint" "Star_Wars_Vector_PCB:GenericComp" (id 2) (at 493.395 119.0752 0)
       (effects (font (size 1.27 1.27)) hide)
     )
@@
     (property "Reference" "R94" (id 0) (at 291.592 101.6 90))
     (property "Value" "820" (id 1) (at 289.56 101.6 90))
-    (property "Footprint" "" (id 2) (at 287.782 101.6 90)
+    (property "Footprint" "Star_Wars_Vector_PCB:GenericComp" (id 2) (at 287.782 101.6 90)
       (effects (font (size 1.27 1.27)) hide)
     )
@@
     (property "Reference" "R75" (id 0) (at 76.708 257.175 90))
     (property "Value" "100K" (id 1) (at 78.74 257.175 90))
-    (property "Footprint" "" (id 2) (at 80.518 257.175 90)
+    (property "Footprint" "Star_Wars_Vector_PCB:GenericComp" (id 2) (at 80.518 257.175 90)
       (effects (font (size 1.27 1.27)) hide)
     )
@@
     (property "Reference" "R101" (id 0) (at 367.411 82.423 90))
     (property "Value" "7.5K" (id 1) (at 367.411 80.391 90))
-    (property "Footprint" "" (id 2) (at 367.411 78.613 90)
+    (property "Footprint" "Star_Wars_Vector_PCB:GenericComp" (id 2) (at 367.411 78.613 90)
       (effects (font (size 1.27 1.27)) hide)
     )
@@
     (property "Reference" "R74" (id 0) (at 72.263 257.175 90))
     (property "Value" "100K" (id 1) (at 74.295 257.175 90))
-    (property "Footprint" "" (id 2) (at 76.073 257.175 90)
+    (property "Footprint" "Star_Wars_Vector_PCB:GenericComp" (id 2) (at 76.073 257.175 90)
       (effects (font (size 1.27 1.27)) hide)
     )
@@
     (property "Reference" "R87" (id 0) (at 166.37 240.792 90))
     (property "Value" "7.5K" (id 1) (at 166.37 238.76 90))
-    (property "Footprint" "" (id 2) (at 166.37 236.982 90)
+    (property "Footprint" "Star_Wars_Vector_PCB:GenericComp" (id 2) (at 166.37 236.982 90)
       (effects (font (size 1.27 1.27)) hide)
     )
@@
     (property "Reference" "R78" (id 0) (at 72.263 226.695 90))
     (property "Value" "100K" (id 1) (at 74.295 226.695 90))
-    (property "Footprint" "" (id 2) (at 76.073 226.695 90)
+    (property "Footprint" "Star_Wars_Vector_PCB:GenericComp" (id 2) (at 76.073 226.695 90)
       (effects (font (size 1.27 1.27)) hide)
     )
@@
     (property "Reference" "R160" (id 0) (at 138.303 180.975 90))
     (property "Value" "1K" (id 1) (at 140.335 180.975 90))
-    (property "Footprint" "" (id 2) (at 142.113 180.975 90)
-      (effects (font (size 1.27 1.27)) hide)
-    )
+    (property "Footprint" "Star_Wars_Vector_PCB:GenericComp" (id 2) (at 142.113 180.975 90)
+      (effects (font (size 1.27 1.27)) hide)
+    )
