File: kicad/atari_gravitar_black_widow/Sheet8A.kicad_sch (KiCad schematic)
At the start: 88 parts, among them Q11 2N3906, Q12 2N3904

Commit message: more resistor placements
Parts:
- R162, R163, R164, R165, R166, R167, R168, R169, R170, R171, R172, R173, R174, R175, R176, R177, R178, R179, R180, R181, R182, R183, R184, R185, R186: footprint (none) -> Star_Wars_Vector_PCB:GenericComp
Changed lines of the file:
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@@
     (property "Reference" "R181" (id 0) (at 434.975 91.44 90))
     (property "Value" "2.7k" (id 1) (at 433.07 91.44 90))
-    (property "Footprint" "" (id 2) (at 434.848 91.44 90)
+    (property "Footprint" "Star_Wars_Vector_PCB:GenericComp" (id 2) (at 434.848 91.44 90)
       (effects (font (size 1.27 1.27)) hide)
     )
@@
     (property "Reference" "R176" (id 0) (at 445.77 91.44 90))
     (property "Value" "470" (id 1) (at 443.865 91.44 90))
-    (property "Footprint" "" (id 2) (at 445.643 91.44 90)
+    (property "Footprint" "Star_Wars_Vector_PCB:GenericComp" (id 2) (at 445.643 91.44 90)
       (effects (font (size 1.27 1.27)) hide)
     )
@@
     (property "Reference" "R164" (id 0) (at 171.323 197.485 90))
     (property "Value" "560" (id 1) (at 173.355 197.485 90))
-    (property "Footprint" "" (id 2) (at 175.133 197.485 90)
+    (property "Footprint" "Star_Wars_Vector_PCB:GenericComp" (id 2) (at 175.133 197.485 90)
       (effects (font (size 1.27 1.27)) hide)
     )
@@
     (property "Reference" "R166" (id 0) (at 209.55 204.47 90))
     (property "Value" "7.5K" (id 1) (at 209.55 206.375 90))
-    (property "Footprint" "" (id 2) (at 209.55 204.597 90)
+    (property "Footprint" "Star_Wars_Vector_PCB:GenericComp" (id 2) (at 209.55 204.597 90)
       (effects (font (size 1.27 1.27)) hide)
     )
@@
     (property "Reference" "R180" (id 0) (at 440.69 91.44 90))
     (property "Value" "680" (id 1) (at 438.785 91.44 90))
-    (property "Footprint" "" (id 2) (at 440.563 91.44 90)
+    (property "Footprint" "Star_Wars_Vector_PCB:GenericComp" (id 2) (at 440.563 91.44 90)
       (effects (font (size 1.27 1.27)) hide)
     )
@@
     (property "Reference" "R185" (id 0) (at 465.455 132.08 90))
     (property "Value" "2.2k" (id 1) (at 465.455 133.985 90))
-    (property "Footprint" "" (id 2) (at 465.455 132.207 90)
+    (property "Footprint" "Star_Wars_Vector_PCB:GenericComp" (id 2) (at 465.455 132.207 90)
       (effects (font (size 1.27 1.27)) hide)
     )
@@
     (property "Reference" "R182" (id 0) (at 481.457 147.32 90))
     (property "Value" "1k" (id 1) (at 479.425 147.32 90))
-    (property "Footprint" "" (id 2) (at 477.647 147.32 90)
+    (property "Footprint" "Star_Wars_Vector_PCB:GenericComp" (id 2) (at 477.647 147.32 90)
       (effects (font (size 1.27 1.27)) hide)
     )
@@
     (property "Reference" "R169" (id 0) (at 438.15 76.2 90))
     (property "Value" "470" (id 1) (at 438.15 78.105 90))
-    (property "Footprint" "" (id 2) (at 438.15 76.327 90)
+    (property "Footprint" "Star_Wars_Vector_PCB:GenericComp" (id 2) (at 438.15 76.327 90)
       (effects (font (size 1.27 1.27)) hide)
     )
@@
     (property "Reference" "R175" (id 0) (at 452.755 66.04 90))
     (property "Value" "2.2k" (id 1) (at 452.755 67.945 90))
-    (property "Footprint" "" (id 2) (at 452.755 66.167 90)
+    (property "Footprint" "Star_Wars_Vector_PCB:GenericComp" (id 2) (at 452.755 66.167 90)
       (effects (font (size 1.27 1.27)) hide)
     )
@@
     (property "Reference" "R174" (id 0) (at 480.06 73.025 90))
     (property "Value" "2.2k" (id 1) (at 478.155 73.025 90))
-    (property "Footprint" "" (id 2) (at 479.933 73.025 90)
+    (property "Footprint" "Star_Wars_Vector_PCB:GenericComp" (id 2) (at 479.933 73.025 90)
       (effects (font (size 1.27 1.27)) hide)
     )
@@
     (property "Reference" "R179" (id 0) (at 468.63 94.615 90))
     (property "Value" "10k" (id 1) (at 466.725 94.615 90))
-    (property "Footprint" "" (id 2) (at 468.503 94.615 90)
+    (property "Footprint" "Star_Wars_Vector_PCB:GenericComp" (id 2) (at 468.503 94.615 90)
       (effects (font (size 1.27 1.27)) hide)
     )
@@
     (property "Reference" "R183" (id 0) (at 453.39 94.615 90))
     (property "Value" "3.9k" (id 1) (at 451.485 94.615 90))
-    (property "Footprint" "" (id 2) (at 453.263 94.615 90)
+    (property "Footprint" "Star_Wars_Vector_PCB:GenericComp" (id 2) (at 453.263 94.615 90)
       (effects (font (size 1.27 1.27)) hide)
     )
@@
     (property "Reference" "R171" (id 0) (at 452.755 132.08 90))
     (property "Value" "2.2K" (id 1) (at 452.755 133.985 90))
-    (property "Footprint" "" (id 2) (at 452.755 132.207 90)
+    (property "Footprint" "Star_Wars_Vector_PCB:GenericComp" (id 2) (at 452.755 132.207 90)
       (effects (font (size 1.27 1.27)) hide)
     )
@@
     (property "Reference" "R170" (id 0) (at 425.831 106.934 90))
     (property "Value" "470" (id 1) (at 422.91 107.315 90))
-    (property "Footprint" "" (id 2) (at 424.688 107.315 90)
+    (property "Footprint" "Star_Wars_Vector_PCB:GenericComp" (id 2) (at 424.688 107.315 90)
       (effects (font (size 1.27 1.27)) hide)
     )
@@
     (property "Reference" "R186" (id 0) (at 443.23 156.21 90))
     (property "Value" "3.9k" (id 1) (at 443.23 158.115 90))
-    (property "Footprint" "" (id 2) (at 443.23 159.893 90)
+    (property "Footprint" "Star_Wars_Vector_PCB:GenericComp" (id 2) (at 443.23 159.893 90)
       (effects (font (size 1.27 1.27)) hide)
     )
@@
     (property "Reference" "R165" (id 0) (at 209.55 190.5 90))
     (property "Value" "7.5k" (id 1) (at 209.55 193.04 90))
-    (property "Footprint" "" (id 2) (at 209.55 191.262 90)
+    (property "Footprint" "Star_Wars_Vector_PCB:GenericComp" (id 2) (at 209.55 191.262 90)
       (effects (font (size 1.27 1.27)) hide)
     )
@@
     (property "Reference" "R184" (id 0) (at 430.53 147.955 90))
     (property "Value" "470" (id 1) (at 430.53 149.86 90))
-    (property "Footprint" "" (id 2) (at 430.53 151.638 90)
+    (property "Footprint" "Star_Wars_Vector_PCB:GenericComp" (id 2) (at 430.53 151.638 90)
       (effects (font (size 1.27 1.27)) hide)
     )
@@
     (property "Reference" "R167" (id 0) (at 209.55 226.06 90))
     (property "Value" "7.5K" (id 1) (at 209.55 227.965 90))
-    (property "Footprint" "" (id 2) (at 209.55 226.187 90)
+    (property "Footprint" "Star_Wars_Vector_PCB:GenericComp" (id 2) (at 209.55 226.187 90)
       (effects (font (size 1.27 1.27)) hide)
     )
@@
     (property "Reference" "R163" (id 0) (at 187.96 198.12 90))
     (property "Value" "7K" (id 1) (at 187.96 195.58 90))
-    (property "Footprint" "" (id 2) (at 187.96 193.802 90)
+    (property "Footprint" "Star_Wars_Vector_PCB:GenericComp" (id 2) (at 187.96 193.802 90)
       (effects (font (size 1.27 1.27)) hide)
     )
@@
     (property "Reference" "R173" (id 0) (at 484.505 73.025 90))
     (property "Value" "2.2k" (id 1) (at 482.6 73.025 90))
-    (property "Footprint" "" (id 2) (at 484.378 73.025 90)
+    (property "Footprint" "Star_Wars_Vector_PCB:GenericComp" (id 2) (at 484.378 73.025 90)
       (effects (font (size 1.27 1.27)) hide)
     )
@@
     (property "Reference" "R177" (id 0) (at 497.205 100.33 90))
     (property "Value" "15k" (id 1) (at 497.205 102.235 90))
-    (property "Footprint" "" (id 2) (at 497.205 100.457 90)
+    (property "Footprint" "Star_Wars_Vector_PCB:GenericComp" (id 2) (at 497.205 100.457 90)
       (effects (font (size 1.27 1.27)) hide)
     )
@@
     (property "Reference" "R178" (id 0) (at 465.455 66.04 90))
     (property "Value" "3.9k" (id 1) (at 465.455 67.945 90))
-    (property "Footprint" "" (id 2) (at 465.455 66.167 90)
+    (property "Footprint" "Star_Wars_Vector_PCB:GenericComp" (id 2) (at 465.455 66.167 90)
       (effects (font (size 1.27 1.27)) hide)
     )
@@
     (property "Reference" "R168" (id 0) (at 209.55 212.09 90))
     (property "Value" "7.5k" (id 1) (at 209.55 214.63 90))
-    (property "Footprint" "" (id 2) (at 209.55 212.852 90)
+    (property "Footprint" "Star_Wars_Vector_PCB:GenericComp" (id 2) (at 209.55 212.852 90)
       (effects (font (size 1.27 1.27)) hide)
     )
@@
     (property "Reference" "R162" (id 0) (at 187.96 187.96 90))
     (property "Value" "7K" (id 1) (at 187.96 190.5 90))
-    (property "Footprint" "" (id 2) (at 187.96 188.722 90)
+    (property "Footprint" "Star_Wars_Vector_PCB:GenericComp" (id 2) (at 187.96 188.722 90)
       (effects (font (size 1.27 1.27)) hide)
     )
@@
     (property "Reference" "R172" (id 0) (at 452.755 126.365 90))
     (property "Value" "100k" (id 1) (at 452.755 128.27 90))
-    (property "Footprint" "" (id 2) (at 452.755 126.492 90)
-      (effects (font (size 1.27 1.27)) hide)
-    )
+    (property "Footprint" "Star_Wars_Vector_PCB:GenericComp" (id 2) (at 452.755 126.492 90)
+      (effects (font (size 1.27 1.27)) hide)
+    )

Commit message: all resistors placed.
Parts:
- R187, R189, R192: footprint (none) -> Star_Wars_Vector_PCB:PotBlue
- R188, R217, R218, R219, RV2: footprint (none) -> Star_Wars_Vector_PCB:GenericComp
Changed lines of the file:
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@@
       (effects (font (size 1.27 1.27)) (justify right))
     )
-    (property "Footprint" "" (id 2) (at 475.615 104.775 0)
+    (property "Footprint" "Star_Wars_Vector_PCB:PotBlue" (id 2) (at 475.615 104.775 0)
       (effects (font (size 1.27 1.27)) hide)
     )
@@
     (property "Reference" "R219" (id 0) (at 537.21 103.886 90))
     (property "Value" "6.8k" (id 1) (at 539.115 104.013 90))
-    (property "Footprint" "" (id 2) (at 537.337 103.886 90)
+    (property "Footprint" "Star_Wars_Vector_PCB:GenericComp" (id 2) (at 537.337 103.886 90)
       (effects (font (size 1.27 1.27)) hide)
     )
@@
     (property "Reference" "R188" (id 0) (at 477.52 95.25 90))
     (property "Value" "5.6k" (id 1) (at 475.615 95.25 90))
-    (property "Footprint" "" (id 2) (at 477.393 95.25 90)
+    (property "Footprint" "Star_Wars_Vector_PCB:GenericComp" (id 2) (at 477.393 95.25 90)
       (effects (font (size 1.27 1.27)) hide)
     )
@@
     (property "Reference" "RV2" (id 0) (at 535.305 87.63 90))
     (property "Value" "VDR" (id 1) (at 528.955 87.63 90))
-    (property "Footprint" "" (id 2) (at 530.352 87.63 90)
+    (property "Footprint" "Star_Wars_Vector_PCB:GenericComp" (id 2) (at 530.352 87.63 90)
       (effects (font (size 1.27 1.27)) hide)
     )
@@
       (effects (font (size 1.27 1.27)) (justify right))
     )
-    (property "Footprint" "" (id 2) (at 523.875 81.915 0)
+    (property "Footprint" "Star_Wars_Vector_PCB:PotBlue" (id 2) (at 523.875 81.915 0)
       (effects (font (size 1.27 1.27)) hide)
     )
@@
       (effects (font (size 1.27 1.27)) (justify right))
     )
-    (property "Footprint" "" (id 2) (at 451.485 104.775 0)
+    (property "Footprint" "Star_Wars_Vector_PCB:PotBlue" (id 2) (at 451.485 104.775 0)
       (effects (font (size 1.27 1.27)) hide)
     )
@@
     (property "Reference" "R217" (id 0) (at 562.229 86.36 90))
     (property "Value" "100" (id 1) (at 562.229 84.455 90))
-    (property "Footprint" "" (id 2) (at 562.229 86.233 90)
+    (property "Footprint" "Star_Wars_Vector_PCB:GenericComp" (id 2) (at 562.229 86.233 90)
       (effects (font (size 1.27 1.27)) hide)
     )
@@
     (property "Reference" "R218" (id 0) (at 547.497 97.282 90))
     (property "Value" "68" (id 1) (at 547.37 99.314 90))
-    (property "Footprint" "" (id 2) (at 547.37 101.092 90)
-      (effects (font (size 1.27 1.27)) hide)
-    )
+    (property "Footprint" "Star_Wars_Vector_PCB:GenericComp" (id 2) (at 547.37 101.092 90)
+      (effects (font (size 1.27 1.27)) hide)
+    )

Commit message: ALL PARTS PLACED!!
Parts:
- CR4: footprint (none) -> quantum_arcade_pcb:Diode
- Q11, Q12: footprint (none) -> quantum_arcade_pcb:GenTrans
Changed lines of the file:
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@@
       (effects (font (size 1.27 1.27)) (justify left))
     )
-    (property "Footprint" "" (id 2) (at 175.895 184.785 0)
+    (property "Footprint" "quantum_arcade_pcb:GenTrans" (id 2) (at 175.895 184.785 0)
       (effects (font (size 1.27 1.27) italic) (justify left) hide)
     )
@@
     (property "Reference" "CR4" (id 0) (at 188.595 214.63 0))
     (property "Value" "1N914" (id 1) (at 188.595 209.55 0))
-    (property "Footprint" "" (id 2) (at 188.595 212.09 0)
+    (property "Footprint" "quantum_arcade_pcb:Diode" (id 2) (at 188.595 212.09 0)
       (effects (font (size 1.27 1.27)) hide)
     )
@@
       (effects (font (size 1.27 1.27)) (justify left))
     )
-    (property "Footprint" "" (id 2) (at 133.985 190.5 0)
-      (effects (font (size 1.27 1.27)) hide)
-    )
+    (property "Footprint" "quantum_arcade_pcb:GenTrans" (id 2) (at 133.985 190.5 0)
+      (effects (font (size 1.27 1.27)) hide)
+    )
