File: kicad/atari_gravitar_black_widow/untitled.kicad_sch (KiCad schematic)
At the start: 53 parts

Commit message: more caps
Parts:
- C65: footprint (none) -> Star_Wars_Vector_PCB:CapBrown
- C66: footprint (none) -> Star_Wars_Vector_PCB:CapYellow
Changed lines of the file:
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@@
       (effects (font (size 1.27 1.27)) (justify left))
     )
-    (property "Footprint" "" (id 2) (at 291.5158 194.691 0)
+    (property "Footprint" "Star_Wars_Vector_PCB:CapBrown" (id 2) (at 291.5158 194.691 0)
       (effects (font (size 1.27 1.27)) hide)
     )
@@
       (effects (font (size 1.27 1.27)) (justify left))
     )
-    (property "Footprint" "" (id 2) (at 297.8658 181.356 0)
-      (effects (font (size 1.27 1.27)) hide)
-    )
+    (property "Footprint" "Star_Wars_Vector_PCB:CapYellow" (id 2) (at 297.8658 181.356 0)
+      (effects (font (size 1.27 1.27)) hide)
+    )

Commit message: more cap placements
Parts:
- C72: footprint (none) -> quantum_arcade_pcb:CapSmall
- C81, C82, C83, C84: footprint (none) -> Star_Wars_Vector_PCB:GenericComp
Changed lines of the file:
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@@
       (effects (font (size 1.27 1.27)) (justify left))
     )
-    (property "Footprint" "" (id 2) (at 331.851 165.1762 0)
+    (property "Footprint" "quantum_arcade_pcb:CapSmall" (id 2) (at 331.851 165.1762 0)
       (effects (font (size 1.27 1.27)) hide)
     )
@@
       (effects (font (size 1.27 1.27)) (justify left))
     )
-    (property "Footprint" "" (id 2) (at 551.3832 223.266 0)
+    (property "Footprint" "Star_Wars_Vector_PCB:GenericComp" (id 2) (at 551.3832 223.266 0)
       (effects (font (size 1.27 1.27)) hide)
     )
@@
       (effects (font (size 1.27 1.27)) (justify left))
     )
-    (property "Footprint" "" (id 2) (at 368.681 199.4662 0)
+    (property "Footprint" "Star_Wars_Vector_PCB:GenericComp" (id 2) (at 368.681 199.4662 0)
       (effects (font (size 1.27 1.27)) hide)
     )
@@
       (effects (font (size 1.27 1.27)) (justify left))
     )
-    (property "Footprint" "" (id 2) (at 543.1282 223.266 0)
+    (property "Footprint" "Star_Wars_Vector_PCB:GenericComp" (id 2) (at 543.1282 223.266 0)
       (effects (font (size 1.27 1.27)) hide)
     )
@@
       (effects (font (size 1.27 1.27)) (justify left))
     )
-    (property "Footprint" "" (id 2) (at 368.681 182.3212 0)
-      (effects (font (size 1.27 1.27)) hide)
-    )
+    (property "Footprint" "Star_Wars_Vector_PCB:GenericComp" (id 2) (at 368.681 182.3212 0)
+      (effects (font (size 1.27 1.27)) hide)
+    )

Commit message: more cap placements
Parts:
- C132, C134: footprint (none) -> Star_Wars_Vector_PCB:CapBrown
- C72: footprint quantum_arcade_pcb:CapSmall -> Star_Wars_Vector_PCB:CapYellow
Changed lines of the file:
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@@
       (effects (font (size 1.27 1.27)) (justify left))
     )
-    (property "Footprint" "quantum_arcade_pcb:CapSmall" (id 2) (at 331.851 165.1762 0)
+    (property "Footprint" "Star_Wars_Vector_PCB:CapYellow" (id 2) (at 331.851 165.1762 0)
       (effects (font (size 1.27 1.27)) hide)
     )
@@
       (effects (font (size 1.27 1.27)) (justify left))
     )
-    (property "Footprint" "" (id 2) (at 496.316 198.1962 0)
+    (property "Footprint" "Star_Wars_Vector_PCB:CapBrown" (id 2) (at 496.316 198.1962 0)
       (effects (font (size 1.27 1.27)) hide)
     )
@@
       (effects (font (size 1.27 1.27)) (justify left))
     )
-    (property "Footprint" "" (id 2) (at 495.9858 232.791 0)
-      (effects (font (size 1.27 1.27)) hide)
-    )
+    (property "Footprint" "Star_Wars_Vector_PCB:CapBrown" (id 2) (at 495.9858 232.791 0)
+      (effects (font (size 1.27 1.27)) hide)
+    )

Commit message: caps placement up to c126
Parts:
- C134: footprint Star_Wars_Vector_PCB:CapBrown -> Star_Wars_Vector_PCB:GenericComp
- C135: footprint (none) -> Star_Wars_Vector_PCB:GenericComp
Changed lines of the file:
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@@
       (effects (font (size 1.27 1.27)) (justify left))
     )
-    (property "Footprint" "" (id 2) (at 471.551 245.1862 0)
+    (property "Footprint" "Star_Wars_Vector_PCB:GenericComp" (id 2) (at 471.551 245.1862 0)
       (effects (font (size 1.27 1.27)) hide)
     )
@@
       (effects (font (size 1.27 1.27)) (justify left))
     )
-    (property "Footprint" "Star_Wars_Vector_PCB:CapBrown" (id 2) (at 495.9858 232.791 0)
-      (effects (font (size 1.27 1.27)) hide)
-    )
+    (property "Footprint" "Star_Wars_Vector_PCB:GenericComp" (id 2) (at 495.9858 232.791 0)
+      (effects (font (size 1.27 1.27)) hide)
+    )

Commit message: resistor placements R1-R153
Parts:
- C130, C131, R83, R84, R96, R97: footprint (none) -> Star_Wars_Vector_PCB:GenericComp
- C136: footprint (none) -> Star_Wars_Vector_PCB:CapBrown
Changed lines of the file:
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@@
       (effects (font (size 1.27 1.27)) (justify left))
     )
-    (property "Footprint" "" (id 2) (at 547.116 181.1782 0)
+    (property "Footprint" "Star_Wars_Vector_PCB:GenericComp" (id 2) (at 547.116 181.1782 0)
       (effects (font (size 1.27 1.27)) hide)
     )
@@
       (effects (font (size 1.27 1.27)) (justify left))
     )
-    (property "Footprint" "" (id 2) (at 547.116 165.3032 0)
+    (property "Footprint" "Star_Wars_Vector_PCB:GenericComp" (id 2) (at 547.116 165.3032 0)
       (effects (font (size 1.27 1.27)) hide)
     )
@@
       (effects (font (size 1.27 1.27)) (justify left))
     )
-    (property "Footprint" "" (id 2) (at 306.7558 194.691 0)
+    (property "Footprint" "Star_Wars_Vector_PCB:CapBrown" (id 2) (at 306.7558 194.691 0)
       (effects (font (size 1.27 1.27)) hide)
     )
@@
     (property "Reference" "R84" (id 0) (at 284.226 197.993 90))
     (property "Value" "820" (id 1) (at 284.226 195.961 90))
-    (property "Footprint" "" (id 2) (at 284.226 194.183 90)
+    (property "Footprint" "Star_Wars_Vector_PCB:GenericComp" (id 2) (at 284.226 194.183 90)
       (effects (font (size 1.27 1.27)) hide)
     )
@@
     (property "Reference" "R97" (id 0) (at 369.824 173.228 90))
     (property "Value" "7.5K" (id 1) (at 369.824 171.196 90))
-    (property "Footprint" "" (id 2) (at 369.824 169.418 90)
+    (property "Footprint" "Star_Wars_Vector_PCB:GenericComp" (id 2) (at 369.824 169.418 90)
       (effects (font (size 1.27 1.27)) hide)
     )
@@
     (property "Reference" "R83" (id 0) (at 294.513 189.611 90))
     (property "Value" "680" (id 1) (at 292.481 189.611 90))
-    (property "Footprint" "" (id 2) (at 290.703 189.611 90)
+    (property "Footprint" "Star_Wars_Vector_PCB:GenericComp" (id 2) (at 290.703 189.611 90)
       (effects (font (size 1.27 1.27)) hide)
     )
@@
     (property "Reference" "R96" (id 0) (at 351.536 187.198 90))
     (property "Value" "7.5K" (id 1) (at 351.536 185.166 90))
-    (property "Footprint" "" (id 2) (at 351.536 183.388 90)
-      (effects (font (size 1.27 1.27)) hide)
-    )
+    (property "Footprint" "Star_Wars_Vector_PCB:GenericComp" (id 2) (at 351.536 183.388 90)
+      (effects (font (size 1.27 1.27)) hide)
+    )

Commit message: all resistors placed.
Parts:
- R190, R191, R193, R194, R196, R197, R198, R199, R200, R201, R202, R203, R204, R205, R206, R207, R208, R209, R211, R214, R215, R216, RV1: footprint (none) -> Star_Wars_Vector_PCB:GenericComp
- R210, R212, R213: footprint (none) -> Star_Wars_Vector_PCB:PotBlue
Changed lines of the file:
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@@
     (property "Reference" "R201" (id 0) (at 471.551 182.626 90))
     (property "Value" "10k" (id 1) (at 469.646 182.626 90))
-    (property "Footprint" "" (id 2) (at 471.424 182.626 90)
+    (property "Footprint" "Star_Wars_Vector_PCB:GenericComp" (id 2) (at 471.424 182.626 90)
       (effects (font (size 1.27 1.27)) hide)
     )
@@
       (effects (font (size 1.27 1.27)) (justify right))
     )
-    (property "Footprint" "" (id 2) (at 454.406 192.786 0)
+    (property "Footprint" "Star_Wars_Vector_PCB:PotBlue" (id 2) (at 454.406 192.786 0)
       (effects (font (size 1.27 1.27)) hide)
     )
@@
     (property "Reference" "R196" (id 0) (at 487.426 161.036 90))
     (property "Value" "2.2k" (id 1) (at 485.521 161.036 90))
-    (property "Footprint" "" (id 2) (at 487.299 161.036 90)
+    (property "Footprint" "Star_Wars_Vector_PCB:GenericComp" (id 2) (at 487.299 161.036 90)
       (effects (font (size 1.27 1.27)) hide)
     )
@@
     (property "Reference" "R209" (id 0) (at 433.451 235.966 90))
     (property "Value" "470" (id 1) (at 433.451 237.871 90))
-    (property "Footprint" "" (id 2) (at 433.451 239.649 90)
+    (property "Footprint" "Star_Wars_Vector_PCB:GenericComp" (id 2) (at 433.451 239.649 90)
       (effects (font (size 1.27 1.27)) hide)
     )
@@
     (property "Reference" "R206" (id 0) (at 456.311 182.626 90))
     (property "Value" "3.9k" (id 1) (at 454.406 182.626 90))
-    (property "Footprint" "" (id 2) (at 456.184 182.626 90)
+    (property "Footprint" "Star_Wars_Vector_PCB:GenericComp" (id 2) (at 456.184 182.626 90)
       (effects (font (size 1.27 1.27)) hide)
     )
@@
     (property "Reference" "R194" (id 0) (at 441.071 164.211 90))
     (property "Value" "470" (id 1) (at 441.071 166.116 90))
-    (property "Footprint" "" (id 2) (at 441.071 164.338 90)
+    (property "Footprint" "Star_Wars_Vector_PCB:GenericComp" (id 2) (at 441.071 164.338 90)
       (effects (font (size 1.27 1.27)) hide)
     )
@@
     (property "Reference" "RV1" (id 0) (at 538.226 175.641 90))
     (property "Value" "VDR" (id 1) (at 531.876 175.641 90))
-    (property "Footprint" "" (id 2) (at 533.273 175.641 90)
+    (property "Footprint" "Star_Wars_Vector_PCB:GenericComp" (id 2) (at 533.273 175.641 90)
       (effects (font (size 1.27 1.27)) hide)
     )
@@
       (effects (font (size 1.27 1.27)) (justify right))
     )
-    (property "Footprint" "" (id 2) (at 478.536 192.786 0)
+    (property "Footprint" "Star_Wars_Vector_PCB:PotBlue" (id 2) (at 478.536 192.786 0)
       (effects (font (size 1.27 1.27)) hide)
     )
@@
       (effects (font (size 1.27 1.27)) (justify right))
     )
-    (property "Footprint" "" (id 2) (at 526.796 169.926 0)
+    (property "Footprint" "Star_Wars_Vector_PCB:PotBlue" (id 2) (at 526.796 169.926 0)
       (effects (font (size 1.27 1.27)) hide)
     )
@@
     (property "Reference" "R211" (id 0) (at 480.441 183.261 90))
     (property "Value" "5.6k" (id 1) (at 478.536 183.261 90))
-    (property "Footprint" "" (id 2) (at 480.314 183.261 90)
+    (property "Footprint" "Star_Wars_Vector_PCB:GenericComp" (id 2) (at 480.314 183.261 90)
       (effects (font (size 1.27 1.27)) hide)
     )
@@
     (property "Reference" "R193" (id 0) (at 427.101 189.484 90))
     (property "Value" "470" (id 1) (at 425.831 195.326 90))
-    (property "Footprint" "" (id 2) (at 427.609 195.326 90)
+    (property "Footprint" "Star_Wars_Vector_PCB:GenericComp" (id 2) (at 427.609 195.326 90)
       (effects (font (size 1.27 1.27)) hide)
     )
@@
     (property "Reference" "R197" (id 0) (at 482.981 161.036 90))
     (property "Value" "2.2k" (id 1) (at 481.076 161.036 90))
-    (property "Footprint" "" (id 2) (at 482.854 161.036 90)
+    (property "Footprint" "Star_Wars_Vector_PCB:GenericComp" (id 2) (at 482.854 161.036 90)
       (effects (font (size 1.27 1.27)) hide)
     )
@@
     (property "Reference" "R205" (id 0) (at 437.896 179.451 90))
     (property "Value" "2.7k" (id 1) (at 435.991 179.451 90))
-    (property "Footprint" "" (id 2) (at 437.769 179.451 90)
+    (property "Footprint" "Star_Wars_Vector_PCB:GenericComp" (id 2) (at 437.769 179.451 90)
       (effects (font (size 1.27 1.27)) hide)
     )
@@
     (property "Reference" "R191" (id 0) (at 455.676 214.376 90))
     (property "Value" "100k" (id 1) (at 455.676 216.281 90))
-    (property "Footprint" "" (id 2) (at 455.676 214.503 90)
+    (property "Footprint" "Star_Wars_Vector_PCB:GenericComp" (id 2) (at 455.676 214.503 90)
       (effects (font (size 1.27 1.27)) hide)
     )
@@
     (property "Reference" "R214" (id 0) (at 562.356 174.371 90))
     (property "Value" "100" (id 1) (at 562.356 172.466 90))
-    (property "Footprint" "" (id 2) (at 562.356 174.244 90)
+    (property "Footprint" "Star_Wars_Vector_PCB:GenericComp" (id 2) (at 562.356 174.244 90)
       (effects (font (size 1.27 1.27)) hide)
     )
@@
     (property "Reference" "R200" (id 0) (at 500.126 188.341 90))
     (property "Value" "12K" (id 1) (at 500.126 190.246 90))
-    (property "Footprint" "" (id 2) (at 500.126 188.468 90)
+    (property "Footprint" "Star_Wars_Vector_PCB:GenericComp" (id 2) (at 500.126 188.468 90)
       (effects (font (size 1.27 1.27)) hide)
     )
@@
     (property "Reference" "R207" (id 0) (at 468.376 220.091 90))
     (property "Value" "2.2k" (id 1) (at 468.376 221.996 90))
-    (property "Footprint" "" (id 2) (at 468.376 220.218 90)
+    (property "Footprint" "Star_Wars_Vector_PCB:GenericComp" (id 2) (at 468.376 220.218 90)
       (effects (font (size 1.27 1.27)) hide)
     )
@@
     (property "Reference" "R215" (id 0) (at 550.672 186.563 90))
     (property "Value" "68" (id 1) (at 550.672 184.658 90))
-    (property "Footprint" "" (id 2) (at 550.672 186.436 90)
+    (property "Footprint" "Star_Wars_Vector_PCB:GenericComp" (id 2) (at 550.672 186.436 90)
       (effects (font (size 1.27 1.27)) hide)
     )
@@
     (property "Reference" "R216" (id 0) (at 540.131 189.103 90))
     (property "Value" "6.8k" (id 1) (at 542.036 189.103 90))
-    (property "Footprint" "" (id 2) (at 540.258 189.103 90)
+    (property "Footprint" "Star_Wars_Vector_PCB:GenericComp" (id 2) (at 540.258 189.103 90)
       (effects (font (size 1.27 1.27)) hide)
     )
@@
     (property "Reference" "R198" (id 0) (at 455.676 154.051 90))
     (property "Value" "2.2k" (id 1) (at 455.676 155.956 90))
-    (property "Footprint" "" (id 2) (at 455.676 154.178 90)
+    (property "Footprint" "Star_Wars_Vector_PCB:GenericComp" (id 2) (at 455.676 154.178 90)
       (effects (font (size 1.27 1.27)) hide)
     )
@@
     (property "Reference" "R190" (id 0) (at 455.676 220.091 90))
     (property "Value" "2.2K" (id 1) (at 455.676 221.996 90))
-    (property "Footprint" "" (id 2) (at 455.676 220.218 90)
+    (property "Footprint" "Star_Wars_Vector_PCB:GenericComp" (id 2) (at 455.676 220.218 90)
       (effects (font (size 1.27 1.27)) hide)
     )
@@
     (property "Reference" "R199" (id 0) (at 448.691 179.451 90))
     (property "Value" "470" (id 1) (at 446.786 179.451 90))
-    (property "Footprint" "" (id 2) (at 448.564 179.451 90)
+    (property "Footprint" "Star_Wars_Vector_PCB:GenericComp" (id 2) (at 448.564 179.451 90)
       (effects (font (size 1.27 1.27)) hide)
     )
@@
     (property "Reference" "R208" (id 0) (at 446.151 244.221 90))
     (property "Value" "3.9k" (id 1) (at 446.151 246.126 90))
-    (property "Footprint" "" (id 2) (at 446.151 247.904 90)
+    (property "Footprint" "Star_Wars_Vector_PCB:GenericComp" (id 2) (at 446.151 247.904 90)
       (effects (font (size 1.27 1.27)) hide)
     )
@@
     (property "Reference" "R203" (id 0) (at 443.611 179.451 90))
     (property "Value" "680" (id 1) (at 441.706 179.451 90))
-    (property "Footprint" "" (id 2) (at 443.484 179.451 90)
+    (property "Footprint" "Star_Wars_Vector_PCB:GenericComp" (id 2) (at 443.484 179.451 90)
       (effects (font (size 1.27 1.27)) hide)
     )
@@
     (property "Reference" "R204" (id 0) (at 484.378 235.331 90))
     (property "Value" "1k" (id 1) (at 482.346 235.331 90))
-    (property "Footprint" "" (id 2) (at 480.568 235.331 90)
+    (property "Footprint" "Star_Wars_Vector_PCB:GenericComp" (id 2) (at 480.568 235.331 90)
       (effects (font (size 1.27 1.27)) hide)
     )
@@
     (property "Reference" "R202" (id 0) (at 468.376 154.051 90))
     (property "Value" "3.9k" (id 1) (at 468.376 155.956 90))
-    (property "Footprint" "" (id 2) (at 468.376 154.178 90)
-      (effects (font (size 1.27 1.27)) hide)
-    )
+    (property "Footprint" "Star_Wars_Vector_PCB:GenericComp" (id 2) (at 468.376 154.178 90)
+      (effects (font (size 1.27 1.27)) hide)
+    )

Commit message: ALL PARTS PLACED!!
Parts:
- C1000: footprint (none) -> Star_Wars_Vector_PCB:GenericComp
Changed lines of the file:
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@@
       (effects (font (size 1.27 1.27)) (justify left))
     )
-    (property "Footprint" "" (id 2) (at 496.316 207.0862 0)
+    (property "Footprint" "Star_Wars_Vector_PCB:GenericComp" (id 2) (at 496.316 207.0862 0)
       (effects (font (size 1.27 1.27)) hide)
     )

Commit message: ROW 7 TOPSIDE TRACES COMPLETED
Parts:
- C66: footprint Star_Wars_Vector_PCB:CapYellow -> Star_Wars_Vector_PCB:GenericComp
Changed lines of the file:
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@@
       (effects (font (size 1.27 1.27)) (justify left))
     )
-    (property "Footprint" "Star_Wars_Vector_PCB:CapYellow" (id 2) (at 297.8658 181.356 0)
+    (property "Footprint" "Star_Wars_Vector_PCB:GenericComp" (id 2) (at 297.8658 181.356 0)
       (effects (font (size 1.27 1.27)) hide)
     )
