File: kicad/atari_gravitar_black_widow/untitled.kicad_sch (KiCad schematic)
At the start: 53 parts

Commit message: Fixed ERC errors and added traces to the edge connectors
Parts:
- renumbered C82 to C81, C81 to C82
Changed lines of the file:
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@@
   (symbol (lib_id "Device:C") (at 550.418 219.456 0) (unit 1)
     (in_bom yes) (on_board yes)
-    (property "Reference" "C82" (id 0) (at 551.053 216.916 0)
+    (property "Reference" "C81" (id 0) (at 551.053 216.916 0)
       (effects (font (size 1.27 1.27)) (justify left))
     )
@@
   (symbol (lib_id "Device:C") (at 542.163 219.456 0) (unit 1)
     (in_bom yes) (on_board yes)
-    (property "Reference" "C81" (id 0) (at 542.798 216.916 0)
-      (effects (font (size 1.27 1.27)) (justify left))
-    )
+    (property "Reference" "C82" (id 0) (at 542.798 216.916 0)
+      (effects (font (size 1.27 1.27)) (justify left))
+    )

Commit message: many traces on back fixed not DVY12 on F9
Connections:
- net DVX10 renamed DVY10
- net DVX11 renamed DVY11
- net DVX3 renamed DVY3
- net DVX4 renamed DVY4
- net DVX5 renamed DVY5
- net DVX6 renamed DVY6
- net DVX7 renamed DVY7
- net DVX8 renamed DVY8
- net DVX9 renamed DVY9
- net ~{DVX12} renamed ~{DVY12}
Changed lines of the file:
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@@
     (effects (font (size 1.27 1.27) (thickness 0.508) bold) (justify left bottom))
   )
-  (global_label "DVX5" (shape input) (at 27.051 193.421 180) (fields_autoplaced)
+  (global_label "DVY5" (shape input) (at 27.051 193.421 180) (fields_autoplaced)
     (effects (font (size 1.27 1.27)) (justify right))
-    (property "Intersheet References" "${INTERSHEET_REFS}" (id 0) (at 19.9492 193.3416 0)
+    (property "Intersheet References" "${INTERSHEET_REFS}" (id 0) (at 20.0701 193.3416 0)
       (effects (font (size 1.27 1.27)) (justify right) hide)
     )
   )
-  (global_label "DVX10" (shape input) (at 27.051 180.721 180) (fields_autoplaced)
+  (global_label "DVY10" (shape input) (at 27.051 180.721 180) (fields_autoplaced)
     (effects (font (size 1.27 1.27)) (justify right))
-    (property "Intersheet References" "${INTERSHEET_REFS}" (id 0) (at 18.7397 180.6416 0)
+    (property "Intersheet References" "${INTERSHEET_REFS}" (id 0) (at 18.8606 180.6416 0)
       (effects (font (size 1.27 1.27)) (justify right) hide)
     )
@@
     )
   )
-  (global_label "DVX4" (shape input) (at 27.051 195.961 180) (fields_autoplaced)
+  (global_label "DVY4" (shape input) (at 27.051 195.961 180) (fields_autoplaced)
     (effects (font (size 1.27 1.27)) (justify right))
-    (property "Intersheet References" "${INTERSHEET_REFS}" (id 0) (at 19.9492 195.8816 0)
+    (property "Intersheet References" "${INTERSHEET_REFS}" (id 0) (at 20.0701 195.8816 0)
       (effects (font (size 1.27 1.27)) (justify right) hide)
     )
   )
-  (global_label "DVX9" (shape input) (at 27.051 183.261 180) (fields_autoplaced)
+  (global_label "DVY9" (shape input) (at 27.051 183.261 180) (fields_autoplaced)
     (effects (font (size 1.27 1.27)) (justify right))
-    (property "Intersheet References" "${INTERSHEET_REFS}" (id 0) (at 19.9492 183.1816 0)
+    (property "Intersheet References" "${INTERSHEET_REFS}" (id 0) (at 20.0701 183.1816 0)
       (effects (font (size 1.27 1.27)) (justify right) hide)
     )
   )
-  (global_label "DVX7" (shape input) (at 27.051 188.341 180) (fields_autoplaced)
+  (global_label "DVY7" (shape input) (at 27.051 188.341 180) (fields_autoplaced)
     (effects (font (size 1.27 1.27)) (justify right))
-    (property "Intersheet References" "${INTERSHEET_REFS}" (id 0) (at 19.9492 188.2616 0)
+    (property "Intersheet References" "${INTERSHEET_REFS}" (id 0) (at 20.0701 188.2616 0)
       (effects (font (size 1.27 1.27)) (justify right) hide)
     )
@@
     )
   )
-  (global_label "DVX8" (shape input) (at 27.051 185.801 180) (fields_autoplaced)
+  (global_label "DVY8" (shape input) (at 27.051 185.801 180) (fields_autoplaced)
     (effects (font (size 1.27 1.27)) (justify right))
-    (property "Intersheet References" "${INTERSHEET_REFS}" (id 0) (at 19.9492 185.7216 0)
+    (property "Intersheet References" "${INTERSHEET_REFS}" (id 0) (at 20.0701 185.7216 0)
       (effects (font (size 1.27 1.27)) (justify right) hide)
     )
   )
-  (global_label "DVX11" (shape input) (at 27.051 178.181 180) (fields_autoplaced)
+  (global_label "DVY11" (shape input) (at 27.051 178.181 180) (fields_autoplaced)
     (effects (font (size 1.27 1.27)) (justify right))
-    (property "Intersheet References" "${INTERSHEET_REFS}" (id 0) (at 18.7397 178.1016 0)
+    (property "Intersheet References" "${INTERSHEET_REFS}" (id 0) (at 18.8606 178.1016 0)
       (effects (font (size 1.27 1.27)) (justify right) hide)
     )
@@
     )
   )
-  (global_label "~{DVX12}" (shape input) (at 27.051 175.641 180) (fields_autoplaced)
+  (global_label "~{DVY12}" (shape input) (at 27.051 175.641 180) (fields_autoplaced)
     (effects (font (size 1.27 1.27)) (justify right))
-    (property "Intersheet References" "${INTERSHEET_REFS}" (id 0) (at 18.7397 175.5616 0)
+    (property "Intersheet References" "${INTERSHEET_REFS}" (id 0) (at 18.8606 175.5616 0)
       (effects (font (size 1.27 1.27)) (justify right) hide)
     )
@@
     )
   )
-  (global_label "DVX3" (shape input) (at 27.051 198.501 180) (fields_autoplaced)
+  (global_label "DVY3" (shape input) (at 27.051 198.501 180) (fields_autoplaced)
     (effects (font (size 1.27 1.27)) (justify right))
-    (property "Intersheet References" "${INTERSHEET_REFS}" (id 0) (at 19.9492 198.4216 0)
+    (property "Intersheet References" "${INTERSHEET_REFS}" (id 0) (at 20.0701 198.4216 0)
       (effects (font (size 1.27 1.27)) (justify right) hide)
     )
   )
-  (global_label "DVX6" (shape input) (at 27.051 190.881 180) (fields_autoplaced)
+  (global_label "DVY6" (shape input) (at 27.051 190.881 180) (fields_autoplaced)
     (effects (font (size 1.27 1.27)) (justify right))
-    (property "Intersheet References" "${INTERSHEET_REFS}" (id 0) (at 19.9492 190.8016 0)
+    (property "Intersheet References" "${INTERSHEET_REFS}" (id 0) (at 20.0701 190.8016 0)
       (effects (font (size 1.27 1.27)) (justify right) hide)
     )

Commit message: finished most all traces in analog
Parts:
- R210, R212, R213: footprint Star_Wars_Vector_PCB:PotBlue -> Star_Wars_Vector_PCB:PotBlk
Changed lines of the file:
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@@
       (effects (font (size 1.27 1.27)) (justify right))
     )
-    (property "Footprint" "Star_Wars_Vector_PCB:PotBlue" (id 2) (at 454.406 192.786 0)
+    (property "Footprint" "Star_Wars_Vector_PCB:PotBlk" (id 2) (at 454.406 192.786 0)
       (effects (font (size 1.27 1.27)) hide)
     )
@@
       (effects (font (size 1.27 1.27)) (justify right))
     )
-    (property "Footprint" "Star_Wars_Vector_PCB:PotBlue" (id 2) (at 478.536 192.786 0)
+    (property "Footprint" "Star_Wars_Vector_PCB:PotBlk" (id 2) (at 478.536 192.786 0)
       (effects (font (size 1.27 1.27)) hide)
     )
@@
       (effects (font (size 1.27 1.27)) (justify right))
     )
-    (property "Footprint" "Star_Wars_Vector_PCB:PotBlue" (id 2) (at 526.796 169.926 0)
-      (effects (font (size 1.27 1.27)) hide)
-    )
+    (property "Footprint" "Star_Wars_Vector_PCB:PotBlk" (id 2) (at 526.796 169.926 0)
+      (effects (font (size 1.27 1.27)) hide)
+    )

Commit message: Analog done but for rev 2 R/Cs
Connections:
- net GND: now also R212.3; no longer R212.1
- net YCOR: no longer R205.1
- net at R211.1: now also R212.1; no longer R212.3
- new net XCOR: R205.1
Changed lines of the file:
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@@
     )
   )
-  (global_label "YCOR" (shape input) (at 435.991 185.166 270) (fields_autoplaced)
-    (effects (font (size 1.27 1.27)) (justify right))
-    (property "Intersheet References" "${INTERSHEET_REFS}" (id 0) (at -65.024 -561.594 0)
-      (effects (font (size 1.27 1.27)) hide)
+  (global_label "XCOR" (shape input) (at 435.991 185.166 270) (fields_autoplaced)
+    (effects (font (size 1.27 1.27)) (justify right))
+    (property "Intersheet References" "${INTERSHEET_REFS}" (id 0) (at 435.9116 192.5702 90)
+      (effects (font (size 1.27 1.27)) (justify right) hide)
     )
   )
@@
     (pin "1")
   )
-  (symbol (lib_id "atari_grav_bw:POT") (at 478.536 192.786 180) (unit 1)
-    (in_bom yes) (on_board yes)
-    (property "Reference" "R212" (id 0) (at 480.568 195.199 90)
+  (symbol (lib_name "POT_1") (lib_id "atari_grav_bw:POT") (at 478.536 192.786 180) (unit 1)
+    (in_bom yes) (on_board yes)
+    (property "Reference" "R212" (id 0) (at 480.6607 195.3003 90)
       (effects (font (size 1.27 1.27)) (justify right))
     )
-    (property "Value" "10k" (id 1) (at 478.536 194.437 90)
+    (property "Value" "10k" (id 1) (at 478.5714 194.3087 90)
       (effects (font (size 1.27 1.27)) (justify right))
     )

Commit message: Just need grounds and rev 2 resistors
Parts:
- added C129: 100pf, Star_Wars_Vector_PCB:CapBrown, symbol Device:C
- C133: renamed from C1000; footprint Star_Wars_Vector_PCB:GenericComp -> Star_Wars_Vector_PCB:CapBrown
- renumbered R202 to R201, R201 to R202
Connections:
- net +6V: now also C129.1
- net at A/B_12.6, R190.1, R191.1: now also C129.2
Changed lines of the file:
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@@
   (junction (at 481.076 167.386) (diameter 0) (color 0 0 0 0)
+  )
+  (junction (at 459.486 216.281) (diameter 0) (color 0 0 0 0)
   )
   (junction (at 454.406 246.126) (diameter 0) (color 0 0 0 0)
@@
     (stroke (width 0) (type default) (color 0 0 0 0))
   )
+  (wire (pts (xy 459.486 216.281) (xy 462.9477 216.281))
+    (stroke (width 0) (type default) (color 0 0 0 0))
+  )
   (wire (pts (xy 427.101 237.871) (xy 427.101 238.506))
     (stroke (width 0) (type default) (color 0 0 0 0))
@@
     (stroke (width 0) (type default) (color 0 0 0 0))
   )
+  (wire (pts (xy 462.9477 212.4393) (xy 462.9477 216.281))
+    (stroke (width 0) (type default) (color 0 0 0 0))
+  )
   (wire (pts (xy 503.936 197.231) (xy 516.636 197.231))
     (stroke (width 0) (type default) (color 0 0 0 0))
@@
   )
   (wire (pts (xy 448.056 232.791) (xy 442.341 232.791))
+    (stroke (width 0) (type default) (color 0 0 0 0))
+  )
+  (wire (pts (xy 462.9477 212.4393) (xy 466.6376 212.4393))
     (stroke (width 0) (type default) (color 0 0 0 0))
   )
@@
   (symbol (lib_id "Device:R") (at 469.646 182.626 180) (unit 1)
     (in_bom yes) (on_board yes)
-    (property "Reference" "R201" (id 0) (at 471.551 182.626 90))
+    (property "Reference" "R202" (id 0) (at 471.551 182.626 90))
     (property "Value" "10k" (id 1) (at 469.646 182.626 90))
     (property "Footprint" "Star_Wars_Vector_PCB:GenericComp" (id 2) (at 471.424 182.626 90)
@@
     )
     (property "Datasheet" "" (id 3) (at 406.146 199.771 0)
+      (effects (font (size 1.27 1.27)) hide)
+    )
+    (pin "1")
+  )
+  (symbol (lib_id "power:+6V") (at 474.2576 212.4393 270) (unit 1)
+    (in_bom yes) (on_board yes)
+    (property "Reference" "#PWR0557" (id 0) (at 470.4476 212.4393 0)
+      (effects (font (size 1.27 1.27)) hide)
+    )
+    (property "Value" "+6V" (id 1) (at 478.6518 212.8203 0))
+    (property "Footprint" "" (id 2) (at 474.2576 212.4393 0)
+      (effects (font (size 1.27 1.27)) hide)
+    )
+    (property "Datasheet" "" (id 3) (at 474.2576 212.4393 0)
       (effects (font (size 1.27 1.27)) hide)
     )
@@
     (pin "2")
   )
+  (symbol (lib_id "Device:C") (at 470.4476 212.4393 270) (unit 1)
+    (in_bom yes) (on_board yes)
+    (property "Reference" "C129" (id 0) (at 471.7176 215.6143 90)
+      (effects (font (size 1.27 1.27)) (justify left))
+    )
+    (property "Value" "100pf" (id 1) (at 465.3676 215.6143 90)
+      (effects (font (size 1.27 1.27)) (justify left))
+    )
+    (property "Footprint" "Star_Wars_Vector_PCB:CapBrown" (id 2) (at 466.6376 213.4045 0)
+      (effects (font (size 1.27 1.27)) hide)
+    )
+    (property "Datasheet" "" (id 3) (at 470.4476 212.4393 0)
+      (effects (font (size 1.27 1.27)) hide)
+    )
+    (pin "1")
+    (pin "2")
+  )
   (symbol (lib_id "Device:C") (at 307.721 198.501 180) (unit 1)
     (in_bom yes) (on_board yes)
@@
   (symbol (lib_id "Device:C") (at 500.126 206.121 270) (unit 1)
     (in_bom yes) (on_board yes)
-    (property "Reference" "C1000" (id 0) (at 501.396 209.296 90)
+    (property "Reference" "C133" (id 0) (at 501.396 209.296 90)
       (effects (font (size 1.27 1.27)) (justify left))
     )
@@
       (effects (font (size 1.27 1.27)) (justify left))
     )
-    (property "Footprint" "Star_Wars_Vector_PCB:GenericComp" (id 2) (at 496.316 207.0862 0)
+    (property "Footprint" "Star_Wars_Vector_PCB:CapBrown" (id 2) (at 496.316 207.0862 0)
       (effects (font (size 1.27 1.27)) hide)
     )
@@
   (symbol (lib_id "Device:R") (at 468.376 155.956 270) (unit 1)
     (in_bom yes) (on_board yes)
-    (property "Reference" "R202" (id 0) (at 468.376 154.051 90))
+    (property "Reference" "R201" (id 0) (at 468.376 154.051 90))
     (property "Value" "3.9k" (id 1) (at 468.376 155.956 90))
     (property "Footprint" "Star_Wars_Vector_PCB:GenericComp" (id 2) (at 468.376 154.178 90)

Commit message: second to last cleanup?
Parts:
- R191: value 100k -> ?
Connections:
- net YLIN: no longer names the net of C132.1, C133.1, D/E_12.7, R200.1, R210.1, R210.2
Other:
- note added: "Atari schematic misnumbers this as R202."
- note added: "Atari schematic shows C1__"
- note added: "Y Center"
- note added: "Y Linearity"
- note added: "Y Size"
Changed lines of the file:
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@@
   (junction (at 516.636 190.246) (diameter 0) (color 0 0 0 0)
-  )
-  (junction (at 280.416 188.341) (diameter 0) (color 0 0 0 0)
   )
   (junction (at 425.831 166.116) (diameter 0) (color 0 0 0 0)
@@
     (stroke (width 0) (type default) (color 0 0 0 0))
   )
+  (text "Atari schematic\nshows C1__" (at 494.5154 218.2438 0)
+    (effects (font (size 1.27 1.27)) (justify left bottom))
+  )
+  (text "Y Linearity" (at 520.5775 164.7888 0)
+    (effects (font (size 1.27 1.27)) (justify left bottom))
+  )
   (text "Y-AXIS OUTPUT" (at 382.016 102.616 0)
     (effects (font (size 2.54 2.54) (thickness 0.508) bold) (justify left bottom))
@@
     (effects (font (size 1.27 1.27)) (justify left bottom))
   )
+  (text "Y Size" (at 442.9475 196.0971 0)
+    (effects (font (size 1.27 1.27)) (justify left bottom))
+  )
   (text "NOT LOADED" (at 449.326 213.106 0)
     (effects (font (size 1.27 1.27)) (justify left bottom))
@@
   (text "NOT LOADED\n" (at 303.276 209.931 0)
     (effects (font (size 1.27 1.27) (thickness 0.508) bold) (justify left bottom))
+  )
+  (text "Atari schematic\nmisnumbers this\nas R202." (at 462.2944 152.0225 0)
+    (effects (font (size 1.27 1.27)) (justify left bottom))
+  )
+  (text "Y Center" (at 465.7463 196.0971 0)
+    (effects (font (size 1.27 1.27)) (justify left bottom))
   )
   (global_label "DVY5" (shape input) (at 27.051 193.421 180) (fields_autoplaced)
@@
     )
   )
-  (global_label "YLIN" (shape input) (at 520.446 166.116 90) (fields_autoplaced)
-    (effects (font (size 1.27 1.27)) (justify left))
-    (property "Intersheet References" "${INTERSHEET_REFS}" (id 0) (at 520.3666 159.7399 90)
-      (effects (font (size 1.27 1.27)) (justify left) hide)
-    )
-  )
   (global_label "DVY4" (shape input) (at 27.051 195.961 180) (fields_autoplaced)
     (effects (font (size 1.27 1.27)) (justify right))
@@
     )
     (property "Datasheet" "" (id 3) (at 542.036 192.913 0)
-      (effects (font (size 1.27 1.27)) hide)
-    )
-    (pin "1")
-  )
-  (symbol (lib_id "power:GND") (at 280.416 188.341 0) (unit 1)
-    (in_bom yes) (on_board yes)
-    (property "Reference" "#PWR0429" (id 0) (at 280.416 194.691 0)
-      (effects (font (size 1.27 1.27)) hide)
-    )
-    (property "Value" "GND" (id 1) (at 284.226 190.246 0))
-    (property "Footprint" "" (id 2) (at 280.416 188.341 0)
-      (effects (font (size 1.27 1.27)) hide)
-    )
-    (property "Datasheet" "" (id 3) (at 280.416 188.341 0)
       (effects (font (size 1.27 1.27)) hide)
     )
@@
       (effects (font (size 1.27 1.27)) hide)
     )
-    (property "Value" "GND" (id 1) (at 280.416 192.151 0))
+    (property "Value" "GND" (id 1) (at 283.9096 190.367 0))
     (property "Footprint" "" (id 2) (at 280.416 188.341 0)
       (effects (font (size 1.27 1.27)) hide)
@@
     (in_bom yes) (on_board yes)
     (property "Reference" "R191" (id 0) (at 455.676 214.376 90))
-    (property "Value" "100k" (id 1) (at 455.676 216.281 90))
+    (property "Value" "?" (id 1) (at 455.676 216.281 90))
     (property "Footprint" "Star_Wars_Vector_PCB:GenericComp" (id 2) (at 455.676 214.503 90)
       (effects (font (size 1.27 1.27)) hide)

Commit message: Fixed various issues and generated gerber files
Other:
- moved on the sheet: R212
Changed lines of the file:
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@@
     (pin "1")
   )
-  (symbol (lib_name "POT_1") (lib_id "atari_grav_bw:POT") (at 478.536 192.786 180) (unit 1)
+  (symbol (lib_id "atari_grav_bw:POT") (at 478.536 192.786 0) (mirror y) (unit 1)
     (in_bom yes) (on_board yes)
-    (property "Reference" "R212" (id 0) (at 480.6607 195.3003 90)
+    (property "Reference" "R212" (id 0) (at 480.6607 190.2717 90)
       (effects (font (size 1.27 1.27)) (justify right))
     )
-    (property "Value" "10k" (id 1) (at 478.5714 194.3087 90)
+    (property "Value" "10k" (id 1) (at 478.5714 191.2633 90)
       (effects (font (size 1.27 1.27)) (justify right))
     )
