File: kicad/atari_gravitar_black_widow/Sheet4B.kicad_sch (KiCad schematic)
At the start: 45 parts

Commit message: resistor placements R1-R153
Parts:
- R1, R10, R11, R12, R13, R14, R15, R16, R17, R18, R2, R21, R3, R4, R5, R6, R7, R8, R9: footprint (none) -> Star_Wars_Vector_PCB:GenericComp
Changed lines of the file:
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@@
       (effects (font (size 1.27 1.27)) (justify left))
     )
-    (property "Footprint" "" (id 2) (at 486.791 256.921 90)
+    (property "Footprint" "Star_Wars_Vector_PCB:GenericComp" (id 2) (at 486.791 256.921 90)
       (effects (font (size 1.27 1.27)) hide)
     )
@@
       (effects (font (size 1.27 1.27)) (justify left))
     )
-    (property "Footprint" "" (id 2) (at 403.606 143.764 90)
+    (property "Footprint" "Star_Wars_Vector_PCB:GenericComp" (id 2) (at 403.606 143.764 90)
       (effects (font (size 1.27 1.27)) hide)
     )
@@
       (effects (font (size 1.27 1.27)) (justify left))
     )
-    (property "Footprint" "" (id 2) (at 486.791 269.621 90)
+    (property "Footprint" "Star_Wars_Vector_PCB:GenericComp" (id 2) (at 486.791 269.621 90)
       (effects (font (size 1.27 1.27)) hide)
     )
@@
       (effects (font (size 1.27 1.27)) (justify left))
     )
-    (property "Footprint" "" (id 2) (at 486.791 264.541 90)
+    (property "Footprint" "Star_Wars_Vector_PCB:GenericComp" (id 2) (at 486.791 264.541 90)
       (effects (font (size 1.27 1.27)) hide)
     )
@@
       (effects (font (size 1.27 1.27)) (justify left))
     )
-    (property "Footprint" "" (id 2) (at 413.766 183.769 90)
+    (property "Footprint" "Star_Wars_Vector_PCB:GenericComp" (id 2) (at 413.766 183.769 90)
       (effects (font (size 1.27 1.27)) hide)
     )
@@
       (effects (font (size 1.27 1.27)) (justify left))
     )
-    (property "Footprint" "" (id 2) (at 423.926 143.764 90)
+    (property "Footprint" "Star_Wars_Vector_PCB:GenericComp" (id 2) (at 423.926 143.764 90)
       (effects (font (size 1.27 1.27)) hide)
     )
@@
       (effects (font (size 1.27 1.27)) (justify left))
     )
-    (property "Footprint" "" (id 2) (at 486.791 251.841 90)
+    (property "Footprint" "Star_Wars_Vector_PCB:GenericComp" (id 2) (at 486.791 251.841 90)
       (effects (font (size 1.27 1.27)) hide)
     )
@@
       (effects (font (size 1.27 1.27)) (justify left))
     )
-    (property "Footprint" "" (id 2) (at 486.791 259.461 90)
+    (property "Footprint" "Star_Wars_Vector_PCB:GenericComp" (id 2) (at 486.791 259.461 90)
       (effects (font (size 1.27 1.27)) hide)
     )
@@
       (effects (font (size 1.27 1.27)) (justify left))
     )
-    (property "Footprint" "" (id 2) (at 418.846 183.769 90)
+    (property "Footprint" "Star_Wars_Vector_PCB:GenericComp" (id 2) (at 418.846 183.769 90)
       (effects (font (size 1.27 1.27)) hide)
     )
@@
       (effects (font (size 1.27 1.27)) (justify left))
     )
-    (property "Footprint" "" (id 2) (at 418.846 143.764 90)
+    (property "Footprint" "Star_Wars_Vector_PCB:GenericComp" (id 2) (at 418.846 143.764 90)
       (effects (font (size 1.27 1.27)) hide)
     )
@@
       (effects (font (size 1.27 1.27)) (justify left))
     )
-    (property "Footprint" "" (id 2) (at 403.606 183.769 90)
+    (property "Footprint" "Star_Wars_Vector_PCB:GenericComp" (id 2) (at 403.606 183.769 90)
       (effects (font (size 1.27 1.27)) hide)
     )
@@
       (effects (font (size 1.27 1.27)) (justify left))
     )
-    (property "Footprint" "" (id 2) (at 486.791 267.081 90)
+    (property "Footprint" "Star_Wars_Vector_PCB:GenericComp" (id 2) (at 486.791 267.081 90)
       (effects (font (size 1.27 1.27)) hide)
     )
@@
       (effects (font (size 1.27 1.27)) (justify left))
     )
-    (property "Footprint" "" (id 2) (at 182.626 181.864 90)
+    (property "Footprint" "Star_Wars_Vector_PCB:GenericComp" (id 2) (at 182.626 181.864 90)
       (effects (font (size 1.27 1.27)) hide)
     )
@@
       (effects (font (size 1.27 1.27)) (justify left))
     )
-    (property "Footprint" "" (id 2) (at 486.791 262.001 90)
+    (property "Footprint" "Star_Wars_Vector_PCB:GenericComp" (id 2) (at 486.791 262.001 90)
       (effects (font (size 1.27 1.27)) hide)
     )
@@
       (effects (font (size 1.27 1.27)) (justify left))
     )
-    (property "Footprint" "" (id 2) (at 408.686 183.769 90)
+    (property "Footprint" "Star_Wars_Vector_PCB:GenericComp" (id 2) (at 408.686 183.769 90)
       (effects (font (size 1.27 1.27)) hide)
     )
@@
       (effects (font (size 1.27 1.27)) (justify left))
     )
-    (property "Footprint" "" (id 2) (at 486.791 254.381 90)
+    (property "Footprint" "Star_Wars_Vector_PCB:GenericComp" (id 2) (at 486.791 254.381 90)
       (effects (font (size 1.27 1.27)) hide)
     )
@@
       (effects (font (size 1.27 1.27)) (justify left))
     )
-    (property "Footprint" "" (id 2) (at 408.686 143.764 90)
+    (property "Footprint" "Star_Wars_Vector_PCB:GenericComp" (id 2) (at 408.686 143.764 90)
       (effects (font (size 1.27 1.27)) hide)
     )
@@
       (effects (font (size 1.27 1.27)) (justify left))
     )
-    (property "Footprint" "" (id 2) (at 398.526 143.764 90)
+    (property "Footprint" "Star_Wars_Vector_PCB:GenericComp" (id 2) (at 398.526 143.764 90)
       (effects (font (size 1.27 1.27)) hide)
     )
@@
       (effects (font (size 1.27 1.27)) (justify left))
     )
-    (property "Footprint" "" (id 2) (at 413.766 143.764 90)
-      (effects (font (size 1.27 1.27)) hide)
-    )
+    (property "Footprint" "Star_Wars_Vector_PCB:GenericComp" (id 2) (at 413.766 143.764 90)
+      (effects (font (size 1.27 1.27)) hide)
+    )

Commit message: ALL PARTS PLACED!!
Parts:
- CR1, CR2: footprint (none) -> quantum_arcade_pcb:Diode
- L2, L3: footprint (none) -> Star_Wars_Vector_PCB:Inductor1
Changed lines of the file:
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@@
       (effects (font (size 1.27 1.27)) (justify left))
     )
-    (property "Footprint" "" (id 2) (at 416.56 95.885 0)
+    (property "Footprint" "quantum_arcade_pcb:Diode" (id 2) (at 416.56 95.885 0)
       (effects (font (size 1.27 1.27)) hide)
     )
@@
     (property "Reference" "L2" (id 0) (at 401.955 78.0755 0))
     (property "Value" "100uh" (id 1) (at 401.955 80.8506 0))
-    (property "Footprint" "" (id 2) (at 401.955 83.185 0)
+    (property "Footprint" "Star_Wars_Vector_PCB:Inductor1" (id 2) (at 401.955 83.185 0)
       (effects (font (size 1.27 1.27)) hide)
     )
@@
       (effects (font (size 1.27 1.27)) (justify left))
     )
-    (property "Footprint" "" (id 2) (at 423.545 99.695 0)
+    (property "Footprint" "quantum_arcade_pcb:Diode" (id 2) (at 423.545 99.695 0)
       (effects (font (size 1.27 1.27)) hide)
     )
@@
     (property "Reference" "L3" (id 0) (at 468.63 81.2505 0))
     (property "Value" "100uh" (id 1) (at 468.63 84.0256 0))
-    (property "Footprint" "" (id 2) (at 468.63 86.36 0)
-      (effects (font (size 1.27 1.27)) hide)
-    )
+    (property "Footprint" "Star_Wars_Vector_PCB:Inductor1" (id 2) (at 468.63 86.36 0)
+      (effects (font (size 1.27 1.27)) hide)
+    )

Commit message: Row 2 routing and schematic fixes
EAROM (M2) had duplicate pins and no footprint :(
N8 pins were in wrong order
Parts:
- M_2: footprint (none) -> Package_DIP:DIP-22_W10.16mm
Connections:
- net +5V: no longer M_2.21 (VCC)
- net GND: no longer M_2.12 (GND)
- net at P_2.7 (3Q), R1.2: now also M_2.11 (A1); no longer M_2.12 (GND)
Other:
- moved on the sheet: C16
Changed lines of the file:
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@@
   (junction (at 141.605 88.9) (diameter 0) (color 0 0 0 0)
   )
-  (junction (at 438.785 99.695) (diameter 0) (color 0 0 0 0)
-  )
   (junction (at 80.645 111.76) (diameter 0) (color 0 0 0 0)
   )
@@
   (junction (at 478.79 203.2) (diameter 0) (color 0 0 0 0)
   )
-  (junction (at 438.785 135.89) (diameter 0) (color 0 0 0 0)
-  )
   (junction (at 141.732 111.633) (diameter 0) (color 0 0 0 0)
   )
-  (junction (at 438.785 86.36) (diameter 0) (color 0 0 0 0)
-  )
   (junction (at 490.855 258.445) (diameter 0) (color 0 0 0 0)
   )
@@
   (junction (at 182.245 125.73) (diameter 0) (color 0 0 0 0)
   )
+  (junction (at 438.15 135.89) (diameter 0) (color 0 0 0 0)
+  )
   (junction (at 490.855 260.985) (diameter 0) (color 0 0 0 0)
   )
@@
   (junction (at 182.245 130.81) (diameter 0) (color 0 0 0 0)
   )
+  (junction (at 438.15 86.36) (diameter 0) (color 0 0 0 0)
+  )
   (junction (at 181.61 185.42) (diameter 0) (color 0 0 0 0)
   )
@@
   (junction (at 416.56 99.695) (diameter 0) (color 0 0 0 0)
   )
-  (junction (at 438.785 127) (diameter 0) (color 0 0 0 0)
-  )
   (junction (at 141.605 114.3) (diameter 0) (color 0 0 0 0)
   )
@@
   (junction (at 121.285 125.73) (diameter 0) (color 0 0 0 0)
   )
+  (junction (at 438.15 99.695) (diameter 0) (color 0 0 0 0)
+  )
   (junction (at 60.325 93.98) (diameter 0) (color 0 0 0 0)
   )
@@
   (junction (at 60.325 86.36) (diameter 0) (color 0 0 0 0)
   )
+  (junction (at 438.15 127) (diameter 0) (color 0 0 0 0)
+  )
   (junction (at 100.965 135.89) (diameter 0) (color 0 0 0 0)
   )
@@
     (stroke (width 0) (type default) (color 0 0 0 0))
   )
-  (wire (pts (xy 438.785 135.89) (xy 438.785 140.97))
+  (wire (pts (xy 438.15 99.695) (xy 438.15 127))
     (stroke (width 0) (type default) (color 0 0 0 0))
   )
@@
     (stroke (width 0) (type default) (color 0 0 0 0))
   )
-  (wire (pts (xy 427.355 99.695) (xy 438.785 99.695))
+  (wire (pts (xy 427.355 99.695) (xy 438.15 99.695))
     (stroke (width 0) (type default) (color 0 0 0 0))
   )
@@
     (stroke (width 0) (type default) (color 0 0 0 0))
   )
-  (wire (pts (xy 438.785 127) (xy 438.785 135.89))
-    (stroke (width 0) (type default) (color 0 0 0 0))
-  )
   (wire (pts (xy 214.63 146.05) (xy 214.63 151.765))
     (stroke (width 0) (type default) (color 0 0 0 0))
@@
     (stroke (width 0) (type default) (color 0 0 0 0))
   )
-  (wire (pts (xy 438.785 86.36) (xy 450.85 86.36))
+  (wire (pts (xy 438.15 86.36) (xy 450.85 86.36))
     (stroke (width 0) (type default) (color 0 0 0 0))
   )
@@
     (stroke (width 0) (type default) (color 0 0 0 0))
   )
+  (wire (pts (xy 438.15 135.89) (xy 438.15 140.97))
+    (stroke (width 0) (type default) (color 0 0 0 0))
+  )
   (wire (pts (xy 524.51 205.74) (xy 546.735 205.74))
     (stroke (width 0) (type default) (color 0 0 0 0))
@@
     (stroke (width 0) (type default) (color 0 0 0 0))
   )
-  (wire (pts (xy 438.785 135.89) (xy 464.185 135.89))
+  (wire (pts (xy 438.15 135.89) (xy 464.185 135.89))
     (stroke (width 0) (type default) (color 0 0 0 0))
   )
@@
     (stroke (width 0) (type default) (color 0 0 0 0))
   )
-  (wire (pts (xy 416.56 86.36) (xy 438.785 86.36))
+  (wire (pts (xy 416.56 86.36) (xy 438.15 86.36))
     (stroke (width 0) (type default) (color 0 0 0 0))
   )
@@
     (stroke (width 0) (type default) (color 0 0 0 0))
   )
-  (wire (pts (xy 436.245 212.09) (xy 417.83 212.09))
-    (stroke (width 0) (type default) (color 0 0 0 0))
-  )
   (wire (pts (xy 58.42 312.42) (xy 140.97 312.42))
     (stroke (width 0) (type default) (color 0 0 0 0))
@@
     (stroke (width 0) (type default) (color 0 0 0 0))
   )
-  (wire (pts (xy 438.785 93.98) (xy 438.785 99.695))
+  (wire (pts (xy 438.15 93.98) (xy 438.15 99.695))
     (stroke (width 0) (type default) (color 0 0 0 0))
   )
@@
     (stroke (width 0) (type default) (color 0 0 0 0))
   )
-  (wire (pts (xy 438.785 127) (xy 546.735 127))
+  (wire (pts (xy 438.15 127) (xy 546.735 127))
     (stroke (width 0) (type default) (color 0 0 0 0))
   )
@@
     (stroke (width 0) (type default) (color 0 0 0 0))
   )
+  (wire (pts (xy 417.83 212.09) (xy 438.15 212.09))
+    (stroke (width 0) (type default) (color 0 0 0 0))
+  )
   (wire (pts (xy 417.83 153.67) (xy 431.165 153.67))
     (stroke (width 0) (type default) (color 0 0 0 0))
@@
     (stroke (width 0) (type default) (color 0 0 0 0))
   )
+  (wire (pts (xy 438.15 127) (xy 438.15 135.89))
+    (stroke (width 0) (type default) (color 0 0 0 0))
+  )
   (wire (pts (xy 141.605 86.36) (xy 161.925 86.36))
     (stroke (width 0) (type default) (color 0 0 0 0))
@@
     (stroke (width 0) (type default) (color 0 0 0 0))
   )
-  (wire (pts (xy 438.785 99.695) (xy 438.785 127))
-    (stroke (width 0) (type default) (color 0 0 0 0))
-  )
   (wire (pts (xy 58.42 163.83) (xy 106.045 163.83))
     (stroke (width 0) (type default) (color 0 0 0 0))
@@
     (pin "1")
   )
-  (symbol (lib_id "power:GND") (at 446.405 212.09 0) (unit 1)
-    (in_bom yes) (on_board yes)
-    (property "Reference" "#PWR0318" (id 0) (at 446.405 218.44 0)
-      (effects (font (size 1.27 1.27)) hide)
-    )
-    (property "Value" "GND" (id 1) (at 450.215 213.995 0))
-    (property "Footprint" "" (id 2) (at 446.405 212.09 0)
-      (effects (font (size 1.27 1.27)) hide)
-    )
-    (property "Datasheet" "" (id 3) (at 446.405 212.09 0)
-      (effects (font (size 1.27 1.27)) hide)
-    )
-    (pin "1")
-  )
   (symbol (lib_id "Device:D") (at 416.56 95.885 270) (unit 1)
     (in_bom yes) (on_board yes)
@@
       (effects (font (size 1.27 1.27)) hide)
     )
-    (property "Value" "+5V" (id 1) (at 458.47 156.845 0))
+    (property "Value" "+5V" (id 1) (at 462.28 153.67 90))
     (property "Footprint" "" (id 2) (at 456.565 153.67 0)
       (effects (font (size 1.27 1.27)) hide)
@@
       (effects (font (size 1.27 1.27)) (justify right))
     )
-    (property "Footprint" "" (id 2) (at 441.325 167.64 0)
+    (property "Footprint" "Package_DIP:DIP-22_W10.16mm" (id 2) (at 441.325 167.64 0)
       (effects (font (size 1.27 1.27)) hide)
     )
@@
     (pin "1")
     (pin "10")
-    (pin "12")
-    (pin "12")
+    (pin "11")
     (pin "12")
     (pin "13")
@@
     (pin "20")
     (pin "21")
-    (pin "21")
     (pin "22")
     (pin "3")
@@
   (symbol (lib_id "Device:C") (at 467.995 135.89 90) (unit 1)
     (in_bom yes) (on_board yes)
-    (property "Reference" "C9" (id 0) (at 466.8266 132.969 0)
+    (property "Reference" "C9" (id 0) (at 468.63 132.08 90)
       (effects (font (size 1.27 1.27)) (justify left))
     )
-    (property "Value" ".1uf" (id 1) (at 469.138 132.969 0)
+    (property "Value" ".1uf" (id 1) (at 469.265 140.335 90)
       (effects (font (size 1.27 1.27)) (justify left))
     )
@@
     (pin "9")
   )
-  (symbol (lib_id "Device:C") (at 438.785 90.17 0) (unit 1)
+  (symbol (lib_id "Device:C") (at 438.15 90.17 0) (unit 1)
     (in_bom yes) (on_board yes)
-    (property "Reference" "C16" (id 0) (at 441.706 89.0016 0)
+    (property "Reference" "C16" (id 0) (at 441.071 89.0016 0)
       (effects (font (size 1.27 1.27)) (justify left))
     )
-    (property "Value" "47uf" (id 1) (at 441.706 91.313 0)
+    (property "Value" "47uf" (id 1) (at 441.071 91.313 0)
       (effects (font (size 1.27 1.27)) (justify left))
     )
-    (property "Footprint" "Star_Wars_Vector_PCB:LargeCap" (id 2) (at 439.7502 93.98 0)
+    (property "Footprint" "Star_Wars_Vector_PCB:LargeCap" (id 2) (at 439.1152 93.98 0)
       (effects (font (size 1.27 1.27)) hide)
     )
-    (property "Datasheet" "~" (id 3) (at 438.785 90.17 0)
+    (property "Datasheet" "~" (id 3) (at 438.15 90.17 0)
       (effects (font (size 1.27 1.27)) hide)
     )
@@
     (pin "2")
   )
-  (symbol (lib_id "power:+5V") (at 446.405 140.97 0) (unit 1)
-    (in_bom yes) (on_board yes)
-    (property "Reference" "#PWR0317" (id 0) (at 446.405 144.78 0)
-      (effects (font (size 1.27 1.27)) hide)
-    )
-    (property "Value" "+5V" (id 1) (at 449.58 139.065 0))
-    (property "Footprint" "" (id 2) (at 446.405 140.97 0)
-      (effects (font (size 1.27 1.27)) hide)
-    )
-    (property "Datasheet" "" (id 3) (at 446.405 140.97 0)
-      (effects (font (size 1.27 1.27)) hide)
-    )
-    (pin "1")
-  )
   (symbol (lib_id "power:+5V") (at 448.31 245.745 0) (unit 1)
