File: kicad/atari_gravitar_black_widow/Sheet6B.kicad_sch (KiCad schematic)
At the start: 20 parts

Commit message: caps polarity, c39, c38, transistors holes to .125 mil
Connections:
- net ST3: now also A_7.9 (2Q); no longer A_7.8 (~{2Q})
Changed lines of the file:
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@@
   (junction (at 412.75 366.395) (diameter 0) (color 0 0 0 0)
   )
-  (junction (at 357.505 236.22) (diameter 0) (color 0 0 0 0)
-  )
   (junction (at 403.86 236.22) (diameter 0) (color 0 0 0 0)
   )
@@
   )
   (junction (at 390.525 82.55) (diameter 0) (color 0 0 0 0)
+  )
+  (junction (at 357.505 231.14) (diameter 0) (color 0 0 0 0)
   )
   (junction (at 196.215 196.215) (diameter 0) (color 0 0 0 0)
@@
   (no_connect (at 398.78 231.14))
   (no_connect (at 407.67 280.67))
-  (no_connect (at 351.79 231.14))
+  (no_connect (at 351.79 236.22))
   (no_connect (at 137.16 203.835))
   (no_connect (at 398.78 228.6))
@@
     (stroke (width 0) (type default) (color 0 0 0 0))
   )
-  (wire (pts (xy 357.505 213.36) (xy 357.505 236.22))
+  (wire (pts (xy 357.505 213.36) (xy 357.505 231.14))
     (stroke (width 0) (type default) (color 0 0 0 0))
   )
@@
     (stroke (width 0) (type default) (color 0 0 0 0))
   )
-  (wire (pts (xy 351.79 236.22) (xy 357.505 236.22))
+  (wire (pts (xy 351.79 231.14) (xy 357.505 231.14))
     (stroke (width 0) (type default) (color 0 0 0 0))
   )
@@
     (stroke (width 0) (type default) (color 0 0 0 0))
   )
+  (wire (pts (xy 357.505 231.14) (xy 357.505 236.22))
+    (stroke (width 0) (type default) (color 0 0 0 0))
+  )

Commit message: Fixed schematic and PCB errors. Added BOM
Connections:
- net ST3: now also A_7.8 (~{2Q}); no longer A_7.9 (2Q)
Changed lines of the file:
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@@
   (junction (at 412.75 366.395) (diameter 0) (color 0 0 0 0)
   )
+  (junction (at 357.505 236.22) (diameter 0) (color 0 0 0 0)
+  )
   (junction (at 403.86 236.22) (diameter 0) (color 0 0 0 0)
   )
@@
   (junction (at 390.525 82.55) (diameter 0) (color 0 0 0 0)
   )
-  (junction (at 357.505 231.14) (diameter 0) (color 0 0 0 0)
-  )
   (junction (at 196.215 196.215) (diameter 0) (color 0 0 0 0)
   )
@@
   )
   (no_connect (at 398.78 231.14))
+  (no_connect (at 351.79 231.14))
   (no_connect (at 407.67 280.67))
-  (no_connect (at 351.79 236.22))
   (no_connect (at 137.16 203.835))
   (no_connect (at 398.78 228.6))
@@
     (stroke (width 0) (type default) (color 0 0 0 0))
   )
+  (wire (pts (xy 351.79 236.22) (xy 357.505 236.22))
+    (stroke (width 0) (type default) (color 0 0 0 0))
+  )
   (wire (pts (xy 309.88 290.83) (xy 309.88 335.915))
     (stroke (width 0) (type default) (color 0 0 0 0))
@@
     (stroke (width 0) (type default) (color 0 0 0 0))
   )
-  (wire (pts (xy 357.505 213.36) (xy 357.505 231.14))
+  (wire (pts (xy 357.505 213.36) (xy 357.505 236.22))
     (stroke (width 0) (type default) (color 0 0 0 0))
   )
@@
     (stroke (width 0) (type default) (color 0 0 0 0))
   )
-  (wire (pts (xy 351.79 231.14) (xy 357.505 231.14))
-    (stroke (width 0) (type default) (color 0 0 0 0))
-  )
   (wire (pts (xy 367.03 259.715) (xy 363.22 259.715))
     (stroke (width 0) (type default) (color 0 0 0 0))
@@
     (stroke (width 0) (type default) (color 0 0 0 0))
   )
-  (wire (pts (xy 357.505 231.14) (xy 357.505 236.22))
-    (stroke (width 0) (type default) (color 0 0 0 0))
-  )
