File: address_decoders/kicad/GAL_to_bipolar/GAL_to_bipolar.kicad_sch (KiCad schematic)
At the start: 2 parts, among them J1 EPROM, J2 GAL

Commit message: Fixed the reversed address bits in the GAL adapter PCB
Connections:
- net A0: now also J1.10 (A0), J2.1 (IO0); no longer J1.14 (A4), J2.5 (IO4)
- net A1: now also J1.11 (A1), J2.2 (IO1); no longer J1.13 (A3), J2.4 (IO3)
- net A3: now also J1.13 (A3), J2.4 (IO3); no longer J1.11 (A1), J2.2 (IO1)
- net A4: now also J1.14 (A4), J2.5 (IO4); no longer J1.10 (A0), J2.1 (IO0)
Changed lines of the file:
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@@
     )
   )
-  (global_label "A3" (shape input) (at 151.13 83.82 180) (fields_autoplaced)
+  (global_label "A3" (shape input) (at 151.13 88.9 180) (fields_autoplaced)
     (effects (font (size 1.27 1.27)) (justify right))
-    (property "Intersheet References" "${INTERSHEET_REFS}" (id 0) (at 146.4188 83.7406 0)
+    (property "Intersheet References" "${INTERSHEET_REFS}" (id 0) (at 146.4188 88.8206 0)
       (effects (font (size 1.27 1.27)) (justify right) hide)
     )
   )
-  (global_label "A4" (shape input) (at 113.03 93.98 180) (fields_autoplaced)
+  (global_label "A4" (shape input) (at 113.03 83.82 180) (fields_autoplaced)
     (effects (font (size 1.27 1.27)) (justify right))
-    (property "Intersheet References" "${INTERSHEET_REFS}" (id 0) (at 108.3188 93.9006 0)
+    (property "Intersheet References" "${INTERSHEET_REFS}" (id 0) (at 108.3188 83.7406 0)
       (effects (font (size 1.27 1.27)) (justify right) hide)
     )
@@
     )
   )
-  (global_label "A0" (shape input) (at 156.21 91.44 180) (fields_autoplaced)
+  (global_label "A0" (shape input) (at 156.21 81.28 180) (fields_autoplaced)
     (effects (font (size 1.27 1.27)) (justify right))
-    (property "Intersheet References" "${INTERSHEET_REFS}" (id 0) (at 151.4988 91.3606 0)
+    (property "Intersheet References" "${INTERSHEET_REFS}" (id 0) (at 151.4988 81.2006 0)
       (effects (font (size 1.27 1.27)) (justify right) hide)
     )
@@
     )
   )
-  (global_label "A0" (shape input) (at 113.03 83.82 180) (fields_autoplaced)
+  (global_label "A0" (shape input) (at 113.03 93.98 180) (fields_autoplaced)
     (effects (font (size 1.27 1.27)) (justify right))
-    (property "Intersheet References" "${INTERSHEET_REFS}" (id 0) (at 108.3188 83.7406 0)
+    (property "Intersheet References" "${INTERSHEET_REFS}" (id 0) (at 108.3188 93.9006 0)
       (effects (font (size 1.27 1.27)) (justify right) hide)
     )
   )
-  (global_label "A1" (shape input) (at 107.95 86.36 180) (fields_autoplaced)
+  (global_label "A1" (shape input) (at 107.95 91.44 180) (fields_autoplaced)
     (effects (font (size 1.27 1.27)) (justify right))
-    (property "Intersheet References" "${INTERSHEET_REFS}" (id 0) (at 103.2388 86.2806 0)
+    (property "Intersheet References" "${INTERSHEET_REFS}" (id 0) (at 103.2388 91.3606 0)
       (effects (font (size 1.27 1.27)) (justify right) hide)
     )
@@
     )
   )
-  (global_label "A4" (shape input) (at 156.21 81.28 180) (fields_autoplaced)
+  (global_label "A4" (shape input) (at 156.21 91.44 180) (fields_autoplaced)
     (effects (font (size 1.27 1.27)) (justify right))
-    (property "Intersheet References" "${INTERSHEET_REFS}" (id 0) (at 151.4988 81.2006 0)
+    (property "Intersheet References" "${INTERSHEET_REFS}" (id 0) (at 151.4988 91.3606 0)
       (effects (font (size 1.27 1.27)) (justify right) hide)
     )
@@
     )
   )
-  (global_label "A1" (shape input) (at 151.13 88.9 180) (fields_autoplaced)
+  (global_label "A1" (shape input) (at 151.13 83.82 180) (fields_autoplaced)
     (effects (font (size 1.27 1.27)) (justify right))
-    (property "Intersheet References" "${INTERSHEET_REFS}" (id 0) (at 146.4188 88.8206 0)
+    (property "Intersheet References" "${INTERSHEET_REFS}" (id 0) (at 146.4188 83.7406 0)
       (effects (font (size 1.27 1.27)) (justify right) hide)
     )
@@
     )
   )
-  (global_label "A3" (shape input) (at 107.95 91.44 180) (fields_autoplaced)
+  (global_label "A3" (shape input) (at 107.95 86.36 180) (fields_autoplaced)
     (effects (font (size 1.27 1.27)) (justify right))
-    (property "Intersheet References" "${INTERSHEET_REFS}" (id 0) (at 103.2388 91.3606 0)
+    (property "Intersheet References" "${INTERSHEET_REFS}" (id 0) (at 103.2388 86.2806 0)
       (effects (font (size 1.27 1.27)) (justify right) hide)
     )
